File: DESIGN FILES/power.kicad_sch (KiCad schematic)
At the start: 49 parts, among them U1 MIMXRT1064CVL5B, Y1 24MHz, Y2 32.768KHz

Commit message: Adding voltage monitor and manual reset circuit
Parts:
- removed R2: 100k, MIMXRT1064 MCU Module:0402WGF1003TCE, symbol MIMXRT1064 MCU Module:0402WGF1003TCE
- added ?: UM805RE, symbol MIMXRT1064 MCU Module:UM805RE
- added ?: UM803RS, symbol MIMXRT1064 MCU Module:UM803RS
- added C34, C? (x2): 100nF, symbol MIMXRT1064 MCU Module:CL05B104KB54PNC
- added D? (x4): RB521S30_R1_00001, symbol MIMXRT1064 MCU Module:RB521S30_R1_00001
- added R8: 1.5k, symbol MIMXRT1064 MCU Module:CQ02WGF1501TCE
Connections:
- net +3V3: now also ?.3 (VCC), C34.1, D?.2 (A), R8.1
- net +5V: no longer VR1.1 (EN)
- net GND: now also ?.1 (GND), ?.1 (GND), C34.2, C?.2, C?.2
- net at U1.M7 (POR_B): now also ?.2 (~{RESET}), R8.2
- net PMIC_ON_REQ renamed LDO_EN
- net LDO_EN: now also VR1.1 (EN), ?.2 (~{RESET})
- net VDD_SNVS_IN: no longer names the net of C6.1, U1.M9 (VDD_SNVS_IN)
- net VDD_SNVS_IN: now also D?.1 (K), D?.1 (K)
- new net: ?.4 (VCC), C?.1
- new net: ?.3 (~{MR}), C?.1, D?.2 (A), D?.2 (A)
- new net EXT_POR_SWITCH: D?.1 (K)
- new net VDD_COIN_CELL: D?.2 (A)
- new net WATCHDOG_B: D?.1 (K)
Other:
- note removed: "EXTERNAL BATT"
- note removed: "EXTERNAL COIN CELL BATT"
- moved on the sheet: C10, C2, C4
