File: DESIGN FILES/supply_pmic.kicad_sch (KiCad schematic)
At the start: 24 parts, among them U6 UM803RS, U7 UM805RE

Commit message: vcc check
Connections:
- net +3V3: now also C69.1, U7.4 (VCC)
Other:
- note added: "DISABLE 3V3 LDO & ON-CHIP PMIC THROUGHT MANUAL RESET"
- note removed: "DISABLE 3V3 LDO & ONC-CHIP PMIC THROUGHT MANUAL RESET"
- moved on the sheet: C69
Changed lines of the file:
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@@
   (junction (at 66.04 129.54) (diameter 0) (color 0 0 0 0)
   )
+  (junction (at 80.01 114.3) (diameter 0) (color 0 0 0 0)
+  )
   (junction (at 201.93 55.88) (diameter 0) (color 0 0 0 0)
   )
@@
   (junction (at 85.09 55.88) (diameter 0) (color 0 0 0 0)
   )
+  (junction (at 182.88 147.32) (diameter 0) (color 0 0 0 0)
+  )
   (junction (at 121.92 43.18) (diameter 0) (color 0 0 0 0)
   )
@@
   (junction (at 111.76 55.88) (diameter 0) (color 0 0 0 0)
   )
-  (junction (at 182.88 146.05) (diameter 0) (color 0 0 0 0)
-  )
   (junction (at 166.37 43.18) (diameter 0) (color 0 0 0 0)
   )
@@
     (stroke (width 0) (type default) (color 0 0 0 0))
   )
+  (wire (pts (xy 166.37 147.32) (xy 182.88 147.32))
+    (stroke (width 0) (type default) (color 0 0 0 0))
+  )
   (wire (pts (xy 64.77 55.88) (xy 64.77 58.42))
     (stroke (width 0) (type default) (color 0 0 0 0))
@@
     (stroke (width 0) (type default) (color 0 0 0 0))
   )
-  (wire (pts (xy 80.01 116.84) (xy 80.01 105.41))
+  (wire (pts (xy 80.01 111.76) (xy 80.01 114.3))
     (stroke (width 0) (type default) (color 0 0 0 0))
   )
@@
     (stroke (width 0) (type default) (color 0 0 0 0))
   )
+  (wire (pts (xy 80.01 114.3) (xy 80.01 116.84))
+    (stroke (width 0) (type default) (color 0 0 0 0))
+  )
   (wire (pts (xy 91.44 129.54) (xy 102.87 129.54))
     (stroke (width 0) (type default) (color 0 0 0 0))
@@
     (stroke (width 0) (type default) (color 0 0 0 0))
   )
-  (wire (pts (xy 102.87 116.84) (xy 102.87 119.38))
-    (stroke (width 0) (type default) (color 0 0 0 0))
-  )
-  (wire (pts (xy 166.37 135.89) (xy 166.37 146.05))
+  (wire (pts (xy 166.37 135.89) (xy 166.37 147.32))
     (stroke (width 0) (type default) (color 0 0 0 0))
   )
@@
     (stroke (width 0) (type default) (color 0 0 0 0))
   )
+  (wire (pts (xy 92.71 114.3) (xy 90.17 114.3))
+    (stroke (width 0) (type default) (color 0 0 0 0))
+  )
   (polyline (pts (xy 19.05 26.67) (xy 132.08 26.67))
     (stroke (width 1) (type default) (color 0 0 0 0))
@@
     (stroke (width 0) (type default) (color 0 0 0 0))
   )
-  (wire (pts (xy 80.01 105.41) (xy 102.87 105.41))
-    (stroke (width 0) (type default) (color 0 0 0 0))
-  )
   (wire (pts (xy 78.74 50.8) (xy 78.74 55.88))
     (stroke (width 0) (type default) (color 0 0 0 0))
   )
+  (wire (pts (xy 80.01 114.3) (xy 82.55 114.3))
+    (stroke (width 0) (type default) (color 0 0 0 0))
+  )
   (wire (pts (xy 57.15 50.8) (xy 54.61 50.8))
     (stroke (width 0) (type default) (color 0 0 0 0))
@@
     (stroke (width 0) (type default) (color 0 0 0 0))
   )
+  (wire (pts (xy 92.71 116.84) (xy 92.71 114.3))
+    (stroke (width 0) (type default) (color 0 0 0 0))
+  )
   (wire (pts (xy 201.93 45.72) (xy 201.93 43.18))
     (stroke (width 0) (type default) (color 0 0 0 0))
   )
-  (wire (pts (xy 182.88 146.05) (xy 182.88 147.32))
-    (stroke (width 0) (type default) (color 0 0 0 0))
-  )
   (wire (pts (xy 43.18 125.73) (xy 48.26 125.73))
     (stroke (width 0) (type default) (color 0 0 0 0))
@@
     (stroke (width 1) (type default) (color 0 0 0 0))
   )
-  (wire (pts (xy 182.88 144.78) (xy 182.88 146.05))
+  (wire (pts (xy 182.88 144.78) (xy 182.88 147.32))
     (stroke (width 0) (type default) (color 0 0 0 0))
   )
@@
     (stroke (width 0) (type default) (color 0 0 0 0))
   )
+  (wire (pts (xy 182.88 147.32) (xy 182.88 149.86))
+    (stroke (width 0) (type default) (color 0 0 0 0))
+  )
   (wire (pts (xy 195.58 50.8) (xy 195.58 55.88))
     (stroke (width 0) (type default) (color 0 0 0 0))
@@
     (stroke (width 0) (type default) (color 0 0 0 0))
   )
-  (wire (pts (xy 166.37 146.05) (xy 182.88 146.05))
-    (stroke (width 0) (type default) (color 0 0 0 0))
-  )
   (wire (pts (xy 111.76 55.88) (xy 111.76 58.42))
     (stroke (width 0) (type default) (color 0 0 0 0))
   )
   (wire (pts (xy 181.61 55.88) (xy 181.61 58.42))
-    (stroke (width 0) (type default) (color 0 0 0 0))
-  )
-  (wire (pts (xy 102.87 105.41) (xy 102.87 109.22))
     (stroke (width 0) (type default) (color 0 0 0 0))
   )
@@
     (effects (font (size 3 3) bold italic) (justify left bottom))
   )
-  (text "DISABLE 3V3 LDO & ONC-CHIP PMIC\nTHROUGHT MANUAL RESET"
+  (text "DISABLE 3V3 LDO & ON-CHIP PMIC\nTHROUGHT MANUAL RESET"
     (at 29.21 111.76 0)
     (effects (font (size 1.27 1.27) bold italic) (justify left bottom))
@@
     )
   )
-  (symbol (lib_id "power:GND") (at 182.88 147.32 0) (unit 1)
-    (in_bom yes) (on_board yes) (fields_autoplaced)
-    (property "Reference" "#PWR069" (id 0) (at 182.88 153.67 0)
-      (effects (font (size 1.27 1.27)) hide)
-    )
-    (property "Value" "GND" (id 1) (at 182.88 152.4 0))
-    (property "Footprint" "" (id 2) (at 182.88 147.32 0)
-      (effects (font (size 1.27 1.27)) hide)
-    )
-    (property "Datasheet" "" (id 3) (at 182.88 147.32 0)
+  (symbol (lib_id "power:GND") (at 182.88 149.86 0) (unit 1)
+    (in_bom yes) (on_board yes) (fields_autoplaced)
+    (property "Reference" "#PWR069" (id 0) (at 182.88 156.21 0)
+      (effects (font (size 1.27 1.27)) hide)
+    )
+    (property "Value" "GND" (id 1) (at 182.88 154.94 0))
+    (property "Footprint" "" (id 2) (at 182.88 149.86 0)
+      (effects (font (size 1.27 1.27)) hide)
+    )
+    (property "Datasheet" "" (id 3) (at 182.88 149.86 0)
       (effects (font (size 1.27 1.27)) hide)
     )
@@
   )
   (symbol (lib_id "MIMXRT1064 MCU Module:CL05B104KB54PNC") (at 66.04 135.89 0) (unit 1)
-    (in_bom yes) (on_board yes) (fields_autoplaced)
-    (property "Reference" "C68" (id 0) (at 69.85 134.6199 0)
-      (effects (font (size 1.27 1.27)) (justify left))
-    )
-    (property "Value" "100nF" (id 1) (at 69.85 137.1599 0)
+    (in_bom yes) (on_board yes)
+    (property "Reference" "C68" (id 0) (at 68.58 135.89 0)
+      (effects (font (size 1.27 1.27)) (justify left))
+    )
+    (property "Value" "100nF" (id 1) (at 68.58 138.43 0)
       (effects (font (size 1.27 1.27)) (justify left))
     )
@@
     (pin "1")
   )
-  (symbol (lib_id "MIMXRT1064 MCU Module:CL05B104KB54PNC") (at 102.87 113.03 0) (unit 1)
-    (in_bom yes) (on_board yes) (fields_autoplaced)
-    (property "Reference" "C69" (id 0) (at 106.68 111.7599 0)
-      (effects (font (size 1.27 1.27)) (justify left))
-    )
-    (property "Value" "100nF" (id 1) (at 106.68 114.2999 0)
-      (effects (font (size 1.27 1.27)) (justify left))
-    )
-    (property "Footprint" "" (id 2) (at 103.8352 116.84 0)
-      (effects (font (size 1.27 1.27)) hide)
-    )
-    (property "Datasheet" "~" (id 3) (at 102.87 113.03 0)
-      (effects (font (size 1.27 1.27)) hide)
-    )
-    (pin "1")
-    (pin "2")
+  (symbol (lib_id "MIMXRT1064 MCU Module:CL05B104KB54PNC") (at 86.36 114.3 90) (unit 1)
+    (in_bom yes) (on_board yes)
+    (property "Reference" "C69" (id 0) (at 90.17 110.49 90))
+    (property "Value" "100nF" (id 1) (at 91.44 113.03 90))
+    (property "Footprint" "" (id 2) (at 90.17 113.3348 0)
+      (effects (font (size 1.27 1.27)) hide)
+    )
+    (property "Datasheet" "~" (id 3) (at 86.36 114.3 0)
+      (effects (font (size 1.27 1.27)) hide)
+    )
+    (pin "1")
+    (pin "2")
+  )
+  (symbol (lib_id "power:+3V3") (at 80.01 111.76 0) (unit 1)
+    (in_bom yes) (on_board yes) (fields_autoplaced)
+    (property "Reference" "#PWR?" (id 0) (at 80.01 115.57 0)
+      (effects (font (size 1.27 1.27)) hide)
+    )
+    (property "Value" "+3V3" (id 1) (at 80.01 106.68 0))
+    (property "Footprint" "" (id 2) (at 80.01 111.76 0)
+      (effects (font (size 1.27 1.27)) hide)
+    )
+    (property "Datasheet" "" (id 3) (at 80.01 111.76 0)
+      (effects (font (size 1.27 1.27)) hide)
+    )
+    (pin "1")
   )
   (symbol (lib_id "MIMXRT1064 MCU Module:CL10A226MQ8NRNC") (at 238.76 49.53 0) (unit 1)
@@
     (pin "2")
   )
-  (symbol (lib_id "power:GND") (at 102.87 119.38 0) (unit 1)
-    (in_bom yes) (on_board yes) (fields_autoplaced)
-    (property "Reference" "#PWR079" (id 0) (at 102.87 125.73 0)
-      (effects (font (size 1.27 1.27)) hide)
-    )
-    (property "Value" "GND" (id 1) (at 102.87 124.46 0))
-    (property "Footprint" "" (id 2) (at 102.87 119.38 0)
-      (effects (font (size 1.27 1.27)) hide)
-    )
-    (property "Datasheet" "" (id 3) (at 102.87 119.38 0)
-      (effects (font (size 1.27 1.27)) hide)
-    )
+  (symbol (lib_id "power:GND") (at 92.71 116.84 0) (unit 1)
+    (in_bom yes) (on_board yes) (fields_autoplaced)
+    (property "Reference" "#PWR079" (id 0) (at 92.71 123.19 0)
+      (effects (font (size 1.27 1.27)) hide)
+    )
+    (property "Value" "GND" (id 1) (at 92.71 121.92 0))
+    (property "Footprint" "" (id 2) (at 92.71 116.84 0)
+      (effects (font (size 1.27 1.27)) hide)
+    )
+    (property "Datasheet" "" (id 3) (at 92.71 116.84 0)
+      (effects (font (size 1.27 1.27)) hide)
+    )
