File: DESIGN FILES/supply_pmic.kicad_sch (KiCad schematic)
At the start: 24 parts, among them U6 UM803RS, U7 UM805RE

Commit message: schematic and lib edit
Parts:
- C63: renamed from C68; footprint (none) -> MIMXRT1064 MCU Module:0402_CL05B104KB54PNC
- C64: renamed from C69; footprint (none) -> MIMXRT1064 MCU Module:0402_CL05B104KB54PNC
- C69: renamed from C63; footprint (none) -> MIMXRT1064 MCU Module:0402_CL05B104KB54PNC
- D3, D4: footprint (none) -> MIMXRT1064 MCU Module:RB521S30_R1_00001
- R11: renamed from R9; footprint (none) -> MIMXRT1064 MCU Module:CQ02WGF1501TCE
- U5: renamed from U7; footprint (none) -> MIMXRT1064 MCU Module:UM805RE
- U6: footprint (none) -> MIMXRT1064 MCU Module:UM803RS
- renumbered C64 to C65, C65 to C66, C66 to C67, C67 to C68, R11 to R10, R10 to R9
Changed lines of the file:
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@@
   (symbol (lib_id "power:GND") (at 182.88 149.86 0) (unit 1)
     (in_bom yes) (on_board yes) (fields_autoplaced)
-    (property "Reference" "#PWR069" (id 0) (at 182.88 156.21 0)
+    (property "Reference" "#PWR078" (id 0) (at 182.88 156.21 0)
       (effects (font (size 1.27 1.27)) hide)
     )
@@
   (symbol (lib_id "power:GND") (at 111.76 58.42 0) (unit 1)
     (in_bom yes) (on_board yes) (fields_autoplaced)
-    (property "Reference" "#PWR071" (id 0) (at 111.76 64.77 0)
+    (property "Reference" "#PWR072" (id 0) (at 111.76 64.77 0)
       (effects (font (size 1.27 1.27)) hide)
     )
@@
   (symbol (lib_id "power:+3V3") (at 166.37 40.64 0) (unit 1)
     (in_bom yes) (on_board yes) (fields_autoplaced)
-    (property "Reference" "#PWR073" (id 0) (at 166.37 44.45 0)
+    (property "Reference" "#PWR074" (id 0) (at 166.37 44.45 0)
       (effects (font (size 1.27 1.27)) hide)
     )
@@
       (effects (font (size 1.27 1.27)) hide)
     )
-    (property "Footprint" "" (id 2) (at 52.07 121.285 0)
+    (property "Footprint" "MIMXRT1064 MCU Module:RB521S30_R1_00001" (id 2) (at 52.07 121.285 0)
       (effects (font (size 1.27 1.27)) hide)
     )
@@
   (symbol (lib_id "MIMXRT1064 MCU Module:CL10A226MQ8NRNC") (at 111.76 49.53 0) (unit 1)
     (in_bom yes) (on_board yes)
-    (property "Reference" "C65" (id 0) (at 114.3 48.26 0)
+    (property "Reference" "C66" (id 0) (at 114.3 48.26 0)
       (effects (font (size 1.27 1.27)) (justify left))
     )
@@
   (symbol (lib_id "MIMXRT1064 MCU Module:UM805RE") (at 78.74 132.08 0) (unit 1)
     (in_bom yes) (on_board yes)
-    (property "Reference" "U7" (id 0) (at 74.93 120.65 0))
+    (property "Reference" "U5" (id 0) (at 74.93 120.65 0))
     (property "Value" "UM805RE" (id 1) (at 85.09 120.65 0))
-    (property "Footprint" "" (id 2) (at 60.96 130.81 0)
+    (property "Footprint" "MIMXRT1064 MCU Module:UM805RE" (id 2) (at 60.96 130.81 0)
       (effects (font (size 1.27 1.27)) hide)
     )
@@
   (symbol (lib_id "MIMXRT1064 MCU Module:0402WGF2202TCE") (at 85.09 62.23 0) (unit 1)
     (in_bom yes) (on_board yes) (fields_autoplaced)
-    (property "Reference" "R11" (id 0) (at 87.63 60.9599 0)
+    (property "Reference" "R10" (id 0) (at 87.63 60.9599 0)
       (effects (font (size 1.27 1.27)) (justify left))
     )
@@
   (symbol (lib_id "MIMXRT1064 MCU Module:CL05B104KB54PNC") (at 66.04 135.89 0) (unit 1)
     (in_bom yes) (on_board yes)
-    (property "Reference" "C68" (id 0) (at 68.58 135.89 0)
+    (property "Reference" "C63" (id 0) (at 68.58 135.89 0)
       (effects (font (size 1.27 1.27)) (justify left))
     )
@@
       (effects (font (size 1.27 1.27)) (justify left))
     )
-    (property "Footprint" "" (id 2) (at 67.0052 139.7 0)
+    (property "Footprint" "MIMXRT1064 MCU Module:0402_CL05B104KB54PNC" (id 2) (at 67.0052 139.7 0)
       (effects (font (size 1.27 1.27)) hide)
     )
@@
       (effects (font (size 1.27 1.27)) hide)
     )
-    (property "Footprint" "" (id 2) (at 52.07 128.905 0)
+    (property "Footprint" "MIMXRT1064 MCU Module:RB521S30_R1_00001" (id 2) (at 52.07 128.905 0)
       (effects (font (size 1.27 1.27)) hide)
     )
@@
   (symbol (lib_id "power:GND") (at 66.04 142.24 0) (unit 1)
     (in_bom yes) (on_board yes) (fields_autoplaced)
-    (property "Reference" "#PWR075" (id 0) (at 66.04 148.59 0)
+    (property "Reference" "#PWR067" (id 0) (at 66.04 148.59 0)
       (effects (font (size 1.27 1.27)) hide)
     )
@@
   (symbol (lib_id "power:GND") (at 166.37 58.42 0) (unit 1)
     (in_bom yes) (on_board yes) (fields_autoplaced)
-    (property "Reference" "#PWR074" (id 0) (at 166.37 64.77 0)
+    (property "Reference" "#PWR075" (id 0) (at 166.37 64.77 0)
       (effects (font (size 1.27 1.27)) hide)
     )
@@
   (symbol (lib_id "MIMXRT1064 MCU Module:CL05B104KB54PNC") (at 86.36 114.3 90) (unit 1)
     (in_bom yes) (on_board yes)
-    (property "Reference" "C69" (id 0) (at 90.17 110.49 90))
+    (property "Reference" "C64" (id 0) (at 90.17 110.49 90))
     (property "Value" "100nF" (id 1) (at 91.44 113.03 90))
-    (property "Footprint" "" (id 2) (at 90.17 113.3348 0)
+    (property "Footprint" "MIMXRT1064 MCU Module:0402_CL05B104KB54PNC" (id 2) (at 90.17 113.3348 0)
       (effects (font (size 1.27 1.27)) hide)
     )
@@
   (symbol (lib_id "power:+3V3") (at 80.01 111.76 0) (unit 1)
     (in_bom yes) (on_board yes) (fields_autoplaced)
-    (property "Reference" "#PWR?" (id 0) (at 80.01 115.57 0)
+    (property "Reference" "#PWR068" (id 0) (at 80.01 115.57 0)
       (effects (font (size 1.27 1.27)) hide)
     )
@@
   (symbol (lib_id "MIMXRT1064 MCU Module:CL10A226MQ8NRNC") (at 166.37 50.8 0) (unit 1)
     (in_bom yes) (on_board yes)
-    (property "Reference" "C67" (id 0) (at 158.75 49.53 0)
+    (property "Reference" "C68" (id 0) (at 158.75 49.53 0)
       (effects (font (size 1.27 1.27)) (justify left))
     )
@@
   (symbol (lib_id "power:+3V3") (at 182.88 114.3 0) (unit 1)
     (in_bom yes) (on_board yes) (fields_autoplaced)
-    (property "Reference" "#PWR068" (id 0) (at 182.88 118.11 0)
+    (property "Reference" "#PWR077" (id 0) (at 182.88 118.11 0)
       (effects (font (size 1.27 1.27)) hide)
     )
@@
   (symbol (lib_id "power:GND") (at 64.77 58.42 0) (unit 1)
     (in_bom yes) (on_board yes) (fields_autoplaced)
-    (property "Reference" "#PWR067" (id 0) (at 64.77 64.77 0)
+    (property "Reference" "#PWR066" (id 0) (at 64.77 64.77 0)
       (effects (font (size 1.27 1.27)) hide)
     )
@@
   (symbol (lib_id "power:+3V3") (at 121.92 40.64 0) (unit 1)
     (in_bom yes) (on_board yes) (fields_autoplaced)
-    (property "Reference" "#PWR072" (id 0) (at 121.92 44.45 0)
+    (property "Reference" "#PWR073" (id 0) (at 121.92 44.45 0)
       (effects (font (size 1.27 1.27)) hide)
     )
@@
   (symbol (lib_id "MIMXRT1064 MCU Module:CL10A226MQ8NRNC") (at 121.92 49.53 0) (unit 1)
     (in_bom yes) (on_board yes)
-    (property "Reference" "C66" (id 0) (at 124.46 48.26 0)
+    (property "Reference" "C67" (id 0) (at 124.46 48.26 0)
       (effects (font (size 1.27 1.27)) (justify left))
     )
@@
   (symbol (lib_id "MIMXRT1064 MCU Module:0402WGF1003TCE") (at 85.09 49.53 0) (unit 1)
     (in_bom yes) (on_board yes) (fields_autoplaced)
-    (property "Reference" "R10" (id 0) (at 87.63 48.2599 0)
+    (property "Reference" "R9" (id 0) (at 87.63 48.2599 0)
       (effects (font (size 1.27 1.27)) (justify left))
     )
@@
   (symbol (lib_id "MIMXRT1064 MCU Module:CL05B104KB54PNC") (at 166.37 132.08 0) (unit 1)
     (in_bom yes) (on_board yes) (fields_autoplaced)
-    (property "Reference" "C63" (id 0) (at 170.18 130.8099 0)
+    (property "Reference" "C69" (id 0) (at 170.18 130.8099 0)
       (effects (font (size 1.27 1.27)) (justify left))
     )
@@
       (effects (font (size 1.27 1.27)) (justify left))
     )
-    (property "Footprint" "" (id 2) (at 167.3352 135.89 0)
+    (property "Footprint" "MIMXRT1064 MCU Module:0402_CL05B104KB54PNC" (id 2) (at 167.3352 135.89 0)
       (effects (font (size 1.27 1.27)) hide)
     )
@@
   (symbol (lib_id "power:GND") (at 80.01 144.78 0) (unit 1)
     (in_bom yes) (on_board yes) (fields_autoplaced)
-    (property "Reference" "#PWR077" (id 0) (at 80.01 151.13 0)
+    (property "Reference" "#PWR069" (id 0) (at 80.01 151.13 0)
       (effects (font (size 1.27 1.27)) hide)
     )
@@
       (effects (font (size 1.27 1.27)) (justify right))
     )
-    (property "Footprint" "" (id 2) (at 171.45 134.62 0)
+    (property "Footprint" "MIMXRT1064 MCU Module:UM803RS" (id 2) (at 171.45 134.62 0)
       (effects (font (size 1.27 1.27)) hide)
     )
@@
   (symbol (lib_id "MIMXRT1064 MCU Module:CQ02WGF1501TCE") (at 196.85 125.73 0) (unit 1)
     (in_bom yes) (on_board yes) (fields_autoplaced)
-    (property "Reference" "R9" (id 0) (at 199.39 124.4599 0)
+    (property "Reference" "R11" (id 0) (at 199.39 124.4599 0)
       (effects (font (size 1.27 1.27)) (justify left))
     )
@@
       (effects (font (size 1.27 1.27)) (justify left))
     )
-    (property "Footprint" "" (id 2) (at 195.072 125.73 90)
+    (property "Footprint" "MIMXRT1064 MCU Module:CQ02WGF1501TCE" (id 2) (at 195.072 125.73 90)
       (effects (font (size 1.27 1.27)) hide)
     )
@@
   (symbol (lib_id "power:GND") (at 92.71 116.84 0) (unit 1)
     (in_bom yes) (on_board yes) (fields_autoplaced)
-    (property "Reference" "#PWR079" (id 0) (at 92.71 123.19 0)
+    (property "Reference" "#PWR071" (id 0) (at 92.71 123.19 0)
       (effects (font (size 1.27 1.27)) hide)
     )
@@
   (symbol (lib_id "power:+5V") (at 35.56 40.64 0) (unit 1)
     (in_bom yes) (on_board yes) (fields_autoplaced)
-    (property "Reference" "#PWR065" (id 0) (at 35.56 44.45 0)
+    (property "Reference" "#PWR064" (id 0) (at 35.56 44.45 0)
       (effects (font (size 1.27 1.27)) hide)
     )
@@
   (symbol (lib_id "power:GND") (at 35.56 58.42 0) (unit 1)
     (in_bom yes) (on_board yes) (fields_autoplaced)
-    (property "Reference" "#PWR066" (id 0) (at 35.56 64.77 0)
+    (property "Reference" "#PWR065" (id 0) (at 35.56 64.77 0)
       (effects (font (size 1.27 1.27)) hide)
     )
@@
   (symbol (lib_id "MIMXRT1064 MCU Module:0402CG220J500NT") (at 95.25 49.53 0) (unit 1)
     (in_bom yes) (on_board yes)
-    (property "Reference" "C64" (id 0) (at 97.79 48.26 0)
+    (property "Reference" "C65" (id 0) (at 97.79 48.26 0)
       (effects (font (size 1.27 1.27)) (justify left))
     )
@@
   (symbol (lib_id "power:GND") (at 201.93 68.58 0) (unit 1)
     (in_bom yes) (on_board yes) (fields_autoplaced)
-    (property "Reference" "#PWR078" (id 0) (at 201.93 74.93 0)
-      (effects (font (size 1.27 1.27)) hide)
-    )
+    (property "Reference" "#PWR079" (id 0) (at 201.93 74.93 0)
+      (effects (font (size 1.27 1.27)) hide)
+    )

Commit message: work
Changed lines of the file:
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@@
   (symbol (lib_id "MIMXRT1064 MCU Module:UM803RS") (at 171.45 134.62 0) (unit 1)
     (in_bom yes) (on_board yes)
-    (property "Reference" "U6" (id 0) (at 191.77 135.89 0)
+    (property "Reference" "U6" (id 0) (at 179.07 123.19 0)
       (effects (font (size 1.27 1.27)) (justify right))
     )
-    (property "Value" "UM803RS" (id 1) (at 199.39 138.43 0)
+    (property "Value" "UM803RS" (id 1) (at 193.04 123.19 0)
       (effects (font (size 1.27 1.27)) (justify right))
     )

Commit message: work
Parts:
- added C?: 100nF, symbol MIMXRT1064 MCU Module:CL05B104KB54PNC
- added C? (x3): 1uF, symbol MIMXRT1064 MCU Module:CL05A105KA5NQNC
- added C?: 10uF, symbol MIMXRT1064 MCU Module:CL10A106KP8NNNC
- added L?: 10nH, symbol MIMXRT1064 MCU Module:MLG1005S10NHT000
- added R?: 220R, symbol MIMXRT1064 MCU Module:0603WAF2200T5E
- added VR?: TPS79333DBVR, Package_TO_SOT_SMD:SOT-23-5, symbol MIMXRT1064 MCU Module:TPS79333DBVR
Connections:
- net +5V: now also C?.1, L?.2, R?.1
- net GND: now also C?.2, C?.2, C?.2, C?.2, C?.2, VR?.2 (GND)
- net BUCK_FB: now reaches C65.2, R10.1, R9.2, VR1.5 (FB)
- net BUCK_SW: now reaches L2.1, VR1.3 (LX)
- new net: C?.1, VR?.4 (NR)
- new net: C?.1, R?.2, VR?.1 (IN), VR?.3 (EN)
- new net +3.3VA: C?.1, VR?.5 (OUT)
- new net VBUS: C?.1, L?.1
Other:
- note added: "0603 1/8W"
- note added: "2 : SUPPLY & PMIC"
- note added: "DCR = 0R22"
- note added: "I(DC) = 500mA"
- note added: "Input Filtering & Analogue and Digital Supplies"
- company: (none) -> Soundsom
- title: (none) -> Supply & PMIC
- moved on the sheet: C62, C63, C64, C65, C66, C67, C68, C69, C70, C71, C72, D3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

Commit message: adding datasheet
Parts:
- removed C62, C66, C67, C68, C71, C72: 22uF, MIMXRT1064 MCU Module:0603_CL10A226MQ8NRNC, symbol MIMXRT1064 MCU Module:CL10A226MQ8NRNC
- removed C65, C70: 22pF, MIMXRT1064 MCU Module:0402CG220J500NT, symbol MIMXRT1064 MCU Module:0402CG220J500NT
- removed L2, L3: 2.2uH, MIMXRT1064 MCU Module:CD32YP0302-2R2M_SMD3.5x3x2.1mm, symbol MIMXRT1064 MCU Module:CD32YP0302-2R2M
- removed R10: 22k, MIMXRT1064 MCU Module:0402WGF2202TCE, symbol MIMXRT1064 MCU Module:0402WGF2202TCE
- removed R12: 200k, MIMXRT1064 MCU Module:0402WGF2003TCE, symbol MIMXRT1064 MCU Module:0402WGF2003TCE
- removed R13, R9: 100k, MIMXRT1064 MCU Module:0402WGF1003TCE, symbol MIMXRT1064 MCU Module:0402WGF1003TCE
- removed VR1, VR2: SY8089AAAC, MIMXRT1064 MCU Module:SY8089AAAC_SOT-23-5, symbol MIMXRT1064 MCU Module:SY8089AAAC
- added C? (x4): 22uF, MIMXRT1064 MCU Module:0603_CL10A226MQ8NRNC, symbol MIMXRT1064 MCU Module:CL10A226MQ8NRNC
- added C? (x2): DNP, MIMXRT1064 MCU Module:0603_CL10A226MQ8NRNC, symbol MIMXRT1064 MCU Module:CL10A226MQ8NRNC
- added L? (x2): 68uH, symbol MIMXRT1064 MCU Module:MPIT4030-680M-LF
- added R? (x2): 100k, MIMXRT1064 MCU Module:0402WGF1003TCE, symbol MIMXRT1064 MCU Module:0402WGF1003TCE
- added R?: 200k, MIMXRT1064 MCU Module:0402WGF2003TCE, symbol MIMXRT1064 MCU Module:0402WGF2003TCE
- added R?: 22k, MIMXRT1064 MCU Module:0402WGF2202TCE, symbol MIMXRT1064 MCU Module:0402WGF2202TCE
- added U? (x2): TLV62569DBV, Package_TO_SOT_SMD:SOT-23-5, symbol MIMXRT1064 MCU Module:TLV62569DBV
Connections:
- net +1V8: now also C?.1, C?.1, L?.2, R?.1
- net +3V3: now also C?.1, C?.1, C?.1, L?.2, R?.1, U?.1 (EN), U?.4 (VIN)
- net +5V: now also C?.1, U?.4 (VIN)
- net GND: now also C?.2, C?.2, C?.2, C?.2, R?.2, R?.2, U?.2 (GND), U?.2 (GND)
- net LDO_EN: now also U?.1 (EN)
- new net: C?.2, R?.1, R?.2, U?.5 (FB) (x2)
- new net: L?.1, U?.3 (SW) (x2)

Commit message: TLV62569DBVR symbol check
Parts:
- removed U? (x2): TLV62569DBV, Package_TO_SOT_SMD:SOT-23-5, symbol MIMXRT1064 MCU Module:TLV62569DBV
- added VR? (x2): TLV62569DBV, Package_TO_SOT_SMD:SOT-23-5, symbol MIMXRT1064 MCU Module:TLV62569DBV
Connections:
- net +3V3: now also VR?.1 (EN), VR?.4 (VIN)
- net +5V: now also VR?.4 (VIN)
- net GND: now also VR?.2 (GND), VR?.2 (GND)
- net LDO_EN: now also VR?.1 (EN)
- net at C?.2, R?.1, R?.2: now also VR?.5 (FB) (x2)
- net at L?.1: now also VR?.3 (SW) (x2)

Commit message: Adding power on led
Parts:
- added D?: Blue LED, symbol MIMXRT1064 MCU Module:19-218_BHC-ZL1M2QY_3T
- added R?: 2.2k, symbol MIMXRT1064 MCU Module:0402WGF2201TCE
Connections:
- net +3V3: now also D?.2 (A)
- net GND: now also R?.2
- new net: D?.1 (K), R?.1
Changed lines of the file:
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@@
+    (stroke (width 0) (type default) (color 0 0 0 0))
+  )
+  (wire (pts (xy 138.43 50.8) (xy 138.43 48.26))
     (stroke (width 0) (type default) (color 0 0 0 0))
   )
@@
     (stroke (width 0) (type default) (color 0 0 0 0))
   )
+  (wire (pts (xy 138.43 68.58) (xy 138.43 69.85))
+    (stroke (width 0) (type default) (color 0 0 0 0))
+  )
   (wire (pts (xy 215.9 58.42) (xy 208.28 58.42))
     (stroke (width 0) (type default) (color 0 0 0 0))
@@
     (stroke (width 0) (type default) (color 0 0 0 0))
   )
+  (wire (pts (xy 138.43 48.26) (xy 124.46 48.26))
+    (stroke (width 0) (type default) (color 0 0 0 0))
+  )
   (wire (pts (xy 88.9 48.26) (xy 90.17 48.26))
     (stroke (width 0) (type default) (color 0 0 0 0))
@@
   )
   (wire (pts (xy 124.46 62.23) (xy 124.46 69.85))
+    (stroke (width 0) (type default) (color 0 0 0 0))
+  )
+  (wire (pts (xy 138.43 58.42) (xy 138.43 60.96))
     (stroke (width 0) (type default) (color 0 0 0 0))
   )
@@
     (pin "1")
   )
+  (symbol (lib_id "MIMXRT1064 MCU Module:0402WGF2201TCE") (at 138.43 64.77 0) (unit 1)
+    (in_bom yes) (on_board yes) (fields_autoplaced)
+    (property "Reference" "R?" (id 0) (at 140.97 63.4999 0)
+      (effects (font (size 1.27 1.27)) (justify left))
+    )
+    (property "Value" "2.2k" (id 1) (at 140.97 66.0399 0)
+      (effects (font (size 1.27 1.27)) (justify left))
+    )
+    (property "Footprint" "" (id 2) (at 136.652 64.77 90)
+      (effects (font (size 1.27 1.27)) hide)
+    )
+    (property "Datasheet" "~" (id 3) (at 138.43 64.77 0)
+      (effects (font (size 1.27 1.27)) hide)
+    )
+    (pin "1")
+    (pin "2")
+  )
   (symbol (lib_id "MIMXRT1064 MCU Module:RB521S30_R1_00001") (at 52.07 160.02 0) (mirror x) (unit 1)
     (in_bom yes) (on_board yes)
@@
     (pin "1")
   )
+  (symbol (lib_id "power:GND") (at 138.43 69.85 0) (unit 1)
+    (in_bom yes) (on_board yes) (fields_autoplaced)
+    (property "Reference" "#PWR?" (id 0) (at 138.43 76.2 0)
+      (effects (font (size 1.27 1.27)) hide)
+    )
+    (property "Value" "GND" (id 1) (at 138.43 74.93 0))
+    (property "Footprint" "" (id 2) (at 138.43 69.85 0)
+      (effects (font (size 1.27 1.27)) hide)
+    )
+    (property "Datasheet" "" (id 3) (at 138.43 69.85 0)
+      (effects (font (size 1.27 1.27)) hide)
+    )
+    (pin "1")
+  )
   (symbol (lib_id "MIMXRT1064 MCU Module:MLG1005S10NHT000") (at 34.29 48.26 90) (unit 1)
     (in_bom yes) (on_board yes) (fields_autoplaced)
@@
       (effects (font (size 1.27 1.27)) hide)
     )
+    (pin "1")
+    (pin "2")
+  )
+  (symbol (lib_id "MIMXRT1064 MCU Module:19-218_BHC-ZL1M2QY_3T") (at 138.43 54.61 90) (unit 1)
+    (in_bom yes) (on_board yes) (fields_autoplaced)
+    (property "Reference" "D?" (id 0) (at 142.24 54.9274 90)
+      (effects (font (size 1.27 1.27)) (justify right))
+    )
+    (property "Value" "Blue LED" (id 1) (at 142.24 57.4674 90)
+      (effects (font (size 1.27 1.27)) (justify right))
+    )
+    (property "Footprint" "" (id 2) (at 138.43 54.61 0)
+      (effects (font (size 1.27 1.27)) hide)
+    )
+    (property "Datasheet" "~" (id 3) (at 138.43 54.61 0)
+      (effects (font (size 1.27 1.27)) hide)
+    )
