File: DESIGN FILES/MIMXRT1064 MCU Module.kicad_sch (KiCad schematic)
At the start: 0 parts

Commit message: Refactoring schematic
Other:
- sheet audio renamed audio codec
- sheet mcu pinout renamed mcu gpio & memory signals & USB
- sheet memory renamed memory ICs
- sheet power renamed mcu power & crystals
- added sheet supply & pmic (supply_pmic.kicad_sch)
- sheet mcu power & crystals: file power.kicad_sch -> mcu_power_crystals.kicad_sch
- note added: "PAGE 6"

Commit message: work
Other:
- sheet memory ICs renamed memory
Changed lines of the file:
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@@
     (stroke (width 1) (type solid) (color 0 0 0 0))
     (fill (color 0 0 0 0.0000))
-    (property "Sheet name" "memory ICs" (id 0) (at 77.47 156.21 0)
+    (property "Sheet name" "memory" (id 0) (at 77.47 156.21 0)
       (effects (font (size 3 3) bold italic) (justify left bottom))
     )

Commit message: work
Other:
- sheet mcu gpio & memory signals & USB renamed mcu gpio & memory signals
- sheet memory renamed memory & USB
- sheet memory & USB: file memory.kicad_sch -> memory_usb.kicad_sch
- note added: "MIMXRT1064 MCU Module - TABLE OF CONTENTS"
- note added: "__________________________________________________________________________________"
- note removed: "TABLE OF CONTENTS"
- note removed: "_________________________________"
- company: (none) -> Soundsom
