File: DESIGN FILES/MIMXRT1064 MCU Module.kicad_sch (KiCad schematic)
At the start: 0 parts

Commit message: schematic changes
Other:
- sheet MCU GPIO renamed MCU GPIO & BUS
- sheet MEMORY renamed MEMORY 

Commit message: changes and adding schematic pdf
Other:
- added sheet MEZZANNINE (mezzannine.kicad_sch)
- note added: "PAGE 7"
- company: Soundsom -> Joël Ucedo
- title: Table on contents -> MIMXRT1064 MCU Module
Changed lines of the file:
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@@
   (paper "A3")
   (title_block
-    (title "Table on contents")
-    (date "2023-05-19")
+    (title "MIMXRT1064 MCU Module")
+    (date "2023-05-23")
     (rev "0")
-    (company "Soundsom")
+    (company "Joël Ucedo")
   )
   (text "MIMXRT1064 MCU Module - TABLE OF CONTENTS" (at 22.86 26.67 0)
@@
   )
   (text "PAGE 6" (at 24.13 157.48 0)
+    (effects (font (size 5 5) bold italic) (justify left bottom))
+  )
+  (text "PAGE 7" (at 24.13 182.88 0)
     (effects (font (size 5 5) bold italic) (justify left bottom))
   )
@@
     )
     (property "Sheet file" "memory.kicad_sch" (id 1) (at 63.5 161.0284 0)
+      (effects (font (size 1.27 1.27)) (justify left top) hide)
+    )
+  )
+  (sheet (at 63.5 172.72) (size 12.7 13.97)
+    (stroke (width 1) (type solid) (color 0 0 0 0))
+    (fill (color 0 0 0 0.0000))
+    (property "Sheet name" "MEZZANNINE" (id 0) (at 77.47 181.61 0)
+      (effects (font (size 3 3) bold italic) (justify left bottom))
+    )
+    (property "Sheet file" "mezzannine.kicad_sch" (id 1) (at 63.5 187.6984 0)
       (effects (font (size 1.27 1.27)) (justify left top) hide)
     )
@@
     (path "/574a2f6c-1db5-4366-bd73-1f4d156f4a53" (page "5"))
     (path "/a2f401b1-e3ca-4fba-8477-437af9831272" (page "6"))
+    (path "/d10fccf0-29f0-4392-b875-5cee27b3fc14" (page "7"))
   )
   (symbol_instances
@@
       (reference "#PWR0404") (unit 1) (value "GND") (footprint "")
     )
-    (path "/829b3f95-6b61-404e-b99c-998f91300f3b/e5359e96-d77a-4c98-a2f9-0d78025e8457"
-      (reference "#PWR0405") (unit 1) (value "VDD_SNVS_3V3") (footprint "")
-    )
     (path "/829b3f95-6b61-404e-b99c-998f91300f3b/009a49bb-70c2-47ac-bda5-07d9269c6bdf"
       (reference "#PWR0406") (unit 1) (value "+3V3") (footprint "")
@@
       (reference "C619") (unit 1) (value "100n") (footprint "MIMXRT1064 MCU Module:0402_CL05B104KB54PNC")
     )
-    (path "/829b3f95-6b61-404e-b99c-998f91300f3b/024e7b2e-36a7-4292-933c-2f0388895000"
-      (reference "D401") (unit 1) (value "RB521S30_R1_00001") (footprint "MIMXRT1064 MCU Module:RB521S30_R1_00001")
-    )
-    (path "/829b3f95-6b61-404e-b99c-998f91300f3b/29b21083-cdd8-49c4-a279-864e7e56279e"
-      (reference "D402") (unit 1) (value "RB521S30_R1_00001") (footprint "MIMXRT1064 MCU Module:RB521S30_R1_00001")
-    )
     (path "/829b3f95-6b61-404e-b99c-998f91300f3b/8e9a58e1-077c-4adc-8e20-9823eceab5dc"

Commit message: updates
Other:
- sheet MEZZANNINE renamed M.2 CONNECTOR
- sheet M.2 CONNECTOR: file mezzannine.kicad_sch -> m2_connector.kicad_sch
Changed lines of the file:
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@@
     (stroke (width 1) (type solid) (color 0 0 0 0))
     (fill (color 0 0 0 0.0000))
-    (property "Sheet name" "MEZZANNINE" (id 0) (at 77.47 181.61 0)
+    (property "Sheet name" "M.2 CONNECTOR" (id 0) (at 77.47 181.61 0)
       (effects (font (size 3 3) bold italic) (justify left bottom))
     )
-    (property "Sheet file" "mezzannine.kicad_sch" (id 1) (at 63.5 187.6984 0)
+    (property "Sheet file" "m2_connector.kicad_sch" (id 1) (at 63.5 187.6984 0)
       (effects (font (size 1.27 1.27)) (justify left top) hide)
     )

Commit message: updates
Other:
- sheet M.2 CONNECTOR renamed AUDIO
- added sheet EXTENSION IO (extension_io.kicad_sch)
- added sheet MIDI (midi.kicad_sch)
- added sheet USB - JTAG (usb_jtag.kicad_sch)
- sheet AUDIO: file m2_connector.kicad_sch -> audio.kicad_sch
- note added: "PAGE 1 COVER"
- note added: "PAGE 10"
- note added: "PAGE 8"
- note added: "PAGE 9"

Commit message: updates
Other:
- sheet EXTENSION IO renamed POTS & ENCODER & LEDS
- sheet POTS & ENCODER & LEDS: file extension_io.kicad_sch -> pots_enc_leds.kicad_sch
