File: DESIGN FILES/audio.kicad_sch (KiCad schematic)
At the start: 9 parts, among them U5 WM8978CGEFL{slash}RV

Commit message: Adding voltage monitor and manual reset circuit
Parts:
- renumbered C65 to C66, C66 to C67, C67 to C68, C68 to C69, C69 to C70, R11 to R12, R12 to R13, R13 to R14, U5 to U7
Changed lines of the file:
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@@
   (symbol (lib_id "MIMXRT1064 MCU Module:CL05A475MP5NRNC") (at 203.2 85.09 0) (unit 1)
     (in_bom yes) (on_board yes) (fields_autoplaced)
-    (property "Reference" "C66" (id 0) (at 207.01 83.8199 0)
+    (property "Reference" "C67" (id 0) (at 207.01 83.8199 0)
       (effects (font (size 1.27 1.27)) (justify left))
     )
@@
   (symbol (lib_id "MIMXRT1064 MCU Module:CL05A475MP5NRNC") (at 228.6 39.37 0) (unit 1)
     (in_bom yes) (on_board yes) (fields_autoplaced)
-    (property "Reference" "C68" (id 0) (at 232.41 38.0999 0)
+    (property "Reference" "C69" (id 0) (at 232.41 38.0999 0)
       (effects (font (size 1.27 1.27)) (justify left))
     )
@@
   (symbol (lib_id "MIMXRT1064 MCU Module:0402WGF2201TCE") (at 96.52 114.3 0) (unit 1)
     (in_bom yes) (on_board yes) (fields_autoplaced)
-    (property "Reference" "R12" (id 0) (at 99.06 113.0299 0)
+    (property "Reference" "R13" (id 0) (at 99.06 113.0299 0)
       (effects (font (size 1.27 1.27)) (justify left))
     )
@@
   (symbol (lib_id "MIMXRT1064 MCU Module:CL05A475MP5NRNC") (at 214.63 39.37 0) (unit 1)
     (in_bom yes) (on_board yes) (fields_autoplaced)
-    (property "Reference" "C67" (id 0) (at 218.44 38.0999 0)
+    (property "Reference" "C68" (id 0) (at 218.44 38.0999 0)
       (effects (font (size 1.27 1.27)) (justify left))
     )
@@
   (symbol (lib_id "MIMXRT1064 MCU Module:WM8978CGEFL{brace}slash}RV") (at 146.05 95.25 0) (unit 1)
     (in_bom yes) (on_board yes) (fields_autoplaced)
-    (property "Reference" "U5" (id 0) (at 147.32 53.34 0)
+    (property "Reference" "U7" (id 0) (at 147.32 53.34 0)
       (effects (font (size 1.524 1.524)))
     )
@@
   (symbol (lib_id "MIMXRT1064 MCU Module:CL05A475MP5NRNC") (at 195.58 39.37 0) (unit 1)
     (in_bom yes) (on_board yes) (fields_autoplaced)
-    (property "Reference" "C65" (id 0) (at 199.39 38.0999 0)
+    (property "Reference" "C66" (id 0) (at 199.39 38.0999 0)
       (effects (font (size 1.27 1.27)) (justify left))
     )
@@
   (symbol (lib_id "MIMXRT1064 MCU Module:0402WGF1002TCE") (at 195.58 130.81 0) (unit 1)
     (in_bom yes) (on_board yes) (fields_autoplaced)
-    (property "Reference" "R13" (id 0) (at 198.12 129.5399 0)
+    (property "Reference" "R14" (id 0) (at 198.12 129.5399 0)
       (effects (font (size 1.27 1.27)) (justify left))
     )
@@
   (symbol (lib_id "MIMXRT1064 MCU Module:CL05A475MP5NRNC") (at 245.11 39.37 0) (unit 1)
     (in_bom yes) (on_board yes) (fields_autoplaced)
-    (property "Reference" "C69" (id 0) (at 248.92 38.0999 0)
+    (property "Reference" "C70" (id 0) (at 248.92 38.0999 0)
       (effects (font (size 1.27 1.27)) (justify left))
     )
@@
   (symbol (lib_id "MIMXRT1064 MCU Module:0402WGF2201TCE") (at 91.44 114.3 0) (unit 1)
     (in_bom yes) (on_board yes)
-    (property "Reference" "R11" (id 0) (at 87.63 113.03 0)
-      (effects (font (size 1.27 1.27)) (justify left))
-    )
+    (property "Reference" "R12" (id 0) (at 87.63 113.03 0)
+      (effects (font (size 1.27 1.27)) (justify left))
+    )

Commit message: Refactoring schematic
Parts:
- renumbered C66 to C57, C67 to C58, C68 to C59, C69 to C60, C70 to C61, R12 to R6, R13 to R7, R14 to R8, U7 to U5
Changed lines of the file:
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@@
   (symbol (lib_id "power:+3V3") (at 214.63 33.02 0) (unit 1)
     (in_bom yes) (on_board yes) (fields_autoplaced)
-    (property "Reference" "#PWR070" (id 0) (at 214.63 36.83 0)
+    (property "Reference" "#PWR059" (id 0) (at 214.63 36.83 0)
       (effects (font (size 1.27 1.27)) hide)
     )
@@
   (symbol (lib_id "power:GND") (at 177.8 139.7 0) (unit 1)
     (in_bom yes) (on_board yes) (fields_autoplaced)
-    (property "Reference" "#PWR065" (id 0) (at 177.8 146.05 0)
+    (property "Reference" "#PWR054" (id 0) (at 177.8 146.05 0)
       (effects (font (size 1.27 1.27)) hide)
     )
@@
   (symbol (lib_id "MIMXRT1064 MCU Module:CL05A475MP5NRNC") (at 203.2 85.09 0) (unit 1)
     (in_bom yes) (on_board yes) (fields_autoplaced)
-    (property "Reference" "C67" (id 0) (at 207.01 83.8199 0)
+    (property "Reference" "C58" (id 0) (at 207.01 83.8199 0)
       (effects (font (size 1.27 1.27)) (justify left))
     )
@@
   (symbol (lib_id "power:GND") (at 203.2 91.44 0) (unit 1)
     (in_bom yes) (on_board yes) (fields_autoplaced)
-    (property "Reference" "#PWR069" (id 0) (at 203.2 97.79 0)
+    (property "Reference" "#PWR058" (id 0) (at 203.2 97.79 0)
       (effects (font (size 1.27 1.27)) hide)
     )
@@
   (symbol (lib_id "power:+3V3") (at 114.3 50.8 0) (unit 1)
     (in_bom yes) (on_board yes) (fields_autoplaced)
-    (property "Reference" "#PWR063" (id 0) (at 114.3 54.61 0)
+    (property "Reference" "#PWR052" (id 0) (at 114.3 54.61 0)
       (effects (font (size 1.27 1.27)) hide)
     )
@@
   (symbol (lib_id "power:+5V") (at 101.6 50.8 0) (unit 1)
     (in_bom yes) (on_board yes) (fields_autoplaced)
-    (property "Reference" "#PWR062" (id 0) (at 101.6 54.61 0)
+    (property "Reference" "#PWR051" (id 0) (at 101.6 54.61 0)
       (effects (font (size 1.27 1.27)) hide)
     )
@@
   (symbol (lib_id "power:GND") (at 195.58 139.7 0) (unit 1)
     (in_bom yes) (on_board yes) (fields_autoplaced)
-    (property "Reference" "#PWR068" (id 0) (at 195.58 146.05 0)
+    (property "Reference" "#PWR057" (id 0) (at 195.58 146.05 0)
       (effects (font (size 1.27 1.27)) hide)
     )
@@
   (symbol (lib_id "MIMXRT1064 MCU Module:CL05A475MP5NRNC") (at 228.6 39.37 0) (unit 1)
     (in_bom yes) (on_board yes) (fields_autoplaced)
-    (property "Reference" "C69" (id 0) (at 232.41 38.0999 0)
+    (property "Reference" "C60" (id 0) (at 232.41 38.0999 0)
       (effects (font (size 1.27 1.27)) (justify left))
     )
@@
   (symbol (lib_id "power:GND") (at 170.18 69.85 0) (unit 1)
     (in_bom yes) (on_board yes)
-    (property "Reference" "#PWR064" (id 0) (at 170.18 76.2 0)
+    (property "Reference" "#PWR053" (id 0) (at 170.18 76.2 0)
       (effects (font (size 1.27 1.27)) hide)
     )
@@
   (symbol (lib_id "power:+3V3") (at 91.44 107.95 0) (unit 1)
     (in_bom yes) (on_board yes) (fields_autoplaced)
-    (property "Reference" "#PWR060" (id 0) (at 91.44 111.76 0)
+    (property "Reference" "#PWR049" (id 0) (at 91.44 111.76 0)
       (effects (font (size 1.27 1.27)) hide)
     )
@@
   (symbol (lib_id "power:GND") (at 228.6 45.72 0) (unit 1)
     (in_bom yes) (on_board yes) (fields_autoplaced)
-    (property "Reference" "#PWR073" (id 0) (at 228.6 52.07 0)
+    (property "Reference" "#PWR062" (id 0) (at 228.6 52.07 0)
       (effects (font (size 1.27 1.27)) hide)
     )
@@
   (symbol (lib_id "power:+5V") (at 245.11 33.02 0) (unit 1)
     (in_bom yes) (on_board yes) (fields_autoplaced)
-    (property "Reference" "#PWR074" (id 0) (at 245.11 36.83 0)
+    (property "Reference" "#PWR063" (id 0) (at 245.11 36.83 0)
       (effects (font (size 1.27 1.27)) hide)
     )
@@
   (symbol (lib_id "MIMXRT1064 MCU Module:0402WGF2201TCE") (at 96.52 114.3 0) (unit 1)
     (in_bom yes) (on_board yes) (fields_autoplaced)
-    (property "Reference" "R13" (id 0) (at 99.06 113.0299 0)
+    (property "Reference" "R7" (id 0) (at 99.06 113.0299 0)
       (effects (font (size 1.27 1.27)) (justify left))
     )
@@
   (symbol (lib_id "power:+3.3VA") (at 88.9 50.8 0) (unit 1)
     (in_bom yes) (on_board yes) (fields_autoplaced)
-    (property "Reference" "#PWR059" (id 0) (at 88.9 54.61 0)
+    (property "Reference" "#PWR048" (id 0) (at 88.9 54.61 0)
       (effects (font (size 1.27 1.27)) hide)
     )
@@
   (symbol (lib_id "MIMXRT1064 MCU Module:CL05A475MP5NRNC") (at 214.63 39.37 0) (unit 1)
     (in_bom yes) (on_board yes) (fields_autoplaced)
-    (property "Reference" "C68" (id 0) (at 218.44 38.0999 0)
+    (property "Reference" "C59" (id 0) (at 218.44 38.0999 0)
       (effects (font (size 1.27 1.27)) (justify left))
     )
@@
   (symbol (lib_id "power:GND") (at 214.63 45.72 0) (unit 1)
     (in_bom yes) (on_board yes) (fields_autoplaced)
-    (property "Reference" "#PWR071" (id 0) (at 214.63 52.07 0)
+    (property "Reference" "#PWR060" (id 0) (at 214.63 52.07 0)
       (effects (font (size 1.27 1.27)) hide)
     )
@@
   (symbol (lib_id "power:GND") (at 195.58 45.72 0) (unit 1)
     (in_bom yes) (on_board yes) (fields_autoplaced)
-    (property "Reference" "#PWR067" (id 0) (at 195.58 52.07 0)
+    (property "Reference" "#PWR056" (id 0) (at 195.58 52.07 0)
       (effects (font (size 1.27 1.27)) hide)
     )
@@
   (symbol (lib_id "MIMXRT1064 MCU Module:WM8978CGEFL{brace}slash}RV") (at 146.05 95.25 0) (unit 1)
     (in_bom yes) (on_board yes) (fields_autoplaced)
-    (property "Reference" "U7" (id 0) (at 147.32 53.34 0)
+    (property "Reference" "U5" (id 0) (at 147.32 53.34 0)
       (effects (font (size 1.524 1.524)))
     )
@@
   (symbol (lib_id "MIMXRT1064 MCU Module:CL05A475MP5NRNC") (at 195.58 39.37 0) (unit 1)
     (in_bom yes) (on_board yes) (fields_autoplaced)
-    (property "Reference" "C66" (id 0) (at 199.39 38.0999 0)
+    (property "Reference" "C57" (id 0) (at 199.39 38.0999 0)
       (effects (font (size 1.27 1.27)) (justify left))
     )
@@
   (symbol (lib_id "MIMXRT1064 MCU Module:0402WGF1002TCE") (at 195.58 130.81 0) (unit 1)
     (in_bom yes) (on_board yes) (fields_autoplaced)
-    (property "Reference" "R14" (id 0) (at 198.12 129.5399 0)
+    (property "Reference" "R8" (id 0) (at 198.12 129.5399 0)
       (effects (font (size 1.27 1.27)) (justify left))
     )
@@
   (symbol (lib_id "power:+3.3VA") (at 195.58 33.02 0) (unit 1)
     (in_bom yes) (on_board yes) (fields_autoplaced)
-    (property "Reference" "#PWR066" (id 0) (at 195.58 36.83 0)
+    (property "Reference" "#PWR055" (id 0) (at 195.58 36.83 0)
       (effects (font (size 1.27 1.27)) hide)
     )
@@
   (symbol (lib_id "power:+3V3") (at 96.52 107.95 0) (unit 1)
     (in_bom yes) (on_board yes) (fields_autoplaced)
-    (property "Reference" "#PWR061" (id 0) (at 96.52 111.76 0)
+    (property "Reference" "#PWR050" (id 0) (at 96.52 111.76 0)
       (effects (font (size 1.27 1.27)) hide)
     )
@@
   (symbol (lib_id "power:+3V3") (at 228.6 33.02 0) (unit 1)
     (in_bom yes) (on_board yes) (fields_autoplaced)
-    (property "Reference" "#PWR072" (id 0) (at 228.6 36.83 0)
+    (property "Reference" "#PWR061" (id 0) (at 228.6 36.83 0)
       (effects (font (size 1.27 1.27)) hide)
     )
@@
   (symbol (lib_id "MIMXRT1064 MCU Module:CL05A475MP5NRNC") (at 245.11 39.37 0) (unit 1)
     (in_bom yes) (on_board yes) (fields_autoplaced)
-    (property "Reference" "C70" (id 0) (at 248.92 38.0999 0)
+    (property "Reference" "C61" (id 0) (at 248.92 38.0999 0)
       (effects (font (size 1.27 1.27)) (justify left))
     )
@@
   (symbol (lib_id "MIMXRT1064 MCU Module:0402WGF2201TCE") (at 91.44 114.3 0) (unit 1)
     (in_bom yes) (on_board yes)
-    (property "Reference" "R12" (id 0) (at 87.63 113.03 0)
+    (property "Reference" "R6" (id 0) (at 87.63 113.03 0)
       (effects (font (size 1.27 1.27)) (justify left))
     )
@@
   (symbol (lib_id "power:GND") (at 245.11 45.72 0) (unit 1)
     (in_bom yes) (on_board yes) (fields_autoplaced)
-    (property "Reference" "#PWR075" (id 0) (at 245.11 52.07 0)
-      (effects (font (size 1.27 1.27)) hide)
-    )
+    (property "Reference" "#PWR064" (id 0) (at 245.11 52.07 0)
+      (effects (font (size 1.27 1.27)) hide)
+    )

Commit message: schematic and lib edit
Parts:
- renumbered U5 to U4
Changed lines of the file:
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@@
   (symbol (lib_id "power:+3V3") (at 214.63 33.02 0) (unit 1)
     (in_bom yes) (on_board yes) (fields_autoplaced)
-    (property "Reference" "#PWR059" (id 0) (at 214.63 36.83 0)
+    (property "Reference" "#PWR058" (id 0) (at 214.63 36.83 0)
       (effects (font (size 1.27 1.27)) hide)
     )
@@
   (symbol (lib_id "power:GND") (at 177.8 139.7 0) (unit 1)
     (in_bom yes) (on_board yes) (fields_autoplaced)
-    (property "Reference" "#PWR054" (id 0) (at 177.8 146.05 0)
+    (property "Reference" "#PWR053" (id 0) (at 177.8 146.05 0)
       (effects (font (size 1.27 1.27)) hide)
     )
@@
   (symbol (lib_id "power:GND") (at 203.2 91.44 0) (unit 1)
     (in_bom yes) (on_board yes) (fields_autoplaced)
-    (property "Reference" "#PWR058" (id 0) (at 203.2 97.79 0)
+    (property "Reference" "#PWR057" (id 0) (at 203.2 97.79 0)
       (effects (font (size 1.27 1.27)) hide)
     )
@@
   (symbol (lib_id "power:+3V3") (at 114.3 50.8 0) (unit 1)
     (in_bom yes) (on_board yes) (fields_autoplaced)
-    (property "Reference" "#PWR052" (id 0) (at 114.3 54.61 0)
+    (property "Reference" "#PWR051" (id 0) (at 114.3 54.61 0)
       (effects (font (size 1.27 1.27)) hide)
     )
@@
   (symbol (lib_id "power:+5V") (at 101.6 50.8 0) (unit 1)
     (in_bom yes) (on_board yes) (fields_autoplaced)
-    (property "Reference" "#PWR051" (id 0) (at 101.6 54.61 0)
+    (property "Reference" "#PWR050" (id 0) (at 101.6 54.61 0)
       (effects (font (size 1.27 1.27)) hide)
     )
@@
   (symbol (lib_id "power:GND") (at 195.58 139.7 0) (unit 1)
     (in_bom yes) (on_board yes) (fields_autoplaced)
-    (property "Reference" "#PWR057" (id 0) (at 195.58 146.05 0)
+    (property "Reference" "#PWR056" (id 0) (at 195.58 146.05 0)
       (effects (font (size 1.27 1.27)) hide)
     )
@@
   (symbol (lib_id "power:GND") (at 170.18 69.85 0) (unit 1)
     (in_bom yes) (on_board yes)
-    (property "Reference" "#PWR053" (id 0) (at 170.18 76.2 0)
+    (property "Reference" "#PWR052" (id 0) (at 170.18 76.2 0)
       (effects (font (size 1.27 1.27)) hide)
     )
@@
   (symbol (lib_id "power:+3V3") (at 91.44 107.95 0) (unit 1)
     (in_bom yes) (on_board yes) (fields_autoplaced)
-    (property "Reference" "#PWR049" (id 0) (at 91.44 111.76 0)
+    (property "Reference" "#PWR048" (id 0) (at 91.44 111.76 0)
       (effects (font (size 1.27 1.27)) hide)
     )
@@
   (symbol (lib_id "power:GND") (at 228.6 45.72 0) (unit 1)
     (in_bom yes) (on_board yes) (fields_autoplaced)
-    (property "Reference" "#PWR062" (id 0) (at 228.6 52.07 0)
+    (property "Reference" "#PWR061" (id 0) (at 228.6 52.07 0)
       (effects (font (size 1.27 1.27)) hide)
     )
@@
   (symbol (lib_id "power:+5V") (at 245.11 33.02 0) (unit 1)
     (in_bom yes) (on_board yes) (fields_autoplaced)
-    (property "Reference" "#PWR063" (id 0) (at 245.11 36.83 0)
+    (property "Reference" "#PWR062" (id 0) (at 245.11 36.83 0)
       (effects (font (size 1.27 1.27)) hide)
     )
@@
   (symbol (lib_id "power:+3.3VA") (at 88.9 50.8 0) (unit 1)
     (in_bom yes) (on_board yes) (fields_autoplaced)
-    (property "Reference" "#PWR048" (id 0) (at 88.9 54.61 0)
+    (property "Reference" "#PWR047" (id 0) (at 88.9 54.61 0)
       (effects (font (size 1.27 1.27)) hide)
     )
@@
   (symbol (lib_id "power:GND") (at 214.63 45.72 0) (unit 1)
     (in_bom yes) (on_board yes) (fields_autoplaced)
-    (property "Reference" "#PWR060" (id 0) (at 214.63 52.07 0)
+    (property "Reference" "#PWR059" (id 0) (at 214.63 52.07 0)
       (effects (font (size 1.27 1.27)) hide)
     )
@@
   (symbol (lib_id "power:GND") (at 195.58 45.72 0) (unit 1)
     (in_bom yes) (on_board yes) (fields_autoplaced)
-    (property "Reference" "#PWR056" (id 0) (at 195.58 52.07 0)
+    (property "Reference" "#PWR055" (id 0) (at 195.58 52.07 0)
       (effects (font (size 1.27 1.27)) hide)
     )
@@
   (symbol (lib_id "MIMXRT1064 MCU Module:WM8978CGEFL{brace}slash}RV") (at 146.05 95.25 0) (unit 1)
     (in_bom yes) (on_board yes) (fields_autoplaced)
-    (property "Reference" "U5" (id 0) (at 147.32 53.34 0)
+    (property "Reference" "U4" (id 0) (at 147.32 53.34 0)
       (effects (font (size 1.524 1.524)))
     )
@@
   (symbol (lib_id "power:+3.3VA") (at 195.58 33.02 0) (unit 1)
     (in_bom yes) (on_board yes) (fields_autoplaced)
-    (property "Reference" "#PWR055" (id 0) (at 195.58 36.83 0)
+    (property "Reference" "#PWR054" (id 0) (at 195.58 36.83 0)
       (effects (font (size 1.27 1.27)) hide)
     )
@@
   (symbol (lib_id "power:+3V3") (at 96.52 107.95 0) (unit 1)
     (in_bom yes) (on_board yes) (fields_autoplaced)
-    (property "Reference" "#PWR050" (id 0) (at 96.52 111.76 0)
+    (property "Reference" "#PWR049" (id 0) (at 96.52 111.76 0)
       (effects (font (size 1.27 1.27)) hide)
     )
@@
   (symbol (lib_id "power:+3V3") (at 228.6 33.02 0) (unit 1)
     (in_bom yes) (on_board yes) (fields_autoplaced)
-    (property "Reference" "#PWR061" (id 0) (at 228.6 36.83 0)
+    (property "Reference" "#PWR060" (id 0) (at 228.6 36.83 0)
       (effects (font (size 1.27 1.27)) hide)
     )
@@
   (symbol (lib_id "power:GND") (at 245.11 45.72 0) (unit 1)
     (in_bom yes) (on_board yes) (fields_autoplaced)
-    (property "Reference" "#PWR064" (id 0) (at 245.11 52.07 0)
-      (effects (font (size 1.27 1.27)) hide)
-    )
+    (property "Reference" "#PWR063" (id 0) (at 245.11 52.07 0)
+      (effects (font (size 1.27 1.27)) hide)
+    )

Commit message: work
Other:
- note added: "6 : AUDIO CODEC"
- company: (none) -> Soundsom
- title: (none) -> Audio codec
- moved on the sheet: C57, C59, C60, C61

Commit message: Removing audio codec from project
Parts:
- removed C57, C58, C59, C60, C61: 4.7uF, MIMXRT1064 MCU Module:0402_CL05A475MP5NRNC, symbol MIMXRT1064 MCU Module:CL05A475MP5NRNC
- removed R6, R7: 2.2k, MIMXRT1064 MCU Module:0402WGF2201TCE, symbol MIMXRT1064 MCU Module:0402WGF2201TCE
- removed R8: 10k, MIMXRT1064 MCU Module:0402WGF1002TCE, symbol MIMXRT1064 MCU Module:0402WGF1002TCE
- removed U4: WM8978CGEFL/RV, MIMXRT1064 MCU Module:WM8978CGEFL_RV_WQFN-32, symbol MIMXRT1064 MCU Module:WM8978CGEFL{brace}slash}RV
Connections:
- no-connect marks 1 -> 0
Other:
- note removed: "6 : AUDIO CODEC"
- note removed: "AVDD"
- note removed: "DBVDD"
- note removed: "DCVDD"
- note removed: "SPKVDD"
