File: DESIGN FILES/audio.kicad_sch (KiCad schematic)
At the start: 22 parts

Commit message: updates
Parts:
- removed C? (x5): (no value), symbol MY CAPACITOR LIBRARY:CL21A475KAQNNNE
- removed C? (x4): (no value), symbol MY CAPACITOR LIBRARY:CL10A105KB8NNNC
- removed C? (x2): (no value), symbol MY CAPACITOR LIBRARY:RVT1A221M0605
- removed J? (x3): (no value), symbol MY CONNECTOR LIBRARY:PJ-342B-TX-SMT
- removed R? (x2): (no value), symbol MY RESISTOR LIBRARY:0603WAF4702T5E
- removed R? (x2): (no value), symbol MY RESISTOR LIBRARY:0805W8F1000T5E
- removed R? (x2): (no value), symbol MY RESISTOR LIBRARY:0805W8F2201T5E
- removed U?: (no value), symbol MY AUDIO CODEC LIBRARY:WM8978CGEFL{brace}brace}brace}slash}RV
- added C701, C702, C703, C704, C705: 4.7u, MY CAPACITOR LIBRARY:0402_CL05A475MP5NRNC, symbol MY CAPACITOR LIBRARY:CL05A475MP5NRNC
- added C706, C707: 220u, MY CAPACITOR LIBRARY:RVT1A221M0605, symbol MY CAPACITOR LIBRARY:RVT1A221M0605
- added C708, C709, C710, C711: 1u, MY CAPACITOR LIBRARY:0402_CL05A105KA5NQNC, symbol MY CAPACITOR LIBRARY:CL05A105KA5NQNC
- added J701, J702, J703: PJ-342B-TX-SMT, MY CONNECTOR LIBRARY:PJ-342B-TX-SMT, symbol MY CONNECTOR LIBRARY:PJ-342B-TX-SMT
- added R701, R702: 2.2k, MY RESISTOR LIBRARY:0402WGF2201TCE, symbol MY RESISTOR LIBRARY:0402WGF2201TCE
- added R704, R705: 100R, MY RESISTOR LIBRARY:0805W8F1000T5E, symbol MY RESISTOR LIBRARY:0805W8F1000T5E
- added R706, R707: 47k, MY RESISTOR LIBRARY:0402WGF4702TCE, symbol MY RESISTOR LIBRARY:0402WGF4702TCE
- added U701: WM8978CGEFL_RV, MY AUDIO CODEC LIBRARY:WM8978CGEFL_RV_WQFN-32, symbol MY AUDIO CODEC LIBRARY:WM8978CGEFL_RV
- R703: renamed from R?; value (none) -> 10k; footprint (none) -> MY RESISTOR LIBRARY:0402WGF1002TCE
Connections:
- net +3.3VA: now also C701.1, U701.31 (AVDD)
- net +3V3: now also C702.1, C703.1, R701.1, R702.1, U701.13 (DCVDD), U701.14 (DBVDD)
- net +5V: now also C704.1, U701.26 (SPKVDD)
- net ADCDAT: now also U701.9 (ADCDAT)
- net BCLK: now also U701.8 (BCLK)
- net CODEC_SCLK: now also R702.2, U701.16 (SCLK)
- net CODEC_SDIN: now also R701.2, U701.17 (SDIN)
- net DACDAT: now also U701.10 (DACDAT)
- net GND: now also C701.2, C702.2, C703.2, C704.2, C705.2, J701.2, J702.2, J703.2, R706.2, R707.2, U701.12 (DGND), U701.24 (SPKGND), U701.28 (AGND), U701.33 (AGND)
- net HP_L: now also C707.1, U701.30 (LOUT1)
- net HP_R: now also C706.1, U701.29 (ROUT1)
- net LRC: now also U701.7 (LRC)
- net Line_In_L: now also C709.2, U701.3 (L2/GPIO2)
- net Line_In_R: now also C708.2, U701.6 (R2/GPIO3)
- net Line_Out_L: now also C711.2, U701.22 (OUT3)
- net Line_Out_R: now also C710.2, U701.21 (OUT4)
- net MCLK: now also U701.11 (MCLK)
- net SDRAM_3V3: now also C705.1, U701.27 (VMID)
- net at R703.2: now also U701.18 (MODE)
- new net: C707.2, J701.3
- new net: C706.2, J701.6
- new net: J703.6, R704.1
- new net: C710.1, R704.2, R707.1
- new net: C709.1, J702.3
- new net: C708.1, J702.6
- new net: C711.1, R705.2, R706.1
- new net: J703.3, R705.1
- no-connect marks 16 -> 19
Other:
- note added: "AVDD"
- note added: "DBVDD"
- note added: "DCVDD"
- note added: "SPKVDD"

Commit message: updates
Parts:
- removed R703: 10k, MY RESISTOR LIBRARY:0402WGF1002TCE, symbol MY RESISTOR LIBRARY:0603WAF1002T5E
- added R703: 10k, MY RESISTOR LIBRARY:0402WGF1002TCE, symbol MY RESISTOR LIBRARY:0402WGF1002TCE
Connections:
- net GND: now also R703.2
- net at U701.18 (MODE): now also R703.1
- net ADCDAT renamed I2S_ADCDAT
- net BCLK renamed I2S_BCLK
- net CODEC_SCLK renamed CODEC_SCL
- net CODEC_SDIN renamed CODEC_SDA
- net DACDAT renamed I2S_DACDAT
- net LRC renamed I2S_LRC
- net MCLK renamed I2S_MCLK
- net SDRAM_3V3 renamed VMID
Other:
- title: MIMXRT1064 MCU Module -> MIMXRT1064 Audio Board

Commit message: up
Parts:
- R704, R705: footprint MY RESISTOR LIBRARY:0805W8F1000T5E -> MY RESISTOR LIBRARY:0603WAF1000T5E
Changed lines of the file:
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@@
     (property "Reference" "R704" (id 0) (at 278.13 154.94 90))
     (property "Value" "100R" (id 1) (at 278.13 160.02 90))
-    (property "Footprint" "MY RESISTOR LIBRARY:0805W8F1000T5E" (id 2) (at 278.13 159.258 90)
+    (property "Footprint" "MY RESISTOR LIBRARY:0603WAF1000T5E" (id 2) (at 278.13 159.258 90)
       (effects (font (size 1.27 1.27)) hide)
     )
@@
     (property "Reference" "R705" (id 0) (at 278.13 162.56 90))
     (property "Value" "100R" (id 1) (at 278.13 167.64 90))
-    (property "Footprint" "MY RESISTOR LIBRARY:0805W8F1000T5E" (id 2) (at 278.13 166.878 90)
-      (effects (font (size 1.27 1.27)) hide)
-    )
+    (property "Footprint" "MY RESISTOR LIBRARY:0603WAF1000T5E" (id 2) (at 278.13 166.878 90)
+      (effects (font (size 1.27 1.27)) hide)
+    )

Commit message: updates
Parts:
- removed C708, C709: 1u, MY CAPACITOR LIBRARY:0402_CL05A105KA5NQNC, symbol MY CAPACITOR LIBRARY:CL05A105KA5NQNC
- removed J702: PJ-342B-TX-SMT, MY CONNECTOR LIBRARY:PJ-342B-TX-SMT, symbol MY CONNECTOR LIBRARY:PJ-342B-TX-SMT
- renumbered C710 to C708, C711 to C709, J703 to J701, J701 to J702
Connections:
- no-connect marks 19 -> 16
Other:
- moved on the sheet: C706, C707, C708, C709, J701, J702, R704, R705, R706, R707
