File: DESIGN FILES/mcu_power_crystals.kicad_sch (KiCad schematic)
At the start: 34 parts, among them U1 MIMXRT1064CVL5B, Y1 24MHz, Y2 32.768KHz

Commit message: Refactoring schematic
Parts:
- C1, C10, C11, C13, C14, C15, C16, C18, C19, C21, C24, C6, C7: value 220nF -> (none); footprint MIMXRT1064 MCU Module:0402_CL05B224KO5NNNC -> (none)
- C12, C17, C2, C20, C23: value 4.7uF -> (none); footprint MIMXRT1064 MCU Module:0402_CL05A475MP5NRNC -> (none)
- C22: value 10uF -> (none); footprint MIMXRT1064 MCU Module:0603_CL10A106KP8NNNC -> (none)
- C25: value 22uF -> (none); footprint MIMXRT1064 MCU Module:0603_CL10A226MQ8NRNC -> (none)
- C3, C4: value 12pF -> (none); footprint MIMXRT1064 MCU Module:0402_GRM1555C1H120GA01D -> (none)
- C5, C8: value 8pF -> (none); footprint MIMXRT1064 MCU Module:0402_GCM1555C1H8R0DA16D -> (none)
- C9: value 1uF -> (none); footprint MIMXRT1064 MCU Module:0402_CL05A105KA5NQNC -> (none)
- D1, D2: value RB521S30_R1_00001 -> (none)
- FB1: value 120R -> (none); footprint MIMXRT1064 MCU Module:0603_BLM18AG121SN1D -> (none)
- L1: value 4.7uH -> (none); footprint MIMXRT1064 MCU Module:CD32YP0302-4R7M -> (none)
- R1: value 2.2M -> (none); footprint MIMXRT1064 MCU Module:0402WGJ0225TCE -> (none)
- R2: value 30k -> (none); footprint MIMXRT1064 MCU Module:TC0225F3002TCE -> (none)
- U1: value MIMXRT1064CVL5B -> (none); footprint MIMXRT1064 MCU Module:MIMXRT1064CVL5B -> (none)
- Y1: value 24MHz -> (none); footprint MIMXRT1064 MCU Module:XL7EL89CMI-111YLC-24M -> (none)
- Y2: value 32.768KHz -> (none); footprint MIMXRT1064 MCU Module:X201232768KJD2SI -> (none)

Commit message: vcc check
Changed lines of the file:
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@@
     (stroke (width 0) (type default) (color 0 0 0 0))
   )
-  (wire (pts (xy 261.62 38.1) (xy 261.62 40.64))
+  (wire (pts (xy 269.24 38.1) (xy 269.24 40.64))
     (stroke (width 0) (type default) (color 0 0 0 0))
   )
@@
     (stroke (width 0) (type default) (color 0 0 0 0))
   )
-  (wire (pts (xy 259.08 40.64) (xy 261.62 40.64))
+  (wire (pts (xy 259.08 40.64) (xy 269.24 40.64))
     (stroke (width 0) (type default) (color 0 0 0 0))
   )
@@
   (symbol (lib_id "MIMXRT1064 MCU Module:BLM18AG121SN1D") (at 255.27 40.64 90) (unit 1)
     (in_bom yes) (on_board yes)
-    (property "Reference" "FB1" (id 0) (at 259.08 38.1 90))
+    (property "Reference" "FB1" (id 0) (at 260.35 38.1 90))
     (property "Value" "" (id 1) (at 251.46 38.1 90))
     (property "Footprint" "" (id 2) (at 257.048 40.64 90)
@@
     (pin "2")
   )
-  (symbol (lib_id "power:+3V3") (at 261.62 38.1 0) (unit 1)
+  (symbol (lib_id "power:+3V3") (at 269.24 38.1 0) (unit 1)
     (in_bom yes) (on_board yes)
-    (property "Reference" "#PWR019" (id 0) (at 261.62 41.91 0)
-      (effects (font (size 1.27 1.27)) hide)
-    )
-    (property "Value" "" (id 1) (at 261.62 34.29 0))
-    (property "Footprint" "" (id 2) (at 261.62 38.1 0)
-      (effects (font (size 1.27 1.27)) hide)
-    )
-    (property "Datasheet" "" (id 3) (at 261.62 38.1 0)
-      (effects (font (size 1.27 1.27)) hide)
-    )
+    (property "Reference" "#PWR019" (id 0) (at 269.24 41.91 0)
+      (effects (font (size 1.27 1.27)) hide)
+    )
+    (property "Value" "" (id 1) (at 269.24 34.29 0))
+    (property "Footprint" "" (id 2) (at 269.24 38.1 0)
+      (effects (font (size 1.27 1.27)) hide)
+    )
+    (property "Datasheet" "" (id 3) (at 269.24 38.1 0)
+      (effects (font (size 1.27 1.27)) hide)
+    )

Commit message: schematic and lib edit
Parts:
- D1, D2: footprint (none) -> MIMXRT1064 MCU Module:RB521S30_R1_00001
Changed lines of the file:
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@@
       (effects (font (size 1.27 1.27)) hide)
     )
-    (property "Footprint" "" (id 2) (at 85.09 142.875 0)
+    (property "Footprint" "MIMXRT1064 MCU Module:RB521S30_R1_00001" (id 2) (at 85.09 142.875 0)
       (effects (font (size 1.27 1.27)) hide)
     )
@@
       (effects (font (size 1.27 1.27)) hide)
     )
-    (property "Footprint" "" (id 2) (at 85.09 135.255 0)
-      (effects (font (size 1.27 1.27)) hide)
-    )
+    (property "Footprint" "MIMXRT1064 MCU Module:RB521S30_R1_00001" (id 2) (at 85.09 135.255 0)
+      (effects (font (size 1.27 1.27)) hide)
+    )

Commit message: work
Parts:
- C1, C10, C11, C13, C14, C15, C16, C18, C19, C21, C24, C6, C7: value (none) -> 220nF; footprint (none) -> MIMXRT1064 MCU Module:0402_CL05B224KO5NNNC
- C12, C17, C2, C20, C23: value (none) -> 4.7uF; footprint (none) -> MIMXRT1064 MCU Module:0402_CL05A475MP5NRNC
- C22: value (none) -> 10uF; footprint (none) -> MIMXRT1064 MCU Module:0603_CL10A106KP8NNNC
- C25: value (none) -> 22uF; footprint (none) -> MIMXRT1064 MCU Module:0603_CL10A226MQ8NRNC
- C3, C4: value (none) -> 12pF; footprint (none) -> MIMXRT1064 MCU Module:0402_GRM1555C1H120GA01D
- C5, C8: value (none) -> 8pF; footprint (none) -> MIMXRT1064 MCU Module:0402_GCM1555C1H8R0DA16D
- C9: value (none) -> 1uF; footprint (none) -> MIMXRT1064 MCU Module:0402_CL05A105KA5NQNC
- D1, D2: value (none) -> RB521S30_R1_00001
- FB1: value (none) -> 120R; footprint (none) -> MIMXRT1064 MCU Module:0603_BLM18AG121SN1D
- L1: value (none) -> 4.7uH; footprint (none) -> MIMXRT1064 MCU Module:CD32YP0302-4R7M
- R1: value (none) -> 2.2M; footprint (none) -> MIMXRT1064 MCU Module:0402WGJ0225TCE
- R2: value (none) -> 30k; footprint (none) -> MIMXRT1064 MCU Module:TC0225F3002TCE
- U1: value (none) -> MIMXRT1064CVL5B; footprint (none) -> MIMXRT1064 MCU Module:MIMXRT1064CVL5B
- Y1: value (none) -> 24MHz; footprint (none) -> MIMXRT1064 MCU Module:XL7EL89CMI-111YLC-24M
- Y2: value (none) -> 32.768KHz; footprint (none) -> MIMXRT1064 MCU Module:X201232768KJD2SI

Commit message: edits
Parts:
- FB1: value 120R -> BLM18AG121SN1D
- Y1: value 24MHz -> XL7EL89CMI-111YLC-24M
- Y2: value 32.768KHz -> X201232768KJD2SI
Connections:
- net GND: now also Y1.2 (GND); no longer Y1.GND (2)

Commit message: work
Other:
- note added: "3 : MCU POWER & CRYSTALS"
- company: (none) -> Soundsom
- title: Power -> MCU Power & Crystals
Changed lines of the file:
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@@
   (paper "A4")
   (title_block
-    (title "Power")
+    (title "MCU Power & Crystals")
     (date "2023-05-12")
     (rev "0")
+    (company "Soundsom")
   )
   (junction (at 184.15 129.54) (diameter 0) (color 0 0 0 0)
@@
     (effects (font (size 1.27 1.27) bold italic) (justify left bottom))
   )
+  (text "3 : MCU POWER & CRYSTALS" (at 168.91 22.86 0)
+    (effects (font (size 5 5) bold italic) (justify left bottom))
+  )
   (global_label "VDD_COIN_CELL" (shape input) (at 78.74 138.43 180) (fields_autoplaced)

Commit message: schematic edit
Parts:
- removed Y1: XL7EL89CMI-111YLC-24M, MIMXRT1064 MCU Module:XL7EL89CMI-111YLC-24M, symbol MIMXRT1064 MCU Module:XL7EL89CMI-111YLC-24M
- added Y?: 7V24000026, symbol MIMXRT1064 MCU Module:7V24000026
Connections:
- net GND: now also Y?.2 (GND), Y?.4 (GND)
- net at C3.1, R1.1, U1.P11 (XTALI): now also Y?.1
- net at C4.1, U1.N11 (XTALO): now also Y?.3
Changed lines of the file:
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@@
     (pin "2")
+  )
+  (symbol (lib_id "MIMXRT1064 MCU Module:7V24000026") (at 67.31 63.5 0) (unit 1)
+    (in_bom yes) (on_board yes) (fields_autoplaced)
+    (property "Reference" "Y?" (id 0) (at 67.31 54.61 0))
+    (property "Value" "7V24000026" (id 1) (at 67.31 57.15 0))
+    (property "Footprint" "" (id 2) (at 67.31 63.5 0)
+      (effects (font (size 1.27 1.27)) hide)
+    )
+    (property "Datasheet" "~" (id 3) (at 67.31 63.5 0)
+      (effects (font (size 1.27 1.27)) hide)
+    )
+    (pin "1")
+    (pin "2")
+    (pin "3")
+    (pin "4")
   )
   (symbol (lib_id "MIMXRT1064 MCU Module:CL05A475MP5NRNC") (at 208.28 130.81 0) (unit 1)
@@
     (pin "2")
   )
-  (symbol (lib_id "MIMXRT1064 MCU Module:XL7EL89CMI-111YLC-24M") (at 67.31 63.5 0) (unit 1)
-    (in_bom yes) (on_board yes) (fields_autoplaced)
-    (property "Reference" "Y1" (id 0) (at 67.31 54.61 0))
-    (property "Value" "XL7EL89CMI-111YLC-24M" (id 1) (at 67.31 57.15 0))
-    (property "Footprint" "MIMXRT1064 MCU Module:XL7EL89CMI-111YLC-24M" (id 2) (at 67.31 63.5 0)
-      (effects (font (size 1.27 1.27)) hide)
-    )
-    (property "Datasheet" "~" (id 3) (at 67.31 63.5 0)
-      (effects (font (size 1.27 1.27)) hide)
-    )
-    (pin "1")
-    (pin "2")
-    (pin "3")
-    (pin "4")
-  )
   (symbol (lib_id "power:GND") (at 64.77 38.1 0) (unit 1)

Commit message: crystals edit
Parts:
- removed Y?: 7V24000026, symbol MIMXRT1064 MCU Module:7V24000026
- added Y?: 7V24000026, symbol MIMXRT1064 MCU Module:7V24000026
Connections:
- net at C3.1, R1.1, U1.P11 (XTALI): now also Y?.1
- net at C4.1, U1.N11 (XTALO): now also Y?.3
Changed lines of the file:
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@@
   (junction (at 161.29 111.76) (diameter 0) (color 0 0 0 0)
   )
-  (junction (at 71.12 71.12) (diameter 0) (color 0 0 0 0)
-  )
   (junction (at 77.47 63.5) (diameter 0) (color 0 0 0 0)
   )
   (junction (at 93.98 74.93) (diameter 0) (color 0 0 0 0)
-  )
-  (junction (at 71.12 78.74) (diameter 0) (color 0 0 0 0)
   )
   (junction (at 196.85 142.24) (diameter 0) (color 0 0 0 0)
@@
     (stroke (width 0) (type default) (color 0 0 0 0))
   )
-  (wire (pts (xy 71.12 78.74) (xy 77.47 78.74))
+  (wire (pts (xy 57.15 78.74) (xy 77.47 78.74))
     (stroke (width 0) (type default) (color 0 0 0 0))
   )
@@
     (stroke (width 0) (type default) (color 0 0 0 0))
   )
-  (wire (pts (xy 71.12 71.12) (xy 71.12 78.74))
-    (stroke (width 0) (type default) (color 0 0 0 0))
-  )
   (wire (pts (xy 158.75 101.6) (xy 161.29 101.6))
     (stroke (width 0) (type default) (color 0 0 0 0))
@@
     (stroke (width 0) (type default) (color 0 0 0 0))
   )
-  (wire (pts (xy 63.5 68.58) (xy 63.5 71.12))
-    (stroke (width 0) (type default) (color 0 0 0 0))
-  )
   (wire (pts (xy 173.99 48.26) (xy 176.53 48.26))
     (stroke (width 0) (type default) (color 0 0 0 0))
@@
     (stroke (width 0) (type default) (color 0 0 0 0))
   )
-  (wire (pts (xy 71.12 68.58) (xy 71.12 71.12))
-    (stroke (width 0) (type default) (color 0 0 0 0))
-  )
   (wire (pts (xy 240.03 109.22) (xy 240.03 111.76))
     (stroke (width 0) (type default) (color 0 0 0 0))
@@
     (stroke (width 0) (type default) (color 0 0 0 0))
   )
-  (wire (pts (xy 63.5 71.12) (xy 71.12 71.12))
-    (stroke (width 0) (type default) (color 0 0 0 0))
-  )
   (wire (pts (xy 208.28 124.46) (xy 220.98 124.46))
     (stroke (width 0) (type default) (color 0 0 0 0))
@@
   )
   (wire (pts (xy 74.93 63.5) (xy 77.47 63.5))
-    (stroke (width 0) (type default) (color 0 0 0 0))
-  )
-  (wire (pts (xy 57.15 78.74) (xy 71.12 78.74))
     (stroke (width 0) (type default) (color 0 0 0 0))
   )
@@
     (pin "2")
   )
-  (symbol (lib_id "MIMXRT1064 MCU Module:7V24000026") (at 67.31 63.5 0) (unit 1)
-    (in_bom yes) (on_board yes) (fields_autoplaced)
-    (property "Reference" "Y?" (id 0) (at 67.31 54.61 0))
-    (property "Value" "7V24000026" (id 1) (at 67.31 57.15 0))
-    (property "Footprint" "" (id 2) (at 67.31 63.5 0)
-      (effects (font (size 1.27 1.27)) hide)
-    )
-    (property "Datasheet" "~" (id 3) (at 67.31 63.5 0)
-      (effects (font (size 1.27 1.27)) hide)
-    )
-    (pin "1")
-    (pin "2")
-    (pin "3")
-    (pin "4")
-  )
   (symbol (lib_id "MIMXRT1064 MCU Module:CL05A475MP5NRNC") (at 208.28 130.81 0) (unit 1)
     (in_bom yes) (on_board yes) (fields_autoplaced)
@@
     (pin "2")
   )
+  (symbol (lib_id "MIMXRT1064 MCU Module:7V24000026") (at 67.31 63.5 0) (unit 1)
+    (in_bom yes) (on_board yes) (fields_autoplaced)
+    (property "Reference" "Y?" (id 0) (at 67.31 54.61 0))
+    (property "Value" "7V24000026" (id 1) (at 67.31 57.15 0))
+    (property "Footprint" "" (id 2) (at 67.31 63.5 0)
+      (effects (font (size 1.27 1.27)) hide)
+    )
+    (property "Datasheet" "~" (id 3) (at 67.31 63.5 0)
+      (effects (font (size 1.27 1.27)) hide)
+    )
+    (pin "1")
+    (pin "2")
+    (pin "3")
+    (pin "4")
+  )
   (symbol (lib_id "power:GND") (at 196.85 144.78 0) (unit 1)
