File: DESIGN FILES/mcu_power_crystals.kicad_sch (KiCad schematic)
At the start: 34 parts, among them U1 MIMXRT1064CVL5B, Y2 X201232768KJD2SI

Commit message: schematic edit
Parts:
- FB1: value BLM18AG121SN1D -> 120R
- Y1: renamed from Y?; footprint (none) -> MIMXRT1064 MCU Module:7V24000026
Connections:
- net POR_B: now reaches U1.M7 (POR_B)
Other:
- note removed: "Normalement c'est 30k"
- note removed: "Suivi Paul"
- moved on the sheet: FB1, R2
Changed lines of the file:
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@@
   (junction (at 161.29 106.68) (diameter 0) (color 0 0 0 0)
   )
-  (junction (at 201.93 40.64) (diameter 0) (color 0 0 0 0)
-  )
   (junction (at 114.3 151.13) (diameter 0) (color 0 0 0 0)
   )
   (junction (at 161.29 146.05) (diameter 0) (color 0 0 0 0)
+  )
+  (junction (at 189.23 40.64) (diameter 0) (color 0 0 0 0)
   )
   (junction (at 114.3 148.59) (diameter 0) (color 0 0 0 0)
@@
     (stroke (width 0) (type default) (color 0 0 0 0))
   )
-  (wire (pts (xy 201.93 40.64) (xy 224.79 40.64))
+  (wire (pts (xy 162.56 40.64) (xy 189.23 40.64))
     (stroke (width 0) (type default) (color 0 0 0 0))
   )
@@
     (stroke (width 0) (type default) (color 0 0 0 0))
   )
+  (wire (pts (xy 189.23 40.64) (xy 224.79 40.64))
+    (stroke (width 0) (type default) (color 0 0 0 0))
+  )
   (wire (pts (xy 196.85 142.24) (xy 196.85 139.7))
     (stroke (width 0) (type default) (color 0 0 0 0))
@@
     (stroke (width 0) (type default) (color 0 0 0 0))
   )
-  (wire (pts (xy 259.08 40.64) (xy 269.24 40.64))
+  (wire (pts (xy 265.43 40.64) (xy 269.24 40.64))
     (stroke (width 0) (type default) (color 0 0 0 0))
   )
@@
     (stroke (width 0) (type default) (color 0 0 0 0))
   )
-  (wire (pts (xy 248.92 40.64) (xy 251.46 40.64))
+  (wire (pts (xy 248.92 40.64) (xy 257.81 40.64))
     (stroke (width 0) (type default) (color 0 0 0 0))
   )
@@
     (stroke (width 0) (type default) (color 0 0 0 0))
   )
+  (wire (pts (xy 104.14 30.48) (xy 116.84 30.48))
+    (stroke (width 0) (type default) (color 0 0 0 0))
+  )
   (wire (pts (xy 161.29 153.67) (xy 161.29 156.21))
     (stroke (width 0) (type default) (color 0 0 0 0))
@@
     (stroke (width 0) (type default) (color 0 0 0 0))
   )
-  (wire (pts (xy 189.23 55.88) (xy 191.77 55.88))
+  (wire (pts (xy 189.23 55.88) (xy 189.23 53.34))
     (stroke (width 0) (type default) (color 0 0 0 0))
   )
@@
     (stroke (width 0) (type default) (color 0 0 0 0))
   )
-  (wire (pts (xy 199.39 55.88) (xy 201.93 55.88))
+  (wire (pts (xy 189.23 40.64) (xy 189.23 45.72))
     (stroke (width 0) (type default) (color 0 0 0 0))
   )
@@
     (stroke (width 0) (type default) (color 0 0 0 0))
   )
-  (wire (pts (xy 201.93 40.64) (xy 201.93 55.88))
-    (stroke (width 0) (type default) (color 0 0 0 0))
-  )
   (wire (pts (xy 104.14 40.64) (xy 116.84 40.64))
     (stroke (width 0) (type default) (color 0 0 0 0))
@@
     (stroke (width 0) (type default) (color 0 0 0 0))
   )
-  (wire (pts (xy 162.56 40.64) (xy 201.93 40.64))
-    (stroke (width 0) (type default) (color 0 0 0 0))
-  )
   (wire (pts (xy 114.3 158.75) (xy 116.84 158.75))
     (stroke (width 0) (type default) (color 0 0 0 0))
@@
   (wire (pts (xy 116.84 163.83) (xy 114.3 163.83))
     (stroke (width 0) (type default) (color 0 0 0 0))
-  )
-  (text "Normalement c'est 30k" (at 191.77 59.69 0)
-    (effects (font (size 1.27 1.27) bold italic) (justify left bottom))
-  )
-  (text "Suivi Paul" (at 257.81 44.45 0)
-    (effects (font (size 1.27 1.27) bold italic) (justify left bottom))
   )
   (text "3 : MCU POWER & CRYSTALS" (at 168.91 22.86 0)
@@
     (effects (font (size 1.27 1.27) bold italic) (justify right))
     (property "Intersheet References" "${INTERSHEET_REFS}" (id 0) (at 88.339 43.053 0)
+      (effects (font (size 1.27 1.27) bold italic) (justify right) hide)
+    )
+  )
+  (global_label "POR_B" (shape input) (at 104.14 30.48 180) (fields_autoplaced)
+    (effects (font (size 1.27 1.27) bold italic) (justify right))
+    (property "Intersheet References" "${INTERSHEET_REFS}" (id 0) (at 95.1728 30.607 0)
       (effects (font (size 1.27 1.27) bold italic) (justify right) hide)
     )
@@
     (pin "1")
   )
-  (symbol (lib_id "MIMXRT1064 MCU Module:TC0225F3002TCE") (at 195.58 55.88 90) (unit 1)
-    (in_bom yes) (on_board yes) (fields_autoplaced)
-    (property "Reference" "R2" (id 0) (at 195.58 49.53 90))
-    (property "Value" "30k" (id 1) (at 195.58 52.07 90))
-    (property "Footprint" "MIMXRT1064 MCU Module:TC0225F3002TCE" (id 2) (at 195.58 57.658 90)
-      (effects (font (size 1.27 1.27)) hide)
-    )
-    (property "Datasheet" "~" (id 3) (at 195.58 55.88 0)
+  (symbol (lib_id "MIMXRT1064 MCU Module:TC0225F3002TCE") (at 189.23 49.53 180) (unit 1)
+    (in_bom yes) (on_board yes)
+    (property "Reference" "R2" (id 0) (at 193.04 48.26 0))
+    (property "Value" "30k" (id 1) (at 193.04 50.8 0))
+    (property "Footprint" "MIMXRT1064 MCU Module:TC0225F3002TCE" (id 2) (at 191.008 49.53 90)
+      (effects (font (size 1.27 1.27)) hide)
+    )
+    (property "Datasheet" "~" (id 3) (at 189.23 49.53 0)
       (effects (font (size 1.27 1.27)) hide)
     )
@@
     (pin "2")
   )
-  (symbol (lib_id "MIMXRT1064 MCU Module:BLM18AG121SN1D") (at 255.27 40.64 90) (unit 1)
-    (in_bom yes) (on_board yes) (fields_autoplaced)
-    (property "Reference" "FB1" (id 0) (at 255.2192 35.56 90))
-    (property "Value" "BLM18AG121SN1D" (id 1) (at 250.19 40.6908 90)
-      (effects (font (size 1.27 1.27)) hide)
-    )
-    (property "Footprint" "MIMXRT1064 MCU Module:0603_BLM18AG121SN1D" (id 2) (at 257.048 40.64 90)
-      (effects (font (size 1.27 1.27)) hide)
-    )
-    (property "Datasheet" "~" (id 3) (at 255.27 40.64 0)
+  (symbol (lib_id "MIMXRT1064 MCU Module:BLM18AG121SN1D") (at 261.62 40.64 90) (unit 1)
+    (in_bom yes) (on_board yes)
+    (property "Reference" "FB1" (id 0) (at 261.5692 35.56 90))
+    (property "Value" "120R" (id 1) (at 261.62 45.72 90))
+    (property "Footprint" "MIMXRT1064 MCU Module:0603_BLM18AG121SN1D" (id 2) (at 263.398 40.64 90)
+      (effects (font (size 1.27 1.27)) hide)
+    )
+    (property "Datasheet" "~" (id 3) (at 261.62 40.64 0)
       (effects (font (size 1.27 1.27)) hide)
     )
@@
   (symbol (lib_id "MIMXRT1064 MCU Module:7V24000026") (at 67.31 63.5 0) (unit 1)
     (in_bom yes) (on_board yes) (fields_autoplaced)
-    (property "Reference" "Y?" (id 0) (at 67.31 54.61 0))
+    (property "Reference" "Y1" (id 0) (at 67.31 54.61 0))
     (property "Value" "7V24000026" (id 1) (at 67.31 57.15 0))
-    (property "Footprint" "" (id 2) (at 67.31 63.5 0)
-      (effects (font (size 1.27 1.27)) hide)
-    )
+    (property "Footprint" "MIMXRT1064 MCU Module:7V24000026" (id 2) (at 67.31 63.5 0)
+      (effects (font (size 1.27 1.27)) hide)
+    )
