File: DESIGN FILES/mcu_pinout.kicad_sch (KiCad schematic)
At the start: 16 parts, among them U1 MIMXRT1064CVL5B

Commit message: Adding voltage monitor and manual reset circuit
Parts:
- renumbered C34 to C35, C35 to C36, C36 to C37, C37 to C38, C38 to C39, C39 to C40, C40 to C41, C41 to C42, C42 to C43, C43 to C44, C44 to C45, C45 to C46, C46 to C47, C47 to C48, C48 to C49
Changed lines of the file:
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@@
   (symbol (lib_id "MIMXRT1064 MCU Module:CL05B104KB54PNC") (at 262.89 152.4 0) (unit 1)
     (in_bom yes) (on_board yes) (fields_autoplaced)
-    (property "Reference" "C47" (id 0) (at 266.7 151.1299 0)
+    (property "Reference" "C48" (id 0) (at 266.7 151.1299 0)
       (effects (font (size 1.27 1.27)) (justify left))
     )
@@
   (symbol (lib_id "MIMXRT1064 MCU Module:CL05B104KB54PNC") (at 35.56 170.18 0) (unit 1)
     (in_bom yes) (on_board yes) (fields_autoplaced)
-    (property "Reference" "C38" (id 0) (at 39.37 168.9099 0)
+    (property "Reference" "C39" (id 0) (at 39.37 168.9099 0)
       (effects (font (size 1.27 1.27)) (justify left))
     )
@@
   (symbol (lib_id "MIMXRT1064 MCU Module:CL05A475MP5NRNC") (at 33.02 151.13 0) (unit 1)
     (in_bom yes) (on_board yes) (fields_autoplaced)
-    (property "Reference" "C37" (id 0) (at 36.83 149.8599 0)
+    (property "Reference" "C38" (id 0) (at 36.83 149.8599 0)
       (effects (font (size 1.27 1.27)) (justify left))
     )
@@
   (symbol (lib_id "MIMXRT1064 MCU Module:CL05A475MP5NRNC") (at 16.51 31.75 0) (unit 1)
     (in_bom yes) (on_board yes) (fields_autoplaced)
-    (property "Reference" "C34" (id 0) (at 20.32 30.4799 0)
+    (property "Reference" "C35" (id 0) (at 20.32 30.4799 0)
       (effects (font (size 1.27 1.27)) (justify left))
     )
@@
   (symbol (lib_id "MIMXRT1064 MCU Module:CL05B104KB54PNC") (at 152.4 30.48 0) (unit 1)
     (in_bom yes) (on_board yes) (fields_autoplaced)
-    (property "Reference" "C43" (id 0) (at 156.21 29.2099 0)
+    (property "Reference" "C44" (id 0) (at 156.21 29.2099 0)
       (effects (font (size 1.27 1.27)) (justify left))
     )
@@
   (symbol (lib_id "MIMXRT1064 MCU Module:CL05B104KB54PNC") (at 177.8 30.48 0) (unit 1)
     (in_bom yes) (on_board yes) (fields_autoplaced)
-    (property "Reference" "C46" (id 0) (at 181.61 29.2099 0)
+    (property "Reference" "C47" (id 0) (at 181.61 29.2099 0)
       (effects (font (size 1.27 1.27)) (justify left))
     )
@@
   (symbol (lib_id "MIMXRT1064 MCU Module:CL05A475MP5NRNC") (at 140.97 30.48 0) (unit 1)
     (in_bom yes) (on_board yes) (fields_autoplaced)
-    (property "Reference" "C41" (id 0) (at 144.78 29.2099 0)
+    (property "Reference" "C42" (id 0) (at 144.78 29.2099 0)
       (effects (font (size 1.27 1.27)) (justify left))
     )
@@
   (symbol (lib_id "MIMXRT1064 MCU Module:CL10A106KP8NNNC") (at 275.59 152.4 0) (unit 1)
     (in_bom yes) (on_board yes) (fields_autoplaced)
-    (property "Reference" "C48" (id 0) (at 279.4 151.1299 0)
+    (property "Reference" "C49" (id 0) (at 279.4 151.1299 0)
       (effects (font (size 1.27 1.27)) (justify left))
     )
@@
   (symbol (lib_id "MIMXRT1064 MCU Module:CL05A105KA5NQNC") (at 168.91 156.21 0) (unit 1)
     (in_bom yes) (on_board yes) (fields_autoplaced)
-    (property "Reference" "C45" (id 0) (at 172.72 154.9399 0)
+    (property "Reference" "C46" (id 0) (at 172.72 154.9399 0)
       (effects (font (size 1.27 1.27)) (justify left))
     )
@@
   (symbol (lib_id "MIMXRT1064 MCU Module:CL05B104KB54PNC") (at 20.32 151.13 0) (unit 1)
     (in_bom yes) (on_board yes) (fields_autoplaced)
-    (property "Reference" "C35" (id 0) (at 24.13 149.8599 0)
+    (property "Reference" "C36" (id 0) (at 24.13 149.8599 0)
       (effects (font (size 1.27 1.27)) (justify left))
     )
@@
   (symbol (lib_id "MIMXRT1064 MCU Module:CL05B104KB54PNC") (at 40.64 31.75 0) (unit 1)
     (in_bom yes) (on_board yes) (fields_autoplaced)
-    (property "Reference" "C39" (id 0) (at 44.45 30.4799 0)
+    (property "Reference" "C40" (id 0) (at 44.45 30.4799 0)
       (effects (font (size 1.27 1.27)) (justify left))
     )
@@
   (symbol (lib_id "MIMXRT1064 MCU Module:CL05B104KB54PNC") (at 27.94 31.75 0) (unit 1)
     (in_bom yes) (on_board yes) (fields_autoplaced)
-    (property "Reference" "C36" (id 0) (at 31.75 30.4799 0)
+    (property "Reference" "C37" (id 0) (at 31.75 30.4799 0)
       (effects (font (size 1.27 1.27)) (justify left))
     )
@@
   (symbol (lib_id "MIMXRT1064 MCU Module:CL05A105KA5NQNC") (at 143.51 146.05 0) (unit 1)
     (in_bom yes) (on_board yes) (fields_autoplaced)
-    (property "Reference" "C42" (id 0) (at 147.32 144.7799 0)
+    (property "Reference" "C43" (id 0) (at 147.32 144.7799 0)
       (effects (font (size 1.27 1.27)) (justify left))
     )
@@
   (symbol (lib_id "MIMXRT1064 MCU Module:CL05A475MP5NRNC") (at 48.26 170.18 0) (unit 1)
     (in_bom yes) (on_board yes) (fields_autoplaced)
-    (property "Reference" "C40" (id 0) (at 52.07 168.9099 0)
+    (property "Reference" "C41" (id 0) (at 52.07 168.9099 0)
       (effects (font (size 1.27 1.27)) (justify left))
     )
@@
   (symbol (lib_id "MIMXRT1064 MCU Module:CL05B104KB54PNC") (at 165.1 30.48 0) (unit 1)
     (in_bom yes) (on_board yes) (fields_autoplaced)
-    (property "Reference" "C44" (id 0) (at 168.91 29.2099 0)
-      (effects (font (size 1.27 1.27)) (justify left))
-    )
+    (property "Reference" "C45" (id 0) (at 168.91 29.2099 0)
+      (effects (font (size 1.27 1.27)) (justify left))
+    )

Commit message: Refactoring schematic
Parts:
- renumbered C35 to C26, C36 to C27, C37 to C28, C38 to C29, C39 to C30, C40 to C31, C41 to C32, C42 to C33, C43 to C34, C44 to C35, C45 to C36, C46 to C37, C47 to C38, C48 to C39, C49 to C40
Other:
- note added: "MCU GPIO"
- note added: "QSPI FLASH"
- note added: "SD CARD"
- note added: "SDRAM"
- note added: "USB"
- moved on the sheet: C26, C28, C31, C33, C34, C35, C36, C37, C38, C39, C40, U1C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

Commit message: schematic and lib edit
Parts:
- renumbered C35 to C34, C34 to C35, C38 to C37, C37 to C38
Changed lines of the file:
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@@
   (symbol (lib_id "MIMXRT1064 MCU Module:CL05B104KB54PNC") (at 154.94 30.48 0) (unit 1)
     (in_bom yes) (on_board yes) (fields_autoplaced)
-    (property "Reference" "C35" (id 0) (at 158.75 29.2099 0)
+    (property "Reference" "C34" (id 0) (at 158.75 29.2099 0)
       (effects (font (size 1.27 1.27)) (justify left))
     )
@@
   (symbol (lib_id "MIMXRT1064 MCU Module:CL05B104KB54PNC") (at 180.34 30.48 0) (unit 1)
     (in_bom yes) (on_board yes) (fields_autoplaced)
-    (property "Reference" "C38" (id 0) (at 184.15 29.2099 0)
+    (property "Reference" "C37" (id 0) (at 184.15 29.2099 0)
       (effects (font (size 1.27 1.27)) (justify left))
     )
@@
   (symbol (lib_id "MIMXRT1064 MCU Module:CL05A105KA5NQNC") (at 182.88 152.4 0) (unit 1)
     (in_bom yes) (on_board yes)
-    (property "Reference" "C37" (id 0) (at 185.42 151.13 0)
+    (property "Reference" "C38" (id 0) (at 185.42 151.13 0)
       (effects (font (size 1.27 1.27)) (justify left))
     )
@@
   (symbol (lib_id "MIMXRT1064 MCU Module:CL05A105KA5NQNC") (at 166.37 143.51 0) (unit 1)
     (in_bom yes) (on_board yes) (fields_autoplaced)
-    (property "Reference" "C34" (id 0) (at 170.18 142.2399 0)
-      (effects (font (size 1.27 1.27)) (justify left))
-    )
+    (property "Reference" "C35" (id 0) (at 170.18 142.2399 0)
+      (effects (font (size 1.27 1.27)) (justify left))
+    )

Commit message: work
Parts:
- removed C35, C38: 1uF, MIMXRT1064 MCU Module:0402_CL05A105KA5NQNC, symbol MIMXRT1064 MCU Module:CL05A105KA5NQNC
- removed C39: 100nF, MIMXRT1064 MCU Module:0402_CL05B104KB54PNC, symbol MIMXRT1064 MCU Module:CL05B104KB54PNC
- removed C40: 10uF, MIMXRT1064 MCU Module:0603_CL10A106KP8NNNC, symbol MIMXRT1064 MCU Module:CL10A106KP8NNNC
- removed unit 3 of U1
Other:
- note added: "4 : MCU GPIO & MEMORY SIGNALS"
- note removed: "USB"
- company: (none) -> Soundsom
- title: (none) -> MCU GPIO & Memory signals
- moved on the sheet: C33, C34, C36, C37, U1E

Commit message: schematic edit
Connections:
- net GPIO_AD_B0_06 renamed JTAG_TMS
- net GPIO_AD_B0_07 renamed JTAG_TCK
- net GPIO_AD_B0_09 renamed JTAG_TDI
- net GPIO_AD_B0_10 renamed JTAG_TDO
- net GPIO_AD_B0_11 renamed JTAG_nTRST
Changed lines of the file:
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@@
     )
   )
-  (global_label "GPIO_AD_B0_06" (shape input) (at 189.23 92.71 180) (fields_autoplaced)
-    (effects (font (size 1.27 1.27) bold italic) (justify right))
-    (property "Intersheet References" "${INTERSHEET_REFS}" (id 0) (at 171.7357 92.583 0)
+  (global_label "JTAG_TMS" (shape input) (at 189.23 92.71 180) (fields_autoplaced)
+    (effects (font (size 1.27 1.27) bold italic) (justify right))
+    (property "Intersheet References" "${INTERSHEET_REFS}" (id 0) (at 177.4809 92.583 0)
       (effects (font (size 1.27 1.27) bold italic) (justify right) hide)
     )
@@
     )
   )
-  (global_label "GPIO_AD_B0_09" (shape input) (at 189.23 100.33 180) (fields_autoplaced)
-    (effects (font (size 1.27 1.27) bold italic) (justify right))
-    (property "Intersheet References" "${INTERSHEET_REFS}" (id 0) (at 171.7357 100.203 0)
+  (global_label "JTAG_TDI" (shape input) (at 189.23 100.33 180) (fields_autoplaced)
+    (effects (font (size 1.27 1.27) bold italic) (justify right))
+    (property "Intersheet References" "${INTERSHEET_REFS}" (id 0) (at 178.2671 100.203 0)
       (effects (font (size 1.27 1.27) bold italic) (justify right) hide)
     )
@@
     )
   )
-  (global_label "GPIO_AD_B0_10" (shape input) (at 189.23 102.87 180) (fields_autoplaced)
-    (effects (font (size 1.27 1.27) bold italic) (justify right))
-    (property "Intersheet References" "${INTERSHEET_REFS}" (id 0) (at 171.7357 102.743 0)
+  (global_label "JTAG_TDO" (shape input) (at 189.23 102.87 180) (fields_autoplaced)
+    (effects (font (size 1.27 1.27) bold italic) (justify right))
+    (property "Intersheet References" "${INTERSHEET_REFS}" (id 0) (at 177.5414 102.743 0)
       (effects (font (size 1.27 1.27) bold italic) (justify right) hide)
     )
@@
     )
   )
-  (global_label "GPIO_AD_B0_11" (shape input) (at 189.23 105.41 180) (fields_autoplaced)
-    (effects (font (size 1.27 1.27) bold italic) (justify right))
-    (property "Intersheet References" "${INTERSHEET_REFS}" (id 0) (at 171.7357 105.283 0)
+  (global_label "JTAG_nTRST" (shape input) (at 189.23 105.41 180) (fields_autoplaced)
+    (effects (font (size 1.27 1.27) bold italic) (justify right))
+    (property "Intersheet References" "${INTERSHEET_REFS}" (id 0) (at 175.5457 105.283 0)
       (effects (font (size 1.27 1.27) bold italic) (justify right) hide)
     )
@@
     )
   )
-  (global_label "GPIO_AD_B0_07" (shape input) (at 189.23 95.25 180) (fields_autoplaced)
-    (effects (font (size 1.27 1.27) bold italic) (justify right))
-    (property "Intersheet References" "${INTERSHEET_REFS}" (id 0) (at 171.7357 95.123 0)
-      (effects (font (size 1.27 1.27) bold italic) (justify right) hide)
-    )
+  (global_label "JTAG_TCK" (shape input) (at 189.23 95.25 180) (fields_autoplaced)
+    (effects (font (size 1.27 1.27) bold italic) (justify right))
+    (property "Intersheet References" "${INTERSHEET_REFS}" (id 0) (at 177.6019 95.123 0)
+      (effects (font (size 1.27 1.27) bold italic) (justify right) hide)
+    )

Commit message: schematic edit
Parts:
- renumbered C36 to C35, C37 to C36
Changed lines of the file:
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@@
   (symbol (lib_id "MIMXRT1064 MCU Module:CL05B104KB54PNC") (at 182.88 66.04 0) (unit 1)
     (in_bom yes) (on_board yes) (fields_autoplaced)
-    (property "Reference" "C37" (id 0) (at 186.69 64.7699 0)
+    (property "Reference" "C36" (id 0) (at 186.69 64.7699 0)
       (effects (font (size 1.27 1.27)) (justify left))
     )
@@
   (symbol (lib_id "MIMXRT1064 MCU Module:CL05B104KB54PNC") (at 170.18 66.04 0) (unit 1)
     (in_bom yes) (on_board yes) (fields_autoplaced)
-    (property "Reference" "C36" (id 0) (at 173.99 64.7699 0)
+    (property "Reference" "C35" (id 0) (at 173.99 64.7699 0)
       (effects (font (size 1.27 1.27)) (justify left))
     )
