File: DESIGN FILES/memory_usb.kicad_sch (KiCad schematic)
At the start: 29 parts, among them J1 TF-15x15, Q1 IRLML6401, U2 IS42S16160J-6BLI, U3 IS25WP064A-JBLE

Commit message: work
Parts:
- C41, C54: value 22uF -> (none); footprint MIMXRT1064 MCU Module:0603_CL10A226MQ8NRNC -> (none)
- C42, C55: value 4.7uF -> (none); footprint MIMXRT1064 MCU Module:0402_CL05A475MP5NRNC -> (none)
- C43, C44, C46, C47, C48, C49, C50, C51, C56, C?: value 100nF -> (none); footprint MIMXRT1064 MCU Module:0402_CL05B104KB54PNC -> (none)
- C45, C52, C53, C? (x2): value 1uF -> (none); footprint MIMXRT1064 MCU Module:0402_CL05A105KA5NQNC -> (none)
- C?: value 10uF -> (none); footprint MIMXRT1064 MCU Module:0603_CL10A106KP8NNNC -> (none)
- FB2: value BLM18AG121SN1D -> (none); footprint MIMXRT1064 MCU Module:0603_BLM18AG121SN1D -> (none)
- J1: value TF-15x15 -> (none); footprint MIMXRT1064 MCU Module:TF-15x15_smd -> (none)
- Q1: value IRLML6401 -> (none); footprint MIMXRT1064 MCU Module:IRLML6401 -> (none)
- R3, R4, R5: value 10k -> (none); footprint MIMXRT1064 MCU Module:0402WGF1002TCE -> (none)
- U2: value IS42S16160J-6BLI -> (none); footprint MIMXRT1064 MCU Module:IS42S16160J-6BLI -> (none)
- U3: value IS25WP064A-JBLE -> (none); footprint MIMXRT1064 MCU Module:IS25WP064A-JBLE -> (none)
- U?: value MIMXRT1064CVL5B -> (none); footprint MIMXRT1064 MCU Module:MIMXRT1064CVL5B -> (none)
Other:
- note added: "5 : MEMORY & USB"
- title: Memory -> Memory & USB
- moved on the sheet: C41, C42, C43, C44, C45, C46, C47, C48, C49, C50, C51, C52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

Commit message: removing SY8089AAAC from library
Parts:
- C41, C54: value (none) -> 22uF; footprint (none) -> MIMXRT1064 MCU Module:0603_CL10A226MQ8NRNC
- C42, C55: value (none) -> 4.7uF; footprint (none) -> MIMXRT1064 MCU Module:0402_CL05A475MP5NRNC
- C43, C44, C46, C47, C48, C49, C50, C51, C56, C?: value (none) -> 100nF; footprint (none) -> MIMXRT1064 MCU Module:0402_CL05B104KB54PNC
- C45, C52, C53, C? (x2): value (none) -> 1uF; footprint (none) -> MIMXRT1064 MCU Module:0402_CL05A105KA5NQNC
- C?: value (none) -> 10uF; footprint (none) -> MIMXRT1064 MCU Module:0603_CL10A106KP8NNNC
- FB2: value (none) -> BLM18AG121SN1D; footprint (none) -> MIMXRT1064 MCU Module:0603_BLM18AG121SN1D
- J1: value (none) -> TF-15x15; footprint (none) -> MIMXRT1064 MCU Module:TF-15x15_smd
- Q1: value (none) -> IRLML6401; footprint (none) -> MIMXRT1064 MCU Module:IRLML6401
- R3, R4, R5: value (none) -> 10k; footprint (none) -> MIMXRT1064 MCU Module:0402WGF1002TCE
- U2: value (none) -> IS42S16160J-6BLI; footprint (none) -> MIMXRT1064 MCU Module:IS42S16160J-6BLI
- U3: value (none) -> IS25WP064A-JBLE; footprint (none) -> MIMXRT1064 MCU Module:IS25WP064A-JBLE
- U?: value (none) -> MIMXRT1064CVL5B; footprint (none) -> MIMXRT1064 MCU Module:MIMXRT1064CVL5B

Commit message: schematic edit
Parts:
- gave numbers to parts that had none: 5
- renumbered C41 to C37, C42 to C39, C43 to C41, C44 to C42, C46 to C43, C48 to C44, C49 to C45, C50 to C46, C51 to C48, C52 to C50, C53 to C51, C45 to C52, C47 to C53, R4 to R3, R3 to R4, U3 to U4
