File: DESIGN FILES/pwrpin_crystals.kicad_sch (KiCad schematic)
At the start: 34 parts, among them U1 MIMXRT1064CVL5B, Y401 7V24000026, Y402 Q13FC1350000200

Commit message: changes and adding schematic pdf
Parts:
- removed D401, D402: RB521S30_R1_00001, MIMXRT1064 MCU Module:RB521S30_R1_00001, symbol MIMXRT1064 MCU Module:RB521S30_R1_00001
Other:
- company: Soundsom -> Joël Ucedo
- title: MCU GPIO & Memory signals -> MIMXRT1064 MCU Module
Changed lines of the file:
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@@
   (paper "A3")
   (title_block
-    (title "MCU GPIO & Memory signals")
-    (date "2023-05-19")
+    (title "MIMXRT1064 MCU Module")
+    (date "2023-05-23")
     (rev "0")
-    (company "Soundsom")
+    (company "Joël Ucedo")
   )
   (junction (at 215.9 175.26) (diameter 0) (color 0 0 0 0)
@@
   (junction (at 168.91 212.09) (diameter 0) (color 0 0 0 0)
   )
-  (junction (at 153.67 203.2) (diameter 0) (color 0 0 0 0)
-  )
   (junction (at 168.91 232.41) (diameter 0) (color 0 0 0 0)
   )
@@
   )
   (junction (at 257.81 78.74) (diameter 0) (color 0 0 0 0)
-  )
-  (junction (at 146.05 203.2) (diameter 0) (color 0 0 0 0)
   )
   (junction (at 231.14 167.64) (diameter 0) (color 0 0 0 0)
@@
     (stroke (width 0) (type default) (color 0 0 0 0))
   )
-  (wire (pts (xy 143.51 207.01) (xy 146.05 207.01))
-    (stroke (width 0) (type default) (color 0 0 0 0))
-  )
   (wire (pts (xy 294.64 167.64) (xy 307.34 167.64))
     (stroke (width 0) (type default) (color 0 0 0 0))
@@
     (stroke (width 0) (type default) (color 0 0 0 0))
   )
-  (wire (pts (xy 146.05 203.2) (xy 153.67 203.2))
-    (stroke (width 0) (type default) (color 0 0 0 0))
-  )
   (wire (pts (xy 270.51 78.74) (xy 257.81 78.74))
     (stroke (width 0) (type default) (color 0 0 0 0))
@@
     (stroke (width 0) (type default) (color 0 0 0 0))
   )
-  (wire (pts (xy 146.05 203.2) (xy 146.05 207.01))
-    (stroke (width 0) (type default) (color 0 0 0 0))
-  )
   (wire (pts (xy 213.36 180.34) (xy 215.9 180.34))
     (stroke (width 0) (type default) (color 0 0 0 0))
@@
     (stroke (width 0) (type default) (color 0 0 0 0))
   )
-  (wire (pts (xy 146.05 199.39) (xy 143.51 199.39))
-    (stroke (width 0) (type default) (color 0 0 0 0))
-  )
   (wire (pts (xy 231.14 96.52) (xy 231.14 86.36))
     (stroke (width 0) (type default) (color 0 0 0 0))
@@
     (stroke (width 0) (type default) (color 0 0 0 0))
   )
-  (wire (pts (xy 146.05 199.39) (xy 146.05 203.2))
-    (stroke (width 0) (type default) (color 0 0 0 0))
-  )
   (wire (pts (xy 129.54 101.6) (xy 132.08 101.6))
     (stroke (width 0) (type default) (color 0 0 0 0))
@@
     (stroke (width 0) (type default) (color 0 0 0 0))
   )
-  (wire (pts (xy 133.35 199.39) (xy 135.89 199.39))
-    (stroke (width 0) (type default) (color 0 0 0 0))
-  )
   (wire (pts (xy 243.84 93.98) (xy 243.84 97.79))
     (stroke (width 0) (type default) (color 0 0 0 0))
@@
   )
   (wire (pts (xy 151.13 104.14) (xy 148.59 104.14))
-    (stroke (width 0) (type default) (color 0 0 0 0))
-  )
-  (wire (pts (xy 133.35 207.01) (xy 135.89 207.01))
     (stroke (width 0) (type default) (color 0 0 0 0))
   )
@@
     (effects (font (size 1.27 1.27) bold italic) (justify left bottom))
   )
-  (label "VDD_SNVS_IN" (at 156.21 203.2 0)
-    (effects (font (size 1.27 1.27) bold italic) (justify left bottom))
+  (label "VDD_SNVS_IN" (at 153.67 203.2 180)
+    (effects (font (size 1.27 1.27) bold italic) (justify right bottom))
   )
   (label "XTALI" (at 165.1 86.36 0)
@@
   (label "VDD_SNVS_CAP" (at 215.9 203.2 0)
     (effects (font (size 1.27 1.27) bold italic) (justify left bottom))
-  )
-  (global_label "VDD_COIN_CELL" (shape input) (at 133.35 207.01 180) (fields_autoplaced)
-    (effects (font (size 1.27 1.27) (thickness 0.254) bold italic) (justify right))
-    (property "Intersheet References" "${INTERSHEET_REFS}" (id 0) (at 115.9162 206.883 0)
-      (effects (font (size 1.27 1.27) (thickness 0.254) bold italic) (justify right) hide)
-    )
   )
   (global_label "PMIC_ON_REQ" (shape input) (at 158.75 81.28 180) (fields_autoplaced)
@@
     )
     (pin "1")
-  )
-  (symbol (lib_id "MIMXRT1064 MCU Module:RB521S30_R1_00001") (at 139.7 199.39 0) (mirror y) (unit 1)
-    (in_bom yes) (on_board yes)
-    (property "Reference" "D401" (id 0) (at 139.7 196.85 0))
-    (property "Value" "RB521S30_R1_00001" (id 1) (at 134.62 201.93 0))
-    (property "Footprint" "MIMXRT1064 MCU Module:RB521S30_R1_00001" (id 2) (at 139.7 203.835 0)
-      (effects (font (size 1.27 1.27)) hide)
-    )
-    (property "Datasheet" "" (id 3) (at 139.7 199.39 0)
-      (effects (font (size 1.27 1.27)) hide)
-    )
-    (pin "1")
-    (pin "2")
   )
   (symbol (lib_id "power:PWR_FLAG") (at 236.22 91.44 0) (unit 1)
@@
     )
     (property "Datasheet" "~" (id 3) (at 224.79 86.36 0)
-      (effects (font (size 1.27 1.27)) hide)
-    )
-    (pin "1")
-    (pin "2")
-  )
-  (symbol (lib_id "MIMXRT1064 MCU Module:RB521S30_R1_00001") (at 139.7 207.01 0) (mirror y) (unit 1)
-    (in_bom yes) (on_board yes)
-    (property "Reference" "D402" (id 0) (at 139.7 204.47 0))
-    (property "Value" "RB521S30_R1_00001" (id 1) (at 134.62 210.82 0))
-    (property "Footprint" "MIMXRT1064 MCU Module:RB521S30_R1_00001" (id 2) (at 139.7 211.455 0)
-      (effects (font (size 1.27 1.27)) hide)
-    )
-    (property "Datasheet" "" (id 3) (at 139.7 207.01 0)
       (effects (font (size 1.27 1.27)) hide)
     )
@@
     (pin "2")
   )
-  (symbol (lib_id "MIMXRT1064 MCU Module:VDD_SNVS_3V3") (at 133.35 199.39 90) (unit 1)
-    (in_bom yes) (on_board yes) (fields_autoplaced)
-    (property "Reference" "#PWR0405" (id 0) (at 137.16 199.39 0)
-      (effects (font (size 1.27 1.27)) hide)
-    )
-    (property "Value" "VDD_SNVS_3V3" (id 1) (at 129.54 199.3899 90)
-      (effects (font (size 1.27 1.27)) (justify left))
-    )
-    (property "Footprint" "" (id 2) (at 133.35 199.39 0)
-      (effects (font (size 1.27 1.27)) hide)
-    )
-    (property "Datasheet" "" (id 3) (at 133.35 199.39 0)
-      (effects (font (size 1.27 1.27)) hide)
-    )
-    (pin "1")
-  )
   (symbol (lib_id "power:GND") (at 168.91 234.95 0) (unit 1)

Commit message: updates
Parts:
- removed C401, C415, C417, C421, C424: 4.7u, MIMXRT1064 MCU Module:0402_CL05A475MP5NRNC, symbol MIMXRT1064 MCU Module:CL05A475MP5NRNC
- removed C402, C407, C408, C410, C411, C412, C413, C414, C416, C418, C419, C422, C423: 0.22u, MIMXRT1064 MCU Module:0402_CL05B224KO5NNNC, symbol MIMXRT1064 MCU Module:CL05B224KO5NNNC
- removed C403, C404: 12p, MIMXRT1064 MCU Module:0402_GRM1555C1H120GA01D, symbol MIMXRT1064 MCU Module:GRM1555C1H120GA01D
- removed C405: 1u, MIMXRT1064 MCU Module:0402_CL05A105KA5NQNC, symbol MIMXRT1064 MCU Module:CL05A105KA5NQNC
- removed C406, C409: 8p, MIMXRT1064 MCU Module:0402_GCM1555C1H8R0DA16D, symbol MIMXRT1064 MCU Module:GCM1555C1H8R0DA16D
- removed C420: 10u, MIMXRT1064 MCU Module:0603_CL10A106KP8NNNC, symbol MIMXRT1064 MCU Module:CL10A106KP8NNNC
- removed C425: 22u, MIMXRT1064 MCU Module:0603_CL10A226MQ8NRNC, symbol MIMXRT1064 MCU Module:CL10A226MQ8NRNC
- removed FB401: 120R, MIMXRT1064 MCU Module:0603_BLM18AG121SN1D, symbol MIMXRT1064 MCU Module:BLM18AG121SN1D
- removed L401: 4.7u, MIMXRT1064 MCU Module:LQM21PN4R7MGRD, symbol MIMXRT1064 MCU Module:LQM21PN4R7MGRD
- removed R401: 2.2M, MIMXRT1064 MCU Module:0402WGJ0225TCE, symbol MIMXRT1064 MCU Module:0402WGJ0225TCE
- removed R402: 30k, MIMXRT1064 MCU Module:AF0402FR-0730KL, symbol MIMXRT1064 MCU Module:AF0402FR-0730KL
- removed U1: MIMXRT1064CVL5B, MIMXRT1064 MCU Module:MIMXRT1064CVL5B, symbol MIMXRT1064 MCU Module:MIMXRT1064CVL5B
- removed Y401: 7V24000026, MIMXRT1064 MCU Module:7V24000026, symbol MIMXRT1064 MCU Module:7V24000026
- removed Y402: Q13FC1350000200, MIMXRT1064 MCU Module:Q13FC1350000200, symbol MIMXRT1064 MCU Module:Q13FC1350000200
- added C401, C416, C417, C423, C424: 4.7u, MY CAPACITOR LIBRARY:0402_CL05A475MP5NRNC, symbol MY CAPACITOR LIBRARY:CL05A475MP5NRNC
- added C402, C407, C408, C410, C411, C412, C413, C414, C415, C418, C420, C421, C422: 220n, MY CAPACITOR LIBRARY:0402_CL05B224KO5NNNC, symbol MY CAPACITOR LIBRARY:CL05B224KO5NNNC
- added C403, C404: 12p, MY CAPACITOR LIBRARY:CL10C120JB81PNC, symbol MY CAPACITOR LIBRARY:CL10C120JB81PNC
- added C405: 1u, MY CAPACITOR LIBRARY:0402_CL05A105KA5NQNC, symbol MY CAPACITOR LIBRARY:CL05A105KA5NQNC
- added C406, C409: 8p, MY CAPACITOR LIBRARY:CL10C080DB81PNC, symbol MY CAPACITOR LIBRARY:CL10C080DB81PNC
- added C419: 10u, MY CAPACITOR LIBRARY:0603_CL10A106KP8NNNC, symbol MY CAPACITOR LIBRARY:CL10A106MA8NRNC
- added C425: 22u, MY CAPACITOR LIBRARY:0603_CL10A226MQ8NRNC, symbol MY CAPACITOR LIBRARY:CL10A226MQ8NRNC
- added FB401: 120R, MY FERRITE BEAD LIBRARY:0603_BLM18AG121SN1D, symbol MY FERRITE BEAD LIBRARY:BLM18AG121SN1D
- added L401: 4.7u, MY INDUCTOR LIBRARY:LQM21PN4R7MGRD, symbol MY INDUCTOR LIBRARY:LQM21PN4R7MGRD
- added R401: 2.2M, MY RESISTOR LIBRARY:0402WGJ0225TCE, symbol MY RESISTOR LIBRARY:0402WGJ0225TCE
- added R402: 30k, MY RESISTOR LIBRARY:AF0402FR-0730KL, symbol MY RESISTOR LIBRARY:AF0402FR-0730KL
- added U1: MIMXRT1064CVL5B, MY MICROCONTROLLER LIBRARY:MIMXRT1064CVL5B, symbol MY MICROCONTROLLER LIBRARY:MIMXRT1064CVL5B
- added Y401: 7V24000026, MY CRYSTAL LIBRARY:7V24000026, symbol MY CRYSTAL LIBRARY:7V24000026
- added Y402: Q13FC1350000200, MY CRYSTAL LIBRARY:Q13FC1350000200, symbol MY CRYSTAL LIBRARY:Q13FC1350000200
Connections:
- net +3V3: now also C401.1, C402.1, C405.1, C407.1, C408.1, FB401.2, U1.M9 (VDD_SNVS_IN), U1.N14 (VDDA_ADC_3P3), U1.P12 (VDD_HIGH_IN)
- net DCDC_IN: now also C416.1, C419.1, C422.1, FB401.1, R402.1, U1.K4 (DCDC_IN_Q), U1.L1 (DCDC_IN_1), U1.L2 (DCDC_IN_2)
- net DCDC_PSWITCH: now also C412.1, R402.2, U1.K3 (DCDC_PSWITCH)
- net GND: now also C401.2, C402.2, C403.2, C404.2, C405.2, C406.2, C407.2, C408.2, C409.2, C410.2, C411.2, C412.2, C413.2, C414.2, C415.2, C416.2, C417.2, C418.2, C419.2, C420.2, C421.2, C422.2, C423.2, C424.2, C425.2, R401.2, U1.A1 (VSS_1), U1.A14 (VSS_2), U1.B10 (VSS_4), U1.B5 (VSS_3), U1.E13 (VSS_6), U1.E2 (VSS_5), U1.G7 (VSS_7), U1.G8 (VSS_8), U1.H7 (VSS_9), U1.H8 (VSS_10), U1.J7 (VSS_11), U1.J8 (VSS_12), U1.K13 (VSS_14), U1.K2 (VSS_13), U1.K6 (TEST_MODE), U1.K9 (NGND_KEL0), U1.L9 (VSS_15), U1.N1 (DCDC_GND_1), U1.N2 (DCDC_GND_2), U1.N5 (VSS_16), U1.N8 (VSS_17), U1.P1 (VSS_18), U1.P14 (VSS_19), Y401.2 (GND), Y401.4 (GND)
- net NVCC_PLL: now also C414.1, C417.1, U1.P10 (NVCC_PLL)
- net ONOFF: now also U1.M6 (ONOFF)
- net PMIC_ON_REQ: now also U1.K7 (PMIC_ON_REQ)
- net PMIC_STBY_REQ: now also U1.L7 (PMIC_STBY_REQ)
- net POR_B: now also U1.M7 (POR_B)
- net RTC_XTALI: now also C406.1, U1.N9 (RTC_XTALI), Y402.1
- net RTC_XTALO: now also C409.1, U1.P9 (RTC_XTALO), Y402.2
- net VDD_HIGH_CAP: now also C420.1, C423.1, U1.P8 (VDD_HIGH_CAP)
- net VDD_SNVS_CAP: now also C411.1, U1.M10 (VDD_SNVS_CAP)
- net VDD_SOC_IN: now also C410.1, C413.1, C415.1, C418.1, C421.1, C424.1, C425.1, L401.2, U1.F6 (VDD_SOC_IN_1), U1.F7 (VDD_SOC_IN_2), U1.F8 (VDD_SOC_IN_3), U1.F9 (VDD_SOC_IN_4), U1.G6 (VDD_SOC_IN_5), U1.G9 (VDD_SOC_IN_6), U1.H6 (VDD_SOC_IN_7), U1.H9 (VDD_SOC_IN_8), U1.J5 (DCDC_SENSE), U1.J9 (VDD_SOC_IN_9)
- net WAKEUP: now also U1.L6 (WAKEUP)
- net XTAL0: now also C404.1, U1.N11 (XTALO), Y401.3
- net XTALI: now also C403.1, R401.1, U1.P11 (XTALI), Y401.1
- new net: L401.1, U1.M1 (DCDC_LP_1), U1.M2 (DCDC_LP_2)

Commit message: updates
Connections:
- net ONOFF: no longer names the net of U1.M6 (ONOFF)
- net PMIC_STBY_REQ: no longer names the net of U1.L7 (PMIC_STBY_REQ)
- net WAKEUP: no longer names the net of U1.L6 (WAKEUP)
- no-connect marks 3 -> 6
Other:
- title: MIMXRT1064 MCU Module -> MIMXRT1064 Audio Board
Changed lines of the file:
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@@
   (paper "A3")
   (title_block
-    (title "MIMXRT1064 MCU Module")
-    (date "2023-05-23")
+    (title "MIMXRT1064 Audio Board")
+    (date "2023-06-06")
     (rev "0")
     (company "Joël Ucedo")
@@
   (junction (at 266.7 210.82) (diameter 0) (color 0 0 0 0)
   )
-  (junction (at 170.18 203.2) (diameter 0) (color 0 0 0 0)
-  )
   (junction (at 153.67 203.2) (diameter 0) (color 0 0 0 0)
   )
@@
   (no_connect (at 171.45 101.6))
   (no_connect (at 214.63 66.04))
+  (no_connect (at 171.45 78.74))
+  (no_connect (at 171.45 66.04))
+  (no_connect (at 214.63 73.66))
   (no_connect (at 214.63 68.58))
   (wire (pts (xy 278.13 205.74) (xy 290.83 205.74))
@@
     (stroke (width 0) (type default) (color 0 0 0 0))
   )
-  (wire (pts (xy 158.75 78.74) (xy 171.45 78.74))
-    (stroke (width 0) (type default) (color 0 0 0 0))
-  )
   (wire (pts (xy 294.64 167.64) (xy 307.34 167.64))
     (stroke (width 0) (type default) (color 0 0 0 0))
@@
     (stroke (width 0) (type default) (color 0 0 0 0))
   )
-  (wire (pts (xy 158.75 66.04) (xy 171.45 66.04))
-    (stroke (width 0) (type default) (color 0 0 0 0))
-  )
   (wire (pts (xy 153.67 213.36) (xy 153.67 215.9))
     (stroke (width 0) (type default) (color 0 0 0 0))
@@
     (stroke (width 0) (type default) (color 0 0 0 0))
   )
-  (wire (pts (xy 214.63 73.66) (xy 227.33 73.66))
-    (stroke (width 0) (type default) (color 0 0 0 0))
-  )
   (wire (pts (xy 168.91 224.79) (xy 171.45 224.79))
     (stroke (width 0) (type default) (color 0 0 0 0))
@@
     (stroke (width 0) (type default) (color 0 0 0 0))
   )
-  (wire (pts (xy 171.45 203.2) (xy 170.18 203.2))
-    (stroke (width 0) (type default) (color 0 0 0 0))
-  )
   (wire (pts (xy 236.22 203.2) (xy 236.22 205.74))
     (stroke (width 0) (type default) (color 0 0 0 0))
@@
     (stroke (width 0) (type default) (color 0 0 0 0))
   )
-  (wire (pts (xy 170.18 203.2) (xy 153.67 203.2))
+  (wire (pts (xy 153.67 203.2) (xy 171.45 203.2))
     (stroke (width 0) (type default) (color 0 0 0 0))
   )
@@
   )
   (wire (pts (xy 217.17 101.6) (xy 217.17 104.14))
-    (stroke (width 0) (type default) (color 0 0 0 0))
-  )
-  (wire (pts (xy 170.18 200.66) (xy 170.18 203.2))
     (stroke (width 0) (type default) (color 0 0 0 0))
   )
@@
     )
   )
-  (global_label "WAKEUP" (shape input) (at 227.33 73.66 0) (fields_autoplaced)
-    (effects (font (size 1.27 1.27) bold italic) (justify left))
-    (property "Intersheet References" "${INTERSHEET_REFS}" (id 0) (at 237.7486 73.533 0)
-      (effects (font (size 1.27 1.27) bold italic) (justify left) hide)
-    )
-  )
-  (global_label "PMIC_STBY_REQ" (shape input) (at 158.75 78.74 180) (fields_autoplaced)
-    (effects (font (size 1.27 1.27) bold italic) (justify right))
-    (property "Intersheet References" "${INTERSHEET_REFS}" (id 0) (at 141.0742 78.613 0)
-      (effects (font (size 1.27 1.27) bold italic) (justify right) hide)
-    )
-  )
-  (global_label "ONOFF" (shape input) (at 158.75 66.04 180) (fields_autoplaced)
-    (effects (font (size 1.27 1.27) bold italic) (justify right))
-    (property "Intersheet References" "${INTERSHEET_REFS}" (id 0) (at 149.7223 65.913 0)
-      (effects (font (size 1.27 1.27) bold italic) (justify right) hide)
-    )
-  )
   (global_label "POR_B" (shape input) (at 158.75 68.58 180) (fields_autoplaced)
     (effects (font (size 1.27 1.27) bold italic) (justify right))
@@
       (effects (font (size 1.27 1.27)) hide)
     )
-    (pin "1")
-  )
-  (symbol (lib_id "power:PWR_FLAG") (at 170.18 200.66 0) (unit 1)
-    (in_bom yes) (on_board yes) (fields_autoplaced)
-    (property "Reference" "#FLG0403" (id 0) (at 170.18 198.755 0)
-      (effects (font (size 1.27 1.27)) hide)
-    )
-    (property "Value" "PWR_FLAG" (id 1) (at 170.18 195.58 0))
-    (property "Footprint" "" (id 2) (at 170.18 200.66 0)
-      (effects (font (size 1.27 1.27)) hide)
-    )
-    (property "Datasheet" "~" (id 3) (at 170.18 200.66 0)
-      (effects (font (size 1.27 1.27)) hide)
-    )
