File: DESIGN FILES/pwrpin_crystals.kicad_sch (KiCad schematic)
At the start: 32 parts, among them U1 MIMXRT1064CVL5B, Y401 7V24000026, Y402 Q13FC1350000200

Commit message: updates
Parts:
- renumbered U1 to U401
Connections:
- net ON_OFF: now reaches U401.M6 (ONOFF)
- no-connect marks 6 -> 5
Other:
- note added: "I followed Paul for the caps"
- note added: "NXP reserved pin"
- note added: "See PMIC on carrier"
- note added: "[4] MCU POWER & CRYSTALS"
- note removed: "4 : MCU POWER & CRYSTALS"
- title: MIMXRT1064 Audio Board -> MIMXRT1064 MCU Module
Changed lines of the file:
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@@
   (paper "A3")
   (title_block
-    (title "MIMXRT1064 Audio Board")
-    (date "2023-06-06")
+    (title "MIMXRT1064 MCU Module")
+    (date "2023-06-24")
     (rev "0")
     (company "Joël Ucedo")
@@
   (no_connect (at 214.63 66.04))
   (no_connect (at 171.45 78.74))
-  (no_connect (at 171.45 66.04))
   (no_connect (at 214.63 73.66))
   (no_connect (at 214.63 68.58))
@@
     (stroke (width 0) (type default) (color 0 0 0 0))
   )
+  (wire (pts (xy 158.75 66.04) (xy 171.45 66.04))
+    (stroke (width 0) (type default) (color 0 0 0 0))
+  )
   (wire (pts (xy 213.36 193.04) (xy 278.13 193.04))
     (stroke (width 0) (type default) (color 0 0 0 0))
@@
     (effects (font (size 1.27 1.27) bold italic) (justify left bottom))
   )
-  (text "4 : MCU POWER & CRYSTALS" (at 25.4 29.21 0)
+  (text "I followed Paul\nfor the caps" (at 262.89 96.52 0)
+    (effects (font (size 1.27 1.27) bold italic) (justify left bottom))
+  )
+  (text "[4] MCU POWER & CRYSTALS" (at 25.4 29.21 0)
     (effects (font (size 5 5) bold italic) (justify left bottom))
+  )
+  (text "See PMIC\non carrier" (at 142.24 80.01 0)
+    (effects (font (size 1.27 1.27) bold italic) (justify left bottom))
+  )
+  (text "See PMIC\non carrier" (at 148.59 64.77 0)
+    (effects (font (size 1.27 1.27) bold italic) (justify left bottom))
   )
   (text "CL = 7p" (at 156.21 120.65 0)
@@
     (effects (font (size 1.27 1.27) bold italic) (justify left bottom))
   )
+  (text "NXP reserved pin" (at 132.08 73.66 0)
+    (effects (font (size 1.27 1.27) bold italic) (justify left bottom))
+  )
   (text "max ESR = 40R" (at 116.84 123.19 0)
     (effects (font (size 1.27 1.27) bold italic) (justify left bottom))
@@
   (label "VDD_SNVS_CAP" (at 215.9 203.2 0)
     (effects (font (size 1.27 1.27) bold italic) (justify left bottom))
+  )
+  (global_label "ON_OFF" (shape input) (at 158.75 66.04 180) (fields_autoplaced)
+    (effects (font (size 1.27 1.27) bold italic) (justify right))
+    (property "Intersheet References" "${INTERSHEET_REFS}" (id 0) (at 148.7547 65.913 0)
+      (effects (font (size 1.27 1.27) bold italic) (justify right) hide)
+    )
   )
   (global_label "PMIC_ON_REQ" (shape input) (at 158.75 81.28 180) (fields_autoplaced)
@@
   (symbol (lib_id "power:+3V3") (at 144.78 162.56 0) (unit 1)
     (in_bom yes) (on_board yes) (fields_autoplaced)
-    (property "Reference" "#PWR0406" (id 0) (at 144.78 166.37 0)
+    (property "Reference" "#PWR0405" (id 0) (at 144.78 166.37 0)
       (effects (font (size 1.27 1.27)) hide)
     )
@@
   (symbol (lib_id "power:+3V3") (at 304.8 76.2 0) (unit 1)
     (in_bom yes) (on_board yes) (fields_autoplaced)
-    (property "Reference" "#PWR0418" (id 0) (at 304.8 80.01 0)
+    (property "Reference" "#PWR0417" (id 0) (at 304.8 80.01 0)
       (effects (font (size 1.27 1.27)) hide)
     )
@@
   (symbol (lib_id "power:PWR_FLAG") (at 236.22 91.44 0) (unit 1)
     (in_bom yes) (on_board yes) (fields_autoplaced)
-    (property "Reference" "#FLG0407" (id 0) (at 236.22 89.535 0)
+    (property "Reference" "#FLG0405" (id 0) (at 236.22 89.535 0)
       (effects (font (size 1.27 1.27)) hide)
     )
@@
   (symbol (lib_id "power:GND") (at 215.9 234.95 0) (unit 1)
     (in_bom yes) (on_board yes) (fields_autoplaced)
-    (property "Reference" "#PWR0411" (id 0) (at 215.9 241.3 0)
+    (property "Reference" "#PWR0410" (id 0) (at 215.9 241.3 0)
       (effects (font (size 1.27 1.27)) hide)
     )
@@
   (symbol (lib_id "power:GND") (at 243.84 107.95 0) (unit 1)
     (in_bom yes) (on_board yes) (fields_autoplaced)
-    (property "Reference" "#PWR0414" (id 0) (at 243.84 114.3 0)
+    (property "Reference" "#PWR0413" (id 0) (at 243.84 114.3 0)
       (effects (font (size 1.27 1.27)) hide)
     )
@@
   (symbol (lib_id "power:GND") (at 217.17 107.95 0) (unit 1)
     (in_bom yes) (on_board yes) (fields_autoplaced)
-    (property "Reference" "#PWR0412" (id 0) (at 217.17 114.3 0)
+    (property "Reference" "#PWR0411" (id 0) (at 217.17 114.3 0)
       (effects (font (size 1.27 1.27)) hide)
     )
@@
   (symbol (lib_id "power:GND") (at 148.59 119.38 0) (unit 1)
     (in_bom yes) (on_board yes) (fields_autoplaced)
-    (property "Reference" "#PWR0408" (id 0) (at 148.59 125.73 0)
+    (property "Reference" "#PWR0407" (id 0) (at 148.59 125.73 0)
       (effects (font (size 1.27 1.27)) hide)
     )
@@
   (symbol (lib_id "power:GND") (at 236.22 215.9 0) (unit 1)
     (in_bom yes) (on_board yes) (fields_autoplaced)
-    (property "Reference" "#PWR0413" (id 0) (at 236.22 222.25 0)
+    (property "Reference" "#PWR0412" (id 0) (at 236.22 222.25 0)
       (effects (font (size 1.27 1.27)) hide)
     )
@@
   (symbol (lib_id "power:GND") (at 307.34 182.88 0) (unit 1)
     (in_bom yes) (on_board yes) (fields_autoplaced)
-    (property "Reference" "#PWR0419" (id 0) (at 307.34 189.23 0)
+    (property "Reference" "#PWR0418" (id 0) (at 307.34 189.23 0)
       (effects (font (size 1.27 1.27)) hide)
     )
@@
   (symbol (lib_id "power:GND") (at 283.21 93.98 0) (unit 1)
     (in_bom yes) (on_board yes) (fields_autoplaced)
-    (property "Reference" "#PWR0417" (id 0) (at 283.21 100.33 0)
+    (property "Reference" "#PWR0415" (id 0) (at 283.21 100.33 0)
       (effects (font (size 1.27 1.27)) hide)
     )
@@
   (symbol (lib_id "power:PWR_FLAG") (at 278.13 190.5 0) (unit 1)
     (in_bom yes) (on_board yes) (fields_autoplaced)
-    (property "Reference" "#FLG0410" (id 0) (at 278.13 188.595 0)
+    (property "Reference" "#FLG0409" (id 0) (at 278.13 188.595 0)
       (effects (font (size 1.27 1.27)) hide)
     )
@@
   (symbol (lib_id "power:GND") (at 144.78 180.34 0) (unit 1)
     (in_bom yes) (on_board yes) (fields_autoplaced)
-    (property "Reference" "#PWR0407" (id 0) (at 144.78 186.69 0)
+    (property "Reference" "#PWR0406" (id 0) (at 144.78 186.69 0)
       (effects (font (size 1.27 1.27)) hide)
     )
@@
   (symbol (lib_id "power:PWR_FLAG") (at 243.84 76.2 0) (unit 1)
     (in_bom yes) (on_board yes) (fields_autoplaced)
-    (property "Reference" "#FLG0408" (id 0) (at 243.84 74.295 0)
+    (property "Reference" "#FLG0407" (id 0) (at 243.84 74.295 0)
       (effects (font (size 1.27 1.27)) hide)
     )
@@
   (symbol (lib_id "power:PWR_FLAG") (at 219.71 83.82 0) (unit 1)
     (in_bom yes) (on_board yes)
-    (property "Reference" "#FLG0405" (id 0) (at 219.71 81.915 0)
+    (property "Reference" "#FLG0404" (id 0) (at 219.71 81.915 0)
       (effects (font (size 1.27 1.27)) hide)
     )
@@
   (symbol (lib_id "MY MICROCONTROLLER LIBRARY:MIMXRT1064CVL5B") (at 193.04 83.82 0) (unit 2)
     (in_bom yes) (on_board yes) (fields_autoplaced)
-    (property "Reference" "U1" (id 0) (at 193.04 58.42 0))
+    (property "Reference" "U401" (id 0) (at 193.04 58.42 0))
     (property "Value" "MIMXRT1064CVL5B" (id 1) (at 193.04 60.96 0))
     (property "Footprint" "MY MICROCONTROLLER LIBRARY:MIMXRT1064CVL5B" (id 2) (at 196.85 29.21 0)
@@
   (symbol (lib_id "power:PWR_FLAG") (at 266.7 196.85 0) (unit 1)
     (in_bom yes) (on_board yes)
-    (property "Reference" "#FLG0409" (id 0) (at 266.7 194.945 0)
+    (property "Reference" "#FLG0408" (id 0) (at 266.7 194.945 0)
       (effects (font (size 1.27 1.27)) hide)
     )
@@
   (symbol (lib_id "power:GND") (at 266.7 213.36 0) (unit 1)
     (in_bom yes) (on_board yes) (fields_autoplaced)
-    (property "Reference" "#PWR0415" (id 0) (at 266.7 219.71 0)
+    (property "Reference" "#PWR0414" (id 0) (at 266.7 219.71 0)
       (effects (font (size 1.27 1.27)) hide)
     )
@@
   (symbol (lib_id "power:PWR_FLAG") (at 215.9 163.83 0) (unit 1)
     (in_bom yes) (on_board yes) (fields_autoplaced)
-    (property "Reference" "#FLG0404" (id 0) (at 215.9 161.925 0)
+    (property "Reference" "#FLG0403" (id 0) (at 215.9 161.925 0)
       (effects (font (size 1.27 1.27)) hide)
     )
@@
   (symbol (lib_id "power:GND") (at 168.91 234.95 0) (unit 1)
     (in_bom yes) (on_board yes) (fields_autoplaced)
-    (property "Reference" "#PWR0410" (id 0) (at 168.91 241.3 0)
+    (property "Reference" "#PWR0409" (id 0) (at 168.91 241.3 0)
       (effects (font (size 1.27 1.27)) hide)
     )
@@
   (symbol (lib_id "power:GND") (at 153.67 215.9 0) (unit 1)
     (in_bom yes) (on_board yes) (fields_autoplaced)
-    (property "Reference" "#PWR0409" (id 0) (at 153.67 222.25 0)
+    (property "Reference" "#PWR0408" (id 0) (at 153.67 222.25 0)
       (effects (font (size 1.27 1.27)) hide)
     )
@@
   (symbol (lib_id "MY MICROCONTROLLER LIBRARY:MIMXRT1064CVL5B") (at 191.77 196.85 0) (unit 1)
     (in_bom yes) (on_board yes) (fields_autoplaced)
-    (property "Reference" "U1" (id 0) (at 192.405 157.48 0))
+    (property "Reference" "U401" (id 0) (at 192.405 157.48 0))
     (property "Value" "MIMXRT1064CVL5B" (id 1) (at 192.405 160.02 0))
     (property "Footprint" "MY MICROCONTROLLER LIBRARY:MIMXRT1064CVL5B" (id 2) (at 195.58 142.24 0)

Commit message: updates
Connections:
- net DCDC_LP: now reaches L401.1, U401.M1 (DCDC_LP_1), U401.M2 (DCDC_LP_2)
Changed lines of the file:
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@@
+    (effects (font (size 1.27 1.27) bold italic) (justify left bottom))
+  )
+  (label "DCDC_LP" (at 217.17 88.9 0)
     (effects (font (size 1.27 1.27) bold italic) (justify left bottom))
   )
@@
   (symbol (lib_id "MY INDUCTOR LIBRARY:LQM21PN4R7MGRD") (at 224.79 86.36 0) (unit 1)
     (in_bom yes) (on_board yes)
-    (property "Reference" "L401" (id 0) (at 224.79 83.82 0))
-    (property "Value" "4.7u" (id 1) (at 224.79 87.63 0))
+    (property "Reference" "L401" (id 0) (at 223.52 83.82 0))
+    (property "Value" "4.7u" (id 1) (at 228.6 83.82 0))
     (property "Footprint" "MY INDUCTOR LIBRARY:LQM21PN4R7MGRD" (id 2) (at 224.79 86.36 90)
       (effects (font (size 1.27 1.27)) hide)

Commit message: updates
Parts:
- removed FB401: 120R, MY FERRITE BEAD LIBRARY:0603_BLM18AG121SN1D, symbol MY FERRITE BEAD LIBRARY:BLM18AG121SN1D
- removed L401: 4.7u, MY INDUCTOR LIBRARY:LQM21PN4R7MGRD, symbol MY INDUCTOR LIBRARY:LQM21PN4R7MGRD
- added C425, C426: 220n, MY CAPACITOR LIBRARY:0402_CL05B224KO5NNNC, symbol MY CAPACITOR LIBRARY:CL05B224KO5NNNC
- added L401: VLS4012ET-4R7M, MY INDUCTOR LIBRARY:VLS4012ET-4R7M, symbol MY INDUCTOR LIBRARY:VLS4012ET-4R7M
- renumbered C425 to C427
Connections:
- net DCDC_IN is gone; now on net +3V3: C416.1, C419.1, C422.1, R402.1, U401.K4 (DCDC_IN_Q), U401.L1 (DCDC_IN_1), U401.L2 (DCDC_IN_2)
- net +3V3: now also C425.1, C426.1
- net DCDC_LP: now also L401.1
- net GND: now also C425.2, C426.2
- net VDD_SOC_IN: now also L401.2
Other:
- note removed: "I followed Paul for the caps"
Changed lines of the file:
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@@
   (junction (at 266.7 210.82) (diameter 0) (color 0 0 0 0)
   )
+  (junction (at 295.91 91.44) (diameter 0) (color 0 0 0 0)
+  )
   (junction (at 153.67 203.2) (diameter 0) (color 0 0 0 0)
   )
@@
   (junction (at 215.9 167.64) (diameter 0) (color 0 0 0 0)
   )
+  (junction (at 307.34 78.74) (diameter 0) (color 0 0 0 0)
+  )
   (junction (at 168.91 212.09) (diameter 0) (color 0 0 0 0)
   )
@@
   )
   (junction (at 132.08 101.6) (diameter 0) (color 0 0 0 0)
+  )
+  (junction (at 295.91 78.74) (diameter 0) (color 0 0 0 0)
   )
   (junction (at 219.71 86.36) (diameter 0) (color 0 0 0 0)
@@
     (stroke (width 0) (type default) (color 0 0 0 0))
   )
-  (wire (pts (xy 304.8 76.2) (xy 304.8 78.74))
-    (stroke (width 0) (type default) (color 0 0 0 0))
-  )
   (wire (pts (xy 213.36 224.79) (xy 215.9 224.79))
     (stroke (width 0) (type default) (color 0 0 0 0))
@@
     (stroke (width 0) (type default) (color 0 0 0 0))
   )
-  (wire (pts (xy 300.99 78.74) (xy 304.8 78.74))
-    (stroke (width 0) (type default) (color 0 0 0 0))
-  )
   (wire (pts (xy 243.84 78.74) (xy 257.81 78.74))
     (stroke (width 0) (type default) (color 0 0 0 0))
   )
+  (wire (pts (xy 295.91 91.44) (xy 307.34 91.44))
+    (stroke (width 0) (type default) (color 0 0 0 0))
+  )
   (wire (pts (xy 144.78 162.56) (xy 144.78 165.1))
     (stroke (width 0) (type default) (color 0 0 0 0))
@@
     (stroke (width 0) (type default) (color 0 0 0 0))
   )
+  (wire (pts (xy 307.34 78.74) (xy 307.34 81.28))
+    (stroke (width 0) (type default) (color 0 0 0 0))
+  )
   (wire (pts (xy 215.9 209.55) (xy 215.9 212.09))
     (stroke (width 0) (type default) (color 0 0 0 0))
@@
     (stroke (width 0) (type default) (color 0 0 0 0))
   )
+  (wire (pts (xy 307.34 91.44) (xy 307.34 88.9))
+    (stroke (width 0) (type default) (color 0 0 0 0))
+  )
   (wire (pts (xy 153.67 213.36) (xy 153.67 215.9))
     (stroke (width 0) (type default) (color 0 0 0 0))
@@
     (stroke (width 0) (type default) (color 0 0 0 0))
   )
+  (wire (pts (xy 295.91 78.74) (xy 307.34 78.74))
+    (stroke (width 0) (type default) (color 0 0 0 0))
+  )
   (wire (pts (xy 168.91 232.41) (xy 168.91 234.95))
     (stroke (width 0) (type default) (color 0 0 0 0))
@@
     (stroke (width 0) (type default) (color 0 0 0 0))
   )
-  (wire (pts (xy 283.21 78.74) (xy 293.37 78.74))
+  (wire (pts (xy 283.21 78.74) (xy 295.91 78.74))
     (stroke (width 0) (type default) (color 0 0 0 0))
   )
@@
     (stroke (width 0) (type default) (color 0 0 0 0))
   )
+  (wire (pts (xy 283.21 91.44) (xy 295.91 91.44))
+    (stroke (width 0) (type default) (color 0 0 0 0))
+  )
   (wire (pts (xy 236.22 203.2) (xy 236.22 205.74))
     (stroke (width 0) (type default) (color 0 0 0 0))
@@
     (stroke (width 0) (type default) (color 0 0 0 0))
   )
+  (wire (pts (xy 307.34 73.66) (xy 307.34 78.74))
+    (stroke (width 0) (type default) (color 0 0 0 0))
+  )
   (wire (pts (xy 215.9 219.71) (xy 215.9 222.25))
     (stroke (width 0) (type default) (color 0 0 0 0))
@@
     (stroke (width 0) (type default) (color 0 0 0 0))
   )
+  (wire (pts (xy 295.91 78.74) (xy 295.91 81.28))
+    (stroke (width 0) (type default) (color 0 0 0 0))
+  )
   (wire (pts (xy 269.24 177.8) (xy 269.24 180.34))
     (stroke (width 0) (type default) (color 0 0 0 0))
@@
     (stroke (width 0) (type default) (color 0 0 0 0))
   )
+  (wire (pts (xy 295.91 91.44) (xy 295.91 88.9))
+    (stroke (width 0) (type default) (color 0 0 0 0))
+  )
   (wire (pts (xy 278.13 203.2) (xy 278.13 205.74))
     (stroke (width 0) (type default) (color 0 0 0 0))
@@
   )
   (text "RC DELAY" (at 246.38 93.98 0)
-    (effects (font (size 1.27 1.27) bold italic) (justify left bottom))
-  )
-  (text "I followed Paul\nfor the caps" (at 262.89 96.52 0)
     (effects (font (size 1.27 1.27) bold italic) (justify left bottom))
   )
@@
     (pin "1")
   )
-  (symbol (lib_id "power:+3V3") (at 304.8 76.2 0) (unit 1)
-    (in_bom yes) (on_board yes) (fields_autoplaced)
-    (property "Reference" "#PWR0417" (id 0) (at 304.8 80.01 0)
-      (effects (font (size 1.27 1.27)) hide)
-    )
-    (property "Value" "+3V3" (id 1) (at 304.8 71.12 0))
-    (property "Footprint" "" (id 2) (at 304.8 76.2 0)
-      (effects (font (size 1.27 1.27)) hide)
-    )
-    (property "Datasheet" "" (id 3) (at 304.8 76.2 0)
+  (symbol (lib_id "power:+3V3") (at 307.34 73.66 0) (unit 1)
+    (in_bom yes) (on_board yes) (fields_autoplaced)
+    (property "Reference" "#PWR0417" (id 0) (at 307.34 77.47 0)
+      (effects (font (size 1.27 1.27)) hide)
+    )
+    (property "Value" "+3V3" (id 1) (at 307.34 68.58 0))
+    (property "Footprint" "" (id 2) (at 307.34 73.66 0)
+      (effects (font (size 1.27 1.27)) hide)
+    )
+    (property "Datasheet" "" (id 3) (at 307.34 73.66 0)
       (effects (font (size 1.27 1.27)) hide)
     )
@@
   (symbol (lib_id "MY CAPACITOR LIBRARY:CL10A226MQ8NRNC") (at 307.34 173.99 0) (unit 1)
     (in_bom yes) (on_board yes) (fields_autoplaced)
-    (property "Reference" "C425" (id 0) (at 311.15 172.7199 0)
+    (property "Reference" "C427" (id 0) (at 311.15 172.7199 0)
       (effects (font (size 1.27 1.27)) (justify left))
     )
@@
     )
     (property "Datasheet" "~" (id 3) (at 307.34 173.99 0)
+      (effects (font (size 1.27 1.27)) hide)
+    )
+    (pin "1")
+    (pin "2")
+  )
+  (symbol (lib_id "MY CAPACITOR LIBRARY:CL05B224KO5NNNC") (at 295.91 85.09 0) (unit 1)
+    (in_bom yes) (on_board yes) (fields_autoplaced)
+    (property "Reference" "C425" (id 0) (at 299.72 83.8199 0)
+      (effects (font (size 1.27 1.27)) (justify left))
+    )
+    (property "Value" "220n" (id 1) (at 299.72 86.3599 0)
+      (effects (font (size 1.27 1.27)) (justify left))
+    )
+    (property "Footprint" "MY CAPACITOR LIBRARY:0402_CL05B224KO5NNNC" (id 2) (at 296.8752 88.9 0)
+      (effects (font (size 1.27 1.27)) hide)
+    )
+    (property "Datasheet" "~" (id 3) (at 295.91 85.09 0)
       (effects (font (size 1.27 1.27)) hide)
     )
@@
     )
     (property "Datasheet" "~" (id 3) (at 99.06 199.39 0)
+      (effects (font (size 1.27 1.27)) hide)
+    )
+    (pin "1")
+    (pin "2")
+  )
+  (symbol (lib_id "MY CAPACITOR LIBRARY:CL05B224KO5NNNC") (at 307.34 85.09 0) (unit 1)
+    (in_bom yes) (on_board yes) (fields_autoplaced)
+    (property "Reference" "C426" (id 0) (at 311.15 83.8199 0)
+      (effects (font (size 1.27 1.27)) (justify left))
+    )
+    (property "Value" "220n" (id 1) (at 311.15 86.3599 0)
+      (effects (font (size 1.27 1.27)) (justify left))
+    )
+    (property "Footprint" "MY CAPACITOR LIBRARY:0402_CL05B224KO5NNNC" (id 2) (at 308.3052 88.9 0)
+      (effects (font (size 1.27 1.27)) hide)
+    )
+    (property "Datasheet" "~" (id 3) (at 307.34 85.09 0)
       (effects (font (size 1.27 1.27)) hide)
     )
@@
     (pin "1")
   )
+  (symbol (lib_id "MY INDUCTOR LIBRARY:VLS4012ET-4R7M") (at 224.79 86.36 0) (unit 1)
+    (in_bom yes) (on_board yes)
+    (property "Reference" "L401" (id 0) (at 224.79 83.82 0))
+    (property "Value" "VLS4012ET-4R7M" (id 1) (at 224.79 82.55 0)
+      (effects (font (size 1.27 1.27)) hide)
+    )
+    (property "Footprint" "MY INDUCTOR LIBRARY:VLS4012ET-4R7M" (id 2) (at 224.79 86.36 90)
+      (effects (font (size 1.27 1.27)) hide)
+    )
+    (property "Datasheet" "~" (id 3) (at 224.79 86.36 0)
+      (effects (font (size 1.27 1.27)) hide)
+    )
+    (pin "1")
+    (pin "2")
+  )
   (symbol (lib_id "power:GND") (at 283.21 93.98 0) (unit 1)
     (in_bom yes) (on_board yes) (fields_autoplaced)
@@
     (pin "1")
   )
-  (symbol (lib_id "MY INDUCTOR LIBRARY:LQM21PN4R7MGRD") (at 224.79 86.36 0) (unit 1)
-    (in_bom yes) (on_board yes)
-    (property "Reference" "L401" (id 0) (at 223.52 83.82 0))
-    (property "Value" "4.7u" (id 1) (at 228.6 83.82 0))
-    (property "Footprint" "MY INDUCTOR LIBRARY:LQM21PN4R7MGRD" (id 2) (at 224.79 86.36 90)
-      (effects (font (size 1.27 1.27)) hide)
-    )
-    (property "Datasheet" "~" (id 3) (at 224.79 86.36 0)
-      (effects (font (size 1.27 1.27)) hide)
-    )
-    (pin "1")
-    (pin "2")
-  )
   (symbol (lib_id "power:GND") (at 144.78 180.34 0) (unit 1)
     (in_bom yes) (on_board yes) (fields_autoplaced)
@@
     (pin "1")
   )
-  (symbol (lib_id "MY FERRITE BEAD LIBRARY:BLM18AG121SN1D") (at 297.18 78.74 90) (unit 1)
-    (in_bom yes) (on_board yes)
-    (property "Reference" "FB401" (id 0) (at 297.1292 73.66 90))
-    (property "Value" "120R" (id 1) (at 297.18 83.82 90))
-    (property "Footprint" "MY FERRITE BEAD LIBRARY:0603_BLM18AG121SN1D" (id 2) (at 298.958 78.74 90)
-      (effects (font (size 1.27 1.27)) hide)
-    )
-    (property "Datasheet" "~" (id 3) (at 297.18 78.74 0)
-      (effects (font (size 1.27 1.27)) hide)
-    )
-    (pin "1")
-    (pin "2")
-  )
   (symbol (lib_id "power:PWR_FLAG") (at 243.84 76.2 0) (unit 1)

Commit message: updates
Connections:
- net VDD_SOC_IN: no longer U401.J5 (DCDC_SENSE)
- no-connect marks 5 -> 6
Other:
- note added: "NC on EVK layout"
Changed lines of the file:
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@@
   (junction (at 243.84 93.98) (diameter 0) (color 0 0 0 0)
   )
-  (junction (at 231.14 96.52) (diameter 0) (color 0 0 0 0)
-  )
   (junction (at 215.9 214.63) (diameter 0) (color 0 0 0 0)
   )
@@
   (junction (at 283.21 91.44) (diameter 0) (color 0 0 0 0)
   )
+  (no_connect (at 214.63 96.52))
   (no_connect (at 171.45 101.6))
   (no_connect (at 214.63 66.04))
@@
     (stroke (width 0) (type default) (color 0 0 0 0))
   )
-  (wire (pts (xy 231.14 96.52) (xy 231.14 86.36))
-    (stroke (width 0) (type default) (color 0 0 0 0))
-  )
   (wire (pts (xy 157.48 165.1) (xy 171.45 165.1))
     (stroke (width 0) (type default) (color 0 0 0 0))
@@
     (stroke (width 0) (type default) (color 0 0 0 0))
   )
-  (wire (pts (xy 231.14 96.52) (xy 231.14 167.64))
+  (wire (pts (xy 231.14 86.36) (xy 231.14 167.64))
     (stroke (width 0) (type default) (color 0 0 0 0))
   )
@@
   )
   (wire (pts (xy 215.9 222.25) (xy 215.9 224.79))
-    (stroke (width 0) (type default) (color 0 0 0 0))
-  )
-  (wire (pts (xy 214.63 96.52) (xy 231.14 96.52))
     (stroke (width 0) (type default) (color 0 0 0 0))
   )
@@
     (effects (font (size 1.27 1.27) bold italic) (justify left bottom))
   )
+  (text "NC on EVK layout" (at 213.36 99.06 0)
+    (effects (font (size 1.27 1.27)) (justify left bottom))
+  )
   (text "[4] MCU POWER & CRYSTALS" (at 25.4 29.21 0)
