File: DESIGN FILES/pwrpin_crystals.kicad_sch (KiCad schematic)
At the start: 33 parts, among them U401 MIMXRT1064CVL5B, Y401 7V24000026, Y402 Q13FC1350000200

Commit message: updates
Parts:
- added D401: LED_BLUE, MY LED LIBRARY:19-218_BHC-ZL1M2QY_3T, symbol MY LED LIBRARY:19-218_BHC-ZL1M2QY_3T
- added R401: 2.2k, MY RESISTOR LIBRARY:0603WAF2201T5E, symbol MY RESISTOR LIBRARY:0603WAF2201T5E
- renumbered R401 to R402, R402 to R403
Connections:
- net +3V3: now also R401.1
- net GND: now also D401.1 (K)
- new net: D401.2 (A), R401.2
Changed lines of the file:
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@@
+    (stroke (width 0) (type default) (color 0 0 0 0))
+  )
+  (wire (pts (xy 38.1 53.34) (xy 38.1 57.15))
     (stroke (width 0) (type default) (color 0 0 0 0))
   )
@@
     (stroke (width 0) (type default) (color 0 0 0 0))
   )
+  (wire (pts (xy 38.1 76.2) (xy 38.1 80.01))
+    (stroke (width 0) (type default) (color 0 0 0 0))
+  )
   (wire (pts (xy 213.36 177.8) (xy 215.9 177.8))
     (stroke (width 0) (type default) (color 0 0 0 0))
@@
   )
   (wire (pts (xy 243.84 76.2) (xy 243.84 78.74))
+    (stroke (width 0) (type default) (color 0 0 0 0))
+  )
+  (wire (pts (xy 38.1 64.77) (xy 38.1 68.58))
     (stroke (width 0) (type default) (color 0 0 0 0))
   )
@@
   (symbol (lib_id "power:+3V3") (at 144.78 162.56 0) (unit 1)
     (in_bom yes) (on_board yes) (fields_autoplaced)
-    (property "Reference" "#PWR0405" (id 0) (at 144.78 166.37 0)
+    (property "Reference" "#PWR0407" (id 0) (at 144.78 166.37 0)
       (effects (font (size 1.27 1.27)) hide)
     )
@@
   (symbol (lib_id "power:+3V3") (at 307.34 73.66 0) (unit 1)
     (in_bom yes) (on_board yes) (fields_autoplaced)
-    (property "Reference" "#PWR0417" (id 0) (at 307.34 77.47 0)
+    (property "Reference" "#PWR0419" (id 0) (at 307.34 77.47 0)
       (effects (font (size 1.27 1.27)) hide)
     )
@@
   (symbol (lib_id "power:GND") (at 215.9 234.95 0) (unit 1)
     (in_bom yes) (on_board yes) (fields_autoplaced)
-    (property "Reference" "#PWR0410" (id 0) (at 215.9 241.3 0)
+    (property "Reference" "#PWR0412" (id 0) (at 215.9 241.3 0)
       (effects (font (size 1.27 1.27)) hide)
     )
@@
   (symbol (lib_id "power:GND") (at 132.08 76.2 0) (unit 1)
     (in_bom yes) (on_board yes) (fields_autoplaced)
-    (property "Reference" "#PWR0404" (id 0) (at 132.08 82.55 0)
+    (property "Reference" "#PWR0406" (id 0) (at 132.08 82.55 0)
       (effects (font (size 1.27 1.27)) hide)
     )
@@
   (symbol (lib_id "power:GND") (at 243.84 107.95 0) (unit 1)
     (in_bom yes) (on_board yes) (fields_autoplaced)
-    (property "Reference" "#PWR0413" (id 0) (at 243.84 114.3 0)
+    (property "Reference" "#PWR0415" (id 0) (at 243.84 114.3 0)
       (effects (font (size 1.27 1.27)) hide)
     )
@@
     (pin "1")
   )
+  (symbol (lib_id "power:+3V3") (at 38.1 53.34 0) (unit 1)
+    (in_bom yes) (on_board yes) (fields_autoplaced)
+    (property "Reference" "#PWR0401" (id 0) (at 38.1 57.15 0)
+      (effects (font (size 1.27 1.27)) hide)
+    )
+    (property "Value" "+3V3" (id 1) (at 38.1 48.26 0))
+    (property "Footprint" "" (id 2) (at 38.1 53.34 0)
+      (effects (font (size 1.27 1.27)) hide)
+    )
+    (property "Datasheet" "" (id 3) (at 38.1 53.34 0)
+      (effects (font (size 1.27 1.27)) hide)
+    )
+    (pin "1")
+  )
   (symbol (lib_id "MY CAPACITOR LIBRARY:CL05B224KO5NNNC") (at 243.84 173.99 0) (unit 1)
     (in_bom yes) (on_board yes) (fields_autoplaced)
@@
   (symbol (lib_id "power:GND") (at 217.17 107.95 0) (unit 1)
     (in_bom yes) (on_board yes) (fields_autoplaced)
-    (property "Reference" "#PWR0411" (id 0) (at 217.17 114.3 0)
+    (property "Reference" "#PWR0413" (id 0) (at 217.17 114.3 0)
       (effects (font (size 1.27 1.27)) hide)
     )
@@
   (symbol (lib_id "MY RESISTOR LIBRARY:AF0402FR-0730KL") (at 243.84 85.09 0) (unit 1)
     (in_bom yes) (on_board yes) (fields_autoplaced)
-    (property "Reference" "R402" (id 0) (at 246.38 83.8199 0)
+    (property "Reference" "R403" (id 0) (at 246.38 83.8199 0)
       (effects (font (size 1.27 1.27)) (justify left))
     )
@@
     )
     (property "Datasheet" "~" (id 3) (at 243.84 85.09 0)
+      (effects (font (size 1.27 1.27)) hide)
+    )
+    (pin "1")
+    (pin "2")
+  )
+  (symbol (lib_id "MY LED LIBRARY:19-218_BHC-ZL1M2QY_3T") (at 38.1 72.39 90) (unit 1)
+    (in_bom yes) (on_board yes) (fields_autoplaced)
+    (property "Reference" "D401" (id 0) (at 41.91 72.7074 90)
+      (effects (font (size 1.27 1.27)) (justify right))
+    )
+    (property "Value" "LED_BLUE" (id 1) (at 41.91 75.2474 90)
+      (effects (font (size 1.27 1.27)) (justify right))
+    )
+    (property "Footprint" "MY LED LIBRARY:19-218_BHC-ZL1M2QY_3T" (id 2) (at 38.1 72.39 0)
+      (effects (font (size 1.27 1.27)) hide)
+    )
+    (property "Datasheet" "~" (id 3) (at 38.1 72.39 0)
       (effects (font (size 1.27 1.27)) hide)
     )
@@
   (symbol (lib_id "power:GND") (at 148.59 119.38 0) (unit 1)
     (in_bom yes) (on_board yes) (fields_autoplaced)
-    (property "Reference" "#PWR0407" (id 0) (at 148.59 125.73 0)
+    (property "Reference" "#PWR0409" (id 0) (at 148.59 125.73 0)
       (effects (font (size 1.27 1.27)) hide)
     )
@@
     (pin "2")
   )
+  (symbol (lib_id "MY RESISTOR LIBRARY:0603WAF2201T5E") (at 38.1 60.96 0) (unit 1)
+    (in_bom yes) (on_board yes) (fields_autoplaced)
+    (property "Reference" "R401" (id 0) (at 40.64 59.6899 0)
+      (effects (font (size 1.27 1.27)) (justify left))
+    )
+    (property "Value" "2.2k" (id 1) (at 40.64 62.2299 0)
+      (effects (font (size 1.27 1.27)) (justify left))
+    )
+    (property "Footprint" "MY RESISTOR LIBRARY:0603WAF2201T5E" (id 2) (at 36.322 60.96 90)
+      (effects (font (size 1.27 1.27)) hide)
+    )
+    (property "Datasheet" "~" (id 3) (at 38.1 60.96 0)
+      (effects (font (size 1.27 1.27)) hide)
+    )
+    (pin "1")
+    (pin "2")
+  )
+  (symbol (lib_id "power:GND") (at 38.1 80.01 0) (unit 1)
+    (in_bom yes) (on_board yes) (fields_autoplaced)
+    (property "Reference" "#PWR0402" (id 0) (at 38.1 86.36 0)
+      (effects (font (size 1.27 1.27)) hide)
+    )
+    (property "Value" "GND" (id 1) (at 38.1 85.09 0))
+    (property "Footprint" "" (id 2) (at 38.1 80.01 0)
+      (effects (font (size 1.27 1.27)) hide)
+    )
+    (property "Datasheet" "" (id 3) (at 38.1 80.01 0)
+      (effects (font (size 1.27 1.27)) hide)
+    )
+    (pin "1")
+  )
   (symbol (lib_id "MY CAPACITOR LIBRARY:CL05B224KO5NNNC") (at 307.34 85.09 0) (unit 1)
     (in_bom yes) (on_board yes) (fields_autoplaced)
@@
   (symbol (lib_id "power:GND") (at 236.22 215.9 0) (unit 1)
     (in_bom yes) (on_board yes) (fields_autoplaced)
-    (property "Reference" "#PWR0412" (id 0) (at 236.22 222.25 0)
+    (property "Reference" "#PWR0414" (id 0) (at 236.22 222.25 0)
       (effects (font (size 1.27 1.27)) hide)
     )
@@
   (symbol (lib_id "MY RESISTOR LIBRARY:0402WGJ0225TCE") (at 99.06 110.49 0) (unit 1)
     (in_bom yes) (on_board yes) (fields_autoplaced)
-    (property "Reference" "R401" (id 0) (at 101.6 109.2199 0)
+    (property "Reference" "R402" (id 0) (at 101.6 109.2199 0)
       (effects (font (size 1.27 1.27)) (justify left))
     )
@@
   (symbol (lib_id "power:GND") (at 307.34 182.88 0) (unit 1)
     (in_bom yes) (on_board yes) (fields_autoplaced)
-    (property "Reference" "#PWR0418" (id 0) (at 307.34 189.23 0)
+    (property "Reference" "#PWR0420" (id 0) (at 307.34 189.23 0)
       (effects (font (size 1.27 1.27)) hide)
     )
@@
   (symbol (lib_id "power:GND") (at 283.21 93.98 0) (unit 1)
     (in_bom yes) (on_board yes) (fields_autoplaced)
-    (property "Reference" "#PWR0415" (id 0) (at 283.21 100.33 0)
+    (property "Reference" "#PWR0417" (id 0) (at 283.21 100.33 0)
       (effects (font (size 1.27 1.27)) hide)
     )
@@
   (symbol (lib_id "power:+3V3") (at 86.36 190.5 0) (unit 1)
     (in_bom yes) (on_board yes) (fields_autoplaced)
-    (property "Reference" "#PWR0401" (id 0) (at 86.36 194.31 0)
+    (property "Reference" "#PWR0403" (id 0) (at 86.36 194.31 0)
       (effects (font (size 1.27 1.27)) hide)
     )
@@
   (symbol (lib_id "power:GND") (at 290.83 208.28 0) (unit 1)
     (in_bom yes) (on_board yes) (fields_autoplaced)
-    (property "Reference" "#PWR0416" (id 0) (at 290.83 214.63 0)
+    (property "Reference" "#PWR0418" (id 0) (at 290.83 214.63 0)
       (effects (font (size 1.27 1.27)) hide)
     )
@@
   (symbol (lib_id "power:GND") (at 144.78 180.34 0) (unit 1)
     (in_bom yes) (on_board yes) (fields_autoplaced)
-    (property "Reference" "#PWR0406" (id 0) (at 144.78 186.69 0)
+    (property "Reference" "#PWR0408" (id 0) (at 144.78 186.69 0)
       (effects (font (size 1.27 1.27)) hide)
     )
@@
   (symbol (lib_id "power:GND") (at 111.76 119.38 0) (unit 1)
     (in_bom yes) (on_board yes) (fields_autoplaced)
-    (property "Reference" "#PWR0403" (id 0) (at 111.76 125.73 0)
+    (property "Reference" "#PWR0405" (id 0) (at 111.76 125.73 0)
       (effects (font (size 1.27 1.27)) hide)
     )
@@
   (symbol (lib_id "power:GND") (at 86.36 208.28 0) (unit 1)
     (in_bom yes) (on_board yes) (fields_autoplaced)
-    (property "Reference" "#PWR0402" (id 0) (at 86.36 214.63 0)
+    (property "Reference" "#PWR0404" (id 0) (at 86.36 214.63 0)
       (effects (font (size 1.27 1.27)) hide)
     )
@@
   (symbol (lib_id "power:GND") (at 266.7 213.36 0) (unit 1)
     (in_bom yes) (on_board yes) (fields_autoplaced)
-    (property "Reference" "#PWR0414" (id 0) (at 266.7 219.71 0)
+    (property "Reference" "#PWR0416" (id 0) (at 266.7 219.71 0)
       (effects (font (size 1.27 1.27)) hide)
     )
@@
   (symbol (lib_id "power:GND") (at 168.91 234.95 0) (unit 1)
     (in_bom yes) (on_board yes) (fields_autoplaced)
-    (property "Reference" "#PWR0409" (id 0) (at 168.91 241.3 0)
+    (property "Reference" "#PWR0411" (id 0) (at 168.91 241.3 0)
       (effects (font (size 1.27 1.27)) hide)
     )
@@
   (symbol (lib_id "power:GND") (at 153.67 215.9 0) (unit 1)
     (in_bom yes) (on_board yes) (fields_autoplaced)
-    (property "Reference" "#PWR0408" (id 0) (at 153.67 222.25 0)
-      (effects (font (size 1.27 1.27)) hide)
-    )
+    (property "Reference" "#PWR0410" (id 0) (at 153.67 222.25 0)
+      (effects (font (size 1.27 1.27)) hide)
+    )
