File: DESIGN FILES/gpio.kicad_sch (KiCad schematic)
At the start: 16 parts, among them U1 MIMXRT1064CVL5B

Commit message: updates
Parts:
- removed C501, C504, C507: 4.7u, MIMXRT1064 MCU Module:0402_CL05A475MP5NRNC, symbol MIMXRT1064 MCU Module:CL05A475MP5NRNC
- removed C502, C503, C505, C506, C509, C510, C511, C514: 100n, MIMXRT1064 MCU Module:0402_CL05B104KB54PNC, symbol MIMXRT1064 MCU Module:CL05B104KB54PNC
- removed C513: 1u, MIMXRT1064 MCU Module:0402_CL05A105KA5NQNC, symbol MIMXRT1064 MCU Module:CL05A105KA5NQNC
- removed C515: 10u, MIMXRT1064 MCU Module:0603_CL10A106KP8NNNC, symbol MIMXRT1064 MCU Module:CL10A106KP8NNNC
- removed U1: MIMXRT1064CVL5B, MIMXRT1064 MCU Module:MIMXRT1064CVL5B, symbol MIMXRT1064 MCU Module:MIMXRT1064CVL5B
- added C501, C504, C507: 4.7u, MY CAPACITOR LIBRARY:0402_CL05A475MP5NRNC, symbol MY CAPACITOR LIBRARY:CL05A475MP5NRNC
- added C502, C503, C505, C506, C509, C510, C511, C513: 100n, MY CAPACITOR LIBRARY:0402_CL05B104KB54PNC, symbol MY CAPACITOR LIBRARY:CL05B104KB54PNC
- added C514: 10u, MY CAPACITOR LIBRARY:0603_CL10A106KP8NNNC, symbol MY CAPACITOR LIBRARY:CL10A106KP8NNNC
- added U1: MIMXRT1064CVL5B, MY MICROCONTROLLER LIBRARY:MIMXRT1064CVL5B, symbol MY MICROCONTROLLER LIBRARY:MIMXRT1064CVL5B
Connections:
- net +1V8: now also C505.1, C507.1, U1.K5 (NVCC_SD1)
- net +3V3: now also C501.1, C502.1, C503.1, C504.1, C506.1, C509.1, C510.1, C511.1, U1.E6 (NVCC_EMC_1), U1.F5 (NVCC_EMC_2), U1.J6 (NVCC_SD0)
- net CODEC_SCL: now also U1.J11 (GPIO_AD_B1_00)
- net CODEC_SDA: now also U1.K11 (GPIO_AD_B1_01)
- net FLEXSPI_CLK: now also U1.L4 (GPIO_SD_B1_07)
- net FLEXSPI_D0: now also U1.P3 (GPIO_SD_B1_08)
- net FLEXSPI_D1: now also U1.N4 (GPIO_SD_B1_09)
- net FLEXSPI_D2: now also U1.P4 (GPIO_SD_B1_10)
- net FLEXSPI_D3: now also U1.P5 (GPIO_SD_B1_11)
- net FLEXSPI_SS: now also U1.L3 (GPIO_SD_B1_06)
- net GND: now also C501.2, C502.2, C503.2, C504.2, C505.2, C506.2, C507.2, C509.2, C510.2, C511.2, C513.2, C514.2, U1.E9 (NVCC_GPIO_1), U1.F10 (NVCC_GPIO_2), U1.F13 (GPIO_AD_B0_08), U1.J10 (NVCC_GPIO_3)
- net GPIO_AD_B0_00: now also U1.M14 (GPIO_AD_B0_00)
- net GPIO_AD_B0_01: now also U1.H10 (GPIO_AD_B0_01)
- net GPIO_AD_B0_02: now also U1.M11 (GPIO_AD_B0_02)
- net GPIO_AD_B0_03: now also U1.G11 (GPIO_AD_B0_03)
- net GPIO_AD_B0_04: now also U1.F11 (GPIO_AD_B0_04)
- net GPIO_AD_B0_05: now also U1.G14 (GPIO_AD_B0_05)
- net GPIO_AD_B0_12: now also U1.K14 (GPIO_AD_B0_12)
- net GPIO_AD_B0_13: now also U1.L14 (GPIO_AD_B0_13)
- net GPIO_AD_B0_14: now also U1.H14 (GPIO_AD_B0_14)
- net GPIO_AD_B0_15: now also U1.L10 (GPIO_AD_B0_15)
- net GPIO_AD_B1_02: now also U1.L11 (GPIO_AD_B1_02)
- net GPIO_AD_B1_04: now also U1.L12 (GPIO_AD_B1_04)
- net GPIO_AD_B1_05: now also U1.K12 (GPIO_AD_B1_05)
- net GPIO_AD_B1_06: now also U1.J12 (GPIO_AD_B1_06)
- net GPIO_AD_B1_07: now also U1.K10 (GPIO_AD_B1_07)
- net GPIO_AD_B1_08: now also U1.H13 (GPIO_AD_B1_08)
- net GPIO_AD_B1_10: now also U1.L13 (GPIO_AD_B1_10)
- net GPIO_AD_B1_11: now also U1.J13 (GPIO_AD_B1_11)
- net GPIO_B0_00: now also U1.D7 (GPIO_B0_00)
- net GPIO_B0_01: now also U1.E7 (GPIO_B0_01)
- net GPIO_B0_02: now also U1.E8 (GPIO_B0_02)
- net GPIO_B0_03: now also U1.D8 (GPIO_B0_03)
- net GPIO_B0_04: now also U1.C8 (GPIO_B0_04)
- net GPIO_B0_05: now also U1.B8 (GPIO_B0_05)
- net GPIO_B0_06: now also U1.A8 (GPIO_B0_06)
- net GPIO_B0_07: now also U1.A9 (GPIO_B0_07)
- net GPIO_B0_08: now also U1.B9 (GPIO_B0_08)
- net GPIO_B0_09: now also U1.C9 (GPIO_B0_09)
- net GPIO_B0_10: now also U1.D9 (GPIO_B0_10)
- net GPIO_B0_11: now also U1.A10 (GPIO_B0_11)
- net GPIO_B0_12: now also U1.C10 (GPIO_B0_12)
- net GPIO_B0_13: now also U1.D10 (GPIO_B0_13)
- net GPIO_B0_14: now also U1.E10 (GPIO_B0_14)
- net GPIO_B0_15: now also U1.E11 (GPIO_B0_15)
- net GPIO_B1_00: now also U1.A11 (GPIO_B1_00)
- net GPIO_B1_01: now also U1.B11 (GPIO_B1_01)
- net GPIO_B1_02: now also U1.C11 (GPIO_B1_02)
- net GPIO_B1_03: now also U1.D11 (GPIO_B1_03)
- net GPIO_B1_04: now also U1.E12 (GPIO_B1_04)
- net GPIO_B1_05: now also U1.D12 (GPIO_B1_05)
- net GPIO_B1_06: now also U1.C12 (GPIO_B1_06)
- net GPIO_B1_07: now also U1.B12 (GPIO_B1_07)
- net GPIO_B1_08: now also U1.A12 (GPIO_B1_08)
- net GPIO_B1_09: now also U1.A13 (GPIO_B1_09)
- net GPIO_B1_10: now also U1.B13 (GPIO_B1_10)
- net GPIO_B1_11: now also U1.C13 (GPIO_B1_11)
- net GPIO_B1_13: now also U1.D14 (GPIO_B1_13)
- net GPIO_B1_14: now also U1.C14 (GPIO_B1_14)
- net GPIO_B1_15: now also U1.B14 (GPIO_B1_15)
- net GPIO_EMC_40: now also U1.A7 (GPIO_EMC_40)
- net GPIO_EMC_41: now also U1.C7 (GPIO_EMC_41)
- net I2S_ADCDAT: now also U1.H12 (GPIO_AD_B1_12)
- net I2S_BCLK: now also U1.G12 (GPIO_AD_B1_14)
- net I2S_DACDAT: now also U1.H11 (GPIO_AD_B1_13)
- net I2S_LRC: now also U1.J14 (GPIO_AD_B1_15)
- net I2S_MCLK: now also U1.M13 (GPIO_AD_B1_09)
- net JTAG_TCK: now also U1.F12 (GPIO_AD_B0_07)
- net JTAG_TDI: now also U1.F14 (GPIO_AD_B0_09)
- net JTAG_TDO: now also U1.G13 (GPIO_AD_B0_10)
- net JTAG_TMS: now also U1.E14 (GPIO_AD_B0_06)
- net JTAG_nTRST: now also U1.G10 (GPIO_AD_B0_11)
- net SDRAM_A0: now also U1.C2 (GPIO_EMC_09)
- net SDRAM_A1: now also U1.G1 (GPIO_EMC_10)
- net SDRAM_A10: now also U1.G2 (GPIO_EMC_23)
- net SDRAM_A11: now also U1.B4 (GPIO_EMC_19)
- net SDRAM_A12: now also U1.A3 (GPIO_EMC_20)
- net SDRAM_A2: now also U1.G3 (GPIO_EMC_11)
- net SDRAM_A3: now also U1.H1 (GPIO_EMC_12)
- net SDRAM_A4: now also U1.A6 (GPIO_EMC_13)
- net SDRAM_A5: now also U1.B6 (GPIO_EMC_14)
- net SDRAM_A6: now also U1.B1 (GPIO_EMC_15)
- net SDRAM_A7: now also U1.A5 (GPIO_EMC_16)
- net SDRAM_A8: now also U1.A4 (GPIO_EMC_17)
- net SDRAM_A9: now also U1.B2 (GPIO_EMC_18)
- net SDRAM_BA0: now also U1.C1 (GPIO_EMC_21)
- net SDRAM_BA1: now also U1.F1 (GPIO_EMC_22)
- net SDRAM_CAS: now also U1.D3 (GPIO_EMC_24)
- net SDRAM_CKE: now also U1.A2 (GPIO_EMC_27)
- net SDRAM_CLK: now also U1.B3 (GPIO_EMC_26)
- net SDRAM_CS: now also U1.E1 (GPIO_EMC_29)
- net SDRAM_D0: now also U1.E3 (GPIO_EMC_00)
- net SDRAM_D1: now also U1.F3 (GPIO_EMC_01)
- net SDRAM_D10: now also U1.D5 (GPIO_EMC_32)
- net SDRAM_D11: now also U1.C4 (GPIO_EMC_33)
- net SDRAM_D12: now also U1.D4 (GPIO_EMC_34)
- net SDRAM_D13: now also U1.E5 (GPIO_EMC_35)
- net SDRAM_D14: now also U1.C3 (GPIO_EMC_36)
- net SDRAM_D15: now also U1.E4 (GPIO_EMC_37)
- net SDRAM_D2: now also U1.F4 (GPIO_EMC_02)
- net SDRAM_D3: now also U1.G4 (GPIO_EMC_03)
- net SDRAM_D4: now also U1.F2 (GPIO_EMC_04)
- net SDRAM_D5: now also U1.G5 (GPIO_EMC_05)
- net SDRAM_D6: now also U1.H5 (GPIO_EMC_06)
- net SDRAM_D7: now also U1.H4 (GPIO_EMC_07)
- net SDRAM_D8: now also U1.C6 (GPIO_EMC_30)
- net SDRAM_D9: now also U1.C5 (GPIO_EMC_31)
- net SDRAM_DQMH: now also U1.D6 (GPIO_EMC_38)
- net SDRAM_DQML: now also U1.H3 (GPIO_EMC_08)
- net SDRAM_RAS: now also U1.D2 (GPIO_EMC_25)
- net SDRAM_WE: now also U1.D1 (GPIO_EMC_28)
- net SD_CD_SW: now also U1.D13 (GPIO_B1_12)
- net SD_CLK: now also U1.J3 (GPIO_SD_B0_01)
- net SD_CMD: now also U1.J4 (GPIO_SD_B0_00)
- net SD_DAT0: now also U1.J1 (GPIO_SD_B0_02)
- net SD_DAT1: now also U1.K1 (GPIO_SD_B0_03)
- net SD_DAT2: now also U1.H2 (GPIO_SD_B0_04)
- net SD_DAT3: now also U1.J2 (GPIO_SD_B0_05)
- net SD_PWREN: now also U1.M12 (GPIO_AD_B1_03)
- net USB_OTG1_VBUS renamed +5V
- net +5V: now also U1.N6 (USB_OTG1_VBUS)
- new net: C513.1, C514.1, U1.K8 (VDD_USB_CAP)
- new net USB_D+: U1.L8 (USB_OTG1_DP)
- new net USB_D-: U1.M8 (USB_OTG1_DN)
- no-connect marks 7 -> 11

Commit message: updates
Parts:
- removed C508: 4.7u, MIMXRT1064 MCU Module:0402_CL05A475MP5NRNC, symbol MIMXRT1064 MCU Module:CL05A475MP5NRNC
- removed C512: 1u, MIMXRT1064 MCU Module:0402_CL05A105KA5NQNC, symbol MIMXRT1064 MCU Module:CL05A105KA5NQNC
- added C508: 4.7u, MY CAPACITOR LIBRARY:0402_CL05A475MP5NRNC, symbol MY CAPACITOR LIBRARY:CL05A475MP5NRNC
- added C512: 1u, MY CAPACITOR LIBRARY:0402_CL05A105KA5NQNC, symbol MY CAPACITOR LIBRARY:CL05A105KA5NQNC
Connections:
- net +3V3: now also C508.1
- net +5V: now also C512.1
- net GND: now also C508.2, C512.2
- net GPIO_B1_13 renamed WATCHDOG_B
- net GPIO_EMC_40: no longer names the net of U1.A7 (GPIO_EMC_40)
- net GPIO_EMC_41: no longer names the net of U1.C7 (GPIO_EMC_41)
- net SD_CD_SW renamed GPIO_B1_12
- net SD_CLK: no longer names the net of U1.J3 (GPIO_SD_B0_01)
- net SD_CMD: no longer names the net of U1.J4 (GPIO_SD_B0_00)
- net SD_DAT0: no longer names the net of U1.J1 (GPIO_SD_B0_02)
- net SD_DAT1: no longer names the net of U1.K1 (GPIO_SD_B0_03)
- net SD_DAT2: no longer names the net of U1.H2 (GPIO_SD_B0_04)
- net SD_DAT3: no longer names the net of U1.J2 (GPIO_SD_B0_05)
- net SD_PWREN renamed GPIO_AD_B1_03
- no-connect marks 11 -> 19
Other:
- note removed: "SD CARD BUS"
- title: MIMXRT1064 MCU Module -> MIMXRT1064 Audio Board

Commit message: updates
Parts:
- renumbered C512 to C510, C510 to C511, C511 to C512, U1 to U401
Connections:
- net SD_DAT2: now reaches U401.H2 (GPIO_SD_B0_04)
- net SD_DAT0: now reaches U401.J1 (GPIO_SD_B0_02)
- net SD_DAT3: now reaches U401.J2 (GPIO_SD_B0_05)
- net SD_CLK: now reaches U401.J3 (GPIO_SD_B0_01)
- net SD_CMD: now reaches U401.J4 (GPIO_SD_B0_00)
- net SD_DAT1: now reaches U401.K1 (GPIO_SD_B0_03)
- net +5V renamed VBUS
- net GPIO_AD_B0_00: no longer names the net of U401.M14 (GPIO_AD_B0_00)
- net GPIO_AD_B0_01: no longer names the net of U401.H10 (GPIO_AD_B0_01)
- net GPIO_AD_B0_02: no longer names the net of U401.M11 (GPIO_AD_B0_02)
- net GPIO_AD_B0_03: no longer names the net of U401.G11 (GPIO_AD_B0_03)
- net GPIO_AD_B0_04: no longer names the net of U401.F11 (GPIO_AD_B0_04)
- net GPIO_AD_B0_05: no longer names the net of U401.G14 (GPIO_AD_B0_05)
- net GPIO_AD_B0_12 renamed MIDI_IN
- net GPIO_AD_B0_13 renamed MIDI_OUT
- net GPIO_AD_B0_14: no longer names the net of U401.H14 (GPIO_AD_B0_14)
- net GPIO_AD_B0_15: no longer names the net of U401.L10 (GPIO_AD_B0_15)
- net GPIO_AD_B1_02: no longer names the net of U401.L11 (GPIO_AD_B1_02)
- net GPIO_AD_B1_03: no longer names the net of U401.M12 (GPIO_AD_B1_03)
- net GPIO_AD_B1_04: no longer names the net of U401.L12 (GPIO_AD_B1_04)
- net GPIO_AD_B1_05: no longer names the net of U401.K12 (GPIO_AD_B1_05)
- net GPIO_AD_B1_06: no longer names the net of U401.J12 (GPIO_AD_B1_06)
- net GPIO_AD_B1_07: no longer names the net of U401.K10 (GPIO_AD_B1_07)
- net GPIO_AD_B1_08: no longer names the net of U401.H13 (GPIO_AD_B1_08)
- net GPIO_AD_B1_10: no longer names the net of U401.L13 (GPIO_AD_B1_10)
- net GPIO_AD_B1_11: no longer names the net of U401.J13 (GPIO_AD_B1_11)
- net GPIO_B0_00 renamed SPI_CS
- net GPIO_B0_01 renamed SPI_SIN
- net GPIO_B0_02 renamed SPI_SOUT
- net GPIO_B0_03 renamed SPI_SCK
- net GPIO_B0_04 renamed IO26
- net GPIO_B0_05 renamed IO27
- net GPIO_B0_06 renamed IO28
- net GPIO_B0_07 renamed IO25
- net GPIO_B0_08 renamed IO24
- net GPIO_B0_09 renamed IO23
- net GPIO_B0_10 renamed IO1
- net GPIO_B0_11 renamed IO22
- net GPIO_B0_12 renamed IO21
- net GPIO_B0_13 renamed IO3
- net GPIO_B0_14 renamed IO2
- net GPIO_B0_15 renamed IO4
- net GPIO_B1_00 renamed IO20
- net GPIO_B1_01 renamed IO19
- net GPIO_B1_02 renamed IO6
- net GPIO_B1_03 renamed IO5
- net GPIO_B1_04 renamed IO7
- net GPIO_B1_05 renamed IO8
- net GPIO_B1_06 renamed IO9
- net GPIO_B1_07 renamed IO17
- net GPIO_B1_08 renamed IO18
- net GPIO_B1_09 renamed IO16
- net GPIO_B1_10 renamed IO15
- net GPIO_B1_11 renamed IO11
- net GPIO_B1_12 renamed IO10
- net GPIO_B1_14 renamed IO13
- net GPIO_B1_15 renamed IO14
- net WATCHDOG_B renamed IO12
- no-connect marks 19 -> 30
Other:
- note added: "JTAG_MOD : GND for normal operation"
- note added: "USB OTG (Module is device only)"
- note added: "VBUS from carrier board"
- note added: "[5] MCU GPIO & BUS"
- note added: "uSD BUS"
- note removed: "5 : MCU GPIO & BUS"
- note removed: "USB OTG"
- title: MIMXRT1064 Audio Board -> MIMXRT1064 MCU Module

Commit message: updates
Parts:
- added R501, R502, R503, R504, R505, R506: 0R, symbol MY RESISTOR LIBRARY:0603WAF0000T5E
Connections:
- net FLEXSPI_CLK: now also R503.2; no longer U401.L4 (GPIO_SD_B1_07)
- net I2S_BCLK: now also R505.1; no longer U401.G12 (GPIO_AD_B1_14)
- net I2S_LRC: now also R506.1; no longer U401.J14 (GPIO_AD_B1_15)
- net I2S_MCLK: now also R504.1; no longer U401.M13 (GPIO_AD_B1_09)
- net MIDI_IN: now also U401.L14 (GPIO_AD_B0_13); no longer U401.K14 (GPIO_AD_B0_12)
- net MIDI_OUT: now also U401.K14 (GPIO_AD_B0_12); no longer U401.L14 (GPIO_AD_B0_13)
- net SDRAM_CLK: now also R501.2; no longer U401.B3 (GPIO_EMC_26)
- net SD_CLK: now also R502.2; no longer U401.J3 (GPIO_SD_B0_01)
- new net: R505.2, U401.G12 (GPIO_AD_B1_14)
- new net: R506.2, U401.J14 (GPIO_AD_B1_15)
- new net: R504.2, U401.M13 (GPIO_AD_B1_09)
- new net: R503.1, U401.L4 (GPIO_SD_B1_07)
- new net: R502.1, U401.J3 (GPIO_SD_B0_01)
- new net: R501.1, U401.B3 (GPIO_EMC_26)
Other:
- note added: "Differential pair"

Commit message: updates
Parts:
- R501, R502, R503, R504, R505, R506: footprint (none) -> MY RESISTOR LIBRARY:0603WAF0000T5E
Connections:
- net USB CAP: now reaches C513.1, C514.1, U401.K8 (VDD_USB_CAP)
Changed lines of the file:
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@@
     (effects (font (size 1.27 1.27) bold italic) (justify left bottom))
+  )
+  (label "USB CAP" (at 344.17 219.71 0)
+    (effects (font (size 1.27 1.27) (thickness 0.254) bold italic) (justify left bottom))
   )
   (global_label "SDRAM_D13" (shape input) (at 144.78 146.05 0) (fields_autoplaced)
@@
     (property "Reference" "R503" (id 0) (at 138.43 247.65 90))
     (property "Value" "0R" (id 1) (at 143.51 246.38 90))
-    (property "Footprint" "" (id 2) (at 138.43 249.428 90)
+    (property "Footprint" "MY RESISTOR LIBRARY:0603WAF0000T5E" (id 2) (at 138.43 249.428 90)
       (effects (font (size 1.27 1.27)) hide)
     )
@@
     (property "Reference" "R502" (id 0) (at 138.43 214.63 90))
     (property "Value" "0R" (id 1) (at 142.24 213.36 90))
-    (property "Footprint" "" (id 2) (at 138.43 216.408 90)
+    (property "Footprint" "MY RESISTOR LIBRARY:0603WAF0000T5E" (id 2) (at 138.43 216.408 90)
       (effects (font (size 1.27 1.27)) hide)
     )
@@
     (property "Reference" "R504" (id 0) (at 281.94 142.24 90))
     (property "Value" "0R" (id 1) (at 285.75 140.97 90))
-    (property "Footprint" "" (id 2) (at 281.94 144.018 90)
+    (property "Footprint" "MY RESISTOR LIBRARY:0603WAF0000T5E" (id 2) (at 281.94 144.018 90)
       (effects (font (size 1.27 1.27)) hide)
     )
@@
     (property "Reference" "R501" (id 0) (at 138.43 123.19 90))
     (property "Value" "0R" (id 1) (at 143.51 124.46 90))
-    (property "Footprint" "" (id 2) (at 138.43 124.968 90)
+    (property "Footprint" "MY RESISTOR LIBRARY:0603WAF0000T5E" (id 2) (at 138.43 124.968 90)
       (effects (font (size 1.27 1.27)) hide)
     )
@@
     (property "Reference" "R506" (id 0) (at 281.94 157.48 90))
     (property "Value" "0R" (id 1) (at 285.75 156.21 90))
-    (property "Footprint" "" (id 2) (at 281.94 159.258 90)
+    (property "Footprint" "MY RESISTOR LIBRARY:0603WAF0000T5E" (id 2) (at 281.94 159.258 90)
       (effects (font (size 1.27 1.27)) hide)
     )
@@
     (property "Reference" "R505" (id 0) (at 281.94 154.94 90))
     (property "Value" "0R" (id 1) (at 285.75 153.67 90))
-    (property "Footprint" "" (id 2) (at 281.94 156.718 90)
-      (effects (font (size 1.27 1.27)) hide)
-    )
+    (property "Footprint" "MY RESISTOR LIBRARY:0603WAF0000T5E" (id 2) (at 281.94 156.718 90)
+      (effects (font (size 1.27 1.27)) hide)
+    )

Commit message: updates
Connections:
- net +3V3: now also U401.E9 (NVCC_GPIO_1), U401.F10 (NVCC_GPIO_2), U401.J10 (NVCC_GPIO_3)
- net GND: no longer U401.E9 (NVCC_GPIO_1), U401.F10 (NVCC_GPIO_2), U401.J10 (NVCC_GPIO_3)
Other:
- moved on the sheet: C508, C509, C511, C512

Commit message: updates
Parts:
- renumbered C511 to C510, C510 to C511
Changed lines of the file:
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@@
   (symbol (lib_id "MY CAPACITOR LIBRARY:CL05B104KB54PNC") (at 254 72.39 0) (unit 1)
     (in_bom yes) (on_board yes) (fields_autoplaced)
-    (property "Reference" "C511" (id 0) (at 257.81 71.1199 0)
+    (property "Reference" "C510" (id 0) (at 257.81 71.1199 0)
       (effects (font (size 1.27 1.27)) (justify left))
     )
@@
   (symbol (lib_id "MY CAPACITOR LIBRARY:CL05A105KA5NQNC") (at 254 219.71 0) (unit 1)
     (in_bom yes) (on_board yes) (fields_autoplaced)
-    (property "Reference" "C510" (id 0) (at 257.81 218.4399 0)
-      (effects (font (size 1.27 1.27)) (justify left))
-    )
+    (property "Reference" "C511" (id 0) (at 257.81 218.4399 0)
+      (effects (font (size 1.27 1.27)) (justify left))
+    )

Commit message: updates
Connections:
- net I2S_BCLK_RES: now reaches R505.2, U401.G12 (GPIO_AD_B1_14)
- net I2C_LRC_RES: now reaches R506.2, U401.J14 (GPIO_AD_B1_15)
- net I2S_MCLK_RES: now reaches R504.2, U401.M13 (GPIO_AD_B1_09)
- net FLEXSPI_CLK_RES: now reaches R503.1, U401.L4 (GPIO_SD_B1_07)
- net SD_CLK_RES: now reaches R502.1, U401.J3 (GPIO_SD_B0_01)
- net SDRAM_CLK_RES: now reaches R501.1, U401.B3 (GPIO_EMC_26)
Other:
- note added: "! A trace must be routed !"
- moved on the sheet: R501, R502, R503, R504, R505, R506
