File: DESIGN FILES/gpio.kicad_sch (KiCad schematic)
At the start: 21 parts, among them U401 MIMXRT1064CVL5B

Commit message: updates
Parts:
- renumbered R502 to R501, R501 to R502, R505 to R504, R506 to R505, R504 to R506
Changed lines of the file:
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@@
   (symbol (lib_id "MY RESISTOR LIBRARY:0603WAF0000T5E") (at 158.75 214.63 90) (unit 1)
     (in_bom yes) (on_board yes)
-    (property "Reference" "R502" (id 0) (at 158.75 214.63 90))
+    (property "Reference" "R501" (id 0) (at 158.75 214.63 90))
     (property "Value" "0R" (id 1) (at 162.56 215.9 90))
     (property "Footprint" "MY RESISTOR LIBRARY:0603WAF0000T5E" (id 2) (at 158.75 216.408 90)
@@
   (symbol (lib_id "MY RESISTOR LIBRARY:0603WAF0000T5E") (at 265.43 142.24 90) (unit 1)
     (in_bom yes) (on_board yes)
-    (property "Reference" "R504" (id 0) (at 265.43 142.24 90))
+    (property "Reference" "R506" (id 0) (at 265.43 142.24 90))
     (property "Value" "0R" (id 1) (at 259.08 143.51 90))
     (property "Footprint" "MY RESISTOR LIBRARY:0603WAF0000T5E" (id 2) (at 265.43 144.018 90)
@@
   (symbol (lib_id "MY RESISTOR LIBRARY:0603WAF0000T5E") (at 160.02 123.19 90) (unit 1)
     (in_bom yes) (on_board yes)
-    (property "Reference" "R501" (id 0) (at 160.02 123.19 90))
+    (property "Reference" "R502" (id 0) (at 160.02 123.19 90))
     (property "Value" "0R" (id 1) (at 165.1 124.46 90))
     (property "Footprint" "MY RESISTOR LIBRARY:0603WAF0000T5E" (id 2) (at 160.02 124.968 90)
@@
   (symbol (lib_id "MY RESISTOR LIBRARY:0603WAF0000T5E") (at 264.16 157.48 90) (unit 1)
     (in_bom yes) (on_board yes)
-    (property "Reference" "R506" (id 0) (at 264.16 157.48 90))
+    (property "Reference" "R505" (id 0) (at 264.16 157.48 90))
     (property "Value" "0R" (id 1) (at 259.08 158.75 90))
     (property "Footprint" "MY RESISTOR LIBRARY:0603WAF0000T5E" (id 2) (at 264.16 159.258 90)
@@
   (symbol (lib_id "MY RESISTOR LIBRARY:0603WAF0000T5E") (at 264.16 154.94 90) (unit 1)
     (in_bom yes) (on_board yes)
-    (property "Reference" "R505" (id 0) (at 264.16 154.94 90))
+    (property "Reference" "R504" (id 0) (at 264.16 154.94 90))
     (property "Value" "0R" (id 1) (at 259.08 156.21 90))
     (property "Footprint" "MY RESISTOR LIBRARY:0603WAF0000T5E" (id 2) (at 264.16 156.718 90)

Commit message: updates
Parts:
- removed R502: 0R, MY RESISTOR LIBRARY:0603WAF0000T5E, symbol MY RESISTOR LIBRARY:0603WAF0000T5E
Connections:
- net SDRAM_CLK_RES is gone; now on net SDRAM_CLK: U401.B3 (GPIO_EMC_26)
Changed lines of the file:
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@@
-    (stroke (width 0) (type default) (color 0 0 0 0))
-  )
-  (wire (pts (xy 163.83 123.19) (xy 167.64 123.19))
     (stroke (width 0) (type default) (color 0 0 0 0))
   )
@@
     (stroke (width 0) (type default) (color 0 0 0 0))
   )
-  (wire (pts (xy 132.08 123.19) (xy 156.21 123.19))
+  (wire (pts (xy 132.08 123.19) (xy 167.64 123.19))
     (stroke (width 0) (type default) (color 0 0 0 0))
   )
@@
   )
   (label "FLEXSPI_CLK_RES" (at 133.35 247.65 0)
-    (effects (font (size 1.27 1.27)) (justify left bottom))
-  )
-  (label "SDRAM_CLK_RES" (at 133.35 123.19 0)
     (effects (font (size 1.27 1.27)) (justify left bottom))
   )
@@
     (pin "1")
   )
-  (symbol (lib_id "MY RESISTOR LIBRARY:0603WAF0000T5E") (at 160.02 123.19 90) (unit 1)
-    (in_bom yes) (on_board yes)
-    (property "Reference" "R502" (id 0) (at 160.02 123.19 90))
-    (property "Value" "0R" (id 1) (at 165.1 124.46 90))
-    (property "Footprint" "MY RESISTOR LIBRARY:0603WAF0000T5E" (id 2) (at 160.02 124.968 90)
-      (effects (font (size 1.27 1.27)) hide)
-    )
-    (property "Datasheet" "~" (id 3) (at 160.02 123.19 0)
-      (effects (font (size 1.27 1.27)) hide)
-    )
-    (pin "1")
-    (pin "2")
-  )
   (symbol (lib_id "MY CAPACITOR LIBRARY:CL05A475MP5NRNC") (at 229.87 72.39 0) (unit 1)

Commit message: updates
Parts:
- removed R501, R503: 0R, MY RESISTOR LIBRARY:0603WAF0000T5E, symbol MY RESISTOR LIBRARY:0603WAF0000T5E
Connections:
- net FLEXSPI_CLK_RES is gone; now on net FLEXSPI_CLK: U401.L4 (GPIO_SD_B1_07)
- net SD_CLK_RES is gone; now on net SD_CLK: U401.J3 (GPIO_SD_B0_01)
Changed lines of the file:
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@@
-    (stroke (width 0) (type default) (color 0 0 0 0))
-  )
-  (wire (pts (xy 132.08 247.65) (xy 157.48 247.65))
     (stroke (width 0) (type default) (color 0 0 0 0))
   )
@@
     (stroke (width 0) (type default) (color 0 0 0 0))
   )
-  (wire (pts (xy 162.56 214.63) (xy 165.1 214.63))
-    (stroke (width 0) (type default) (color 0 0 0 0))
-  )
   (wire (pts (xy 335.28 91.44) (xy 347.98 91.44))
     (stroke (width 0) (type default) (color 0 0 0 0))
@@
     (stroke (width 0.5) (type default) (color 0 0 0 0))
   )
+  (wire (pts (xy 132.08 214.63) (xy 144.78 214.63))
+    (stroke (width 0) (type default) (color 0 0 0 0))
+  )
   (wire (pts (xy 229.87 78.74) (xy 229.87 81.28))
     (stroke (width 0) (type default) (color 0 0 0 0))
@@
     (stroke (width 0) (type default) (color 0 0 0 0))
   )
-  (wire (pts (xy 132.08 214.63) (xy 154.94 214.63))
-    (stroke (width 0) (type default) (color 0 0 0 0))
-  )
   (wire (pts (xy 85.09 57.15) (xy 87.63 57.15))
     (stroke (width 0) (type default) (color 0 0 0 0))
@@
     (stroke (width 0) (type default) (color 0 0 0 0))
   )
-  (wire (pts (xy 170.18 247.65) (xy 165.1 247.65))
+  (wire (pts (xy 132.08 247.65) (xy 144.78 247.65))
     (stroke (width 0) (type default) (color 0 0 0 0))
   )
@@
   (text "JTAG_MOD : GND for normal operation" (at 226.06 96.52 0)
     (effects (font (size 1.27 1.27) bold italic) (justify left bottom))
-  )
-  (label "FLEXSPI_CLK_RES" (at 133.35 247.65 0)
-    (effects (font (size 1.27 1.27)) (justify left bottom))
   )
   (label "I2S_BCLK_RES" (at 275.59 154.94 0)
@@
     )
   )
-  (global_label "FLEXSPI_CLK" (shape input) (at 170.18 247.65 0) (fields_autoplaced)
-    (effects (font (size 1.27 1.27) (thickness 0.254) bold italic) (justify left))
-    (property "Intersheet References" "${INTERSHEET_REFS}" (id 0) (at 185.1343 247.523 0)
+  (global_label "FLEXSPI_CLK" (shape input) (at 144.78 247.65 0) (fields_autoplaced)
+    (effects (font (size 1.27 1.27) (thickness 0.254) bold italic) (justify left))
+    (property "Intersheet References" "${INTERSHEET_REFS}" (id 0) (at 159.7343 247.523 0)
       (effects (font (size 1.27 1.27) (thickness 0.254) bold italic) (justify left) hide)
     )
@@
     )
   )
-  (global_label "SD_CLK" (shape input) (at 165.1 214.63 0) (fields_autoplaced)
-    (effects (font (size 1.27 1.27) bold italic) (justify left))
-    (property "Intersheet References" "${INTERSHEET_REFS}" (id 0) (at 174.9743 214.757 0)
+  (global_label "SD_CLK" (shape input) (at 144.78 214.63 0) (fields_autoplaced)
+    (effects (font (size 1.27 1.27) bold italic) (justify left))
+    (property "Intersheet References" "${INTERSHEET_REFS}" (id 0) (at 154.6543 214.757 0)
       (effects (font (size 1.27 1.27) bold italic) (justify left) hide)
     )
@@
     (pin "P5")
   )
-  (symbol (lib_id "MY RESISTOR LIBRARY:0603WAF0000T5E") (at 161.29 247.65 90) (unit 1)
-    (in_bom yes) (on_board yes)
-    (property "Reference" "R503" (id 0) (at 161.29 247.65 90))
-    (property "Value" "0R" (id 1) (at 166.37 248.92 90))
-    (property "Footprint" "MY RESISTOR LIBRARY:0603WAF0000T5E" (id 2) (at 161.29 249.428 90)
-      (effects (font (size 1.27 1.27)) hide)
-    )
-    (property "Datasheet" "~" (id 3) (at 161.29 247.65 0)
-      (effects (font (size 1.27 1.27)) hide)
-    )
-    (pin "1")
-    (pin "2")
-  )
   (symbol (lib_id "MY CAPACITOR LIBRARY:CL05B104KB54PNC") (at 254 72.39 0) (unit 1)
     (in_bom yes) (on_board yes) (fields_autoplaced)
@@
     (pin "1")
   )
-  (symbol (lib_id "MY RESISTOR LIBRARY:0603WAF0000T5E") (at 158.75 214.63 90) (unit 1)
-    (in_bom yes) (on_board yes)
-    (property "Reference" "R501" (id 0) (at 158.75 214.63 90))
-    (property "Value" "0R" (id 1) (at 162.56 215.9 90))
-    (property "Footprint" "MY RESISTOR LIBRARY:0603WAF0000T5E" (id 2) (at 158.75 216.408 90)
-      (effects (font (size 1.27 1.27)) hide)
-    )
-    (property "Datasheet" "~" (id 3) (at 158.75 214.63 0)
-      (effects (font (size 1.27 1.27)) hide)
-    )
-    (pin "1")
-    (pin "2")
-  )
   (symbol (lib_id "MY RESISTOR LIBRARY:0603WAF0000T5E") (at 265.43 142.24 90) (unit 1)

Commit message: up
Parts:
- removed R504, R505, R506: 0R, MY RESISTOR LIBRARY:0603WAF0000T5E, symbol MY RESISTOR LIBRARY:0603WAF0000T5E
Connections:
- net I2C_LRC_RES is gone; now on net I2S_LRC: U401.J14 (GPIO_AD_B1_15)
- net I2S_BCLK_RES is gone; now on net I2S_BCLK: U401.G12 (GPIO_AD_B1_14)
- net I2S_MCLK_RES is gone; now on net I2S_MCLK: U401.M13 (GPIO_AD_B1_09)
- net IO24: now also U401.A9 (GPIO_B0_07); no longer U401.B9 (GPIO_B0_08)
- net IO25: now also U401.B9 (GPIO_B0_08); no longer U401.A9 (GPIO_B0_07)
- net IO27: now also U401.A8 (GPIO_B0_06); no longer U401.B8 (GPIO_B0_05)
- net IO28: now also U401.B8 (GPIO_B0_05); no longer U401.A8 (GPIO_B0_06)
