File: DESIGN FILES/MIMXRT1064 MCU Module.kicad_pcb (KiCad board)
At the start: 2 copper layers, 40.1 x 40 mm, 97 parts, among them J1 TF-15x15, U1 MIMXRT1064CVL5B, U2 IS25WP064A-JBLE, U3 IS42S16160J-6BLI, U4 IRLML6401, U5 WM8978CGEFL/RV, Y1 24MHz, Y2 32.768KHz

Commit message: updates
Parts:
- removed the C10 at (220.5, 96.7)
- removed the C12 at (223.9, 96.5)
- removed the C17 at (216.5, 96.7)
- removed the C20 at (216.5, 99.2)
- removed the C24 at (244.2, 120.2)
- removed the C31 at (257.0, 108.7)
- removed the C32 at (244.2, 117.6)
- removed the C33 at (253.4, 111.1)
- removed the L1 at (176.6, 76.8)
- removed the R2 at (163.2, 57.8)
- removed the R3 at (215.9, 101.5)
- removed the R4 at (219.9, 99.0)
- removed the R6 at (247.7, 117.4)
- removed the R7 at (238.6, 122.4)
- removed the U4 at (259.4, 83.3)
- added C62: 22uF, MIMXRT1064 MCU Module:0603_CL10A226MQ8NRNC, F.Cu at (200.4, 57.8)
- added C63: 100nF, MIMXRT1064 MCU Module:0402_CL05B104KB54PNC, F.Cu at (202.7, 60.1)
- added C64: 100nF, MIMXRT1064 MCU Module:0402_CL05B104KB54PNC, F.Cu at (210.4, 52.6)
- added C65: 22pF, MIMXRT1064 MCU Module:0402CG220J500NT, F.Cu at (206.7, 57.1)
- added C66: 22uF, MIMXRT1064 MCU Module:0603_CL10A226MQ8NRNC, F.Cu at (192.3, 59.8)
- added C67: 22uF, MIMXRT1064 MCU Module:0603_CL10A226MQ8NRNC, F.Cu at (221.2, 42.2)
- added C68: 22uF, MIMXRT1064 MCU Module:0603_CL10A226MQ8NRNC, F.Cu at (196.3, 59.8)
- added C69: 100nF, MIMXRT1064 MCU Module:0402_CL05B104KB54PNC, F.Cu at (203.8, 57.1)
- added C70: 22pF, MIMXRT1064 MCU Module:0402CG220J500NT, F.Cu at (219.5, 46.9)
- added C71: 22uF, MIMXRT1064 MCU Module:0603_CL10A226MQ8NRNC, F.Cu at (216.1, 47.1)
- added C72: 22uF, MIMXRT1064 MCU Module:0603_CL10A226MQ8NRNC, F.Cu at (204.0, 52.8)
- added D1: RB521S30_R1_00001, MIMXRT1064 MCU Module:RB521S30_R1_00001, F.Cu at (229.1, 52.6)
- added D2: RB521S30_R1_00001, MIMXRT1064 MCU Module:RB521S30_R1_00001, F.Cu at (229.1, 50.2)
- added D3: RB521S30_R1_00001, MIMXRT1064 MCU Module:RB521S30_R1_00001, F.Cu at (188.2, 59.7)
- added D4: RB521S30_R1_00001, MIMXRT1064 MCU Module:RB521S30_R1_00001, F.Cu at (194.2, 57.4)
- added L2: 2.2uH, MIMXRT1064 MCU Module:CD32YP0302-2R2M_SMD3.5x3x2.1mm, F.Cu at (216.6, 45.0)
- added Q1: IRLML6401, MIMXRT1064 MCU Module:IRLML6401, F.Cu at (229.0, 43.2)
- added R10: 22k, MIMXRT1064 MCU Module:0402WGF2202TCE, F.Cu at (207.5, 52.6)
- added R11: 1.5k, MIMXRT1064 MCU Module:CQ02WGF1501TCE, F.Cu at (215.5, 49.4)
- added R12: 200k, MIMXRT1064 MCU Module:0402WGF2003TCE, F.Cu at (206.4, 55.1)
- added R13: 100k, MIMXRT1064 MCU Module:0402WGF1003TCE, F.Cu at (203.5, 55.1)
- added R9: 100k, MIMXRT1064 MCU Module:0402WGF1003TCE, F.Cu at (199.8, 60.1)
- added U5: UM805RE, MIMXRT1064 MCU Module:UM805RE, F.Cu at (188.6, 54.7)
- added U6: UM803RS, MIMXRT1064 MCU Module:UM803RS, F.Cu at (194.3, 53.9)
- moved J1 89.6 mm to (158.1, 101.9)
- moved L3 76.3 mm to (199.4, 55.7)
- moved VR2 74.8 mm to (204.7, 47.2)
- moved VR1 29.5 mm to (190.5, 47.2)
- renumbered C2 to C1, C11 to C10, C13 to C11, C14 to C12, C15 to C13, C16 to C14, C18 to C15, C19 to C16, C21 to C17, C22 to C18, C23 to C19, C4 to C2, C25 to C20, C26 to C21, C27 to C22, C28 to C23, C29 to C24, C30 to C25, C34 to C26, C35 to C27, C36 to C28, C37 to C29, C1 to C3, C38 to C30, C39 to C31, C40 to C32, C41 to C33, C43 to C34, C42 to C35, C44 to C36, C46 to C37, C45 to C38, C47 to C39, C3 to C4, C48 to C40, C51 to C41, C52 to C42, C53 to C43, C54 to C44, C49 to C45, C56 to C46, C50 to C47, C58 to C48, C59 to C49, C60 to C50, C61 to C51, C55 to C52, C57 to C53, C62 to C54, C63 to C55, C64 to C56, C65 to C57, C66 to C58, C67 to C59, C68 to C60, C69 to C61, L2 to L1, R5 to R2, R8 to R3, R9 to R4, R10 to R5, R11 to R6, R12 to R7, R13 to R8, U3 to U2, U2 to U3, U5 to U4
Connections:
- net VDD_SNVS_IN renamed Net-(C6-Pad1)
- C54 pad 1: +3V3 -> VSD_3V3
- C55 pad 1: +3V3 -> VSD_3V3
- C56 pad 1: +3V3 -> VSD_3V3
- J1 pad 4: +3V3 -> VSD_3V3
- U1 pad K7: PMIC_ON_REQ -> LDO_EN
- U1 pad M7: Net-(R2-Pad2) -> unconnected-(U1-PadM7)
- VR1 pad 1: +5V -> LDO_EN

Commit message: edits
Parts:
- FB1: value 120R -> BLM18AG121SN1D
- Y1: value 24MHz -> XL7EL89CMI-111YLC-24M
- Y2: value 32.768KHz -> X201232768KJD2SI
- moved C15 113.3 mm to (151.2, 63.0)
- moved R2 113.3 mm to (155.5, 56.4)
- moved C19 112.0 mm to (144.7, 66.0)
- moved Y1 108.4 mm to (156.0, 60.2)
- moved C52 105.4 mm to (145.1, 58.4)
- moved R4 105.4 mm to (142.2, 58.4)
- moved C35 54.6 mm to (223.7, 103.9)
- moved C38 54.6 mm to (223.7, 101.9)
- moved R5 43.1 mm to (217.9, 101.6)
- moved C53 43.1 mm to (222.9, 97.0)
- moved D4 38.6 mm to (203.0, 95.0)
- moved L3 38.6 mm to (208.3, 93.2)
- moved R10 38.6 mm to (216.3, 90.1)
- moved U6 38.6 mm to (203.1, 91.5)
- moved C62 38.6 mm to (209.2, 95.4)
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Connections:
- Y1 pad 2: (no net) -> GND
Other:
- board size 40.1 x 40 mm -> 99.1 x 66 mm

Commit message: work
Parts:
- moved C64 139.7 mm to (81.3, 67.8), turned to -90 degrees
- moved C65 138.5 mm to (82.0, 57.4), turned to -90 degrees
- moved R10 136.7 mm to (83.6, 57.4), turned to 90 degrees
- moved R9 134.3 mm to (80.5, 57.4), turned to -90 degrees
- moved C63 133.1 mm to (81.3, 70.1), turned to -90 degrees
- moved C62 130.0 mm to (85.3, 55.9), turned to -90 degrees
- moved C67 129.6 mm to (76.5, 57.9), turned to -90 degrees
- moved C66 128.9 mm to (78.5, 57.9), turned to -90 degrees
- moved L2 125.6 mm to (75.9, 54.1), turned to -90 degrees
- moved C72 122.0 mm to (95.2, 57.7), turned to -90 degrees
- moved R12 121.3 mm to (99.3, 56.9), turned to -90 degrees
- moved D4 121.1 mm to (84.8, 68.5), turned to -90 degrees
- moved L3 120.2 mm to (94.7, 53.8), turned to -90 degrees
- moved C69 118.1 mm to (98.0, 65.8), turned to 180 degrees
- moved L1 117.5 mm to (67.1, 107.3)
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
Commit message: schematic edit
Parts:
- removed the C35 at (223.7, 103.9)
- removed the C39 at (178.2, 98.6)
- removed the C60 at (223.9, 65.5)
- removed the C61 at (223.8, 69.4)
- removed the C65 at (82.0, 57.4)
- removed C68, C71, C72: 22uF, MIMXRT1064 MCU Module:0603_CL10A226MQ8NRNC
- removed C70: 22pF, MIMXRT1064 MCU Module:0402CG220J500NT
- removed L2, L3: 2.2uH, MIMXRT1064 MCU Module:CD32YP0302-2R2M_SMD3.5x3x2.1mm
- removed R12: 200k, MIMXRT1064 MCU Module:0402WGF2003TCE
- removed R13: 100k, MIMXRT1064 MCU Module:0402WGF1003TCE
- removed R8: 10k, MIMXRT1064 MCU Module:0402WGF1002TCE
- removed the U4 at (183.6, 76.9)
- added C47: 100nF, MIMXRT1064 MCU Module:0402_CL05B104KB54PNC, F.Cu at (132.0, 118.7)
- added C49: 10uF, MIMXRT1064 MCU Module:0603_CL10A106KP8NNNC, F.Cu at (128.6, 119.0)
- added C63: 22uF, MIMXRT1064 MCU Module:0603_CL10A226MQ8NRNC, F.Cu at (119.5, 145.3)
- added C64: 22uF, MIMXRT1064 MCU Module:0603_CL10A226MQ8NRNC, F.Cu at (115.5, 145.3)
- added D5: Blue LED, MIMXRT1064 MCU Module:19-218_BHC-ZL1M2QY_3T, F.Cu at (120.7, 136.5)
- C40: value 10uF -> 1uF; footprint MIMXRT1064 MCU Module:0603_CL10A106KP8NNNC -> MIMXRT1064 MCU Module:0402_CL05A105KA5NQNC
- C57, C58: value 4.7uF -> 1uF; footprint MIMXRT1064 MCU Module:0402_CL05A475MP5NRNC -> MIMXRT1064 MCU Module:0402_CL05A105KA5NQNC
- C59: value 4.7uF -> 22uF; footprint MIMXRT1064 MCU Module:0402_CL05A475MP5NRNC -> MIMXRT1064 MCU Module:0603_CL10A226MQ8NRNC
- C62, C66: value 22uF -> DNP
- R10: value 22k -> 100k; footprint MIMXRT1064 MCU Module:0402WGF2202TCE -> MIMXRT1064 MCU Module:0402WGF1003TCE
- R6: value 2.2k -> 100k; footprint MIMXRT1064 MCU Module:0402WGF2201TCE -> MIMXRT1064 MCU Module:0402WGF1003TCE
- R7: value 2.2k -> 22k; footprint MIMXRT1064 MCU Module:0402WGF2201TCE -> MIMXRT1064 MCU Module:0402WGF2202TCE
- R9: value 100k -> 200k; footprint MIMXRT1064 MCU Module:0402WGF1003TCE -> MIMXRT1064 MCU Module:0402WGF2003TCE
- VR1, VR2: value SY8089AAAC -> TLV62569DBV; footprint MIMXRT1064 MCU Module:SY8089AAAC_SOT-23-5 -> Package_TO_SOT_SMD:SOT-23-5
- Y1: value XL7EL89CMI-111YLC-24M -> 7V24000026; footprint MIMXRT1064 MCU Module:XL7EL89CMI-111YLC-24M -> MIMXRT1064 MCU Module:7V24000026
- moved C57 127.7 mm to (123.0, 145.8)
- moved R7 126.7 mm to (123.0, 143.8)
- moved R6 120.2 mm to (128.2, 136.2)
- moved C58 119.4 mm to (127.0, 141.2)
- moved C59 117.3 mm to (124.7, 136.4)
- moved C38 98.0 mm to (128.0, 123.2)
- moved C67 94.6 mm to (120.7, 141.5), turned to 0 degrees
- moved VR1 94.4 mm to (116.1, 141.9)
- moved R9 93.8 mm to (128.2, 138.2), turned to 0 degrees
- moved R10 93.1 mm to (124.1, 141.2), turned to 0 degrees
- moved C62 91.9 mm to (124.7, 138.9), turned to 0 degrees
- moved C66 91.4 mm to (120.7, 139.0), turned to 0 degrees
- moved VR2 85.2 mm to (116.1, 137.4)
- moved Y1 67.7 mm to (141.9, 120.3)
- moved C40 56.5 mm to (128.0, 121.2)
- renumbered C36 to C35, C37 to C36, C41 to C37, C42 to C39, C43 to C41, C44 to C42, C46 to C43, C48 to C44, C49 to C45, C50 to C46, C51 to C48, C52 to C50, C53 to C51, C45 to C52, C47 to C53, C63 to C60, C64 to C61, C69 to C65, R4 to R3, R3 to R4, U3 to U4
Connections:
- net GPIO_AD_B0_06 renamed JTAG_TMS
- net GPIO_AD_B0_07 renamed JTAG_TCK
- net GPIO_AD_B0_09 renamed JTAG_TDI
- net GPIO_AD_B0_10 renamed JTAG_TDO
- net GPIO_AD_B0_11 renamed JTAG_nTRST
- C38 pad 1: USB_OTG2_VBUS -> USB_OTG1_VBUS
- C40 pad 1: Net-(C39-Pad1) -> USB_OTG2_VBUS
- C57 pad 1: +3.3VA -> VBUS
- C58 pad 1: Net-(C58-Pad1) -> +5V
- C59 pad 1: +3V3 -> +5V
- C62 pad 1: +5V -> +3V3
- C62 pad 2: GND -> Net-(C62-Pad2)
- C66 pad 1: +3V3 -> +1V8
- C66 pad 2: GND -> Net-(C66-Pad2)
- C67 pad 1: +3V3 -> +1V8
- R10 pad 1: Net-(C65-Pad2) -> Net-(C66-Pad2)
- R6 pad 2: CODEC_SDA -> Net-(C62-Pad2)
- R7 pad 1: +3V3 -> Net-(C62-Pad2)
- R7 pad 2: CODEC_SCL -> GND
- R9 pad 1: +3V3 -> +1V8
- R9 pad 2: Net-(C65-Pad2) -> Net-(C66-Pad2)
- U1 pad K8: Net-(C39-Pad1) -> Net-(C47-Pad1)
- VR1 pad 5: Net-(C65-Pad2) -> Net-(C62-Pad2)
- VR2 pad 5: Net-(C70-Pad2) -> Net-(C66-Pad2)
- Y1 pad 2: GND -> unconnected-(Y1-Pad2)
- Y1 pad 4: GND -> unconnected-(Y1-Pad4)

Commit message: schematic changes
Parts:
- removed C1, C10, C11, C13, C14, C15, C16, C18, C19, C21, C24, C6, C7: 220nF, MIMXRT1064 MCU Module:0402_CL05B224KO5NNNC
- removed C12, C17, C2, C20, C23, C26, C29, C32, C33, C39, C55: 4.7uF, MIMXRT1064 MCU Module:0402_CL05A475MP5NRNC
- removed C22, C49: 10uF, MIMXRT1064 MCU Module:0603_CL10A106KP8NNNC
- removed C25, C37, C54, C59, C63, C64, C67: 22uF, MIMXRT1064 MCU Module:0603_CL10A226MQ8NRNC
- removed C27, C28, C30, C31, C34, C35, C36, C41, C42, C43, C44, C45, C46, C47, C48, C53, C56, C60, C61, C65: 100nF, MIMXRT1064 MCU Module:0402_CL05B104KB54PNC
- removed C3, C4: 12pF, MIMXRT1064 MCU Module:0402_GRM1555C1H120GA01D
- removed C38, C40, C50, C51, C52, C57, C58, C9: 1uF, MIMXRT1064 MCU Module:0402_CL05A105KA5NQNC
- removed C5, C8: 8pF, MIMXRT1064 MCU Module:0402_GCM1555C1H8R0DA16D
- removed C62, C66: DNP, MIMXRT1064 MCU Module:0603_CL10A226MQ8NRNC
- removed D1, D2, D3, D4: RB521S30_R1_00001, MIMXRT1064 MCU Module:RB521S30_R1_00001
- removed D5: Blue LED, MIMXRT1064 MCU Module:19-218_BHC-ZL1M2QY_3T
- removed FB1, FB2: BLM18AG121SN1D, MIMXRT1064 MCU Module:0603_BLM18AG121SN1D
- removed J1: TF-15x15, MIMXRT1064 MCU Module:TF-15x15_smd
- removed L1: 4.7uH, MIMXRT1064 MCU Module:CD32YP0302-4R7M
- removed Q1: IRLML6401, MIMXRT1064 MCU Module:IRLML6401
- removed R1: 2.2M, MIMXRT1064 MCU Module:0402WGJ0225TCE
- removed R10, R6: 100k, MIMXRT1064 MCU Module:0402WGF1003TCE
- removed R11: 1.5k, MIMXRT1064 MCU Module:CQ02WGF1501TCE
- removed R2: 30k, MIMXRT1064 MCU Module:TC0225F3002TCE
- removed R3, R4, R5: 10k, MIMXRT1064 MCU Module:0402WGF1002TCE
- removed R7: 22k, MIMXRT1064 MCU Module:0402WGF2202TCE
- removed R9: 200k, MIMXRT1064 MCU Module:0402WGF2003TCE
- removed U2: IS42S16160J-6BLI, MIMXRT1064 MCU Module:IS42S16160J-6BLI
- removed U4: IS25WP064A-JBLE, MIMXRT1064 MCU Module:IS25WP064A-JBLE
- removed U5: UM805RE, MIMXRT1064 MCU Module:UM805RE
- removed U6: UM803RS, MIMXRT1064 MCU Module:UM803RS
- removed VR1, VR2: TLV62569DBV, Package_TO_SOT_SMD:SOT-23-5
- removed Y1: 7V24000026, MIMXRT1064 MCU Module:7V24000026
- removed Y2: X201232768KJD2SI, MIMXRT1064 MCU Module:X201232768KJD2SI
- added C301: 1u, MIMXRT1064 MCU Module:0402_CL05A105KA5NQNC, F.Cu at (159.8, 92.7)
- added C302: 1u, MIMXRT1064 MCU Module:0402_CL05A105KA5NQNC, F.Cu at (153.5, 99.6)
- added C303: 22u, MIMXRT1064 MCU Module:0603_CL10A226MQ8NRNC, F.Cu at (157.5, 90.5)
- added C304: 100n, MIMXRT1064 MCU Module:0402_CL05B104KB54PNC, F.Cu at (163.9, 90.2)
- added C305: 100n, MIMXRT1064 MCU Module:0402_CL05B104KB54PNC, F.Cu at (151.6, 102.1)
- added C306: 10u, MIMXRT1064 MCU Module:0603_CL10A106KP8NNNC, F.Cu at (161.5, 88.0)
- added C307: 100n, MIMXRT1064 MCU Module:0402_CL05B104KB54PNC, F.Cu at (156.9, 98.6)
- added C308: 22u, MIMXRT1064 MCU Module:0603_CL10A226MQ8NRNC, F.Cu at (157.5, 88.0)
- added C309: 10u, MIMXRT1064 MCU Module:0603_CL10A106KP8NNNC, F.Cu at (150.5, 97.4)
- added C310: 1u, MIMXRT1064 MCU Module:0402_CL05A105KA5NQNC, F.Cu at (156.9, 96.7)
- added C311: 10n, MIMXRT1064 MCU Module:0402_CL05B103KB5NNNC, F.Cu at (159.7, 94.7)
- added C312: 10u, MIMXRT1064 MCU Module:0402_CL05B103KB5NNNC, F.Cu at (156.9, 94.7)
- added C401: 4.7u, MIMXRT1064 MCU Module:0402_CL05A475MP5NRNC, F.Cu at (202.1, 73.9)
- added C402: 0.22u, MIMXRT1064 MCU Module:0402_CL05B224KO5NNNC, F.Cu at (210.2, 64.5)
- added C403: 12p, MIMXRT1064 MCU Module:0402_GRM1555C1H120GA01D, F.Cu at (216.0, 60.1)
- added C404: 12p, MIMXRT1064 MCU Module:0402_GRM1555C1H120GA01D, F.Cu at (213.1, 64.5)
- added C405: 1u, MIMXRT1064 MCU Module:0402_CL05A105KA5NQNC, F.Cu at (206.2, 71.0)
- added C406: 8p, MIMXRT1064 MCU Module:0402_GCM1555C1H8R0DA16D, F.Cu at (210.2, 66.5)
- added C407: 0.22u, MIMXRT1064 MCU Module:0402_CL05B224KO5NNNC, F.Cu at (200.5, 70.0)
- added C408: 0.22u, MIMXRT1064 MCU Module:0402_CL05B224KO5NNNC, F.Cu at (200.5, 72.0)
- added C409: 8p, MIMXRT1064 MCU Module:0402_GCM1555C1H8R0DA16D, F.Cu at (203.4, 72.0)
- added C410: 0.22u, MIMXRT1064 MCU Module:0402_CL05B224KO5NNNC, F.Cu at (204.5, 67.0)
- added C411: 0.22u, MIMXRT1064 MCU Module:0402_CL05B224KO5NNNC, F.Cu at (199.2, 73.9)
- added C412: 0.22u, MIMXRT1064 MCU Module:0402_CL05B224KO5NNNC, F.Cu at (206.2, 69.0)
- added C413: 0.22u, MIMXRT1064 MCU Module:0402_CL05B224KO5NNNC, F.Cu at (207.4, 67.0)
- added C414: 0.22u, MIMXRT1064 MCU Module:0402_CL05B224KO5NNNC, F.Cu at (212.0, 62.5)
- added C415: 4.7u, MIMXRT1064 MCU Module:0402_CL05A475MP5NRNC, F.Cu at (195.5, 76.1)
- added C416: 0.22u, MIMXRT1064 MCU Module:0402_CL05B224KO5NNNC, F.Cu at (213.2, 60.1)
- added C417: 4.7u, MIMXRT1064 MCU Module:0402_CL05A475MP5NRNC, F.Cu at (204.5, 65.0)
- added C418: 0.22u, MIMXRT1064 MCU Module:0402_CL05B224KO5NNNC, F.Cu at (209.1, 62.6)
- added C419: 0.22u, MIMXRT1064 MCU Module:0402_CL05B224KO5NNNC, F.Cu at (201.2, 75.9)
- added C420: 10u, MIMXRT1064 MCU Module:0603_CL10A106KP8NNNC, F.Cu at (206.2, 60.3)
- added C421: 4.7u, MIMXRT1064 MCU Module:0402_CL05A475MP5NRNC, F.Cu at (198.3, 75.9)
- added C422: 0.22u, MIMXRT1064 MCU Module:0402_CL05B224KO5NNNC, F.Cu at (203.4, 70.0)
- added C423: 0.22u, MIMXRT1064 MCU Module:0402_CL05B224KO5NNNC, F.Cu at (207.4, 65.0)
- added C424: 4.7u, MIMXRT1064 MCU Module:0402_CL05A475MP5NRNC, F.Cu at (214.9, 62.0)
- added C425: 22u, MIMXRT1064 MCU Module:0603_CL10A226MQ8NRNC, F.Cu at (201.1, 65.3)
- added C501: 4.7u, MIMXRT1064 MCU Module:0402_CL05A475MP5NRNC, F.Cu at (187.4, 81.5)
- added C502: 100n, MIMXRT1064 MCU Module:0402_CL05B104KB54PNC, F.Cu at (187.4, 83.5)
- added C503: 100n, MIMXRT1064 MCU Module:0402_CL05B104KB54PNC, F.Cu at (190.3, 83.5)
- added C504: 4.7u, MIMXRT1064 MCU Module:0402_CL05A475MP5NRNC, F.Cu at (190.3, 81.5)
- added C505: 100n, MIMXRT1064 MCU Module:0402_CL05B104KB54PNC, F.Cu at (193.2, 83.5)
- added C506: 100n, MIMXRT1064 MCU Module:0402_CL05B104KB54PNC, F.Cu at (190.3, 85.5)
- added C507: 4.7u, MIMXRT1064 MCU Module:0402_CL05A475MP5NRNC, F.Cu at (193.2, 85.5)
- added C508: 4.7u, MIMXRT1064 MCU Module:0402_CL05A475MP5NRNC, F.Cu at (187.4, 85.5)
- added C509: 100n, MIMXRT1064 MCU Module:0402_CL05B104KB54PNC, F.Cu at (196.0, 83.5)
- added C510: 100n, MIMXRT1064 MCU Module:0402_CL05B104KB54PNC, F.Cu at (193.2, 81.5)
- added C511: 100n, MIMXRT1064 MCU Module:0402_CL05B104KB54PNC, F.Cu at (196.0, 81.5)
- added C601: 22u, MIMXRT1064 MCU Module:0603_CL10A226MQ8NRNC, F.Cu at (172.2, 60.3)
- added C602: 4.7u, MIMXRT1064 MCU Module:0402_CL05A475MP5NRNC, F.Cu at (171.6, 68.5)
- added C603: 100n, MIMXRT1064 MCU Module:0402_CL05B104KB54PNC, F.Cu at (156.0, 79.2)
- added C604: 100n, MIMXRT1064 MCU Module:0402_CL05B104KB54PNC, F.Cu at (178.5, 60.1)
- added C605: 100n, MIMXRT1064 MCU Module:0402_CL05B104KB54PNC, F.Cu at (171.6, 66.5)
- added C606: 1u, MIMXRT1064 MCU Module:0402_CL05A105KA5NQNC, F.Cu at (171.6, 64.5)
- added C607: 100n, MIMXRT1064 MCU Module:0402_CL05B104KB54PNC, F.Cu at (151.4, 81.6)
- added C608: 100n, MIMXRT1064 MCU Module:0402_CL05B104KB54PNC, F.Cu at (171.6, 62.6)
- added C609: 100n, MIMXRT1064 MCU Module:0402_CL05B104KB54PNC, F.Cu at (160.0, 80.7)
- added C610: 100n, MIMXRT1064 MCU Module:0402_CL05B104KB54PNC, F.Cu at (164.4, 78.1)
- added C611: 100n, MIMXRT1064 MCU Module:0402_CL05B104KB54PNC, F.Cu at (154.3, 81.1)
- added C612: 1u, MIMXRT1064 MCU Module:0402_CL05A105KA5NQNC, F.Cu at (178.5, 62.0)
- added C613: 1uF, MIMXRT1064 MCU Module:0402_CL05A105KA5NQNC, F.Cu at (157.1, 81.1)
- added C614: 1u, MIMXRT1064 MCU Module:0402_CL05A105KA5NQNC, F.Cu at (153.1, 79.2)
- added C615: 1uF, MIMXRT1064 MCU Module:0402_CL05A105KA5NQNC, F.Cu at (177.3, 64.0)
- added C616: 22uF, MIMXRT1064 MCU Module:0603_CL10A226MQ8NRNC, F.Cu at (161.0, 78.4)
- added C617: 4.7uF, MIMXRT1064 MCU Module:0402_CL05A475MP5NRNC, F.Cu at (174.5, 64.5)
- added C618: 100n, MIMXRT1064 MCU Module:0402_CL05B104KB54PNC, F.Cu at (170.8, 71.2)
- added C619: 100nF, MIMXRT1064 MCU Module:0402_CL05B104KB54PNC, F.Cu at (174.5, 62.6)
- added C620: 10u, MIMXRT1064 MCU Module:0603_CL10A106KP8NNNC, F.Cu at (146.2, 79.4)
- added D301: RB521S30_R1_00001, MIMXRT1064 MCU Module:RB521S30_R1_00001, F.Cu at (150.3, 99.9)
- added D302: RB521S30_R1_00001, MIMXRT1064 MCU Module:RB521S30_R1_00001, F.Cu at (146.1, 100.0)
- added D303: ~, MIMXRT1064 MCU Module:19-218_BHC-ZL1M2QY_3T, F.Cu at (146.5, 97.4)
- added D401: RB521S30_R1_00001, MIMXRT1064 MCU Module:RB521S30_R1_00001, F.Cu at (205.9, 62.8)
- added D402: RB521S30_R1_00001, MIMXRT1064 MCU Module:RB521S30_R1_00001, F.Cu at (200.8, 67.8)
- added FB401: 120R, MIMXRT1064 MCU Module:0603_BLM18AG121SN1D, F.Cu at (209.9, 60.3)
- added FB601: 120R, MIMXRT1064 MCU Module:0603_BLM18AG121SN1D, F.Cu at (149.9, 79.4)
- added J601: TF-15x15, MIMXRT1064 MCU Module:TF-15x15_smd, F.Cu at (149.1, 69.0)
- added L301: 10n, MIMXRT1064 MCU Module:0402_CL05B103KB5NNNC, F.Cu at (162.6, 92.2)
- added L302: 2.2u, MIMXRT1064 MCU Module:CD32YP0302-2R2M_SMD3.5x3x2.1mm, F.Cu at (147.8, 95.2)
- added L303: 2.2u, MIMXRT1064 MCU Module:CD32YP0302-2R2M_SMD3.5x3x2.1mm, F.Cu at (152.9, 95.2)
- added L401: 4.7u, MIMXRT1064 MCU Module:CD32YP0302-4R7M, F.Cu at (201.6, 63.2)
- added Q601: IRLML6401, MIMXRT1064 MCU Module:IRLML6401, F.Cu at (141.7, 80.5)
- added R301: 10k, MIMXRT1064 MCU Module:0402WGF1002TCE, F.Cu at (156.9, 92.7)
- added R302: 100k, MIMXRT1064 MCU Module:0402WGF1003TCE, F.Cu at (161.0, 90.2)
- added R303: 22k, MIMXRT1064 MCU Module:0402WGF2202TCE, F.Cu at (148.7, 102.2)
- added R304: 2.2k, MIMXRT1064 MCU Module:0402WGF2201TCE, F.Cu at (145.8, 102.2)
- added R305: 200k, MIMXRT1064 MCU Module:0402WGF2003TCE, F.Cu at (154.0, 97.1)
- added R306: 100k, MIMXRT1064 MCU Module:0402WGF1003TCE, F.Cu at (165.0, 87.7)
- added R401: 2.2M, MIMXRT1064 MCU Module:0402WGJ0225TCE, F.Cu at (192.6, 76.1)
- added R402: 30k, MIMXRT1064 MCU Module:0402WGF3302TCE, F.Cu at (196.3, 73.1)
- added R601: 10k, MIMXRT1064 MCU Module:0402WGF1002TCE, F.Cu at (175.6, 60.1)
- added R602: 10k, MIMXRT1064 MCU Module:0402WGF1002TCE, F.Cu at (145.6, 81.7)
- added R603: 10k, MIMXRT1064 MCU Module:0402WGF1002TCE, F.Cu at (148.5, 81.7)
- added U301: UM805RE, MIMXRT1064 MCU Module:UM805RE, F.Cu at (142.2, 89.9)
- added U302: UM803RS, MIMXRT1064 MCU Module:UM803RS, F.Cu at (141.8, 96.0)
- added U601: IS42S16160J-6BLI, MIMXRT1064 MCU Module:IS42S16160J-6BLI, F.Cu at (164.6, 64.7)
- added U602: IS25WP064A-JBLE, MIMXRT1064 MCU Module:IS25WP064A-JBLE, F.Cu at (164.2, 73.7)
- added VR301: TLV62569DBV, MIMXRT1064 MCU Module:TLV62569DBVR, F.Cu at (141.8, 100.5)
- added VR302: TLV62569DBV, MIMXRT1064 MCU Module:TLV62569DBVR, F.Cu at (152.9, 88.9)
- added VR303: TPS79333DBVR, MIMXRT1064 MCU Module:TPS79333DBVR_SOT-23-5, F.Cu at (147.8, 88.9)
- added Y401: 7V24000026, MIMXRT1064 MCU Module:7V24000026, F.Cu at (188.9, 74.7)
- added Y402: X201232768KJD2SI, MIMXRT1064 MCU Module:X201232768KJD2SI, F.Cu at (193.0, 73.6)
- moved U1 122.8 mm to (192.5, 65.6)
Connections:
- net Net-(C11-Pad1) renamed /MCU POWER & CRYSTALS/VDD_SOC_IN
- net Net-(C20-Pad1) renamed /MCU POWER & CRYSTALS/DCDC_IN
- U1 pad K3: Net-(C13-Pad1) -> /MCU POWER & CRYSTALS/DCDC_PSWITCH
- U1 pad K7: LDO_EN -> PMIC_ON_REQ
- U1 pad M10: Net-(C10-Pad1) -> /MCU POWER & CRYSTALS/VDD_SNVS_CAP
- U1 pad M7: unconnected-(U1-PadM7) -> POR_B
- U1 pad M9: Net-(C6-Pad1) -> /MCU POWER & CRYSTALS/VDD_SNVS_IN
- U1 pad N11: Net-(C4-Pad1) -> /MCU POWER & CRYSTALS/XTAL0
- U1 pad N3: FLEXSPI_DQS -> unconnected-(U1-PadN3)
- U1 pad N9: Net-(C5-Pad1) -> /MCU POWER & CRYSTALS/RTC_XTALI
- U1 pad P10: Net-(C12-Pad1) -> /MCU POWER & CRYSTALS/NVCC_PLL
- U1 pad P11: Net-(C3-Pad1) -> /MCU POWER & CRYSTALS/XTALI
- U1 pad P8: Net-(C17-Pad1) -> /MCU POWER & CRYSTALS/VDD_HIGH_CAP
- U1 pad P9: Net-(C8-Pad1) -> /MCU POWER & CRYSTALS/RTC_XTALO

Commit message: schematic changes
Parts:
- removed C301, C302, C310, C612, C614: 1u, MIMXRT1064 MCU Module:0402_CL05A105KA5NQNC
- removed C303, C308: 22u, MIMXRT1064 MCU Module:0603_CL10A226MQ8NRNC
- removed C304, C305, C307, C618: 100n, MIMXRT1064 MCU Module:0402_CL05B104KB54PNC
- removed C306, C309, C620: 10u, MIMXRT1064 MCU Module:0603_CL10A106KP8NNNC
- removed C311, L301: 10n, MIMXRT1064 MCU Module:0402_CL05B103KB5NNNC
- removed C312: 10u, MIMXRT1064 MCU Module:0402_CL05B103KB5NNNC
- removed C613, C615: 1uF, MIMXRT1064 MCU Module:0402_CL05A105KA5NQNC
- removed D301, D302: RB521S30_R1_00001, MIMXRT1064 MCU Module:RB521S30_R1_00001
- removed D303: ~, MIMXRT1064 MCU Module:19-218_BHC-ZL1M2QY_3T
- removed L302, L303: 2.2u, MIMXRT1064 MCU Module:CD32YP0302-2R2M_SMD3.5x3x2.1mm
- removed Q601: IRLML6401, MIMXRT1064 MCU Module:IRLML6401
- removed R301, R602: 10k, MIMXRT1064 MCU Module:0402WGF1002TCE
- removed R302, R306: 100k, MIMXRT1064 MCU Module:0402WGF1003TCE
- removed R303: 22k, MIMXRT1064 MCU Module:0402WGF2202TCE
- removed R304: 2.2k, MIMXRT1064 MCU Module:0402WGF2201TCE
- removed R305: 200k, MIMXRT1064 MCU Module:0402WGF2003TCE
- removed U301: UM805RE, MIMXRT1064 MCU Module:UM805RE
- removed U302: UM803RS, MIMXRT1064 MCU Module:UM803RS
- removed VR301, VR302: TLV62569DBV, MIMXRT1064 MCU Module:TLV62569DBVR
- removed VR303: TPS79333DBVR, MIMXRT1064 MCU Module:TPS79333DBVR_SOT-23-5
- added C512: 1u, MIMXRT1064 MCU Module:0402_CL05A105KA5NQNC, F.Cu at (162.3, 78.9)
- added C513: 1u, MIMXRT1064 MCU Module:0402_CL05A105KA5NQNC, F.Cu at (159.5, 78.9)
- added C514: 100n, MIMXRT1064 MCU Module:0402_CL05B104KB54PNC, F.Cu at (163.5, 76.4)
- added C515: 10u, MIMXRT1064 MCU Module:0603_CL10A106KP8NNNC, F.Cu at (160.0, 76.7)
- R402: footprint MIMXRT1064 MCU Module:0402WGF3302TCE -> MIMXRT1064 MCU Module:AF0402FR-0730KL
- Y402: value X201232768KJD2SI -> Q13FC1350000200; footprint MIMXRT1064 MCU Module:X201232768KJD2SI -> MIMXRT1064 MCU Module:Q13FC1350000200
- moved C403 72.6 mm to (157.3, 102.8), turned to 180 degrees
- moved C424 68.5 mm to (158.5, 100.9), turned to 180 degrees
- moved C416 68.1 mm to (160.2, 102.8), turned to 180 degrees
- moved C414 63.2 mm to (161.4, 100.4), turned to 180 degrees
- moved FB401 62.8 mm to (163.4, 102.6), turned to 180 degrees
- moved C404 62.8 mm to (160.3, 98.4), turned to 180 degrees
- moved C418 58.7 mm to (164.2, 100.3), turned to 180 degrees
- moved C402 58.0 mm to (163.1, 98.3), turned to 180 degrees
- moved C420 57.4 mm to (167.2, 102.6), turned to 180 degrees
- moved C406 55.8 mm to (163.1, 96.4), turned to 180 degrees
- moved D401 53.6 mm to (167.4, 100.1), turned to 180 degrees
- moved C422 52.8 mm to (166.0, 97.9), turned to 180 degrees
- moved C413 50.5 mm to (166.0, 95.9), turned to 180 degrees
- moved C417 48.4 mm to (168.9, 97.8), turned to 180 degrees
- moved Y402 47.7 mm to (153.7, 100.6), turned to 90 degrees
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- renumbered C423 to C422, C422 to C423
Connections:
- net USB_OTG1_DN renamed USB_OTG1_D-
- net USB_OTG1_DP renamed USB_OTG1_D+
- net USB_OTG2_DN renamed USB_OTG2_D-
- net USB_OTG2_DP renamed USB_OTG2_D+
- R402 pad 1: /MCU POWER & CRYSTALS/DCDC_PSWITCH -> /MCU POWER & CRYSTALS/DCDC_IN
- R402 pad 2: /MCU POWER & CRYSTALS/DCDC_IN -> /MCU POWER & CRYSTALS/DCDC_PSWITCH
Other:
- board size 99.1 x 66 mm -> 36.8 x 41.1 mm
