File: DESIGN FILES/MIMXRT1064 MCU Module.kicad_pcb (KiCad board)
At the start: 2 copper layers, 36.8 x 41.1 mm, 69 parts, among them J601 TF-15x15, U1 MIMXRT1064CVL5B, U601 IS42S16160J-6BLI, U602 IS25WP064A-JBLE, Y401 7V24000026, Y402 Q13FC1350000200

Commit message: changes and adding schematic pdf
Parts:
- C616: value 22uF -> 22u
- C617: value 4.7uF -> 4.7u
- C619: value 100nF -> 100n
- L401: footprint MIMXRT1064 MCU Module:CD32YP0302-4R7M -> MIMXRT1064 MCU Module:LQM21PN4R7MGRD
- moved L401 1.88 mm to (172.0, 101.6), turned to 0 degrees
Changed lines of the file:
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@@
   (net 93 "JTAG_nTRST")
   (net 94 "JTAG_TDO")
-  (net 95 "Net-(L401-Pad1)")
+  (net 95 "Net-(U1-PadM1)")
   (net 96 "GPIO_B0_06")
   (net 97 "GPIO_B0_07")
@@
     )
   )
+  (footprint "MIMXRT1064 MCU Module:LQM21PN4R7MGRD" (layer "F.Cu")
+    (at 171.958 101.6)
+    (descr "Inductor SMD 0805 (2012 Metric), square (rectangular) end terminal, IPC_7351 nominal, (Body size source: IPC-SM-782 page 80, https://www.pcb-3d.com/wordpress/wp-content/uploads/ipc-sm-782a_amendment_1_and_2.pdf), generated with kicad-footprint-generator")
+    (tags "inductor")
+    (property "Sheetfile" "pwrpin_crystals.kicad_sch")
+    (property "Sheetname" "MCU POWER & CRYSTALS")
+    (attr smd)
+    (fp_text reference "L401" (at 0 -1.55) (layer "F.SilkS")
+      (effects (font (size 1 1) (thickness 0.15)))
+    )
+    (fp_text value "4.7u" (at 0 1.55) (layer "F.Fab")
+      (effects (font (size 1 1) (thickness 0.15)))
+    )
+    (fp_text user "${REFERENCE}" (at 0 0) (layer "F.Fab")
+      (effects (font (size 0.5 0.5) (thickness 0.08)))
+    )
+    (fp_line (start -0.399622 0.56) (end 0.399622 0.56) (layer "F.SilkS") (width 0.12))
+    (fp_line (start -0.399622 -0.56) (end 0.399622 -0.56) (layer "F.SilkS") (width 0.12))
+    (fp_line (start -1.75 0.85) (end -1.75 -0.85) (layer "F.CrtYd") (width 0.05))
+    (fp_line (start 1.75 0.85) (end -1.75 0.85) (layer "F.CrtYd") (width 0.05))
+    (fp_line (start 1.75 -0.85) (end 1.75 0.85) (layer "F.CrtYd") (width 0.05))
+    (fp_line (start -1.75 -0.85) (end 1.75 -0.85) (layer "F.CrtYd") (width 0.05))
+    (fp_line (start 1 -0.45) (end 1 0.45) (layer "F.Fab") (width 0.1))
+    (fp_line (start 1 0.45) (end -1 0.45) (layer "F.Fab") (width 0.1))
+    (fp_line (start -1 0.45) (end -1 -0.45) (layer "F.Fab") (width 0.1))
+    (fp_line (start -1 -0.45) (end 1 -0.45) (layer "F.Fab") (width 0.1))
+    (pad "1" smd roundrect (at -1.0625 0) (size 0.875 1.2) (layers "F.Cu" "F.Paste" "F.Mask") (roundrect_rratio 0.25)
+      (net 95 "Net-(U1-PadM1)") (pinfunction "1") (pintype "passive"))
+    (pad "2" smd roundrect (at 1.0625 0) (size 0.875 1.2) (layers "F.Cu" "F.Paste" "F.Mask") (roundrect_rratio 0.25)
+      (net 21 "/MCU POWER & CRYSTALS/VDD_SOC_IN") (pinfunction "2") (pintype "passive"))
+    (model "${KICAD6_3DMODEL_DIR}/Inductor_SMD.3dshapes/L_0805_2012Metric.wrl"
+      (offset (xyz 0 0 0))
+      (scale (xyz 1 1 1))
+      (rotate (xyz 0 0 0))
+    )
+  )
   (footprint "MIMXRT1064 MCU Module:0402_CL05B104KB54PNC" (layer "F.Cu")
     (at 158.118 92.634 90)
@@
       (effects (font (size 1 1) (thickness 0.15)))
     )
-    (fp_text value "4.7uF" (at 0 1.16) (layer "F.Fab")
+    (fp_text value "4.7u" (at 0 1.16) (layer "F.Fab")
       (effects (font (size 1 1) (thickness 0.15)))
     )
@@
       (net 135 "GPIO_AD_B0_13") (pinfunction "GPIO_AD_B0_13") (pintype "passive"))
     (pad "M1" smd circle (at -4.225 2.925 270) (size 0.29 0.29) (layers "F.Cu" "F.Paste" "F.Mask")
-      (net 95 "Net-(L401-Pad1)") (pinfunction "DCDC_LP_1") (pintype "power_in"))
+      (net 95 "Net-(U1-PadM1)") (pinfunction "DCDC_LP_1") (pintype "power_in"))
     (pad "M2" smd circle (at -3.575 2.925 270) (size 0.29 0.29) (layers "F.Cu" "F.Paste" "F.Mask")
-      (net 95 "Net-(L401-Pad1)") (pinfunction "DCDC_LP_2") (pintype "power_in"))
+      (net 95 "Net-(U1-PadM1)") (pinfunction "DCDC_LP_2") (pintype "power_in"))
     (pad "M3" smd circle (at -2.925 2.925 270) (size 0.29 0.29) (layers "F.Cu" "F.Paste" "F.Mask")
       (net 156 "unconnected-(U1-PadM3)") (pinfunction "GPIO_SD_B1_02") (pintype "passive+no_connect"))
@@
       (effects (font (size 1 1) (thickness 0.15)))
     )
-    (fp_text value "22uF" (at 0 1.43) (layer "F.Fab")
+    (fp_text value "22u" (at 0 1.43) (layer "F.Fab")
       (effects (font (size 1 1) (thickness 0.15)))
     )
@@
       (effects (font (size 1 1) (thickness 0.15)))
     )
-    (fp_text value "100nF" (at 0 1.16) (layer "F.Fab")
+    (fp_text value "100n" (at 0 1.16) (layer "F.Fab")
       (effects (font (size 1 1) (thickness 0.15)))
     )
@@
     )
   )
-  (footprint "MIMXRT1064 MCU Module:CD32YP0302-4R7M" (layer "F.Cu")
-    (at 171.766 99.726 180)
-    (descr "4.7uH Inductor - 1.5A - ±20% - 170mΩ")
-    (property "Sheetfile" "pwrpin_crystals.kicad_sch")
-    (property "Sheetname" "MCU POWER & CRYSTALS")
-    (attr smd)
-    (fp_text reference "L401" (at 0.127 -4.318 180 unlocked) (layer "F.SilkS")
-      (effects (font (size 1 1) (thickness 0.15)))
-    )
-    (fp_text value "4.7u" (at 0 1 180 unlocked) (layer "F.Fab")
-      (effects (font (size 1 1) (thickness 0.15)))
-    )
-    (fp_text user "${REFERENCE}" (at 0 2.5 180 unlocked) (layer "F.Fab")
-      (effects (font (size 1 1) (thickness 0.15)))
-    )
-    (fp_line (start -1.778 -3.429) (end 1.778 -3.429) (layer "F.SilkS") (width 0.12))
-    (fp_line (start -1.778 0.254) (end 1.778 0.254) (layer "F.SilkS") (width 0.12))
-    (fp_rect (start -2.032 -3.556) (end 2.032 0.381) (layer "F.CrtYd") (width 0.05) (fill none))
-    (fp_line (start 1.778 0) (end -1.778 0) (layer "F.Fab") (width 0.1))
-    (fp_line (start -1.778 -3.175) (end 1.778 -3.175) (layer "F.Fab") (width 0.1))
-    (fp_line (start 1.778 -3.175) (end 1.778 0) (layer "F.Fab") (width 0.1))
-    (fp_line (start -1.778 0) (end -1.778 -3.175) (layer "F.Fab") (width 0.1))
-    (pad "1" smd roundrect (at -1.143 -1.5875 270) (size 3.175 1.27) (layers "F.Cu" "F.Paste" "F.Mask") (roundrect_rratio 0.25)
-      (net 95 "Net-(L401-Pad1)") (pinfunction "1") (pintype "passive"))
-    (pad "2" smd roundrect (at 1.143 -1.5875 270) (size 3.175 1.27) (layers "F.Cu" "F.Paste" "F.Mask") (roundrect_rratio 0.25)
-      (net 21 "/MCU POWER & CRYSTALS/VDD_SOC_IN") (pinfunction "2") (pintype "passive"))
-  )
   (footprint "MIMXRT1064 MCU Module:0402_GRM1555C1H120GA01D" (layer "F.Cu")

Commit message: updates
Parts:
- removed D401, D402: RB521S30_R1_00001, MIMXRT1064 MCU Module:RB521S30_R1_00001
- moved C423 65.7 mm to (235.7, 94.5)
- moved C602 54.3 mm to (130.7, 81.6)
- moved C604 54.3 mm to (130.4, 90.7)
- moved C605 54.3 mm to (130.7, 79.6)
- moved C606 54.3 mm to (130.7, 77.6)
- moved C608 54.3 mm to (130.7, 75.6)
- moved C617 54.3 mm to (130.7, 88.8)
- moved C619 54.3 mm to (130.7, 86.9)
- moved R601 54.3 mm to (131.9, 84.4)
- moved C601 54.3 mm to (131.3, 73.4)
- moved C410 47.6 mm to (216.5, 95.9)
- moved C416 47.6 mm to (207.8, 102.8)
- moved C417 47.6 mm to (216.5, 97.8)
- moved C401 47.6 mm to (218.9, 88.9)
- moved C402 47.6 mm to (210.7, 98.3)
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Other:
- board size 36.8 x 41.1 mm -> 30.2 x 41.1 mm
