File: DESIGN FILES/MIMXRT1064 MCU Module.kicad_pcb (KiCad board)
At the start: 2 copper layers, 127 x 127 mm, 163 parts, among them J1001 YTC-TC16S-28, J1002 Conn_02x05_Odd_Even, J701 PJ-342B-TX-SMT, J702 PJ-342B-TX-SMT, J703 PJ-342B-TX-SMT, J801 PJ-342B-TX-SMT, J802 PJ-342B-TX-SMT, J803 PJ-342B-TX-SMT, U1 MIMXRT1064CVL5B, U301 UM805RE, U302 UM803RS, U701 WM8978CGEFL_RV, U801 6N137S1(TA), U802 74HC04D,653, U901 PEC12R-4025F-S0024, Y401 7V24000026, Y402 Q13FC1350000200

Commit message: updates
Parts:
- removed 601601601601: IS42S16160J-6BLI, MY MEMORY AND STORAGE LIBRARY:IS42S16160J-6BLI
- removed 602601601601: IS25WP064A-JBLE, MY MEMORY AND STORAGE LIBRARY:IS25WP064A-JBLE
- added C313: 100n, MY CAPACITOR LIBRARY:0402_CL05B104KB54PNC, F.Cu at (203.6, 74.0)
- added H101: MountingHole, MountingHole:MountingHole_2.5mm, F.Cu at (83.8, 35.7)
- added H102: MountingHole, MountingHole:MountingHole_2.5mm, F.Cu at (204.2, 35.7)
- added H103: MountingHole, MountingHole:MountingHole_2.5mm, F.Cu at (204.2, 156.1)
- added H104: MountingHole, MountingHole:MountingHole_2.5mm, F.Cu at (83.8, 156.1)
- added SW301: TS-1187A-B-A-B, MY SWITCH LIBRARY:TS-1187A-B-A-B_smd, F.Cu at (203.7, 67.9)
- added U601: IS25WP064A-JBLE, MY MEMORY AND STORAGE LIBRARY:IS25WP064A-JBLE, F.Cu at (153.2, 53.3)
- added U602: IS42S16160J-6BLI, MY MEMORY AND STORAGE LIBRARY:IS42S16160J-6BLI, F.Cu at (136.9, 38.4)
- C508: footprint MIMXRT1064 MCU Module:0402_CL05A475MP5NRNC -> MY CAPACITOR LIBRARY:0402_CL05A475MP5NRNC
- C512: footprint MIMXRT1064 MCU Module:0402_CL05A105KA5NQNC -> MY CAPACITOR LIBRARY:0402_CL05A105KA5NQNC
- D901, D902: value LED_RGBK -> WP154A4SUREQBFZGW
- J1002: value Conn_02x05_Odd_Even -> PZ127VS-12-10-H10-A38
- R1001: footprint MY RESISTOR LIBRARY:CQ03WAJ0152T5E -> MY RESISTOR LIBRARY:CQ02WGF1501TCE
- moved J1002 348.9 mm to (142.5, 154.5)
- moved C308 299.4 mm to (96.5, 68.5), turned to 90 degrees
- moved C310 295.1 mm to (93.5, 65.1), turned to 180 degrees
- moved VR303 285.3 mm to (93.1, 68.0)
- moved C305 281.0 mm to (90.2, 67.5), turned to -90 degrees
- moved R601 266.2 mm to (244.8, 151.3)
- moved RV912 265.8 mm to (158.4, 152.7), turned to 90 degrees
- moved RV916 265.3 mm to (192.3, 152.7), turned to 90 degrees
- moved C601 264.2 mm to (216.3, 130.0)
- moved C604 264.2 mm to (222.7, 131.7)
- moved C608 264.2 mm to (222.7, 129.7)
- moved C602 264.2 mm to (218.6, 132.2)
- moved C603 264.2 mm to (218.6, 134.2)
- moved C606 264.2 mm to (215.8, 132.2)
- moved C609 264.2 mm to (215.8, 134.2)
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Connections:
- net Net-(VR303-Pad4) renamed /SUPPLIES & PMIC/LDO_NR
- net SD_CD_SW renamed GPIO_B1_12
- net SD_PWREN renamed GPIO_AD_B1_03
- C705 pad 1: SDRAM_3V3 -> VMID
- D901 pad 2: Net-(D901-Pad2) -> GND
- D901 pad 4: GND -> Net-(D901-Pad4)
- D902 pad 2: Net-(D902-Pad2) -> GND
- D902 pad 4: GND -> Net-(D902-Pad4)
- R306 pad 1: EXT_POR_BUT -> RESET_SWITCH
- R701 pad 2: CODEC_SDIN -> CODEC_SDA
- R702 pad 2: CODEC_SCLK -> CODEC_SCL
- R703 pad 1: GND -> Net-(R703-Pad1)
- R703 pad 2: Net-(R703-Pad2) -> GND
- R902 pad 2: Net-(D901-Pad2) -> Net-(D901-Pad3)
- R903 pad 2: Net-(D901-Pad3) -> Net-(D901-Pad4)
- R905 pad 2: Net-(D902-Pad2) -> Net-(D902-Pad3)
- R906 pad 2: Net-(D902-Pad3) -> Net-(D902-Pad4)
- U1 pad A7: GPIO_EMC_40 -> unconnected-(U1-PadA7)
- U1 pad C7: GPIO_EMC_41 -> unconnected-(U1-PadC7)
- U1 pad D14: GPIO_B1_13 -> WATCHDOG_B
- U1 pad H2: SD_DAT2 -> unconnected-(U1-PadH2)
- U1 pad J1: SD_DAT0 -> unconnected-(U1-PadJ1)
- U1 pad J2: SD_DAT3 -> unconnected-(U1-PadJ2)
- U1 pad J3: SD_CLK -> unconnected-(U1-PadJ3)
- U1 pad J4: SD_CMD -> unconnected-(U1-PadJ4)
- U1 pad K1: SD_DAT1 -> unconnected-(U1-PadK1)
- U1 pad L6: WAKEUP -> unconnected-(U1-PadL6)
- U1 pad L7: PMIC_STBY_REQ -> unconnected-(U1-PadL7)
- U1 pad M6: ONOFF -> unconnected-(U1-PadM6)
- U701 pad 10: DACDAT -> I2S_DACDAT
- U701 pad 11: MCLK -> I2S_MCLK
- U701 pad 16: CODEC_SCLK -> CODEC_SCL
- U701 pad 17: CODEC_SDIN -> CODEC_SDA
- U701 pad 18: Net-(R703-Pad2) -> Net-(R703-Pad1)
- U701 pad 27: SDRAM_3V3 -> VMID
- U701 pad 7: LRC -> I2S_LRC
- U701 pad 8: BCLK -> I2S_BCLK
- U701 pad 9: ADCDAT -> I2S_ADCDAT

Commit message: up
Parts:
- R306, R704, R705: footprint MY RESISTOR LIBRARY:0805W8F1000T5E -> MY RESISTOR LIBRARY:0603WAF1000T5E
- R803, R804, R805, R806: footprint MY RESISTOR LIBRARY:0805W8F330JT5E -> MY RESISTOR LIBRARY:0603WAF330JT5E
- moved C610 64.3 mm to (260.5, 93.0)
- moved C611 64.3 mm to (264.4, 93.5)
- moved R601 64.3 mm to (265.4, 90.5)
- moved L301 58.6 mm to (228.1, 77.9)
- moved R301 58.6 mm to (222.7, 73.2)
- moved R302 58.6 mm to (222.5, 81.7)
- moved VR301 58.6 mm to (228.2, 81.2)
- moved C301 58.6 mm to (223.6, 76.8)
- moved C303 58.6 mm to (221.5, 76.7)
- moved C312 50.2 mm to (268.3, 53.1)
- moved U302 50.2 mm to (274.4, 54.6)
- moved R309 50.2 mm to (268.5, 56.3)
- moved C601 46.7 mm to (237.3, 88.2)
- moved C605 46.7 mm to (246.9, 91.9)
- moved C604 46.7 mm to (243.7, 89.9)
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
Commit message: updates
Parts:
- removed C1001: 4.7u, MY CAPACITOR LIBRARY:CL10A475KO8NNNC_0603
- removed C1002: 1uF, MY CAPACITOR LIBRARY:CL10A105KB8NNNC_0603
- removed C301, C302: 22u, MY CAPACITOR LIBRARY:0603_CL10A226MQ8NRNC
- removed C303, C304, C310: 10u, MY CAPACITOR LIBRARY:0603_CL10A106KP8NNNC
- removed C305, C306, C708, C709, C710, C711: 1u, MY CAPACITOR LIBRARY:0402_CL05A105KA5NQNC
- removed C307: 1n, MY CAPACITOR LIBRARY:CL05B102KB5VPNC
- removed C308, C309, C311, C312, C313, C801, C802: 100n, MY CAPACITOR LIBRARY:0402_CL05B104KB54PNC
- removed C701, C702, C703, C704, C705: 4.7u, MY CAPACITOR LIBRARY:0402_CL05A475MP5NRNC
- removed C706, C707: 220u, MY CAPACITOR LIBRARY:RVT1A221M0605
- removed D1001: SP0503BAHTG, MY DIODE LIBRARY:SP0503BAHTG_SOT-143
- removed D301: LED, MY LED LIBRARY:LED_D3.0mm
- removed D302, D303: RB521S30_R1_00001, MY DIODE LIBRARY:RB521S30_R1_00001
- removed D801: 1N4148W, MY DIODE LIBRARY:1N4148W_SOD-123
- removed D901, D902: WP154A4SUREQBFZGW, MY LED LIBRARY:WP154A4SUREQBFZGW
- removed F1001: SMD0805P020TF, MY FUSE LIBRARY:0805_SMD0805P020TF
- removed FB1001: 120R, MY FERRITE BEAD LIBRARY:0603_BLM18AG121SN1D
- removed H101, H102, H103, H104: MountingHole, MountingHole:MountingHole_2.5mm
- removed J1001: YTC-TC16S-28, MY CONNECTOR LIBRARY:YTC-TC16S-28
- removed J1002: PZ127VS-12-10-H10-A38, MY CONNECTOR LIBRARY:PZ127VS-12-10-H10-A38
- removed J701, J702, J703, J801, J802, J803: PJ-342B-TX-SMT, MY CONNECTOR LIBRARY:PJ-342B-TX-SMT
- removed L301, L302: 2.2u, MY INDUCTOR LIBRARY:CD32YP0302-2R2M
- removed R1001, R309: 1.5k, MY RESISTOR LIBRARY:CQ02WGF1501TCE
- removed R1002, R1003: 5.1k, MY RESISTOR LIBRARY:0603WAF5101T5E
- removed R301: 200k, MY RESISTOR LIBRARY:0402WGF2003TCE
- removed R302, R303: 100k, MY RESISTOR LIBRARY:0402WGF1003TCE
- removed R304: 22k, MY RESISTOR LIBRARY:0402WGF2202TCE
- removed R305, R701, R702, R901, R902, R903, R904, R905, R906: 2.2k, MY RESISTOR LIBRARY:0402WGF2201TCE
- removed R306, R704, R705: 100R, MY RESISTOR LIBRARY:0603WAF1000T5E
- removed R307: 1M, MY RESISTOR LIBRARY:0402WGF1004TCE
- removed R308, R703, R802: 10k, MY RESISTOR LIBRARY:0402WGF1002TCE
- removed R706, R707: 47k, MY RESISTOR LIBRARY:0402WGF4702TCE
- removed R801: 220R, MY RESISTOR LIBRARY:0603WAF2200T5E
- removed R803, R804, R805, R806: 33R, MY RESISTOR LIBRARY:0603WAF330JT5E
- removed RV901: POT_A1, MY POTENTIOMETER LIBRARY:RK09D1130C2P
- removed RV902: POT_B1, MY POTENTIOMETER LIBRARY:RK09D1130C2P
- removed RV903: POT_C1, MY POTENTIOMETER LIBRARY:RK09D1130C2P
- removed RV904: POT_D1, MY POTENTIOMETER LIBRARY:RK09D1130C2P
- removed RV905: POT_A2, MY POTENTIOMETER LIBRARY:RK09D1130C2P
- removed RV906: POT_B2, MY POTENTIOMETER LIBRARY:RK09D1130C2P
- removed RV907: POT_C2, MY POTENTIOMETER LIBRARY:RK09D1130C2P
- removed RV908: POT_D2, MY POTENTIOMETER LIBRARY:RK09D1130C2P
- removed RV909: POT_A3, MY POTENTIOMETER LIBRARY:RK09D1130C2P
- removed RV910: POT_B3, MY POTENTIOMETER LIBRARY:RK09D1130C2P
- removed RV911: POT_C3, MY POTENTIOMETER LIBRARY:RK09D1130C2P
- removed RV912: POT_D3, MY POTENTIOMETER LIBRARY:RK09D1130C2P
- removed RV913: POT_A4, MY POTENTIOMETER LIBRARY:RK09D1130C2P
- removed RV914: POT_B4, MY POTENTIOMETER LIBRARY:RK09D1130C2P
- removed RV915: POT_C4, MY POTENTIOMETER LIBRARY:RK09D1130C2P
- removed RV916: POT_D4, MY POTENTIOMETER LIBRARY:RK09D1130C2P
- removed SW301: TS-1187A-B-A-B, MY SWITCH LIBRARY:TS-1187A-B-A-B_smd
- removed U301: UM805RE, MY PMIC LIBRARY:UM805RE
- removed U302: UM803RS, MY PMIC LIBRARY:UM803RS
- removed U801: 6N137S1(TA), MY OPTO IC LIBRARY:6N137S1_TA_SMD-8P
- removed U802: 74HC04D,653, MY IC LIBRARY:74HC04D_653_SOIC-14
- removed U901: PEC12R-4025F-S0024, MY ENCODER LIBRARY:ENC_PEC12R-4025F-S0024
- removed VR301, VR302: TLV62569DBV, MY REGULATOR LIBRARY:TLV62569DBVR
- removed VR303: TPS79333DBVR, MY REGULATOR LIBRARY:TPS79333DBVR_SOT-23-5
- added C612: 22u, MY CAPACITOR LIBRARY:0603_CL10A226MQ8NRNC, F.Cu at (573.8, 124.4)
- added C613: 4.7u, MY CAPACITOR LIBRARY:0402_CL05A475MP5NRNC, F.Cu at (573.2, 126.6)
- added C614: 100n, MY CAPACITOR LIBRARY:0402_CL05B104KB54PNC, F.Cu at (577.2, 126.6)
- added FB602: UPZ1608U601-1R3TF, MY FERRITE BEAD LIBRARY:UPZ1608U601-1R3TF_0603, F.Cu at (577.6, 124.4)
- added J601: TF-15x15, MY CONNECTOR LIBRARY:TF-15x15_smd, F.Cu at (144.7, 84.7)
- U701: value WM8978CGEFL_RV -> M.2-B-KEY; footprint MY AUDIO CODEC LIBRARY:WM8978CGEFL_RV_WQFN-32 -> MY CONNECTOR LIBRARY:M.2-B-KEY
- moved C611 347.7 mm to (583.7, 69.8), turned to 90 degrees
- moved C607 343.5 mm to (579.6, 69.6), turned to 90 degrees
- moved C603 340.7 mm to (579.6, 72.1), turned to 90 degrees
- moved C610 340.4 mm to (583.6, 72.2), turned to 90 degrees
- moved C609 339.5 mm to (581.5, 69.7), turned to 90 degrees
- moved C601 338.4 mm to (575.2, 71.4), turned to 90 degrees
- moved C602 338.4 mm to (577.5, 72.0), turned to 90 degrees
- moved C604 338.3 mm to (581.5, 72.1), turned to 90 degrees
- moved C605 331.2 mm to (577.4, 69.6), turned to 90 degrees
- moved FB601 325.7 mm to (572.4, 71.5), turned to 90 degrees
- moved C606 315.0 mm to (575.4, 87.0), turned to 90 degrees
- moved C608 313.2 mm to (577.5, 87.0), turned to 90 degrees
- moved R601 306.3 mm to (571.7, 87.0), turned to 90 degrees
- moved C409 262.3 mm to (485.1, 61.6), turned to 90 degrees
- moved L401 259.4 mm to (485.7, 84.4), turned to 90 degrees
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- renumbered C512 to C510, C510 to C511, C511 to C512, C610 to C606, C606 to C607, C611 to C608, C607 to C609, C608 to C610, C609 to C611, U1 to U401
Connections:
- U401 pad A10: GPIO_B0_11 -> IO22
- U401 pad A11: GPIO_B1_00 -> IO20
- U401 pad A12: GPIO_B1_08 -> IO18
- U401 pad A13: GPIO_B1_09 -> IO16
- U401 pad A8: GPIO_B0_06 -> IO28
- U401 pad A9: GPIO_B0_07 -> IO25
- U401 pad B11: GPIO_B1_01 -> IO19
- U401 pad B12: GPIO_B1_07 -> IO17
- U401 pad B13: GPIO_B1_10 -> IO15
- U401 pad B14: GPIO_B1_15 -> IO14
- U401 pad B8: GPIO_B0_05 -> IO27
- U401 pad B9: GPIO_B0_08 -> IO24
- U401 pad C10: GPIO_B0_12 -> IO21
- U401 pad C11: GPIO_B1_02 -> IO6
- U401 pad C12: GPIO_B1_06 -> IO9
- U401 pad C13: GPIO_B1_11 -> IO11
- U401 pad C14: GPIO_B1_14 -> IO13
- U401 pad C8: GPIO_B0_04 -> IO26
- U401 pad C9: GPIO_B0_09 -> IO23
- U401 pad D10: GPIO_B0_13 -> IO3
- U401 pad D11: GPIO_B1_03 -> IO5
- U401 pad D12: GPIO_B1_05 -> IO8
- U401 pad D13: GPIO_B1_12 -> IO10
- U401 pad D14: WATCHDOG_B -> IO12
- U401 pad D7: GPIO_B0_00 -> SPI_CS
- U401 pad D8: GPIO_B0_03 -> SPI_SCK
- U401 pad D9: GPIO_B0_10 -> IO1
- U401 pad E10: GPIO_B0_14 -> IO2
- U401 pad E11: GPIO_B0_15 -> IO4
- U401 pad E12: GPIO_B1_04 -> IO7
- U401 pad E7: GPIO_B0_01 -> SPI_SIN
- U401 pad E8: GPIO_B0_02 -> SPI_SOUT
- U401 pad F11: GPIO_AD_B0_04 -> unconnected-(U401-PadF11)
- U401 pad G11: GPIO_AD_B0_03 -> unconnected-(U401-PadG11)
- U401 pad G14: GPIO_AD_B0_05 -> unconnected-(U401-PadG14)
- U401 pad H10: GPIO_AD_B0_01 -> unconnected-(U401-PadH10)
- U401 pad H13: GPIO_AD_B1_08 -> unconnected-(U401-PadH13)
- U401 pad H14: GPIO_AD_B0_14 -> unconnected-(U401-PadH14)
- U401 pad H2: unconnected-(U1-PadH2) -> SD_DAT2
- U401 pad J1: unconnected-(U1-PadJ1) -> SD_DAT0
- U401 pad J12: GPIO_AD_B1_06 -> unconnected-(U401-PadJ12)
- U401 pad J13: GPIO_AD_B1_11 -> unconnected-(U401-PadJ13)
- U401 pad J2: unconnected-(U1-PadJ2) -> SD_DAT3
- U401 pad J3: unconnected-(U1-PadJ3) -> SD_CLK
- U401 pad J4: unconnected-(U1-PadJ4) -> SD_CMD
- U401 pad K1: unconnected-(U1-PadK1) -> SD_DAT1
- U401 pad K10: GPIO_AD_B1_07 -> unconnected-(U401-PadK10)
- U401 pad K12: GPIO_AD_B1_05 -> unconnected-(U401-PadK12)
- U401 pad K14: GPIO_AD_B0_12 -> MIDI_IN
- U401 pad L10: GPIO_AD_B0_15 -> unconnected-(U401-PadL10)
- U401 pad L11: GPIO_AD_B1_02 -> unconnected-(U401-PadL11)
- U401 pad L12: GPIO_AD_B1_04 -> unconnected-(U401-PadL12)
- U401 pad L13: GPIO_AD_B1_10 -> unconnected-(U401-PadL13)
- U401 pad L14: GPIO_AD_B0_13 -> MIDI_OUT
- U401 pad M11: GPIO_AD_B0_02 -> unconnected-(U401-PadM11)
- U401 pad M12: GPIO_AD_B1_03 -> unconnected-(U401-PadM12)
- U401 pad M14: GPIO_AD_B0_00 -> unconnected-(U401-PadM14)
- U401 pad M6: unconnected-(U1-PadM6) -> ON_OFF
Other:
- board size 127 x 127 mm -> 22 x 62 mm
- board text added: "1V8"
- board text added: "DCDC IN"
- board text added: "DCDC_LP"
- board text added: "MCU OTHER CIRCUITS"
- board text added: "MCU POWER SUPPLY DECOUPLING"
- board text added: "NVCC PLL"
- board text added: "NVCC_EMC"
- board text added: "NVCC_GPIO"
- board text added: "NVCC_SD0"
- board text added: "NVCC_SD1"
- board text added: "QSPI FLASH"
- board text added: "RC DELAY"
- board text added: "RESET CIRCUIT"
- board text added: "SDRAM"
- board text added: "SDRAM - FLASH"
- board text added: "USB"
- board text added: "VDDA_ADC_3P3"
- board text added: "VDD_HIGH_CAP"
- board text added: "VDD_HIGH_IN"
- board text added: "VDD_SNVS_CAP"
- board text added: "VDD_SNVS_IN"
- board text added: "VDD_SOC_IN"
- board text added: "XTAL"

Commit message: updates
Parts:
- moved J601 6.00 mm to (144.5, 90.7)
- moved U401 3.02 mm to (143.8, 120.0)
- moved U601 1.59 mm to (136.9, 107.8)
- moved U602 1.17 mm to (150.8, 107.8)
Connections:
- C510 pad 1: +5V -> VBUS
- U401 pad K14: MIDI_IN -> MIDI_OUT
- U401 pad L14: MIDI_OUT -> MIDI_IN
- U401 pad N6: +5V -> VBUS
- U701 pad MOUNTING-HOLE: unconnected-(U701-PadMOUNTING-HOLE) -> GND
Other:
- board size 22 x 62 mm -> 22 x 60 mm
- copper layers 2 -> 6
- board text removed: "1V8"
- board text removed: "RESET CIRCUIT"

Commit message: updates
Parts:
- added R501: 0R, MY RESISTOR LIBRARY:0603WAF0000T5E, F.Cu at (458.5, 128.5)
- added R502: 0R, MY RESISTOR LIBRARY:0603WAF0000T5E, F.Cu at (454.5, 128.5)
- added R503: 0R, MY RESISTOR LIBRARY:0603WAF0000T5E, F.Cu at (454.5, 126.0)
- added R504: 0R, MY RESISTOR LIBRARY:0603WAF0000T5E, F.Cu at (458.5, 126.0)
- added R505: 0R, MY RESISTOR LIBRARY:0603WAF0000T5E, F.Cu at (462.5, 128.5)
- added R506: 0R, MY RESISTOR LIBRARY:0603WAF0000T5E, F.Cu at (462.5, 126.0)
- moved U601 1.15 mm to (138.1, 107.9)
- moved C410 0.61 mm to (322.7, 63.7)
- moved Y402 0.35 mm to (477.4, 61.7)
Connections:
- net Net-(C513-Pad1) renamed /MCU GPIO & BUS/USB CAP
- net Net-(L401-Pad1) renamed /MCU POWER & CRYSTALS/DCDC_LP
- U401 pad B3: SDRAM_CLK -> Net-(R501-Pad1)
- U401 pad G12: I2S_BCLK -> Net-(R505-Pad2)
- U401 pad J14: I2S_LRC -> Net-(R506-Pad2)
- U401 pad J3: SD_CLK -> Net-(R502-Pad1)
- U401 pad L4: FLEXSPI_CLK -> Net-(R503-Pad1)
- U401 pad M13: I2S_MCLK -> Net-(R504-Pad2)
Other:
- board text added: "FLASH"
- board text added: "MCU"
- board text added: "Terminaison resistor"

Commit message: updates
Parts:
- C410, C411, C412, C413, C415, C418, C422, C424, C504, C508: moved to B.Cu
- moved C601 439.6 mm to (140.8, 138.3)
- moved C602 439.6 mm to (143.0, 138.9)
- moved C603 439.6 mm to (145.2, 139.0)
- moved C604 439.6 mm to (147.0, 139.0)
- moved C605 439.6 mm to (142.9, 136.5)
- moved C606 439.6 mm to (140.9, 153.8)
- moved C607 439.6 mm to (145.1, 136.5)
- moved C608 439.6 mm to (143.0, 153.9)
- moved C610 439.6 mm to (149.2, 139.1)
- moved C611 439.6 mm to (149.2, 136.7)
- moved FB601 439.6 mm to (137.9, 138.4)
- moved R601 439.6 mm to (137.2, 153.8)
- moved C609 439.6 mm to (147.1, 136.6)
- moved C613 433.1 mm to (141.9, 166.3)
- moved FB602 433.1 mm to (146.3, 164.0)
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Connections:
- U401 pad E9: GND -> +3V3
- U401 pad F10: GND -> +3V3
- U401 pad J10: GND -> +3V3
Routing:
- net GND: track 0.00 -> 28.2 mm, vias 0 -> 11
- net +3V3: track 0.00 -> 16.9 mm, vias 0 -> 5
- net /MCU POWER & CRYSTALS/VDD_SOC_IN: track 0.00 -> 14.7 mm, vias 0 -> 8
- net SDRAM_D13: track 0.00 -> 7.26 mm, vias 0 -> 1
- net SDRAM_D5: track 0.00 -> 6.74 mm, vias 0 -> 1
- net SDRAM_D6: track 0.00 -> 4.02 mm, vias 0 -> 1
- net USB_D+: track 0.00 -> 3.90 mm, vias 0 -> 1
- net SDRAM_D12: track 0.00 -> 3.64 mm, vias 0 -> 1
- net SDRAM_D15: track 0.00 -> 3.53 mm, vias 0 -> 1
- net SDRAM_D2: track 0.00 -> 3.51 mm, vias 0 -> 1
- net SDRAM_D3: track 0.00 -> 3.46 mm, vias 0 -> 1
- net SDRAM_D10: track 0.00 -> 3.41 mm, vias 0 -> 1
- net SDRAM_DQMH: track 0.00 -> 3.41 mm, vias 0 -> 1
- net SPI_SIN: track 0.00 -> 3.33 mm, vias 0 -> 1
- net I2S_DACDAT: track 0.00 -> 3.29 mm, vias 0 -> 1
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- added copper zone on B.Cu, net /MCU POWER & CRYSTALS/VDD_SOC_IN
- added copper zone on B.Cu, net GND
Other:
- board size 22 x 60 mm -> 60 x 22 mm
- board text added: "SD CARD"
- board text removed: "RC DELAY"

Commit message: up
Parts:
- moved R402 77.3 mm to (158.4, 102.9)
- moved C407 30.5 mm to (257.5, 44.2)
- moved C502 17.6 mm to (257.1, 100.1)
- moved C414 8.98 mm to (244.3, 100.8)
- moved C417 8.98 mm to (241.3, 100.7)
- moved C421 6.27 mm to (221.0, 45.2)
- moved C509 1.49 mm to (229.5, 103.7)
- moved C511 1.49 mm to (229.5, 99.5)
- moved C512 1.49 mm to (225.8, 99.5)
Other:
- board text removed: "NVCC_SD1"
- board text removed: "VDD_SNVS_CAP"
Changed lines of the file:
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@@
   )
   (footprint "MY CAPACITOR LIBRARY:0402_CL05B224KO5NNNC" (layer "F.Cu")
-    (at 230.66 58.73 90)
+    (at 257.46 44.19 90)
     (descr "0402 - SMD MLCC")
     (tags "capacitor")
@@
   )
   (footprint "MY RESISTOR LIBRARY:AF0402FR-0730KL" (layer "F.Cu")
-    (at 89.7 67.48 -90)
+    (at 158.45 102.88 -90)
     (descr "0402 SMD Resistor")
     (tags "resistor")
@@
   )
   (footprint "MY CAPACITOR LIBRARY:0402_CL05B104KB54PNC" (layer "F.Cu")
-    (at 231.01 103.86 90)
+    (at 229.53 103.71 90)
     (descr "0402 - SMD MLCC")
     (tags "capacitor")
@@
   )
   (footprint "MY CAPACITOR LIBRARY:0402_CL05A475MP5NRNC" (layer "F.Cu")
-    (at 250.26 101.76 90)
+    (at 241.34 100.73 90)
     (descr "0402 - SMD MLCC")
     (tags "capacitor")
@@
   )
   (footprint "MY CAPACITOR LIBRARY:0402_CL05B224KO5NNNC" (layer "F.Cu")
-    (at 214.75 45.59 90)
+    (at 221.01 45.19 90)
     (descr "0402 - SMD MLCC")
     (tags "capacitor")
@@
   )
   (footprint "MY CAPACITOR LIBRARY:0402_CL05B104KB54PNC" (layer "F.Cu")
-    (at 246.07 86.47 90)
+    (at 257.14 100.09 90)
     (descr "0402 - SMD MLCC")
     (tags "capacitor")
@@
   )
   (footprint "MY CAPACITOR LIBRARY:0402_CL05B104KB54PNC" (layer "F.Cu")
-    (at 227.26 99.66 90)
+    (at 225.78 99.51 90)
     (descr "0402 - SMD MLCC")
     (tags "capacitor")
@@
   )
   (footprint "MY CAPACITOR LIBRARY:0402_CL05B104KB54PNC" (layer "F.Cu")
-    (at 231.01 99.66 90)
+    (at 229.53 99.51 90)
     (descr "0402 - SMD MLCC")
     (tags "capacitor")
@@
   )
   (footprint "MY CAPACITOR LIBRARY:0402_CL05B224KO5NNNC" (layer "F.Cu")
-    (at 253.26 101.86 90)
+    (at 244.34 100.83 90)
     (descr "0402 - SMD MLCC")
     (tags "capacitor")
@@
   (gr_rect (start 237.36 47.78) (end 225.91 40.13) (layer "User.2") (width 1) (fill none))
   (gr_rect (start 219.37 90.51) (end 204.02 80.61) (layer "User.2") (width 1) (fill none))
-  (gr_rect (start 226.31 55.48) (end 234.61 62.43) (layer "User.2") (width 1) (fill none))
+  (gr_rect (start 253.11 40.94) (end 261.41 47.89) (layer "User.2") (width 1) (fill none))
   (gr_rect (start 187.215 59.14) (end 151.615 42.89) (layer "User.2") (width 1) (fill none))
   (gr_rect (start 152.86 143.69) (end 133.81 131.89) (layer "User.2") (width 1) (fill none))
   (gr_rect (start 146.76 158.44) (end 133.86 149.89) (layer "User.2") (width 1) (fill none))
-  (gr_rect (start 250.57 90.59) (end 239.77 82.59) (layer "User.2") (width 1) (fill none))
-  (gr_rect (start 253.41 62.58) (end 243.86 55.83) (layer "User.2") (width 1) (fill none))
+  (gr_rect (start 261.64 104.21) (end 250.84 96.21) (layer "User.2") (width 1) (fill none))
   (gr_rect (start 271.13 111.51) (end 200.2 34.99) (layer "User.2") (width 1) (fill none))
   (gr_rect (start 226.77 135.38) (end 201.31 118.66) (layer "User.2") (width 2) (fill none))
@@
   (gr_rect (start 187.915 79.34) (end 175.965 71.04) (layer "User.2") (width 1) (fill none))
   (gr_rect (start 192.525 82) (end 142.795 34.74) (layer "User.2") (width 1) (fill none))
-  (gr_rect (start 267.24 91.27) (end 255.34 82.47) (layer "User.2") (width 1) (fill none))
-  (gr_rect (start 257.41 106.16) (end 245.86 97.16) (layer "User.2") (width 1) (fill none))
-  (gr_rect (start 236.21 107.21) (end 223.46 96.21) (layer "User.2") (width 1) (fill none))
+  (gr_rect (start 248.49 105.13) (end 236.94 96.13) (layer "User.2") (width 1) (fill none))
+  (gr_rect (start 234.73 107.06) (end 221.98 96.06) (layer "User.2") (width 1) (fill none))
   (gr_rect (start 223.25 50.49) (end 203.3 40.29) (layer "User.2") (width 1) (fill none))
   (gr_rect (start 239.96 47.81) (end 251.01 40.56) (layer "User.2") (width 1) (fill none))
@@
     (effects (font (size 2 2) (thickness 0.5) italic))
   )
-  (gr_text "VDD_SNVS_IN" (at 230.66 54.28) (layer "User.2")
-    (effects (font (size 1 1) (thickness 0.15) italic))
-  )
-  (gr_text "VDD_SNVS_CAP" (at 248.71 54.68) (layer "User.2")
+  (gr_text "VDD_SNVS_IN" (at 257.46 39.74) (layer "User.2")
     (effects (font (size 1 1) (thickness 0.15) italic))
   )
@@
     (effects (font (size 1 1) (thickness 0.15) italic))
   )
-  (gr_text "NVCC_SD0" (at 243.17 81.34) (layer "User.2")
+  (gr_text "NVCC_SD0" (at 254.24 94.96) (layer "User.2")
     (effects (font (size 1 1) (thickness 0.15) italic))
   )
@@
     (effects (font (size 1 1) (thickness 0.15) italic))
   )
-  (gr_text "NVCC_SD1" (at 258.79 81.17) (layer "User.2")
-    (effects (font (size 1 1) (thickness 0.15) italic))
-  )
   (gr_text "MCU POWER SUPPLY\nDECOUPLING" (at 238.53 24.69) (layer "User.2")
     (effects (font (size 5 5) (thickness 1) italic))
@@
     (effects (font (size 1 1) (thickness 0.15) italic))
   )
-  (gr_text "NVCC_GPIO" (at 227.21 95.01) (layer "User.2")
+  (gr_text "NVCC_GPIO" (at 225.73 94.86) (layer "User.2")
     (effects (font (size 1 1) (thickness 0.15) italic))
   )
@@
     (effects (font (size 1 1) (thickness 0.15) italic))
   )
-  (gr_text "NVCC PLL" (at 249.01 96.01) (layer "User.2")
+  (gr_text "NVCC PLL" (at 240.09 94.98) (layer "User.2")
     (effects (font (size 1 1) (thickness 0.15) italic))
   )

Commit message: updates
Parts:
- removed FB401: 120R, MY FERRITE BEAD LIBRARY:0603_BLM18AG121SN1D
- added C425: 220n, MY CAPACITOR LIBRARY:0402_CL05B224KO5NNNC, F.Cu at (149.1, 105.3)
- added C426: 220n, MY CAPACITOR LIBRARY:0402_CL05B224KO5NNNC, F.Cu at (148.1, 105.4)
- C407, C416, C505, C507, C513, C514, C601, C602, C604, C607, C610, C611, C613, C614, FB601, FB602, R402, R601: moved to B.Cu
- L401: value 4.7u -> VLS4012ET-4R7M; footprint MY INDUCTOR LIBRARY:LQM21PN4R7MGRD -> MY INDUCTOR LIBRARY:VLS4012ET-4R7M
- moved C407 106.3 mm to (171.2, 106.3), turned to -90 degrees
- moved C423 101.8 mm to (166.0, 106.5), turned to 0 degrees
- moved C420 99.2 mm to (166.0, 105.7), turned to 0 degrees
- moved C502 98.9 mm to (158.3, 105.4), turned to 0 degrees
- moved C402 93.0 mm to (172.1, 104.0)
- moved C421 88.7 mm to (155.7, 105.2), turned to -90 degrees
- moved C427 86.1 mm to (156.8, 105.5), turned to -90 degrees
- moved C514 85.5 mm to (169.2, 106.8), turned to 0 degrees
- moved C513 84.8 mm to (167.8, 105.7), turned to 0 degrees
- moved C401 84.0 mm to (171.2, 104.0)
- moved C507 81.0 mm to (161.6, 105.8), turned to -90 degrees
- moved C505 80.7 mm to (163.1, 104.2), turned to 0 degrees
- moved C419 79.9 mm to (150.3, 105.6), turned to -90 degrees
- moved C414 79.1 mm to (166.0, 111.4), turned to 0 degrees
- moved C417 76.3 mm to (165.9, 112.4), turned to 0 degrees
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- renumbered C425 to C427, C511 to C510, C510 to C511
Connections:
- C416 pad 1: /MCU POWER & CRYSTALS/DCDC_IN -> +3V3
- C419 pad 1: /MCU POWER & CRYSTALS/DCDC_IN -> +3V3
- C422 pad 1: /MCU POWER & CRYSTALS/DCDC_IN -> +3V3
- R402 pad 1: /MCU POWER & CRYSTALS/DCDC_IN -> +3V3
- U401 pad K4: /MCU POWER & CRYSTALS/DCDC_IN -> +3V3
- U401 pad L1: /MCU POWER & CRYSTALS/DCDC_IN -> +3V3
- U401 pad L2: /MCU POWER & CRYSTALS/DCDC_IN -> +3V3
Routing:
- net SD_CMD: track 3.27 -> 0.00 mm, vias 1 -> 0
- net GND: track 28.2 -> 31.4 mm, vias 11 -> 12
- net /MCU POWER & CRYSTALS/DCDC_IN: track 1.83 -> 0.00 mm, vias 2 -> 0
- net +3V3: track 16.9 -> 18.7 mm, vias 5 -> 7
Other:
- board text removed: "DCDC IN"
- board text removed: "DCDC_LP"
- board text removed: "MCU OTHER CIRCUITS"
- board text removed: "MCU POWER SUPPLY DECOUPLING"
- board text removed: "NVCC PLL"
- board text removed: "NVCC_EMC"
- board text removed: "NVCC_GPIO"
- board text removed: "NVCC_SD0"
- board text removed: "QSPI FLASH"
- board text removed: "SDRAM - FLASH"
- board text removed: "Terminaison resistor"
- board text removed: "USB"
- board text removed: "VDDA_ADC_3P3"
- board text removed: "VDD_HIGH_CAP"
- board text removed: "VDD_HIGH_IN"
- board text removed: "VDD_SNVS_IN"
- board text removed: "VDD_SOC_IN"
- board text removed: "XTAL"
