File: DESIGN FILES/MIMXRT1064 MCU Module.kicad_pcb (KiCad board)
At the start: 6 copper layers, 60 x 22 mm, 74 parts, among them J601 TF-15x15, U401 MIMXRT1064CVL5B, U601 IS25WP064A-JBLE, U602 IS42S16160J-6BLI, U701 M.2-B-KEY, Y401 7V24000026, Y402 Q13FC1350000200

Commit message: updates
Parts:
- moved C602 3.27 mm to (144.3, 95.7)
- moved C601 3.27 mm to (141.7, 97.0)
- moved C603 3.27 mm to (150.3, 95.9)
- moved C605 3.27 mm to (150.9, 98.7)
- moved C609 3.27 mm to (150.9, 99.9)
- moved C611 3.27 mm to (141.9, 99.5)
- moved U602 3.27 mm to (145.6, 97.1)
- moved C604 3.27 mm to (146.1, 95.7)
- moved C607 3.27 mm to (148.6, 97.3)
- moved C610 3.27 mm to (146.4, 98.3)
- moved FB601 3.27 mm to (144.3, 94.7)
- moved U601 1.94 mm to (154.2, 110.1)
- moved R601 1.93 mm to (154.2, 111.8)
- moved C606 1.89 mm to (148.4, 111.3)
- moved C608 1.87 mm to (148.4, 112.4)
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Connections:
- net Net-(R501-Pad1) renamed /MCU GPIO & BUS/SDRAM_CLK_RES
- net Net-(R502-Pad1) renamed /MCU GPIO & BUS/SD_CLK_RES
- net Net-(R503-Pad1) renamed /MCU GPIO & BUS/FLEXSPI_CLK_RES
- net Net-(R504-Pad2) renamed /MCU GPIO & BUS/I2S_MCLK_RES
- net Net-(R505-Pad2) renamed /MCU GPIO & BUS/I2S_BCLK_RES
- net Net-(R506-Pad2) renamed /MCU GPIO & BUS/I2C_LRC_RES
- U401 pad J5: /MCU POWER & CRYSTALS/VDD_SOC_IN -> unconnected-(U401-PadJ5)
- U701 pad P$62: +5V -> VBUS
Routing:
- net GND: track 31.4 -> 20.8 mm, vias 12 -> 18
- net /MCU POWER & CRYSTALS/VDD_SOC_IN: track 14.7 -> 7.22 mm, vias 8 -> 7
- net +1V8: track 0.45 -> 7.88 mm, vias 1 -> 4
- net VBUS: track 1.71 -> 6.49 mm, vias 0 -> 3
- net SD_CMD: track 0.00 -> 3.49 mm, vias 0 -> 1
- net PMIC_ON_REQ: track 0.45 -> 3.88 mm
- net /MCU GPIO & BUS/USB CAP: track 0.45 -> 3.87 mm
- net JTAG_nTRST: track 0.45 -> 3.34 mm
- net IO2: track 0.45 -> 3.33 mm
- net SPI_SOUT: track 0.45 -> 3.33 mm
- net SDRAM_D2: track 3.51 -> 6.38 mm
- net SDRAM_D15: track 3.53 -> 6.41 mm
- net SDRAM_D13: track 7.26 -> 4.39 mm
- net SDRAM_D5: track 6.74 -> 3.87 mm
- net SDRAM_D3: track 3.46 -> 6.34 mm
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- added copper zone on In3.Cu, net +1V8
- added copper zone on In3.Cu, net +3V3
- added copper zone on In1.Cu, net GND
- added copper zone on In4.Cu, net GND
- added copper zone on In3.Cu, net VBUS

Commit message: updates
Parts:
- added D401: LED_BLUE, MY LED LIBRARY:19-218_BHC-ZL1M2QY_3T, F.Cu at (172.7, 93.6)
- added R401: 2.2k, MY RESISTOR LIBRARY:0603WAF2201T5E, F.Cu at (169.8, 93.6)
- added REF**: OSHW-Logo_5.7x6mm_SilkScreen, Symbol:OSHW-Logo_5.7x6mm_SilkScreen, F.Cu at (143.9, 107.5)
- added REF**: TestPoint_Pad_D1.0mm, TestPoint:TestPoint_Pad_D1.0mm, F.Cu at (182.4, 107.0)
- moved C407 0.68 mm to (171.3, 106.5)
- renumbered R401 to R402, R402 to R403, R502 to R501, R501 to R502, R505 to R504, R506 to R505, R504 to R506
Routing:
- net +1V8: track 7.88 -> 4.09 mm, vias 4 -> 3
- net /MCU GPIO & BUS/FLEXSPI_CLK_RES: track 0.00 -> 2.55 mm, vias 0 -> 1
- net VBUS: track 6.49 -> 4.34 mm
- net +3V3: track 18.9 -> 19.6 mm, vias 13 -> 14
Other:
- board text added: "JU REVA 07/23"
- board text added: "SOLAR AUDIO"
- board text added: "uSD"
- board text removed: "SD CARD"

Commit message: updates
Parts:
- removed R502: 0R, MY RESISTOR LIBRARY:0603WAF0000T5E
- removed REF**: OSHW-Logo_5.7x6mm_SilkScreen, Symbol:OSHW-Logo_5.7x6mm_SilkScreen
- removed REF**: TestPoint_Pad_D1.0mm, TestPoint:TestPoint_Pad_D1.0mm
- C603, C605, C609: moved to B.Cu
- moved U601 13.9 mm to (142.5, 102.7), turned to -90 degrees
- moved L401 13.1 mm to (142.3, 110.4)
- moved C427 11.2 mm to (162.1, 115.7)
- moved C421 10.6 mm to (159.3, 115.3)
- moved C425 10.3 mm to (149.1, 115.2)
- moved C426 10.2 mm to (147.8, 115.1)
- moved C419 9.98 mm to (150.8, 115.2)
- moved C601 9.70 mm to (150.5, 100.9)
- moved C602 9.26 mm to (149.9, 103.1), turned to 180 degrees
- moved C502 8.86 mm to (160.8, 114.2)
- moved FB601 8.19 mm to (148.1, 102.0), turned to 180 degrees
- moved R501 7.39 mm to (139.5, 94.2)
- moved U602 7.31 mm to (150.4, 102.6)
- moved R503 6.48 mm to (159.9, 111.6), turned to 90 degrees
- moved R403 6.42 mm to (163.8, 108.5), turned to -90 degrees
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Connections:
- U401 pad B3: /MCU GPIO & BUS/SDRAM_CLK_RES -> SDRAM_CLK
Routing:
- net SDRAM_CLK: track 0.00 -> 34.5 mm
- net SDRAM_A4: track 0.47 -> 32.5 mm
- net SDRAM_A1: track 0.47 -> 31.9 mm
- net SDRAM_CKE: track 0.47 -> 30.8 mm
- net SDRAM_A3: track 0.47 -> 30.3 mm
- net SDRAM_BA1: track 0.47 -> 29.5 mm
- net SDRAM_A5: track 1.26 -> 30.3 mm
- net SDRAM_CS: track 0.47 -> 29.2 mm
- net SDRAM_BA0: track 0.47 -> 28.7 mm
- net SDRAM_A12: track 0.47 -> 28.2 mm
- net SDRAM_WE: track 0.47 -> 27.9 mm
- net SDRAM_A10: track 1.80 -> 29.2 mm
- net SDRAM_RAS: track 1.24 -> 28.1 mm
- net SDRAM_A7: track 0.47 -> 27.3 mm
- net SDRAM_A2: track 2.45 -> 28.9 mm
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
Commit message: updates
Parts:
- removed R501, R503: 0R, MY RESISTOR LIBRARY:0603WAF0000T5E
- C419, C420, C423, C425, C426, C502, C511, C606, C608, C612: moved to B.Cu
- C603, C604: moved to F.Cu
- moved R601 18.0 mm to (143.9, 97.4), turned to 0 degrees
- moved C427 17.4 mm to (145.2, 111.2), turned to 90 degrees
- moved C426 16.6 mm to (162.8, 108.0), turned to 90 degrees
- moved C608 16.0 mm to (143.7, 103.3)
- moved C419 15.4 mm to (164.9, 109.1)
- moved C606 13.7 mm to (143.7, 104.3)
- moved C604 13.7 mm to (155.6, 105.0), turned to 90 degrees
- moved C421 13.6 mm to (146.3, 111.5), turned to 90 degrees
- moved C425 13.0 mm to (160.9, 109.8)
- moved C603 9.84 mm to (154.9, 105.0), turned to -90 degrees
- moved C612 9.78 mm to (135.3, 101.5), turned to 180 degrees
- moved R402 7.19 mm to (166.7, 110.9), turned to 180 degrees
- moved C605 6.94 mm to (152.5, 102.4)
- moved C502 6.28 mm to (161.8, 108.0), turned to 90 degrees
- moved C609 6.15 mm to (150.5, 102.4)
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Connections:
- U401 pad J3: /MCU GPIO & BUS/SD_CLK_RES -> SD_CLK
- U401 pad L4: /MCU GPIO & BUS/FLEXSPI_CLK_RES -> FLEXSPI_CLK
Routing:
- net GND: track 20.8 -> 30.5 mm, vias 18 -> 22
- net +3V3: track 19.6 -> 24.7 mm, vias 14 -> 15
- net FLEXSPI_CLK: track 0.00 -> 2.55 mm, vias 0 -> 1
- net /MCU GPIO & BUS/FLEXSPI_CLK_RES: track 2.55 -> 0.00 mm, vias 1 -> 0
- net SD_CLK: track 0.00 -> 2.04 mm, vias 0 -> 1
- net /MCU GPIO & BUS/SD_CLK_RES: track 2.04 -> 0.00 mm, vias 1 -> 0
- net VBUS: track 4.34 -> 5.37 mm
- added copper zone on F.Cu, net +3V3

Commit message: up
Parts:
- removed R504, R505, R506: 0R, MY RESISTOR LIBRARY:0603WAF0000T5E
- C401, C402, C405, C408, C414, C417: moved to B.Cu
- R601: moved to F.Cu
- moved C511 6.68 mm to (173.2, 108.3), turned to 90 degrees
- moved C406 5.11 mm to (164.9, 111.6), turned to -90 degrees
- moved C417 4.13 mm to (169.0, 108.5), turned to -90 degrees
- moved C414 4.05 mm to (168.0, 108.5), turned to -90 degrees
- moved C409 3.51 mm to (161.4, 111.6), turned to -90 degrees
- moved C502 3.26 mm to (161.4, 111.3), turned to -90 degrees
- moved C419 2.49 mm to (164.0, 111.4), turned to 0 degrees
- moved R403 2.33 mm to (161.9, 107.7), turned to 0 degrees
- moved C416 2.24 mm to (164.0, 109.4)
- moved C425 2.19 mm to (163.1, 109.4)
- moved C506 2.11 mm to (165.9, 94.0), turned to -90 degrees
- moved C407 2.10 mm to (171.7, 106.2)
- moved C408 2.04 mm to (173.5, 105.4)
- moved C514 1.82 mm to (170.5, 108.6), turned to -90 degrees
- moved C426 1.60 mm to (162.1, 109.5), turned to -90 degrees
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Connections:
- U401 pad A8: IO28 -> IO27
- U401 pad A9: IO25 -> IO24
- U401 pad B8: IO27 -> IO28
- U401 pad B9: IO24 -> IO25
- U401 pad G12: /MCU GPIO & BUS/I2S_BCLK_RES -> I2S_BCLK
- U401 pad J14: /MCU GPIO & BUS/I2C_LRC_RES -> I2S_LRC
- U401 pad M13: /MCU GPIO & BUS/I2S_MCLK_RES -> I2S_MCLK
- U701 pad P$10: JTAG_TDI -> unconnected-(U701-PadP$10)
- U701 pad P$2: USB_D+ -> SPI_SIN
- U701 pad P$20: JTAG_TCK -> GND
- U701 pad P$21: IO23 -> IO22
- U701 pad P$22: JTAG_TDO -> IO23
- U701 pad P$23: IO22 -> IO20
- U701 pad P$24: JTAG_nTRST -> IO1
- U701 pad P$25: IO21 -> IO19
- U701 pad P$26: GND -> IO21
- U701 pad P$27: IO20 -> IO18
- U701 pad P$28: GND -> IO3
- U701 pad P$29: IO19 -> IO17
- U701 pad P$3: IO26 -> IO28
- U701 pad P$30: I2S_BCLK -> IO6
- U701 pad P$31: IO18 -> IO16
- U701 pad P$32: I2S_ADCDAT -> IO9
- U701 pad P$33: IO17 -> IO14
- U701 pad P$34: I2S_DACDAT -> IO5
- U701 pad P$35: IO16 -> IO15
- U701 pad P$36: I2S_LRC -> IO8
- U701 pad P$37: IO15 -> IO13
- U701 pad P$38: I2S_MCLK -> IO4
- U701 pad P$39: IO14 -> IO11
- U701 pad P$4: USB_D- -> SPI_CS
- U701 pad P$41: IO13 -> IO12
- U701 pad P$42: CODEC_SCL -> IO7
- U701 pad P$43: IO12 -> IO10
- U701 pad P$44: CODEC_SDA -> IO2
- U701 pad P$45: IO11 -> JTAG_TMS
- U701 pad P$47: IO10 -> JTAG_TCK
- U701 pad P$48: MIDI_IN -> CODEC_SCL
- U701 pad P$49: IO9 -> JTAG_TDI
- U701 pad P$50: MIDI_OUT -> CODEC_SDA
- U701 pad P$51: IO8 -> JTAG_TDO
- U701 pad P$53: IO7 -> JTAG_nTRST
- U701 pad P$55: IO6 -> I2S_BCLK
- U701 pad P$57: IO5 -> I2S_DACDAT
- U701 pad P$59: IO4 -> I2S_ADCDAT
- U701 pad P$6: GND -> SPI_SOUT
- U701 pad P$61: IO3 -> I2S_LRC
- U701 pad P$63: IO2 -> I2S_MCLK
- U701 pad P$65: IO1 -> MIDI_OUT
- U701 pad P$67: SPI_SCK -> MIDI_IN
- U701 pad P$69: SPI_SOUT -> GND
- U701 pad P$7: IO28 -> IO26
- U701 pad P$71: SPI_SIN -> USB_D+
- U701 pad P$73: SPI_CS -> USB_D-
- U701 pad P$8: JTAG_TMS -> SPI_SCK
Routing:
- net GND: track 30.5 -> 124.9 mm, vias 22 -> 48
- net SD_CLK: track 2.04 -> 45.3 mm, vias 1 -> 6
- net SD_DAT2: track 1.25 -> 42.8 mm, vias 0 -> 2
- net SD_DAT1: track 0.47 -> 41.6 mm, vias 0 -> 4
- net SD_DAT0: track 0.47 -> 37.8 mm, vias 0 -> 2
- net FLEXSPI_D2: track 0.47 -> 37.1 mm, vias 0 -> 2
- net /MCU POWER & CRYSTALS/VDD_SOC_IN: track 7.22 -> 42.7 mm, vias 7 -> 8
- net SD_DAT3: track 1.24 -> 36.3 mm, vias 0 -> 2
- net /MCU POWER & CRYSTALS/DCDC_LP: track 1.20 -> 33.5 mm, vias 0 -> 2
- net SD_CMD: track 3.03 -> 32.4 mm, vias 1 -> 2
- net FLEXSPI_D1: track 1.26 -> 30.6 mm, vias 0 -> 2
- net FLEXSPI_D3: track 0.47 -> 29.7 mm, vias 0 -> 2
- net FLEXSPI_D0: track 0.47 -> 26.9 mm, vias 0 -> 2
- net FLEXSPI_SS: track 2.56 -> 28.2 mm, vias 1 -> 2
- net FLEXSPI_CLK: track 2.55 -> 24.9 mm, vias 1 -> 2
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- added copper zone on In3.Cu, net SDRAM_3V3

Commit message: up
Parts:
- U602: value IS42S16160J-6BLI -> BGA54C80P9X9_800X800X120
Routing:
- net GND: track 124.9 -> 125.7 mm

Commit message: up
Parts:
- moved R401 1.08 mm to (170.5, 94.4), turned to 90 degrees
- moved C603 0.40 mm to (156.1, 105.7)
- moved C503 0.39 mm to (167.0, 93.7)
- moved C506 0.38 mm to (166.0, 93.7)
- moved C501 0.38 mm to (168.0, 93.7)
- moved C604 0.36 mm to (156.1, 104.7)
- moved R601 0.36 mm to (143.9, 97.4)
- moved C510 0.11 mm to (172.7, 97.2), turned to -90 degrees
- moved C509 0.08 mm to (173.6, 97.2), turned to -90 degrees
- moved C512 0.07 mm to (171.7, 97.1), turned to -90 degrees
Routing:
- net GND: track 125.7 -> 67.1 mm, vias 48 -> 66
- net +3V3: track 40.4 -> 16.8 mm, vias 17 -> 28
- net SDRAM_3V3: track 16.6 -> 6.05 mm, vias 7 -> 10
- net /MEMORY /SD_VDD: track 6.35 -> 0.02 mm
- net +1V8: track 14.1 -> 9.58 mm, vias 5 -> 6
- net /MCU POWER & CRYSTALS/VDD_HIGH_CAP: track 2.77 -> 1.22 mm
- net /MCU POWER & CRYSTALS/NVCC_PLL: track 2.95 -> 1.46 mm
- net /MCU POWER & CRYSTALS/VDD_SOC_IN: track 42.7 -> 44.0 mm
- net VBUS: track 3.04 -> 2.22 mm
- net IO25: track 14.3 -> 13.6 mm
- net SPI_CS: track 17.4 -> 18.0 mm
- net SPI_SOUT: track 17.5 -> 18.1 mm
- net /MCU POWER & CRYSTALS/DCDC_LP: track 33.5 -> 33.1 mm, vias 2 -> 0
- added copper zone on B.Cu, net +1V8
- added copper zone on F.Cu, net +1V8
- added copper zone on B.Cu, net +3V3
- added copper zone on B.Cu, net /MCU POWER & CRYSTALS/NVCC_PLL
- added copper zone on B.Cu, net /MCU POWER & CRYSTALS/VDD_HIGH_CAP
- added copper zone on B.Cu, net /MEMORY /SD_VDD
- added copper zone on F.Cu, net /MEMORY /SD_VDD
- added copper zone on F.Cu, net GND
- added copper zone on B.Cu, net SDRAM_3V3
- added copper zone on F.Cu, net SDRAM_3V3
- added copper zone on B.Cu, net VBUS
