File: DESIGN FILES/supplies_pmic.kicad_sch (KiCad schematic)
At the start: 29 parts

Commit message: schematic changes
Parts:
- removed C?: ~, symbol MIMXRT1064 MCU Module:CL05A105KA5NQNC
- removed U?: ~, symbol MIMXRT1064 MCU Module:UM803RS
- added C301: 1u, symbol MIMXRT1064 MCU Module:CL05A105KA5NQNC
- added U302: UM803RS, symbol MIMXRT1064 MCU Module:UM803RS
- C302, C310: renamed from C?; value ~ -> 1u
- C303, C308: renamed from C?; value ~ -> 22u
- C304, C305, C307: renamed from C?; value ~ -> 100n
- C306, C309, C312: renamed from C?; value ~ -> 10u
- C311: renamed from C?; value ~ -> 10n
- D301, D302: renamed from D?; value ~ -> RB521S30_R1_00001
- L301: renamed from L?; value ~ -> 10n
- L302, L303: renamed from L?; value ~ -> 2.2u
- R301: renamed from R?; value ~ -> 10k
- R302, R306: renamed from R?; value ~ -> 100k
- R303: renamed from R?; value ~ -> 22k
- R304: renamed from R?; value ~ -> 2.2k
- R305: renamed from R?; value ~ -> 200k
- U301: renamed from U?; value ~ -> UM805RE
- VR301, VR302: renamed from VR?; value ~ -> TLV62569DBV
- VR303: renamed from VR?; value ~ -> TPS79333DBVR
- gave numbers to parts that had none: 1
Connections:
- net +3V3: now also U302.3 (VCC)
- net GND: now also C301.2, U302.1 (GND)
- net POR_B: now also U302.2 (~{RESET})
- net VBUS: now also C301.1
Other:
- note added: "DISABLE 3V3 OUT LDO THROUGHT MANUAL RESET (POR Button & Watchdog) OR PMIC ON LOW STATE"
- note added: "Input filtering & supplies"
- note added: "SNVS LDO : 5V > 3V3"
- note added: "V(out) = 0.6*(1+100k/22k) =3.327V"
- note added: "V(out) = 0.6*(1+200k/100k) =1.8V"
- note added: "Voltage monitor & reset circuit"
- note removed: "DISABLE 3V3 LDO THROUGHT MANUAL RESET OR PMIC LOW STATE"
- note removed: "Input Filtering & Digital Supplies"
- note removed: "SNVS LDO"
- note removed: "Supervisory circuit"
- note removed: "V(out) = 0.6*(1+100k/22k)=3.327V"
- note removed: "V(out) = 0.6*(1+200k/100k)=1.8V"
- moved on the sheet: C302, C303, C304, C305, C306, C307, C308, C309, C310, C311, C312, D301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

Commit message: schematic changes
Parts:
- C301, C302, C310: footprint (none) -> MIMXRT1064 MCU Module:0402_CL05A105KA5NQNC
- C303, C308: footprint (none) -> MIMXRT1064 MCU Module:0603_CL10A226MQ8NRNC
- C304, C305, C307: footprint (none) -> MIMXRT1064 MCU Module:0402_CL05B104KB54PNC
- C306, C309: footprint (none) -> MIMXRT1064 MCU Module:0603_CL10A106KP8NNNC
- C311, C312, L301: footprint (none) -> MIMXRT1064 MCU Module:0402_CL05B103KB5NNNC
- D301, D302: footprint (none) -> MIMXRT1064 MCU Module:RB521S30_R1_00001
- D303: footprint (none) -> MIMXRT1064 MCU Module:19-218_BHC-ZL1M2QY_3T
- L302, L303: footprint (none) -> MIMXRT1064 MCU Module:CD32YP0302-2R2M_SMD3.5x3x2.1mm
- R301: footprint (none) -> MIMXRT1064 MCU Module:0402WGF1002TCE
- R302, R306: footprint (none) -> MIMXRT1064 MCU Module:0402WGF1003TCE
- R303: footprint (none) -> MIMXRT1064 MCU Module:0402WGF2202TCE
- R304: footprint (none) -> MIMXRT1064 MCU Module:0402WGF2201TCE
- R305: footprint (none) -> MIMXRT1064 MCU Module:0402WGF2003TCE
- U301: footprint (none) -> MIMXRT1064 MCU Module:UM805RE
- U302: footprint (none) -> MIMXRT1064 MCU Module:UM803RS
- VR301, VR302: footprint (none) -> MIMXRT1064 MCU Module:TLV62569DBVR
- VR303: footprint (none) -> MIMXRT1064 MCU Module:TPS79333DBVR_SOT-23-5
Changed lines of the file:
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@@
     (property "Reference" "L302" (id 0) (at 127 68.58 0))
     (property "Value" "2.2u" (id 1) (at 127 71.12 0))
-    (property "Footprint" "" (id 2) (at 127 73.66 90)
+    (property "Footprint" "MIMXRT1064 MCU Module:CD32YP0302-2R2M_SMD3.5x3x2.1mm" (id 2) (at 127 73.66 90)
       (effects (font (size 1.27 1.27)) hide)
     )
@@
     (property "Reference" "U301" (id 0) (at 102.87 166.37 0))
     (property "Value" "UM805RE" (id 1) (at 113.03 166.37 0))
-    (property "Footprint" "" (id 2) (at 88.9 173.99 0)
+    (property "Footprint" "MIMXRT1064 MCU Module:UM805RE" (id 2) (at 88.9 173.99 0)
       (effects (font (size 1.27 1.27)) hide)
     )
@@
       (effects (font (size 1.27 1.27)) (justify left))
     )
-    (property "Footprint" "" (id 2) (at 33.9852 86.36 0)
+    (property "Footprint" "MIMXRT1064 MCU Module:0402_CL05A105KA5NQNC" (id 2) (at 33.9852 86.36 0)
       (effects (font (size 1.27 1.27)) hide)
     )
@@
       (effects (font (size 1.27 1.27)) (justify left))
     )
-    (property "Footprint" "" (id 2) (at 167.132 82.55 90)
+    (property "Footprint" "MIMXRT1064 MCU Module:0402WGF2201TCE" (id 2) (at 167.132 82.55 90)
       (effects (font (size 1.27 1.27)) hide)
     )
@@
     (property "Reference" "D302" (id 0) (at 81.28 181.61 0))
     (property "Value" "RB521S30_R1_00001" (id 1) (at 77.47 187.96 0))
-    (property "Footprint" "" (id 2) (at 81.28 179.705 0)
+    (property "Footprint" "MIMXRT1064 MCU Module:RB521S30_R1_00001" (id 2) (at 81.28 179.705 0)
       (effects (font (size 1.27 1.27)) hide)
     )
@@
       (effects (font (size 1.27 1.27)) (justify left))
     )
-    (property "Footprint" "" (id 2) (at 340.0552 90.17 0)
+    (property "Footprint" "MIMXRT1064 MCU Module:0402_CL05B103KB5NNNC" (id 2) (at 340.0552 90.17 0)
       (effects (font (size 1.27 1.27)) hide)
     )
@@
       (effects (font (size 1.27 1.27)) (justify left))
     )
-    (property "Footprint" "" (id 2) (at 61.9252 86.36 0)
+    (property "Footprint" "MIMXRT1064 MCU Module:0402_CL05A105KA5NQNC" (id 2) (at 61.9252 86.36 0)
       (effects (font (size 1.27 1.27)) hide)
     )
@@
       (effects (font (size 1.27 1.27)) (justify left))
     )
-    (property "Footprint" "" (id 2) (at 293.0652 88.9 0)
+    (property "Footprint" "MIMXRT1064 MCU Module:0402_CL05A105KA5NQNC" (id 2) (at 293.0652 88.9 0)
       (effects (font (size 1.27 1.27)) hide)
     )
@@
       (effects (font (size 1.27 1.27)) (justify left))
     )
-    (property "Footprint" "" (id 2) (at 191.4652 86.36 0)
+    (property "Footprint" "MIMXRT1064 MCU Module:0603_CL10A226MQ8NRNC" (id 2) (at 191.4652 86.36 0)
       (effects (font (size 1.27 1.27)) hide)
     )
@@
       (effects (font (size 1.27 1.27)) (justify left))
     )
-    (property "Footprint" "" (id 2) (at 239.7252 82.55 0)
+    (property "Footprint" "MIMXRT1064 MCU Module:0603_CL10A106KP8NNNC" (id 2) (at 239.7252 82.55 0)
       (effects (font (size 1.27 1.27)) hide)
     )
@@
       (effects (font (size 1.27 1.27)) (justify left))
     )
-    (property "Footprint" "" (id 2) (at 249.682 82.55 90)
+    (property "Footprint" "MIMXRT1064 MCU Module:0402WGF2003TCE" (id 2) (at 249.682 82.55 90)
       (effects (font (size 1.27 1.27)) hide)
     )
@@
     (property "Reference" "L303" (id 0) (at 232.41 68.58 0))
     (property "Value" "2.2u" (id 1) (at 232.41 71.12 0))
-    (property "Footprint" "" (id 2) (at 232.41 73.66 90)
+    (property "Footprint" "MIMXRT1064 MCU Module:CD32YP0302-2R2M_SMD3.5x3x2.1mm" (id 2) (at 232.41 73.66 90)
       (effects (font (size 1.27 1.27)) hide)
     )
@@
   (symbol (lib_id "MIMXRT1064 MCU Module:CL05B104KB54PNC") (at 114.3 160.02 90) (unit 1)
     (in_bom yes) (on_board yes)
-    (property "Reference" "C305" (id 0) (at 118.11 156.21 90))
+    (property "Reference" "C305" (id 0) (at 119.38 156.21 90))
     (property "Value" "100n" (id 1) (at 119.38 158.75 90))
-    (property "Footprint" "" (id 2) (at 118.11 159.0548 0)
+    (property "Footprint" "MIMXRT1064 MCU Module:0402_CL05B104KB54PNC" (id 2) (at 118.11 159.0548 0)
       (effects (font (size 1.27 1.27)) hide)
     )
@@
     (property "Reference" "VR303" (id 0) (at 314.96 68.58 0))
     (property "Value" "TPS79333DBVR" (id 1) (at 314.96 71.12 0))
-    (property "Footprint" "" (id 2) (at 334.01 87.63 0)
+    (property "Footprint" "MIMXRT1064 MCU Module:TPS79333DBVR_SOT-23-5" (id 2) (at 334.01 87.63 0)
       (effects (font (size 1.27 1.27) italic) hide)
     )
@@
   (symbol (lib_id "MIMXRT1064 MCU Module:0402WGF2202TCE") (at 156.21 90.17 90) (unit 1)
     (in_bom yes) (on_board yes)
-    (property "Reference" "R303" (id 0) (at 156.21 87.63 90)
+    (property "Reference" "R303" (id 0) (at 158.75 87.63 90)
       (effects (font (size 1.27 1.27)) (justify left))
     )
@@
       (effects (font (size 1.27 1.27)) (justify left))
     )
-    (property "Footprint" "" (id 2) (at 156.21 91.948 90)
+    (property "Footprint" "MIMXRT1064 MCU Module:0402WGF2202TCE" (id 2) (at 156.21 91.948 90)
       (effects (font (size 1.27 1.27)) hide)
     )
@@
     (property "Reference" "D303" (id 0) (at 162.56 69.85 0))
     (property "Value" "~" (id 1) (at 163.83 77.47 0))
-    (property "Footprint" "" (id 2) (at 162.56 73.66 0)
+    (property "Footprint" "MIMXRT1064 MCU Module:19-218_BHC-ZL1M2QY_3T" (id 2) (at 162.56 73.66 0)
       (effects (font (size 1.27 1.27)) hide)
     )
@@
     (property "Reference" "VR301" (id 0) (at 100.33 66.04 0))
     (property "Value" "TLV62569DBV" (id 1) (at 100.33 68.58 0))
-    (property "Footprint" "" (id 2) (at 101.6 82.55 0)
+    (property "Footprint" "MIMXRT1064 MCU Module:TLV62569DBVR" (id 2) (at 101.6 82.55 0)
       (effects (font (size 1.27 1.27) italic) (justify left) hide)
     )
@@
       (effects (font (size 1.27 1.27)) (justify left))
     )
-    (property "Footprint" "" (id 2) (at 120.142 186.69 90)
+    (property "Footprint" "MIMXRT1064 MCU Module:0402WGF1002TCE" (id 2) (at 120.142 186.69 90)
       (effects (font (size 1.27 1.27)) hide)
     )
@@
     (property "Reference" "VR302" (id 0) (at 205.74 66.04 0))
     (property "Value" "TLV62569DBV" (id 1) (at 205.74 68.58 0))
-    (property "Footprint" "" (id 2) (at 207.01 82.55 0)
+    (property "Footprint" "MIMXRT1064 MCU Module:TLV62569DBVR" (id 2) (at 207.01 82.55 0)
       (effects (font (size 1.27 1.27) italic) (justify left) hide)
     )
@@
       (effects (font (size 1.27 1.27)) (justify left))
     )
-    (property "Footprint" "" (id 2) (at 94.9452 185.42 0)
+    (property "Footprint" "MIMXRT1064 MCU Module:0402_CL05B104KB54PNC" (id 2) (at 94.9452 185.42 0)
       (effects (font (size 1.27 1.27)) hide)
     )
@@
       (effects (font (size 1.27 1.27)) (justify left))
     )
-    (property "Footprint" "" (id 2) (at 326.0852 90.17 0)
+    (property "Footprint" "MIMXRT1064 MCU Module:0402_CL05B103KB5NNNC" (id 2) (at 326.0852 90.17 0)
       (effects (font (size 1.27 1.27)) hide)
     )
@@
     (property "Reference" "D301" (id 0) (at 81.28 162.56 0))
     (property "Value" "RB521S30_R1_00001" (id 1) (at 77.47 168.91 0))
-    (property "Footprint" "" (id 2) (at 81.28 160.655 0)
+    (property "Footprint" "MIMXRT1064 MCU Module:RB521S30_R1_00001" (id 2) (at 81.28 160.655 0)
       (effects (font (size 1.27 1.27)) hide)
     )
@@
       (effects (font (size 1.27 1.27)) (justify left))
     )
-    (property "Footprint" "" (id 2) (at 186.3852 179.07 0)
+    (property "Footprint" "MIMXRT1064 MCU Module:0402_CL05B104KB54PNC" (id 2) (at 186.3852 179.07 0)
       (effects (font (size 1.27 1.27)) hide)
     )
@@
       (effects (font (size 1.27 1.27)) (justify left))
     )
-    (property "Footprint" "" (id 2) (at 135.5852 82.55 0)
+    (property "Footprint" "MIMXRT1064 MCU Module:0603_CL10A106KP8NNNC" (id 2) (at 135.5852 82.55 0)
       (effects (font (size 1.27 1.27)) hide)
     )
@@
       (effects (font (size 1.27 1.27)) (justify left))
     )
-    (property "Footprint" "" (id 2) (at 143.002 82.55 90)
+    (property "Footprint" "MIMXRT1064 MCU Module:0402WGF1003TCE" (id 2) (at 143.002 82.55 90)
       (effects (font (size 1.27 1.27)) hide)
     )
@@
     (property "Reference" "L301" (id 0) (at 52.07 68.58 90))
     (property "Value" "10n" (id 1) (at 52.07 71.12 90))
-    (property "Footprint" "" (id 2) (at 52.07 73.66 0)
+    (property "Footprint" "MIMXRT1064 MCU Module:0402_CL05B103KB5NNNC" (id 2) (at 52.07 73.66 0)
       (effects (font (size 1.27 1.27)) hide)
     )
@@
       (effects (font (size 1.27 1.27)) (justify right))
     )
-    (property "Footprint" "" (id 2) (at 190.5 177.8 0)
+    (property "Footprint" "MIMXRT1064 MCU Module:UM803RS" (id 2) (at 190.5 177.8 0)
       (effects (font (size 1.27 1.27)) hide)
     )
@@
   (symbol (lib_id "MIMXRT1064 MCU Module:0402WGF1003TCE") (at 260.35 90.17 90) (unit 1)
     (in_bom yes) (on_board yes)
-    (property "Reference" "R306" (id 0) (at 261.62 87.63 90)
+    (property "Reference" "R306" (id 0) (at 262.89 87.63 90)
       (effects (font (size 1.27 1.27)) (justify left))
     )
@@
       (effects (font (size 1.27 1.27)) (justify left))
     )
-    (property "Footprint" "" (id 2) (at 260.35 91.948 90)
+    (property "Footprint" "MIMXRT1064 MCU Module:0402WGF1003TCE" (id 2) (at 260.35 91.948 90)
       (effects (font (size 1.27 1.27)) hide)
     )
@@
       (effects (font (size 1.27 1.27)) (justify left))
     )
-    (property "Footprint" "" (id 2) (at 77.1652 86.36 0)
-      (effects (font (size 1.27 1.27)) hide)
-    )
+    (property "Footprint" "MIMXRT1064 MCU Module:0603_CL10A226MQ8NRNC" (id 2) (at 77.1652 86.36 0)
+      (effects (font (size 1.27 1.27)) hide)
+    )

Commit message: schematic changes
Changed lines of the file:
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@@
   )
   (polyline (pts (xy 241.3 207.01) (xy 25.4 207.01))
-    (stroke (width 1) (type default) (color 0 0 0 0))
+    (stroke (width 0.5) (type default) (color 0 0 0 0))
   )
   (wire (pts (xy 107.95 76.2) (xy 120.65 76.2))
@@
   )
   (polyline (pts (xy 25.4 207.01) (xy 25.4 139.7))
-    (stroke (width 1) (type default) (color 0 0 0 0))
+    (stroke (width 0.5) (type default) (color 0 0 0 0))
   )
   (wire (pts (xy 292.1 81.28) (xy 292.1 76.2))
@@
   )
   (polyline (pts (xy 25.4 50.8) (xy 361.95 50.8))
-    (stroke (width 1) (type default) (color 0 0 0 0))
+    (stroke (width 0.5) (type default) (color 0 0 0 0))
   )
   (wire (pts (xy 256.54 90.17) (xy 251.46 90.17))
@@
   )
   (polyline (pts (xy 25.4 50.8) (xy 25.4 114.3))
-    (stroke (width 1) (type default) (color 0 0 0 0))
+    (stroke (width 0.5) (type default) (color 0 0 0 0))
   )
   (wire (pts (xy 60.96 78.74) (xy 60.96 73.66))
@@
   )
   (polyline (pts (xy 361.95 50.8) (xy 361.95 114.3))
-    (stroke (width 1) (type default) (color 0 0 0 0))
+    (stroke (width 0.5) (type default) (color 0 0 0 0))
   )
   (wire (pts (xy 160.02 90.17) (xy 168.91 90.17))
@@
   )
   (polyline (pts (xy 25.4 114.3) (xy 361.95 114.3))
-    (stroke (width 1) (type default) (color 0 0 0 0))
+    (stroke (width 0.5) (type default) (color 0 0 0 0))
   )
   (wire (pts (xy 96.52 175.26) (xy 93.98 175.26))
@@
   )
   (polyline (pts (xy 241.3 139.7) (xy 241.3 207.01))
-    (stroke (width 1) (type default) (color 0 0 0 0))
+    (stroke (width 0.5) (type default) (color 0 0 0 0))
   )
   (wire (pts (xy 185.42 190.5) (xy 201.93 190.5))
@@
   )
   (polyline (pts (xy 25.4 139.7) (xy 241.3 139.7))
-    (stroke (width 1) (type default) (color 0 0 0 0))
+    (stroke (width 0.5) (type default) (color 0 0 0 0))
   )
   (wire (pts (xy 121.92 175.26) (xy 139.7 175.26))

Commit message: schematic changes
Parts:
- removed C301, C302, C310: 1u, MIMXRT1064 MCU Module:0402_CL05A105KA5NQNC, symbol MIMXRT1064 MCU Module:CL05A105KA5NQNC
- removed C303, C308: 22u, MIMXRT1064 MCU Module:0603_CL10A226MQ8NRNC, symbol MIMXRT1064 MCU Module:CL10A226MQ8NRNC
- removed C304, C305, C307: 100n, MIMXRT1064 MCU Module:0402_CL05B104KB54PNC, symbol MIMXRT1064 MCU Module:CL05B104KB54PNC
- removed C306, C309: 10u, MIMXRT1064 MCU Module:0603_CL10A106KP8NNNC, symbol MIMXRT1064 MCU Module:CL10A106KP8NNNC
- removed C311: 10n, MIMXRT1064 MCU Module:0402_CL05B103KB5NNNC, symbol MIMXRT1064 MCU Module:CL05B104KB54PNC
- removed C312: 10u, MIMXRT1064 MCU Module:0402_CL05B103KB5NNNC, symbol MIMXRT1064 MCU Module:CL10A106KP8NNNC
- removed D301, D302: RB521S30_R1_00001, MIMXRT1064 MCU Module:RB521S30_R1_00001, symbol MIMXRT1064 MCU Module:RB521S30_R1_00001
- removed D303: ~, MIMXRT1064 MCU Module:19-218_BHC-ZL1M2QY_3T, symbol MIMXRT1064 MCU Module:19-218_BHC-ZL1M2QY_3T
- removed L301: 10n, MIMXRT1064 MCU Module:0402_CL05B103KB5NNNC, symbol MIMXRT1064 MCU Module:MLG1005S10NHT000
- removed L302, L303: 2.2u, MIMXRT1064 MCU Module:CD32YP0302-2R2M_SMD3.5x3x2.1mm, symbol MIMXRT1064 MCU Module:CD32YP0302-2R2M
- removed R301: 10k, MIMXRT1064 MCU Module:0402WGF1002TCE, symbol MIMXRT1064 MCU Module:0402WGF1002TCE
- removed R302, R306: 100k, MIMXRT1064 MCU Module:0402WGF1003TCE, symbol MIMXRT1064 MCU Module:0402WGF1003TCE
- removed R303: 22k, MIMXRT1064 MCU Module:0402WGF2202TCE, symbol MIMXRT1064 MCU Module:0402WGF2202TCE
- removed R304: 2.2k, MIMXRT1064 MCU Module:0402WGF2201TCE, symbol MIMXRT1064 MCU Module:0402WGF2201TCE
- removed R305: 200k, MIMXRT1064 MCU Module:0402WGF2003TCE, symbol MIMXRT1064 MCU Module:0402WGF2003TCE
- removed U301: UM805RE, MIMXRT1064 MCU Module:UM805RE, symbol MIMXRT1064 MCU Module:UM805RE
- removed U302: UM803RS, MIMXRT1064 MCU Module:UM803RS, symbol MIMXRT1064 MCU Module:UM803RS
- removed VR301, VR302: TLV62569DBV, MIMXRT1064 MCU Module:TLV62569DBVR, symbol MIMXRT1064 MCU Module:TLV62569DBV
- removed VR303: TPS79333DBVR, MIMXRT1064 MCU Module:TPS79333DBVR_SOT-23-5, symbol MIMXRT1064 MCU Module:TPS79333DBVR
Other:
- note added: "--> +3V3 --> +3V3 SNVS --> +3V3 SD --> +1V8 --> MANUAL & WATCHDOG RESET --> BELOW THRESHOLD VOLTAGE RESET"
- note added: "SUPPLIES & PMIC ON CARRIER BOARDS"
- note removed: "DCDC : 3V3 > 1V8"
- note removed: "DCDC : 5V > 3V3"
- note removed: "DCR = 0R22"
- note removed: "DISABLE 3V3 OUT LDO THROUGHT MANUAL RESET (POR Button & Watchdog) OR PMIC ON LOW STATE"
- note removed: "I(DC) = 500mA"
- note removed: "Input filtering & supplies"
- note removed: "LP Fc = 1.6MHz"
- note removed: "LP Fc = 34KHz"
- note removed: "RST : Open-drain NMOS output (sinks current only)"
- note removed: "SNVS LDO : 5V > 3V3"
- note removed: "TRIGGER MCU POWER ON RESET WHEN VCC FALL BELOW THRESHOLD (2.63V)"
- note removed: "V(out) = 0.6*(1+100k/22k) =3.327V"
- note removed: "V(out) = 0.6*(1+200k/100k) =1.8V"
- note removed: "VBUS comes from USB Type C connector (carrier board)"
- note removed: "Voltage monitor & reset circuit"

Commit message: changes and adding schematic pdf
Other:
- note removed: "--> +3V3 --> +3V3 SNVS --> +3V3 SD --> +1V8 --> MANUAL & WATCHDOG RESET --> BELOW THRESHOLD VOLTAGE RESET"
- note removed: "3 : SUPPLIES & PMIC"
- company: Soundsom -> Joël Ucedo
- title: MCU Power & Crystals -> MIMXRT1064 MCU Module
Changed lines of the file:
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@@
   (paper "A3")
   (title_block
-    (title "MCU Power & Crystals")
-    (date "2023-05-12")
+    (title "MIMXRT1064 MCU Module")
+    (date "2023-05-23")
     (rev "0")
-    (company "Soundsom")
+    (company "Joël Ucedo")
   )
-  (text "--> +3V3\n--> +3V3 SNVS\n--> +3V3 SD\n--> +1V8\n\n--> MANUAL & WATCHDOG RESET\n--> BELOW THRESHOLD VOLTAGE RESET\n\n"
-    (at 73.66 247.65 0)
+  (text "SUPPLIES & PMIC ON CARRIER BOARDS" (at 60.96 147.32 0)
     (effects (font (size 10 10) (thickness 2) bold italic) (justify left bottom))
   )
-  (text "SUPPLIES & PMIC ON CARRIER BOARDS" (at 73.66 91.44 0)
-    (effects (font (size 10 10) (thickness 2) bold italic) (justify left bottom))
-  )
-  (text "3 : SUPPLIES & PMIC" (at 25.4 26.67 0)
-    (effects (font (size 5 5) (thickness 1) bold italic) (justify left bottom))
-  )
 )

Commit message: updates
Other:
- note added: "SUPPLIES & PMIC ON CARRIER BOARD"
- note removed: "SUPPLIES & PMIC ON CARRIER BOARDS"
Changed lines of the file:
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@@
     (company "Joël Ucedo")
   )
-  (text "SUPPLIES & PMIC ON CARRIER BOARDS" (at 60.96 147.32 0)
+  (text "SUPPLIES & PMIC ON CARRIER BOARD" (at 60.96 147.32 0)
     (effects (font (size 10 10) (thickness 2) bold italic) (justify left bottom))
   )

Commit message: updates
Parts:
- added C?: 100n, symbol MY CAPACITOR LIBRARY:CC0603KRX7R9BB104
- added C?: 1u, MIMXRT1064 Carrier:0402_CL05A105KA5NQNC, symbol MIMXRT1064 Carrier:CL05A105KA5NQNC
- added C? (x3): 100n, MIMXRT1064 Carrier:0402_CL05B104KB54PNC, symbol MIMXRT1064 Carrier:CL05B104KB54PNC
- added C?: 10n, MIMXRT1064 Carrier:0402_CL05B103KB5NNNC, symbol MIMXRT1064 Carrier:CL05B103KB5NNNC
- added C?: 10u, symbol MY CAPACITOR LIBRARY:CL10A106KP8NNNC
- added C? (x2): 22u, MIMXRT1064 Carrier:0603_CL10A226MQ8NRNC, symbol MIMXRT1064 Carrier:CL10A226MQ8NRNC
- added C?: 1uF, symbol MY CAPACITOR LIBRARY:CL10A105KB8NNNC
- added C? (x3): 10u, MIMXRT1064 Carrier:0603_CL10A106KP8NNNC, symbol MIMXRT1064 Carrier:CL10A106KP8NNNC
- added D? (x2): RB521S30_R1_00001, MIMXRT1064 Carrier:RB521S30_R1_00001, symbol MIMXRT1064 Carrier:RB521S30_R1_00001
- added D?: LED, symbol MY LED LIBRARY:LED
- added L? (x2): 2.2u, MIMXRT1064 Carrier:CD32YP0302-2R2M_SMD3.5x3x2.1mm, symbol MIMXRT1064 Carrier:CD32YP0302-2R2M
- added R?: 10k, MIMXRT1064 Carrier:0402WGF1002TCE, symbol MIMXRT1064 Carrier:0402WGF1002TCE
- added R?: 22k, MIMXRT1064 Carrier:0402WGF2202TCE, symbol MIMXRT1064 Carrier:0402WGF2202TCE
- added R?: 200k, MIMXRT1064 Carrier:0402WGF2003TCE, symbol MIMXRT1064 Carrier:0402WGF2003TCE
- added R? (x2): 100k, MIMXRT1064 Carrier:0402WGF1003TCE, symbol MIMXRT1064 Carrier:0402WGF1003TCE
- added R?: 2.2k, MIMXRT1064 Carrier:0402WGF2201TCE, symbol MIMXRT1064 Carrier:0402WGF2201TCE
- added U?: UM803RS, MIMXRT1064 Carrier:UM803RS, symbol MIMXRT1064 Carrier:UM803RS
- added U?: UM805RE, MIMXRT1064 Carrier:UM805RE, symbol MIMXRT1064 Carrier:UM805RE
- added VR? (x2): TLV62569DBV, MIMXRT1064 Carrier:TLV62569DBVR, symbol MIMXRT1064 Carrier:TLV62569DBV
- added VR?: TPS79333DBVR, MIMXRT1064 Carrier:TPS79333DBVR_SOT-23-5, symbol MIMXRT1064 Carrier:TPS79333DBVR
- added VR?: TPS79333DBVR, Package_TO_SOT_SMD:SOT-23-5, symbol MY REGULATOR LIBRARY:TPS79333DBVR
Connections:
- new net: C?.1, VR?.4 (NR)
- new net +1V8: C?.1, L?.2, R?.1
- new net +3.3VA: C?.1, VR?.5 (OUT)
- new net +3V3: C?.1, C?.1, C?.1, D?.2 (A), L?.2, R?.1, U?.3 (VCC), VR?.1 (EN), VR?.4 (VIN)
- new net +5V: C?.1, C?.1, C?.1, VR?.1 (IN), VR?.1 (IN), VR?.3 (EN), VR?.3 (EN), VR?.4 (VIN)
- new net BUCK1_FB: R?.1, R?.2, VR?.5 (FB)
- new net BUCK1_SW: L?.1, VR?.3 (SW)
- new net BUCK2_FB: R?.2, R?.2, VR?.5 (FB)
- new net BUCK2_SW: L?.1, VR?.3 (SW)
- new net EXT_POR_BUT: D?.1 (K)
- new net GND: C?.2, C?.2, C?.2, C?.2, C?.2, C?.2, C?.2, C?.2, C?.2, C?.2, C?.2, C?.2, C?.2, R?.1, R?.2, R?.2, U?.1 (GND), U?.1 (GND), VR?.2 (GND), VR?.2 (GND), VR?.2 (GND), VR?.2 (GND)
- new net LDO_EN: R?.1, U?.2 (~{RESET}), VR?.1 (EN)
- new net LED_PWR_K: D?.1 (K), R?.1
- new net PMIC_ON_REQ: R?.2
- new net POR_B: U?.2 (~{RESET})
- new net SNVS LDO NR: C?.1, VR?.4 (NR)
- new net UM805RE MR: C?.1, D?.2 (A), D?.2 (A), U?.3 (~{MR})
- new net VDD_SNVS_3V3: C?.1, C?.1, U?.4 (VCC), VR?.5 (OUT)
- new net WATCHDOG_B: D?.1 (K)
Other:
- note added: "+ 3V3 > 1V8 FOR QSPI FLASH"
- note added: "+5V USB > +3V3 FOR ANALOG AUDIO CIRCUIT"
- note added: "+5V USB > 3V3 FOR DIGITAL CIRCUIT"
- note added: "Ajouter un switch de reset"
- note added: "DISABLE 3V3 OUT LDO THROUGHT MANUAL RESET (POR Button & Watchdog) RESET WHEN PMIC ON REQ FALL BELOW THRESHOLD (2.63V)"
- note added: "LP Fc = 34KHz"
- note added: "RST : Open-drain NMOS output (sinks current only)"
- note added: "SNVS LDO : 5V > 3V3"
- note added: "TRIGGER MCU POWER ON RESET WHEN VCC FALL BELOW THRESHOLD (2.63V)"
- note added: "V(out) = 0.6*(1+100k/22k) =3.327V"
- note added: "V(out) = 0.6*(1+200k/100k) =1.8V"
- note added: "Voltage monitor & reset circuit"
- note removed: "SUPPLIES & PMIC ON CARRIER BOARD"
