File: DESIGN FILES/supplies_pmic.kicad_sch (KiCad schematic)
At the start: 30 parts

Commit message: updates
Parts:
- removed C?: 100n, symbol MY CAPACITOR LIBRARY:CC0603KRX7R9BB104
- removed C?: 1u, MIMXRT1064 Carrier:0402_CL05A105KA5NQNC, symbol MIMXRT1064 Carrier:CL05A105KA5NQNC
- removed C? (x3): 100n, MIMXRT1064 Carrier:0402_CL05B104KB54PNC, symbol MIMXRT1064 Carrier:CL05B104KB54PNC
- removed C?: 10n, MIMXRT1064 Carrier:0402_CL05B103KB5NNNC, symbol MIMXRT1064 Carrier:CL05B103KB5NNNC
- removed C?: 10u, symbol MY CAPACITOR LIBRARY:CL10A106KP8NNNC
- removed C? (x2): 22u, MIMXRT1064 Carrier:0603_CL10A226MQ8NRNC, symbol MIMXRT1064 Carrier:CL10A226MQ8NRNC
- removed C?: 1uF, symbol MY CAPACITOR LIBRARY:CL10A105KB8NNNC
- removed C? (x3): 10u, MIMXRT1064 Carrier:0603_CL10A106KP8NNNC, symbol MIMXRT1064 Carrier:CL10A106KP8NNNC
- removed D? (x2): RB521S30_R1_00001, MIMXRT1064 Carrier:RB521S30_R1_00001, symbol MIMXRT1064 Carrier:RB521S30_R1_00001
- removed D?: LED, symbol MY LED LIBRARY:LED
- removed L? (x2): 2.2u, MIMXRT1064 Carrier:CD32YP0302-2R2M_SMD3.5x3x2.1mm, symbol MIMXRT1064 Carrier:CD32YP0302-2R2M
- removed R?: 10k, MIMXRT1064 Carrier:0402WGF1002TCE, symbol MIMXRT1064 Carrier:0402WGF1002TCE
- removed R?: 22k, MIMXRT1064 Carrier:0402WGF2202TCE, symbol MIMXRT1064 Carrier:0402WGF2202TCE
- removed R?: 200k, MIMXRT1064 Carrier:0402WGF2003TCE, symbol MIMXRT1064 Carrier:0402WGF2003TCE
- removed R? (x2): 100k, MIMXRT1064 Carrier:0402WGF1003TCE, symbol MIMXRT1064 Carrier:0402WGF1003TCE
- removed R?: 2.2k, MIMXRT1064 Carrier:0402WGF2201TCE, symbol MIMXRT1064 Carrier:0402WGF2201TCE
- removed U?: UM803RS, MIMXRT1064 Carrier:UM803RS, symbol MIMXRT1064 Carrier:UM803RS
- removed U?: UM805RE, MIMXRT1064 Carrier:UM805RE, symbol MIMXRT1064 Carrier:UM805RE
- removed VR? (x2): TLV62569DBV, MIMXRT1064 Carrier:TLV62569DBVR, symbol MIMXRT1064 Carrier:TLV62569DBV
- removed VR?: TPS79333DBVR, MIMXRT1064 Carrier:TPS79333DBVR_SOT-23-5, symbol MIMXRT1064 Carrier:TPS79333DBVR
- added C301, C302: 22u, MY CAPACITOR LIBRARY:0603_CL10A226MQ8NRNC, symbol MY CAPACITOR LIBRARY:CL10A226MQ8NRNC
- added C303, C304, C310: 10u, MY CAPACITOR LIBRARY:0603_CL10A106KP8NNNC, symbol MY CAPACITOR LIBRARY:CL10A106KP8NNNC
- added C305, C306: 1u, MY CAPACITOR LIBRARY:0402_CL05A105KA5NQNC, symbol MY CAPACITOR LIBRARY:CL05A105KA5NQNC
- added C307: 1n, MY CAPACITOR LIBRARY:CL05B102KB5VPNC, symbol MY CAPACITOR LIBRARY:CL05B102KB5VPNC
- added C308, C309, C311, C312: 100n, MY CAPACITOR LIBRARY:0402_CL05B104KB54PNC, symbol MY CAPACITOR LIBRARY:CL05B104KB54PNC
- added D301: LED, MY LED LIBRARY:LED_D3.0mm, symbol MY LED LIBRARY:LED
- added D302, D303: RB521S30_R1_00001, MY DIODE LIBRARY:RB521S30_R1_00001, symbol MY DIODE LIBRARY:RB521S30_R1_00001
- added L301, L302: 2.2u, MY INDUCTOR LIBRARY:CD32YP0302-2R2M, symbol MY INDUCTOR LIBRARY:CD32YP0302-2R2M
- added R301: 200k, MY RESISTOR LIBRARY:0402WGF2003TCE, symbol MY RESISTOR LIBRARY:0402WGF2003TCE
- added R302, R303: 100k, MY RESISTOR LIBRARY:0402WGF1003TCE, symbol MY RESISTOR LIBRARY:0402WGF1003TCE
- added R304: 22k, MY RESISTOR LIBRARY:0402WGF2202TCE, symbol MY RESISTOR LIBRARY:0402WGF2202TCE
- added R305: 2.2k, MY RESISTOR LIBRARY:0402WGF2201TCE, symbol MY RESISTOR LIBRARY:0402WGF2201TCE
- added R306: 100R, MY RESISTOR LIBRARY:0805W8F1000T5E, symbol MY RESISTOR LIBRARY:0805W8F1000T5E
- added R307: 1M, MY RESISTOR LIBRARY:0402WGF1004TCE, symbol MY RESISTOR LIBRARY:0402WGF1004TCE
- added R308: 10k, MY RESISTOR LIBRARY:0402WGF1002TCE, symbol MY RESISTOR LIBRARY:0402WGF1002TCE
- added R309: 1.5k, MY RESISTOR LIBRARY:CQ02WGF1501TCE, symbol MY RESISTOR LIBRARY:CQ02WGF1501TCE
- added U301: UM805RE, MY PMIC LIBRARY:UM805RE, symbol MY PMIC LIBRARY:UM805RE
- added U302: UM803RS, MY PMIC LIBRARY:UM803RS, symbol MY PMIC LIBRARY:UM803RS
- added VR301, VR302: TLV62569DBV, MY REGULATOR LIBRARY:TLV62569DBVR, symbol MY REGULATOR LIBRARY:TLV62569DBV
- VR303: renamed from VR?; footprint Package_TO_SOT_SMD:SOT-23-5 -> MY REGULATOR LIBRARY:TPS79333DBVR_SOT-23-5
Connections:
- net +1V8: now also C303.1, L301.2, R301.1
- net +3.3VA: now also C310.1
- net +3V3: now also C301.1, C304.1, C311.1, D301.2 (A), L302.2, R303.1, R309.1, U301.4 (VCC), VR301.1 (EN), VR301.4 (VIN)
- net +5V: now also C302.1, C305.1, VR302.4 (VIN)
- net BUCK1_FB: now also R303.2, R304.1, VR302.5 (FB)
- net BUCK1_SW: now also L302.1, VR302.3 (SW)
- net BUCK2_FB: now also R301.2, R302.1, VR301.5 (FB)
- net BUCK2_SW: now also L301.1, VR301.3 (SW)
- net EXT_POR_BUT: now also R306.1
- net GND: now also C301.2, C302.2, C303.2, C304.2, C305.2, C307.2, C308.2, C309.2, C310.2, C311.2, C312.1, R302.2, R304.2, R305.2, R307.2, U301.1 (GND), U302.1 (GND), VR301.2 (GND), VR302.2 (GND)
- net LDO_EN: now also R308.1, U301.2 (~{RESET}), VR302.1 (EN)
- net LED_PWR_K: now also D301.1 (K), R305.1
- net PMIC_ON_REQ: now also R308.2
- net POR_B: now also U302.2 (~{RESET})
- net UM805RE MR: now also C309.1, D302.2 (A), D303.2 (A), U301.3 (~{MR})
- net WATCHDOG_B: now also C306.1
- net at VR303.4 (NR): now also C308.1
- new net: C306.2, D303.1 (K), R307.1
- new net: C312.2, R309.2, U302.3 (VCC)
- new net: C307.1, D302.1 (K), R306.2
Other:
- note removed: "SNVS LDO : 5V > 3V3"
