File: DESIGN FILES/supplies_pmic.kicad_sch (KiCad schematic)
At the start: 31 parts, among them U301 UM805RE, U302 UM803RS

Commit message: updates
Parts:
- added C313: 100n, MY CAPACITOR LIBRARY:0402_CL05B104KB54PNC, symbol MY CAPACITOR LIBRARY:CL05B104KB54PNC
- added SW301: TS-1187A-B-A-B, MY SWITCH LIBRARY:TS-1187A-B-A-B_smd, symbol MY SWITCH LIBRARY:TS-1187A-B-A-B
Connections:
- net GND: now also C313.1, SW301.A, SW301.B
- net LDO_NR: now reaches C308.1, VR303.4 (NR)
- net EXT_POR_BUT renamed RESET_SWITCH
- net RESET_SWITCH: now also C313.2, SW301.C, SW301.D
Other:
- note added: "3 : SUPPLIES & PMIC"
- note added: "DISABLE 3V3 OUT LDO THROUGHT MANUAL RESET (POR Button & Watchdog)"
- note added: "RESET SWITCH"
- note removed: "Ajouter un switch de reset"
- note removed: "DISABLE 3V3 OUT LDO THROUGHT MANUAL RESET (POR Button & Watchdog) RESET WHEN PMIC ON REQ FALL BELOW THRESHOLD (2.63V)"
- moved on the sheet: C301, C302, C303, C304, C305, C306, C307, C308, C309, C310, C311, C312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

Commit message: up
Parts:
- R306: footprint MY RESISTOR LIBRARY:0805W8F1000T5E -> MY RESISTOR LIBRARY:0603WAF1000T5E
Changed lines of the file:
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@@
     (property "Reference" "R306" (id 0) (at 236.22 162.56 90))
     (property "Value" "100R" (id 1) (at 236.22 167.64 90))
-    (property "Footprint" "MY RESISTOR LIBRARY:0805W8F1000T5E" (id 2) (at 236.22 166.878 90)
+    (property "Footprint" "MY RESISTOR LIBRARY:0603WAF1000T5E" (id 2) (at 236.22 166.878 90)
       (effects (font (size 1.27 1.27)) hide)
     )

Commit message: updates
Parts:
- removed C301, C302: 22u, MY CAPACITOR LIBRARY:0603_CL10A226MQ8NRNC, symbol MY CAPACITOR LIBRARY:CL10A226MQ8NRNC
- removed C303, C304, C310: 10u, MY CAPACITOR LIBRARY:0603_CL10A106KP8NNNC, symbol MY CAPACITOR LIBRARY:CL10A106KP8NNNC
- removed C305, C306: 1u, MY CAPACITOR LIBRARY:0402_CL05A105KA5NQNC, symbol MY CAPACITOR LIBRARY:CL05A105KA5NQNC
- removed C307: 1n, MY CAPACITOR LIBRARY:CL05B102KB5VPNC, symbol MY CAPACITOR LIBRARY:CL05B102KB5VPNC
- removed C308, C309, C311, C312, C313: 100n, MY CAPACITOR LIBRARY:0402_CL05B104KB54PNC, symbol MY CAPACITOR LIBRARY:CL05B104KB54PNC
- removed D301: LED, MY LED LIBRARY:LED_D3.0mm, symbol MY LED LIBRARY:LED
- removed D302, D303: RB521S30_R1_00001, MY DIODE LIBRARY:RB521S30_R1_00001, symbol MY DIODE LIBRARY:RB521S30_R1_00001
- removed L301, L302: 2.2u, MY INDUCTOR LIBRARY:CD32YP0302-2R2M, symbol MY INDUCTOR LIBRARY:CD32YP0302-2R2M
- removed R301: 200k, MY RESISTOR LIBRARY:0402WGF2003TCE, symbol MY RESISTOR LIBRARY:0402WGF2003TCE
- removed R302, R303: 100k, MY RESISTOR LIBRARY:0402WGF1003TCE, symbol MY RESISTOR LIBRARY:0402WGF1003TCE
- removed R304: 22k, MY RESISTOR LIBRARY:0402WGF2202TCE, symbol MY RESISTOR LIBRARY:0402WGF2202TCE
- removed R305: 2.2k, MY RESISTOR LIBRARY:0402WGF2201TCE, symbol MY RESISTOR LIBRARY:0402WGF2201TCE
- removed R306: 100R, MY RESISTOR LIBRARY:0603WAF1000T5E, symbol MY RESISTOR LIBRARY:0805W8F1000T5E
- removed R307: 1M, MY RESISTOR LIBRARY:0402WGF1004TCE, symbol MY RESISTOR LIBRARY:0402WGF1004TCE
- removed R308: 10k, MY RESISTOR LIBRARY:0402WGF1002TCE, symbol MY RESISTOR LIBRARY:0402WGF1002TCE
- removed R309: 1.5k, MY RESISTOR LIBRARY:CQ02WGF1501TCE, symbol MY RESISTOR LIBRARY:CQ02WGF1501TCE
- removed SW301: TS-1187A-B-A-B, MY SWITCH LIBRARY:TS-1187A-B-A-B_smd, symbol MY SWITCH LIBRARY:TS-1187A-B-A-B
- removed U301: UM805RE, MY PMIC LIBRARY:UM805RE, symbol MY PMIC LIBRARY:UM805RE
- removed U302: UM803RS, MY PMIC LIBRARY:UM803RS, symbol MY PMIC LIBRARY:UM803RS
- removed VR301, VR302: TLV62569DBV, MY REGULATOR LIBRARY:TLV62569DBVR, symbol MY REGULATOR LIBRARY:TLV62569DBV
- removed VR303: TPS79333DBVR, MY REGULATOR LIBRARY:TPS79333DBVR_SOT-23-5, symbol MY REGULATOR LIBRARY:TPS79333DBVR
Other:
- note added: "ON CARRIER BOARD"
- note added: "[3] SUPPLIES & PMIC"
- note removed: "+ 3V3 > 1V8 FOR QSPI FLASH"
- note removed: "+5V USB > +3V3 FOR ANALOG AUDIO CIRCUIT"
- note removed: "+5V USB > 3V3 FOR DIGITAL CIRCUIT"
- note removed: "3 : SUPPLIES & PMIC"
- note removed: "DISABLE 3V3 OUT LDO THROUGHT MANUAL RESET (POR Button & Watchdog)"
- note removed: "LP Fc = 34KHz"
- note removed: "RESET SWITCH"
- note removed: "RST : Open-drain NMOS output (sinks current only)"
- note removed: "TRIGGER MCU POWER ON RESET WHEN VCC FALL BELOW THRESHOLD (2.63V)"
- note removed: "V(out) = 0.6*(1+100k/22k) =3.327V"
- note removed: "V(out) = 0.6*(1+200k/100k) =1.8V"
- note removed: "Voltage monitor & reset circuit"
