File: DESIGN FILES/midi.kicad_sch (KiCad schematic)
At the start: 14 parts

Commit message: updates
Parts:
- removed C? (x2): 100n, symbol MY CAPACITOR LIBRARY:CC0603KRX7R9BB104
- removed D?: 1N4148W, Diode_SMD:D_SOD-123, symbol MY DIODE LIBRARY:1N4148W
- removed J? (x3): PJ-342B-TX-SMT, PJ-342B-TX-SMT_XKB, symbol MY CONNECTOR LIBRARY:PJ-342B-TX-SMT
- removed R? (x4): 33R, symbol MY RESISTOR LIBRARY:0603WAF330JT5E
- removed R?: 220R, symbol MY RESISTOR LIBRARY:0603WAF2200T5E
- removed R?: 10k, symbol MY RESISTOR LIBRARY:0603WAF1002T5E
- removed U?: 6N137S1(TA), digikey-footprints:DIP-8_W7.62mm, symbol MY OPTO IC LIBRARY:6N137S1(TA)
- removed U?: 74HC04D,653, SOIC127P600X175-14N, symbol MY IC LIBRARY:74HC04D,653
- added C801, C802: 100n, MY CAPACITOR LIBRARY:0402_CL05B104KB54PNC, symbol MY CAPACITOR LIBRARY:CL05B104KB54PNC
- added D801: 1N4148W, MY DIODE LIBRARY:1N4148W_SOD-123, symbol MY DIODE LIBRARY:1N4148W
- added J801, J802, J803: PJ-342B-TX-SMT, MY CONNECTOR LIBRARY:PJ-342B-TX-SMT, symbol MY CONNECTOR LIBRARY:PJ-342B-TX-SMT
- added R801: 220R, MY RESISTOR LIBRARY:0603WAF2200T5E, symbol MY RESISTOR LIBRARY:0603WAF2200T5E
- added R802: 10k, MY RESISTOR LIBRARY:0402WGF1002TCE, symbol MY RESISTOR LIBRARY:0402WGF1002TCE
- added R803, R804, R805, R806: 33R, MY RESISTOR LIBRARY:0805W8F330JT5E, symbol MY RESISTOR LIBRARY:0603WAF330JT5E
- added U801: 6N137S1(TA), MY OPTO IC LIBRARY:6N137S1_TA_SMD-8P, symbol MY OPTO IC LIBRARY:6N137S1(TA)
- added U802: 74HC04D,653, MY IC LIBRARY:74HC04D_653_SOIC-14, symbol MY IC LIBRARY:74HC04D,653
Connections:
- net +3V3: now also C802.1, R802.1, R803.2, R805.2, U802.14 (VCC)
- net +5V: now also C801.1, U801.8 (VCC)
- net GND: now also C801.2, C802.2, J802.2, J803.2, U801.5 (GND), U802.7 (GND)
- net MIDI_IN: now also R802.2, U801.6 (VO), U802.1 (1A)
- net MIDI_IN_RING: now also J801.6, R801.2
- net MIDI_IN_TIP: now also D801.2 (A), J801.3, U801.3 (K)
- net MIDI_OUT: now also U802.13 (6A)
- net OUT: now also R804.2, U802.10 (5Y)
- net THRU: now also R806.2, U802.4 (2Y)
- new net: U802.11 (5A), U802.12 (6Y)
- new net: U802.2 (1Y), U802.3 (2A)
- new net: J803.3, R806.1
- new net: J803.6, R805.1
- new net: D801.1 (K), R801.1, U801.2 (A)
- new net: J802.3, R804.1
- new net: J802.6, R803.1

Commit message: updates
Other:
- note added: "8 : MIDI"
- company: (none) -> Joël Ucedo
- title: (none) -> MIMXRT1064 Audio Board
- moved on the sheet: C801, C802, D801, J801, J802, J803, R801, R802, R803, R804, R805, R806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

Commit message: up
Parts:
- R803, R804, R805, R806: footprint MY RESISTOR LIBRARY:0805W8F330JT5E -> MY RESISTOR LIBRARY:0603WAF330JT5E
Changed lines of the file:
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@@
     (property "Reference" "R805" (id 0) (at 302.26 180.34 90))
     (property "Value" "33R" (id 1) (at 302.26 185.42 90))
-    (property "Footprint" "MY RESISTOR LIBRARY:0805W8F330JT5E" (id 2) (at 302.26 184.658 90)
+    (property "Footprint" "MY RESISTOR LIBRARY:0603WAF330JT5E" (id 2) (at 302.26 184.658 90)
       (effects (font (size 1.27 1.27)) hide)
     )
@@
     (property "Reference" "R804" (id 0) (at 302.26 148.59 90))
     (property "Value" "33R" (id 1) (at 302.26 153.67 90))
-    (property "Footprint" "MY RESISTOR LIBRARY:0805W8F330JT5E" (id 2) (at 302.26 152.908 90)
+    (property "Footprint" "MY RESISTOR LIBRARY:0603WAF330JT5E" (id 2) (at 302.26 152.908 90)
       (effects (font (size 1.27 1.27)) hide)
     )
@@
     (property "Reference" "R803" (id 0) (at 302.26 140.97 90))
     (property "Value" "33R" (id 1) (at 302.26 146.05 90))
-    (property "Footprint" "MY RESISTOR LIBRARY:0805W8F330JT5E" (id 2) (at 302.26 145.288 90)
+    (property "Footprint" "MY RESISTOR LIBRARY:0603WAF330JT5E" (id 2) (at 302.26 145.288 90)
       (effects (font (size 1.27 1.27)) hide)
     )
@@
     (property "Reference" "R806" (id 0) (at 302.26 187.96 90))
     (property "Value" "33R" (id 1) (at 302.26 193.04 90))
-    (property "Footprint" "MY RESISTOR LIBRARY:0805W8F330JT5E" (id 2) (at 302.26 192.278 90)
+    (property "Footprint" "MY RESISTOR LIBRARY:0603WAF330JT5E" (id 2) (at 302.26 192.278 90)
       (effects (font (size 1.27 1.27)) hide)
     )
