File: DESIGN FILES/block_diagram.kicad_sch (KiCad schematic)
At the start: 0 parts

Commit message: work
Other:
- note added: "1 : BLOCK DIAGRAM"
- company: (none) -> Soundsom
Changed lines of the file:
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@@
   (title_block
     (title "Block diagram")
-    (date "2023-05-12")
+    (date "2023-05-19")
     (rev "0")
+    (company "Soundsom")
+  )
+  (text "1 : BLOCK DIAGRAM" (at 204.47 27.94 0)
+    (effects (font (size 5 5) (thickness 1) bold italic) (justify left bottom))
   )
 )

Commit message: schematic edit
Other:
- note added: "2 : BLOCK DIAGRAM"
- note removed: "1 : BLOCK DIAGRAM"
Changed lines of the file:
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@@
 (kicad_sch (version 20211123) (generator eeschema)
-  (paper "A4")
+  (paper "A3")
   (title_block
     (title "Block diagram")
@@
     (company "Soundsom")
   )
-  (text "1 : BLOCK DIAGRAM" (at 204.47 27.94 0)
+  (text "2 : BLOCK DIAGRAM" (at 25.4 26.67 0)
     (effects (font (size 5 5) (thickness 1) bold italic) (justify left bottom))
   )

Commit message: changes and adding schematic pdf
Other:
- company: Soundsom -> Joël Ucedo
- title: Block diagram -> MIMXRT1064 MCU Module
Changed lines of the file:
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@@
   (paper "A3")
   (title_block
-    (title "Block diagram")
-    (date "2023-05-19")
+    (title "MIMXRT1064 MCU Module")
+    (date "2023-05-23")
     (rev "0")
-    (company "Soundsom")
+    (company "Joël Ucedo")
   )
   (text "2 : BLOCK DIAGRAM" (at 25.4 26.67 0)

Commit message: updates
Other:
- title: MIMXRT1064 MCU Module -> MIMXRT1064 Audio Board
Changed lines of the file:
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@@
   (paper "A3")
   (title_block
-    (title "MIMXRT1064 MCU Module")
-    (date "2023-05-23")
+    (title "MIMXRT1064 Audio Board")
+    (date "2023-06-06")
     (rev "0")
     (company "Joël Ucedo")

Commit message: updates
Other:
- note added: "[2] BLOCK DIAGRAM"
- note removed: "2 : BLOCK DIAGRAM"
- title: MIMXRT1064 Audio Board -> MIMXRT1064 MCU Module
Changed lines of the file:
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@@
   (paper "A3")
   (title_block
-    (title "MIMXRT1064 Audio Board")
-    (date "2023-06-06")
+    (title "MIMXRT1064 MCU Module")
+    (date "2023-06-24")
     (rev "0")
     (company "Joël Ucedo")
   )
-  (text "2 : BLOCK DIAGRAM" (at 25.4 26.67 0)
+  (text "[2] BLOCK DIAGRAM" (at 25.4 26.67 0)
     (effects (font (size 5 5) (thickness 1) bold italic) (justify left bottom))
   )
