File: DESIGN FILES/pots_enc_leds.kicad_sch (KiCad schematic)
At the start: 25 parts, among them U901 PEC12R-4025F-S0024

Commit message: updates
Parts:
- removed D901, D902: LED_RGBK, MY LED LIBRARY:WP154A4SUREQBFZGW, symbol MY LED LIBRARY:LED_RGBK
- added D901, D902: WP154A4SUREQBFZGW, MY LED LIBRARY:WP154A4SUREQBFZGW, symbol MY LED LIBRARY:WP154A4SUREQBFZGW
Connections:
- net GND: now also D901.2 (K), D902.2 (K)
- net at R905.2: now also D902.3 (GA)
- net at R901.2: now also D901.1 (RA)
- net at R902.2: now also D901.3 (GA)
- net at R904.2: now also D902.1 (RA)
- net at R906.2: now also D902.4 (BA)
- net at R903.2: now also D901.4 (BA)
Other:
- note added: "9 : POTS & ENCODER & LEDS"
Changed lines of the file:
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@@
+    (effects (font (size 5 5) bold italic) (justify left bottom))
+  )
+  (text "9 : POTS & ENCODER & LEDS" (at 25.4 25.4 0)
     (effects (font (size 5 5) bold italic) (justify left bottom))
   )
@@
     (pin "1")
   )
+  (symbol (lib_id "MY LED LIBRARY:WP154A4SUREQBFZGW") (at 340.36 177.8 0) (mirror y) (unit 1)
+    (in_bom yes) (on_board yes) (fields_autoplaced)
+    (property "Reference" "D902" (id 0) (at 340.36 163.83 0))
+    (property "Value" "WP154A4SUREQBFZGW" (id 1) (at 340.36 166.37 0))
+    (property "Footprint" "MY LED LIBRARY:WP154A4SUREQBFZGW" (id 2) (at 340.36 179.07 0)
+      (effects (font (size 1.27 1.27)) hide)
+    )
+    (property "Datasheet" "~" (id 3) (at 340.36 179.07 0)
+      (effects (font (size 1.27 1.27)) hide)
+    )
+    (pin "1")
+    (pin "2")
+    (pin "3")
+    (pin "4")
+  )
   (symbol (lib_id "MY POTENTIOMETER LIBRARY:RK09D1130C2P") (at 204.47 91.44 0) (unit 1)
     (in_bom yes) (on_board yes) (fields_autoplaced)
@@
     (pin "1")
   )
-  (symbol (lib_id "MY LED LIBRARY:LED_RGBK") (at 340.36 177.8 0) (mirror y) (unit 1)
-    (in_bom yes) (on_board yes) (fields_autoplaced)
-    (property "Reference" "D902" (id 0) (at 340.36 163.83 0))
-    (property "Value" "LED_RGBK" (id 1) (at 340.36 166.37 0))
-    (property "Footprint" "MY LED LIBRARY:WP154A4SUREQBFZGW" (id 2) (at 340.36 179.07 0)
-      (effects (font (size 1.27 1.27)) hide)
-    )
-    (property "Datasheet" "~" (id 3) (at 340.36 179.07 0)
-      (effects (font (size 1.27 1.27)) hide)
-    )
-    (pin "1")
-    (pin "2")
-    (pin "3")
-    (pin "4")
-  )
-  (symbol (lib_id "MY LED LIBRARY:LED_RGBK") (at 340.36 139.7 0) (mirror y) (unit 1)
+  (symbol (lib_id "MY LED LIBRARY:WP154A4SUREQBFZGW") (at 340.36 139.7 0) (mirror y) (unit 1)
     (in_bom yes) (on_board yes) (fields_autoplaced)
     (property "Reference" "D901" (id 0) (at 340.36 125.73 0))
-    (property "Value" "LED_RGBK" (id 1) (at 340.36 128.27 0))
+    (property "Value" "WP154A4SUREQBFZGW" (id 1) (at 340.36 128.27 0))
     (property "Footprint" "MY LED LIBRARY:WP154A4SUREQBFZGW" (id 2) (at 340.36 140.97 0)
       (effects (font (size 1.27 1.27)) hide)

Commit message: updates
Parts:
- removed D901, D902: WP154A4SUREQBFZGW, MY LED LIBRARY:WP154A4SUREQBFZGW, symbol MY LED LIBRARY:WP154A4SUREQBFZGW
- removed R901, R902, R903, R904, R905, R906: 2.2k, MY RESISTOR LIBRARY:0402WGF2201TCE, symbol MY RESISTOR LIBRARY:0603WAF2201T5E
- removed RV902: POT_B1, MY POTENTIOMETER LIBRARY:RK09D1130C2P, symbol MY POTENTIOMETER LIBRARY:RK09D1130C2P
- removed RV903: POT_C1, MY POTENTIOMETER LIBRARY:RK09D1130C2P, symbol MY POTENTIOMETER LIBRARY:RK09D1130C2P
- removed RV904: POT_D1, MY POTENTIOMETER LIBRARY:RK09D1130C2P, symbol MY POTENTIOMETER LIBRARY:RK09D1130C2P
- removed RV906: POT_B2, MY POTENTIOMETER LIBRARY:RK09D1130C2P, symbol MY POTENTIOMETER LIBRARY:RK09D1130C2P
- removed RV907: POT_C2, MY POTENTIOMETER LIBRARY:RK09D1130C2P, symbol MY POTENTIOMETER LIBRARY:RK09D1130C2P
- removed RV908: POT_D2, MY POTENTIOMETER LIBRARY:RK09D1130C2P, symbol MY POTENTIOMETER LIBRARY:RK09D1130C2P
- removed RV910: POT_B3, MY POTENTIOMETER LIBRARY:RK09D1130C2P, symbol MY POTENTIOMETER LIBRARY:RK09D1130C2P
- removed RV911: POT_C3, MY POTENTIOMETER LIBRARY:RK09D1130C2P, symbol MY POTENTIOMETER LIBRARY:RK09D1130C2P
- removed RV912: POT_D3, MY POTENTIOMETER LIBRARY:RK09D1130C2P, symbol MY POTENTIOMETER LIBRARY:RK09D1130C2P
- removed RV914: POT_B4, MY POTENTIOMETER LIBRARY:RK09D1130C2P, symbol MY POTENTIOMETER LIBRARY:RK09D1130C2P
- removed RV915: POT_C4, MY POTENTIOMETER LIBRARY:RK09D1130C2P, symbol MY POTENTIOMETER LIBRARY:RK09D1130C2P
- removed RV916: POT_D4, MY POTENTIOMETER LIBRARY:RK09D1130C2P, symbol MY POTENTIOMETER LIBRARY:RK09D1130C2P
- added U902, U903, U904, U905, U906, U907, U908: PEC12R-4025F-S0024, MY ENCODER LIBRARY:ENC_PEC12R-4025F-S0024, symbol MY ENCODER LIBRARY:PEC12R-4025F-S0024
- renumbered RV905 to RV902, RV909 to RV903, RV913 to RV904
Connections:
- net GND: now also U902.1 (S1), U902.C (COM), U903.1 (S1), U903.C (COM), U904.1 (S1), U904.C (COM), U905.1 (S1), U905.C (COM), U906.1 (S1), U906.C (COM), U907.1 (S1), U907.C (COM), U908.1 (S1), U908.C (COM)
- net ENC_CHA renamed ENC_MENU_CHA
- net ENC_CHB renamed ENC_MENU_CHB
- net ENC_SW renamed ENC_MENU_SW
- net POT_A1 renamed POT_CUT
- net POT_A2 renamed POT_RES
- net POT_A3 renamed POT_MIX
- net POT_A4 renamed POT_VOL
- new net ENC1_CHA: U902.A (CHA)
- new net ENC1_CHB: U902.B (CHB)
- new net ENC1_SW: U902.2 (S2)
- new net ENC2_CHA: U905.A (CHA)
- new net ENC2_CHB: U905.B (CHB)
- new net ENC2_SW: U905.2 (S2)
- new net ENC3_CHA: U907.A (CHA)
- new net ENC3_CHB: U907.B (CHB)
- new net ENC3_SW: U907.2 (S2)
- new net ENC4_CHA: U903.A (CHA)
- new net ENC4_CHB: U903.B (CHB)
- new net ENC4_SW: U903.2 (S2)
- new net ENC5_CHA: U906.A (CHA)
- new net ENC5_CHB: U906.B (CHB)
- new net ENC5_SW: U906.2 (S2)
- new net ENC6_CHA: U908.A (CHA)
- new net ENC6_CHB: U908.B (CHB)
- new net ENC6_SW: U908.2 (S2)
- new net ENCOM_CHA: U904.A (CHA)
- new net ENCOM_CHB: U904.B (CHB)
- new net ENCOM_SW: U904.2 (S2)
Other:
- note removed: "SELECT LEDS"
- moved on the sheet: RV901, RV902, RV903, RV904, U901
