File: DESIGN FILES/memory.kicad_sch (KiCad schematic)
At the start: 20 parts, among them J601 TF-15x15, U601 IS42S16160J-6BLI, U602 IS25WP064A-JBLE

Commit message: changes and adding schematic pdf
Other:
- company: Soundsom -> Joël Ucedo
- title: Memory -> MIMXRT1064 MCU Module
Changed lines of the file:
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@@
   (paper "A3")
   (title_block
-    (title "Memory")
-    (date "2023-05-19")
+    (title "MIMXRT1064 MCU Module")
+    (date "2023-05-23")
     (rev "0")
-    (company "Soundsom")
+    (company "Joël Ucedo")
   )
   (junction (at 288.29 102.87) (diameter 0) (color 0 0 0 0)

Commit message: updates
Parts:
- removed C601, C616: 22u, MIMXRT1064 MCU Module:0603_CL10A226MQ8NRNC, symbol MIMXRT1064 MCU Module:CL10A226MQ8NRNC
- removed C602, C617: 4.7u, MIMXRT1064 MCU Module:0402_CL05A475MP5NRNC, symbol MIMXRT1064 MCU Module:CL05A475MP5NRNC
- removed C603, C604, C605, C607, C608, C609, C610, C611, C619: 100n, MIMXRT1064 MCU Module:0402_CL05B104KB54PNC, symbol MIMXRT1064 MCU Module:CL05B104KB54PNC
- removed C606: 1u, MIMXRT1064 MCU Module:0402_CL05A105KA5NQNC, symbol MIMXRT1064 MCU Module:CL05A105KA5NQNC
- removed FB601: 120R, MIMXRT1064 MCU Module:0603_BLM18AG121SN1D, symbol MIMXRT1064 MCU Module:BLM18AG121SN1D
- removed J601: TF-15x15, MIMXRT1064 MCU Module:TF-15x15_smd, symbol MIMXRT1064 MCU Module:TF-15x15
- removed R601, R603: 10k, MIMXRT1064 MCU Module:0402WGF1002TCE, symbol MIMXRT1064 MCU Module:0402WGF1002TCE
- removed U601: IS42S16160J-6BLI, MIMXRT1064 MCU Module:IS42S16160J-6BLI, symbol MIMXRT1064 MCU Module:IS42S16160J-6BLI
- removed U602: IS25WP064A-JBLE, MIMXRT1064 MCU Module:IS25WP064A-JBLE, symbol MIMXRT1064 MCU Module:IS25WP064A-JBLE
- added 601601601601: IS42S16160J-6BLI, MY MEMORY AND STORAGE LIBRARY:IS42S16160J-6BLI, symbol MY MEMORY AND STORAGE LIBRARY:IS42S16160J-6BLI
- added 602601601601: IS25WP064A-JBLE, MY MEMORY AND STORAGE LIBRARY:IS25WP064A-JBLE, symbol MY MEMORY AND STORAGE LIBRARY:IS25WP064A-JBLE
- added C601: 22u, MY CAPACITOR LIBRARY:0603_CL10A226MQ8NRNC, symbol MY CAPACITOR LIBRARY:CL10A226MQ8NRNC
- added C602: 4.7u, MY CAPACITOR LIBRARY:0402_CL05A475MP5NRNC, symbol MY CAPACITOR LIBRARY:CL05A475MP5NRNC
- added C603, C604, C605, C606, C607, C608, C609, C611: 100n, MY CAPACITOR LIBRARY:0402_CL05B104KB54PNC, symbol MY CAPACITOR LIBRARY:CL05B104KB54PNC
- added C610: 1u, MY CAPACITOR LIBRARY:0402_CL05A105KA5NQNC, symbol MY CAPACITOR LIBRARY:CL05A105KA5NQNC
- added FB601: 120R, MY FERRITE BEAD LIBRARY:0603_BLM18AG121SN1D, symbol MY FERRITE BEAD LIBRARY:BLM18AG121SN1D
- added R601: 10k, MY RESISTOR LIBRARY:0402WGF1002TCE, symbol MY RESISTOR LIBRARY:0402WGF1002TCE
Connections:
- net +1V8: now also 602601601601.8 (VCC), C610.1, C611.1, R601.1
- net +3V3: now also FB601.1
- net FLEXSPI_CLK: now also 602601601601.6 (SCK)
- net FLEXSPI_D0: now also 602601601601.5 (SI(IO0))
- net FLEXSPI_D1: now also 602601601601.2 (SO(IO1))
- net FLEXSPI_D2: now also 602601601601.3 (WP#(IO2))
- net FLEXSPI_D3: now also 602601601601.7 (HOLD#)
- net FLEXSPI_SS: now also 602601601601.1 (CE#), R601.2
- net GND: now also 601601601601.A1 (VSS_1), 601601601601.A3 (VSSQ_1), 601601601601.B7 (VSSQ_2), 601601601601.C3 (VSSQ_3), 601601601601.D7 (VSSQ_4), 601601601601.E3 (VSS_2), 601601601601.J1 (VSS_3), 602601601601.4 (GND), C601.2, C602.2, C603.2, C604.2, C605.2, C606.2, C607.2, C608.2, C609.2, C610.2, C611.2
- net SDRAM_3V3: now also 601601601601.A7 (VDDQ_1), 601601601601.A9 (VDD_1), 601601601601.B3 (VDDQ_2), 601601601601.C7 (VDDQ_3), 601601601601.D3 (VDDQ_4), 601601601601.E7 (VDD_2), 601601601601.J9 (VDD_3), C601.1, C602.1, C603.1, C604.1, C605.1, C606.1, C607.1, C608.1, C609.1, FB601.2
- net SDRAM_A0: now also 601601601601.H7 (A0)
- net SDRAM_A1: now also 601601601601.H8 (A1)
- net SDRAM_A10: now also 601601601601.H9 (A10)
- net SDRAM_A11: now also 601601601601.G2 (A11)
- net SDRAM_A12: now also 601601601601.G1 (A12)
- net SDRAM_A2: now also 601601601601.J8 (A2)
- net SDRAM_A3: now also 601601601601.J7 (A3)
- net SDRAM_A4: now also 601601601601.J3 (A4)
- net SDRAM_A5: now also 601601601601.J2 (A5)
- net SDRAM_A6: now also 601601601601.H3 (A6)
- net SDRAM_A7: now also 601601601601.H2 (A7)
- net SDRAM_A8: now also 601601601601.H1 (A8)
- net SDRAM_A9: now also 601601601601.G3 (A9)
- net SDRAM_BA0: now also 601601601601.G7 (BA0)
- net SDRAM_BA1: now also 601601601601.G8 (BA1)
- net SDRAM_CAS: now also 601601601601.F7 (~{CAS})
- net SDRAM_CKE: now also 601601601601.F3 (CKE)
- net SDRAM_CLK: now also 601601601601.F2 (CLK)
- net SDRAM_CS: now also 601601601601.G9 (~{CS})
- net SDRAM_D0: now also 601601601601.A8 (DQ0)
- net SDRAM_D1: now also 601601601601.B9 (DQ1)
- net SDRAM_D10: now also 601601601601.D1 (DQ10)
- net SDRAM_D11: now also 601601601601.C2 (DQ11)
- net SDRAM_D12: now also 601601601601.C1 (DQ12)
- net SDRAM_D13: now also 601601601601.B2 (DQ13)
- net SDRAM_D14: now also 601601601601.B1 (DQ14)
- net SDRAM_D15: now also 601601601601.A2 (DQ15)
- net SDRAM_D2: now also 601601601601.B8 (DQ2)
- net SDRAM_D3: now also 601601601601.C9 (DQ3)
- net SDRAM_D4: now also 601601601601.C8 (DQ4)
- net SDRAM_D5: now also 601601601601.D9 (DQ5)
- net SDRAM_D6: now also 601601601601.D8 (DQ6)
- net SDRAM_D7: now also 601601601601.E9 (DQ7)
- net SDRAM_D8: now also 601601601601.E1 (DQ8)
- net SDRAM_D9: now also 601601601601.D2 (DQ9)
- net SDRAM_DQMH: now also 601601601601.F1 (DQMH)
- net SDRAM_DQML: now also 601601601601.E8 (DQML)
- net SDRAM_RAS: now also 601601601601.F8 (~{RAS})
- net SDRAM_WE: now also 601601601601.F9 (~{WE})
Other:
- note removed: "CARD INSERT-->SD_CD_SW LOW CARD OFF-->SD_CD_SW HIGH"
- note removed: "FOR SD BOOT, ROM NEED SD_CD_SW PIN KEPT LOW"
- note removed: "uSD CARD"

Commit message: updates
Parts:
- removed 601601601601: IS42S16160J-6BLI, MY MEMORY AND STORAGE LIBRARY:IS42S16160J-6BLI, symbol MY MEMORY AND STORAGE LIBRARY:IS42S16160J-6BLI
- removed 602601601601: IS25WP064A-JBLE, MY MEMORY AND STORAGE LIBRARY:IS25WP064A-JBLE, symbol MY MEMORY AND STORAGE LIBRARY:IS25WP064A-JBLE
- added U601: IS25WP064A-JBLE, MY MEMORY AND STORAGE LIBRARY:IS25WP064A-JBLE, symbol MY MEMORY AND STORAGE LIBRARY:IS25WP064A-JBLE
- added U602: IS42S16160J-6BLI, MY MEMORY AND STORAGE LIBRARY:IS42S16160J-6BLI, symbol MY MEMORY AND STORAGE LIBRARY:IS42S16160J-6BLI
Connections:
- net +1V8: now also U601.8 (VCC)
- net FLEXSPI_CLK: now also U601.6 (SCK)
- net FLEXSPI_D0: now also U601.5 (SI(IO0))
- net FLEXSPI_D1: now also U601.2 (SO(IO1))
- net FLEXSPI_D2: now also U601.3 (WP#(IO2))
- net FLEXSPI_D3: now also U601.7 (HOLD#)
- net FLEXSPI_SS: now also U601.1 (CE#)
- net GND: now also U601.4 (GND), U602.A1 (VSS_1), U602.A3 (VSSQ_1), U602.B7 (VSSQ_2), U602.C3 (VSSQ_3), U602.D7 (VSSQ_4), U602.E3 (VSS_2), U602.J1 (VSS_3)
- net SDRAM_3V3: now also U602.A7 (VDDQ_1), U602.A9 (VDD_1), U602.B3 (VDDQ_2), U602.C7 (VDDQ_3), U602.D3 (VDDQ_4), U602.E7 (VDD_2), U602.J9 (VDD_3)
- net SDRAM_A0: now also U602.H7 (A0)
- net SDRAM_A1: now also U602.H8 (A1)
- net SDRAM_A10: now also U602.H9 (A10)
- net SDRAM_A11: now also U602.G2 (A11)
- net SDRAM_A12: now also U602.G1 (A12)
- net SDRAM_A2: now also U602.J8 (A2)
- net SDRAM_A3: now also U602.J7 (A3)
- net SDRAM_A4: now also U602.J3 (A4)
- net SDRAM_A5: now also U602.J2 (A5)
- net SDRAM_A6: now also U602.H3 (A6)
- net SDRAM_A7: now also U602.H2 (A7)
- net SDRAM_A8: now also U602.H1 (A8)
- net SDRAM_A9: now also U602.G3 (A9)
- net SDRAM_BA0: now also U602.G7 (BA0)
- net SDRAM_BA1: now also U602.G8 (BA1)
- net SDRAM_CAS: now also U602.F7 (~{CAS})
- net SDRAM_CKE: now also U602.F3 (CKE)
- net SDRAM_CLK: now also U602.F2 (CLK)
- net SDRAM_CS: now also U602.G9 (~{CS})
- net SDRAM_D0: now also U602.A8 (DQ0)
- net SDRAM_D1: now also U602.B9 (DQ1)
- net SDRAM_D10: now also U602.D1 (DQ10)
- net SDRAM_D11: now also U602.C2 (DQ11)
- net SDRAM_D12: now also U602.C1 (DQ12)
- net SDRAM_D13: now also U602.B2 (DQ13)
- net SDRAM_D14: now also U602.B1 (DQ14)
- net SDRAM_D15: now also U602.A2 (DQ15)
- net SDRAM_D2: now also U602.B8 (DQ2)
- net SDRAM_D3: now also U602.C9 (DQ3)
- net SDRAM_D4: now also U602.C8 (DQ4)
- net SDRAM_D5: now also U602.D9 (DQ5)
- net SDRAM_D6: now also U602.D8 (DQ6)
- net SDRAM_D7: now also U602.E9 (DQ7)
- net SDRAM_D8: now also U602.E1 (DQ8)
- net SDRAM_D9: now also U602.D2 (DQ9)
- net SDRAM_DQMH: now also U602.F1 (DQMH)
- net SDRAM_DQML: now also U602.E8 (DQML)
- net SDRAM_RAS: now also U602.F8 (~{RAS})
- net SDRAM_WE: now also U602.F9 (~{WE})
Other:
- title: MIMXRT1064 MCU Module -> MIMXRT1064 Audio Board

Commit message: updates
Parts:
- added C612: 22u, MY CAPACITOR LIBRARY:0603_CL10A226MQ8NRNC, symbol MY CAPACITOR LIBRARY:CL10A226MQ8NRNC
- added C613: 4.7u, MY CAPACITOR LIBRARY:0402_CL05A475MP5NRNC, symbol MY CAPACITOR LIBRARY:CL05A475MP5NRNC
- added C614: 100n, MY CAPACITOR LIBRARY:0402_CL05B104KB54PNC, symbol MY CAPACITOR LIBRARY:CL05B104KB54PNC
- added FB602: UPZ1608U601-1R3TF, MY FERRITE BEAD LIBRARY:UPZ1608U601-1R3TF_0603, symbol MY FERRITE BEAD LIBRARY:UPZ1608U601-1R3TF
- added J601: TF-15x15, MY CONNECTOR LIBRARY:TF-15x15_smd, symbol MY CONNECTOR LIBRARY:TF-15x15
- renumbered C610 to C606, C606 to C607, C611 to C608, C607 to C609, C608 to C610, C609 to C611
Connections:
- net +3V3: now also FB602.1
- net GND: now also C612.2, C613.2, C614.2, J601.10 (MP1), J601.11 (MP2), J601.12 (MP3), J601.13 (MP4), J601.6 (VSS)
- new net SD_CLK: J601.5 (CLK)
- new net SD_CMD: J601.3 (CMD)
- new net SD_DAT0: J601.7 (DAT0)
- new net SD_DAT1: J601.8 (DAT1)
- new net SD_DAT2: J601.1 (DAT2)
- new net SD_DAT3: J601.2 (DAT3/CD)
- new net SD_VDD: C612.1, C613.1, C614.1, FB602.2, J601.4 (VDD)
- no-connect marks 0 -> 1
Other:
- note added: "Capacity : Up to 2TByte SDHX card Data transfer rate : Up to 104 MByte/s (UHS-I SDR104)"
- note added: "Memory size : 256Mbit Data Bus Width : 16bit Max clock frequency : 166MHz"
- note added: "Memory size : 64 Mbit Data bus width : 8 bit Max clock frequency : 133MHz"
- note added: "[6] MEMORY"
- note added: "uSD"
- note removed: "6 : MEMORY"
- title: MIMXRT1064 Audio Board -> MIMXRT1064 MCU Module
- moved on the sheet: C601, C602, C603, C604, C605, C606, C607, C608, C609, C610, C611, FB601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

Commit message: updates
Changed lines of the file:
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@@
   (junction (at 266.7 137.16) (diameter 0) (color 0 0 0 0)
+  )
+  (junction (at 317.5 85.09) (diameter 0) (color 0 0 0 0)
   )
   (junction (at 151.13 67.31) (diameter 0) (color 0 0 0 0)
@@
     (stroke (width 0) (type default) (color 0 0 0 0))
   )
+  (wire (pts (xy 317.5 85.09) (xy 317.5 88.9))
+    (stroke (width 0) (type default) (color 0 0 0 0))
+  )
   (wire (pts (xy 74.93 67.31) (xy 87.63 67.31))
     (stroke (width 0) (type default) (color 0 0 0 0))
@@
     (stroke (width 0) (type default) (color 0 0 0 0))
   )
+  (wire (pts (xy 311.15 82.55) (xy 311.15 85.09))
+    (stroke (width 0) (type default) (color 0 0 0 0))
+  )
   (wire (pts (xy 113.03 91.44) (xy 113.03 92.71))
     (stroke (width 0) (type default) (color 0 0 0 0))
@@
     (stroke (width 0.5) (type default) (color 0 0 0 0))
   )
-  (wire (pts (xy 317.5 80.01) (xy 317.5 88.9))
+  (wire (pts (xy 317.5 80.01) (xy 317.5 85.09))
     (stroke (width 0) (type default) (color 0 0 0 0))
   )
@@
   )
   (wire (pts (xy 130.81 120.65) (xy 143.51 120.65))
+    (stroke (width 0) (type default) (color 0 0 0 0))
+  )
+  (wire (pts (xy 311.15 85.09) (xy 317.5 85.09))
     (stroke (width 0) (type default) (color 0 0 0 0))
   )
@@
       (effects (font (size 1.27 1.27)) hide)
     )
+    (pin "1")
+  )
+  (symbol (lib_id "power:PWR_FLAG") (at 311.15 82.55 0) (unit 1)
+    (in_bom yes) (on_board yes) (fields_autoplaced)
+    (property "Reference" "#FLG0602" (id 0) (at 311.15 80.645 0)
+      (effects (font (size 1.27 1.27)) hide)
+    )
+    (property "Value" "PWR_FLAG" (id 1) (at 311.15 77.47 0))
+    (property "Footprint" "" (id 2) (at 311.15 82.55 0)
+      (effects (font (size 1.27 1.27)) hide)
+    )
+    (property "Datasheet" "~" (id 3) (at 311.15 82.55 0)
+      (effects (font (size 1.27 1.27)) hide)
+    )
