File: DESIGN FILES/pinout.kicad_sch (KiCad schematic)
At the start: 1 part, among them U701 M.2-B-KEY

Commit message: updates
Connections:
- net GND: now also U701.MOUNTING-HOLE (MP1)
Changed lines of the file:
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@@
   (junction (at 121.92 125.73) (diameter 0) (color 0 0 0 0)
   )
+  (junction (at 114.3 130.81) (diameter 0) (color 0 0 0 0)
+  )
   (junction (at 133.35 138.43) (diameter 0) (color 0 0 0 0)
   )
@@
   (junction (at 133.35 85.09) (diameter 0) (color 0 0 0 0)
   )
+  (junction (at 168.91 64.77) (diameter 0) (color 0 0 0 0)
+  )
   (wire (pts (xy 133.35 87.63) (xy 133.35 102.87))
     (stroke (width 0) (type default) (color 0 0 0 0))
@@
     (stroke (width 0) (type default) (color 0 0 0 0))
   )
-  (wire (pts (xy 165.1 64.77) (xy 200.66 64.77))
+  (wire (pts (xy 165.1 64.77) (xy 168.91 64.77))
     (stroke (width 0) (type default) (color 0 0 0 0))
   )
@@
     (stroke (width 0) (type default) (color 0 0 0 0))
   )
+  (wire (pts (xy 168.91 50.8) (xy 168.91 64.77))
+    (stroke (width 0) (type default) (color 0 0 0 0))
+  )
   (wire (pts (xy 121.92 123.19) (xy 139.7 123.19))
     (stroke (width 0) (type default) (color 0 0 0 0))
@@
     (stroke (width 0) (type default) (color 0 0 0 0))
   )
+  (wire (pts (xy 152.4 57.15) (xy 152.4 50.8))
+    (stroke (width 0) (type default) (color 0 0 0 0))
+  )
   (wire (pts (xy 133.35 85.09) (xy 133.35 69.85))
     (stroke (width 0) (type default) (color 0 0 0 0))
@@
     (stroke (width 0) (type default) (color 0 0 0 0))
   )
-  (wire (pts (xy 139.7 130.81) (xy 99.06 130.81))
+  (wire (pts (xy 139.7 130.81) (xy 114.3 130.81))
     (stroke (width 0) (type default) (color 0 0 0 0))
   )
@@
     (stroke (width 0) (type default) (color 0 0 0 0))
   )
+  (wire (pts (xy 168.91 64.77) (xy 200.66 64.77))
+    (stroke (width 0) (type default) (color 0 0 0 0))
+  )
   (wire (pts (xy 133.35 128.27) (xy 133.35 133.35))
     (stroke (width 0) (type default) (color 0 0 0 0))
   )
+  (wire (pts (xy 152.4 50.8) (xy 168.91 50.8))
+    (stroke (width 0) (type default) (color 0 0 0 0))
+  )
   (wire (pts (xy 165.1 67.31) (xy 185.42 67.31))
     (stroke (width 0) (type default) (color 0 0 0 0))
@@
     (stroke (width 0) (type default) (color 0 0 0 0))
   )
+  (wire (pts (xy 114.3 129.54) (xy 114.3 130.81))
+    (stroke (width 0) (type default) (color 0 0 0 0))
+  )
   (wire (pts (xy 165.1 138.43) (xy 185.42 138.43))
     (stroke (width 0) (type default) (color 0 0 0 0))
@@
   )
   (wire (pts (xy 165.1 128.27) (xy 185.42 128.27))
+    (stroke (width 0) (type default) (color 0 0 0 0))
+  )
+  (wire (pts (xy 114.3 130.81) (xy 99.06 130.81))
     (stroke (width 0) (type default) (color 0 0 0 0))
   )
@@
       (effects (font (size 1.27 1.27)) hide)
     )
+    (pin "1")
+  )
+  (symbol (lib_id "power:PWR_FLAG") (at 114.3 129.54 0) (unit 1)
+    (in_bom yes) (on_board yes)
+    (property "Reference" "#FLG0701" (id 0) (at 114.3 127.635 0)
+      (effects (font (size 1.27 1.27)) hide)
+    )
+    (property "Value" "PWR_FLAG" (id 1) (at 120.65 128.27 0))
+    (property "Footprint" "" (id 2) (at 114.3 129.54 0)
+      (effects (font (size 1.27 1.27)) hide)
+    )
+    (property "Datasheet" "~" (id 3) (at 114.3 129.54 0)
+      (effects (font (size 1.27 1.27)) hide)
+    )

Commit message: updates
Connections:
- net +5V renamed VBUS
Changed lines of the file:
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@@
     (pin "P$9")
-  )
-  (symbol (lib_id "power:+5V") (at 99.06 62.23 0) (unit 1)
-    (in_bom yes) (on_board yes) (fields_autoplaced)
-    (property "Reference" "#PWR0702" (id 0) (at 99.06 66.04 0)
-      (effects (font (size 1.27 1.27)) hide)
-    )
-    (property "Value" "+5V" (id 1) (at 99.06 57.15 0))
-    (property "Footprint" "" (id 2) (at 99.06 62.23 0)
-      (effects (font (size 1.27 1.27)) hide)
-    )
-    (property "Datasheet" "" (id 3) (at 99.06 62.23 0)
-      (effects (font (size 1.27 1.27)) hide)
-    )
-    (pin "1")
   )
   (symbol (lib_id "power:GND") (at 133.35 154.94 0) (unit 1)
@@
       (effects (font (size 1.27 1.27)) hide)
     )
+    (pin "1")
+  )
+  (symbol (lib_id "power:VBUS") (at 99.06 62.23 0) (unit 1)
+    (in_bom yes) (on_board yes) (fields_autoplaced)
+    (property "Reference" "#PWR0101" (id 0) (at 99.06 66.04 0)
+      (effects (font (size 1.27 1.27)) hide)
+    )
+    (property "Value" "VBUS" (id 1) (at 99.06 57.15 0))
+    (property "Footprint" "" (id 2) (at 99.06 62.23 0)
+      (effects (font (size 1.27 1.27)) hide)
+    )
+    (property "Datasheet" "" (id 3) (at 99.06 62.23 0)
+      (effects (font (size 1.27 1.27)) hide)
+    )

Commit message: up
Connections:
- net CODEC_SCL: now also U701.P$48 (48); no longer U701.P$42 (42)
- net CODEC_SDA: now also U701.P$50 (50); no longer U701.P$44 (44)
- net GND: now also U701.P$20 (20), U701.P$69 (69); no longer U701.P$26 (26), U701.P$28 (28), U701.P$6 (6)
- net I2S_ADCDAT: now also U701.P$59 (59); no longer U701.P$32 (32)
- net I2S_BCLK: now also U701.P$55 (55); no longer U701.P$30 (30)
- net I2S_DACDAT: now also U701.P$57 (57); no longer U701.P$34 (34)
- net I2S_LRC: now also U701.P$61 (61); no longer U701.P$36 (36)
- net I2S_MCLK: now also U701.P$63 (63); no longer U701.P$38 (38)
- net IO1: now also U701.P$24 (24); no longer U701.P$65 (65)
- net IO10: now also U701.P$43 (43); no longer U701.P$47 (47)
- net IO11: now also U701.P$39 (39); no longer U701.P$45 (45)
- net IO12: now also U701.P$41 (41); no longer U701.P$43 (43)
- net IO13: now also U701.P$37 (37); no longer U701.P$41 (41)
- net IO14: now also U701.P$33 (33); no longer U701.P$39 (39)
- net IO15: now also U701.P$35 (35); no longer U701.P$37 (37)
- net IO16: now also U701.P$31 (31); no longer U701.P$35 (35)
- net IO17: now also U701.P$29 (29); no longer U701.P$33 (33)
- net IO18: now also U701.P$27 (27); no longer U701.P$31 (31)
- net IO19: now also U701.P$25 (25); no longer U701.P$29 (29)
- net IO2: now also U701.P$44 (44); no longer U701.P$63 (63)
- net IO20: now also U701.P$23 (23); no longer U701.P$27 (27)
- net IO21: now also U701.P$26 (26); no longer U701.P$25 (25)
- net IO22: now also U701.P$21 (21); no longer U701.P$23 (23)
- net IO23: now also U701.P$22 (22); no longer U701.P$21 (21)
- net IO26: now also U701.P$7 (7); no longer U701.P$3 (3)
- net IO28: now also U701.P$3 (3); no longer U701.P$7 (7)
- net IO3: now also U701.P$28 (28); no longer U701.P$61 (61)
- net IO4: now also U701.P$38 (38); no longer U701.P$59 (59)
- net IO5: now also U701.P$34 (34); no longer U701.P$57 (57)
- net IO6: now also U701.P$30 (30); no longer U701.P$55 (55)
- net IO7: now also U701.P$42 (42); no longer U701.P$53 (53)
- net IO8: now also U701.P$36 (36); no longer U701.P$51 (51)
- net IO9: now also U701.P$32 (32); no longer U701.P$49 (49)
- net JTAG_TCK: now also U701.P$47 (47); no longer U701.P$20 (20)
- net JTAG_TDI: now also U701.P$49 (49); no longer U701.P$10 (10)
- net JTAG_TDO: now also U701.P$51 (51); no longer U701.P$22 (22)
- net JTAG_TMS: now also U701.P$45 (45); no longer U701.P$8 (8)
- net JTAG_nTRST: now also U701.P$53 (53); no longer U701.P$24 (24)
- net MIDI_IN: now also U701.P$67 (67); no longer U701.P$48 (48)
- net MIDI_OUT: now also U701.P$65 (65); no longer U701.P$50 (50)
- net SPI_CS: now also U701.P$4 (4); no longer U701.P$73 (73)
- net SPI_SCK: now also U701.P$8 (8); no longer U701.P$67 (67)
- net SPI_SIN: now also U701.P$2 (2); no longer U701.P$71 (71)
- net SPI_SOUT: now also U701.P$6 (6); no longer U701.P$69 (69)
- net USB_D+: now also U701.P$71 (71); no longer U701.P$2 (2)
- net USB_D-: now also U701.P$73 (73); no longer U701.P$4 (4)
